File: prancha-XIII.sch (KiCad schematic (older format))
At the start: 0 parts

Commit message: trocando pranchas XII <=> XIII
Parts:
- added U? (x7): 7402, ~, symbol 7402
- added U? (x7): 74HC04, ~, symbol 74HC04
- added U? (x5): 74LS10, ~, symbol 74LS10
- added U? (x3): 7400, ~, symbol 7400
- added U?: 74LS13, ~, symbol 74LS13
- added U? (x2): 74LS54, ~, symbol 74LS54
Connections:
- new net: U?.1, U?.2
- new net: U?.2, U?.2 (x2)
- new net: U?.1, U?.1, U?.1 (x2)
- new net: U?.2, U?.3 (x4)
- new net: U?.1, U?.12 (x2)
- new net: U?.12, U?.13, U?.2
- new net: U?.12, U?.2
- new net: U?.12, U?.2, U?.2
- new net: U?.1, U?.3 (x2)
- new net: U?.1, U?.1
- new net: U?.2, U?.4
- new net: U?.2, U?.5
- new net: U?.13, U?.3
- new net: U?.3, U?.4, U?.4
- new net: U?.10, U?.10, U?.6
- new net +(PARTIDA.(-RODA)): U?.1
- new net +F1: U?.1, U?.1, U?.1, U?.1, U?.1, U?.1, U?.1, U?.1, U?.1, U?.13, U?.13, U?.13, U?.2, U?.2, U?.2, U?.2, U?.2, U?.2, U?.2, U?.2, U?.2, U?.3
- new net +PUL: U?.1
- new net +T6: U?.13, U?.13, U?.3, U?.3, U?.5, U?.5, U?.9, U?.9
- new net -F1: U?.3
- new net GND: U?.7 (GND), U?.7 (GND), U?.7 (GND), U?.7 (GND), U?.7 (GND), U?.7 (GND), U?.7 (GND), U?.7 (GND), U?.7 (GND), U?.7 (GND), U?.7 (GND), U?.7 (GND), U?.7 (GND), U?.7 (GND), U?.7 (GND), U?.7 (GND), U?.7 (GND), U?.7 (GND), U?.7 (GND), U?.7 (GND), U?.7 (GND), U?.7 (GND), U?.7 (GND), U?.7 (GND), U?.7 (GND)
- new net VCC: U?.14 (VCC), U?.14 (VCC), U?.14 (VCC), U?.14 (VCC), U?.14 (VCC), U?.14 (VCC), U?.14 (VCC), U?.14 (VCC), U?.14 (VCC), U?.14 (VCC), U?.14 (VCC), U?.14 (VCC), U?.14 (VCC), U?.14 (VCC), U?.14 (VCC), U?.14 (VCC), U?.14 (VCC), U?.14 (VCC), U?.14 (VCC), U?.14 (VCC), U?.14 (VCC), U?.14 (VCC), U?.14 (VCC), U?.14 (VCC), U?.14 (VCC)
- new net aaa: U?.1, U?.2, U?.8, U?.8
Other:
- note added: "Este bloco esta com todos lables errados. Falta colocar os nomes certos."

Commit message: wip
Parts:
- removed U?: 74LS10, ~, symbol 74LS10
- added 2F_P13: 74LS13, ~, symbol 74LS13
- gave numbers to parts that had none: 7
Connections:
- net +F1: now also 3A_P13.3; no longer 2E_P13.1, 2E_P13.1, 2E_P13.13, 2E_P13.13, 2E_P13.2, 2E_P13.2, 3A_P13.1, 3A_P13.13, 3A_P13.2, 3E_P13.2, 4A_P13.1, U?.1, U?.1, U?.1, U?.1, U?.2, U?.2, U?.2, U?.2, U?.2, U?.3
- net +PUL: now also 4A_P13.13; no longer 4A_P13.1
- net +T6: no longer U?.13, U?.13, U?.3, U?.3, U?.5, U?.5
- net -F1: now also 3E_P13.9, U?.1; no longer 3E_P13.3
- net GND: now also 2F_P13.7 (GND)
- net VCC: now also 2F_P13.14 (VCC)
- net at U?.2: now also 3E_P13.10; no longer 3E_P13.1
- net at U?.1: now also 3A_P13.6; no longer 3A_P13.12
- net at 3E_P13.3: now also 1F_P13.13; no longer 1F_P13.1
- net at 3E_P13.1: now also 3F_P13.3; no longer 3F_P13.1
- net at 4D_P13.4: now also 3F_P13.4; no longer 3F_P13.2
- net at 4D_P13.5: now also 3F_P13.6; no longer 3F_P13.2
- net at U?.3: now also 2F_P13.4
- net at U?.3: now also 2F_P13.2, 2F_P13.5
- net aaa renamed PAROP
- net PAROP: no longer U?.8, U?.8
- new net: 3E_P13.8, 4A_P13.12
- new net: 1F_P13.11, 2E_P13.6
- new net: 1F_P13.12, 4A_P13.10
- new net: 2F_P13.6, 3F_P13.5
- new net +CE: U?.1
- new net +CP: U?.3
- new net +F3: 2E_P13.1
- new net +F5: U?.1
- new net +MICG2A: 3A_P13.4
- new net +MP: U?.2
- new net +PLI: U?.2
- new net +PM1: U?.1
- new net +S: 2E_P13.13
- new net +SALMIC: 3A_P13.5
- new net +SUS: 2E_P13.2
- new net +T1: U?.5, U?.5
- new net +T2: U?.13, U?.13
- new net +T4: U?.3, U?.3
- new net -(C_CI)_1: U?.8
- new net -(C_CI)_2: U?.8
- new net -(F2.SAESA.S): 4A_P13.11, U?.2
- new net -(F4.PUG): 2F_P13.1
- new net -(PAN.ACN): 2E_P13.4
- new net -(PARTIDA.(-RODA)): U?.2
- new net -(PAZ.ACZ): 2E_P13.5
- new net -F2: 3E_P13.2, U?.2
- new net -PLI: 2E_P13.3
Other:
- note added: "Este bloco esta com todas referencias de CIs erradas. Falta colocar os numeros certos."
- note removed: "Este bloco esta com todos lables errados. Falta colocar os nomes certos."
Changed lines of the file:
@@
 $Descr A2 23386 16535
 encoding utf-8
-Sheet 4 17
+Sheet 6 17
 Title ""
-Date "1 aug 2016"
+Date "2 aug 2016"
 Rev ""
 Comp ""
@@
 $EndDescr
 $Comp
-L 7402 U?
-U 1 1 5772BFAE
+L 7402 3E_P13
+U 3 1 5772BFAE
 P 12650 1950
-F 0 "U?" H 12650 2000 60  0000 C CNN
+F 0 "3E_P13" H 12650 2000 60  0000 C CNN
 F 1 "7402" H 12700 1900 60  0000 C CNN
 F 2 "~" H 12650 1950 60  0000 C CNN
 F 3 "~" H 12650 1950 60  0000 C CNN
-	1    12650 1950
+	3    12650 1950
 	1    0    0    -1
 $EndComp
@@
 $EndComp
 $Comp
-L 74HC04 U?
-U 1 1 5772BFC3
+L 74HC04 4A_P13
+U 6 1 5772BFC3
 P 11400 1600
-F 0 "U?" H 11550 1700 40  0000 C CNN
+F 0 "4A_P13" H 11550 1700 40  0000 C CNN
 F 1 "74HC04" H 11600 1500 40  0000 C CNN
 F 2 "~" H 11400 1600 60  0000 C CNN
 F 3 "~" H 11400 1600 60  0000 C CNN
-	1    11400 1600
+	6    11400 1600
 	1    0    0    -1
 $EndComp
@@
 	12050 2300 10750 2300
 $Comp
-L 74LS10 U?
-U 1 1 5772C019
+L 74LS10 3A_P13
+U 2 1 5772C019
 P 12650 2450
-F 0 "U?" H 12650 2500 60  0000 C CNN
+F 0 "3A_P13" H 12650 2500 60  0000 C CNN
 F 1 "74LS10" H 12650 2400 60  0000 C CNN
 F 2 "~" H 12650 2450 60  0000 C CNN
 F 3 "~" H 12650 2450 60  0000 C CNN
-	1    12650 2450
-	1    0    0    -1
-$EndComp
-$Comp
-L 74LS10 U?
+	2    12650 2450
+	1    0    0    -1
+$EndComp
+$Comp
+L 74LS10 2E_P13
 U 1 1 5772C030
 P 12650 2950
-F 0 "U?" H 12650 3000 60  0000 C CNN
+F 0 "2E_P13" H 12650 3000 60  0000 C CNN
 F 1 "74LS10" H 12650 2900 60  0000 C CNN
 F 2 "~" H 12650 2950 60  0000 C CNN
@@
 $EndComp
 $Comp
-L 74LS10 U?
-U 1 1 5772C036
+L 74LS10 2E_P13
+U 2 1 5772C036
 P 12650 3450
-F 0 "U?" H 12650 3500 60  0000 C CNN
+F 0 "2E_P13" H 12650 3500 60  0000 C CNN
 F 1 "74LS10" H 12650 3400 60  0000 C CNN
 F 2 "~" H 12650 3450 60  0000 C CNN
 F 3 "~" H 12650 3450 60  0000 C CNN
-	1    12650 3450
+	2    12650 3450
 	1    0    0    -1
 $EndComp
 Text GLabel 10750 2800 0    60   Input ~ 0
-+F1
++F3
 Wire Wire Line
 	12050 2800 10750 2800
 Text GLabel 10750 2450 0    60   Input ~ 0
-+F1
++MICG2A
 Wire Wire Line
 	12050 2450 10750 2450
 Text GLabel 10750 2600 0    60   Input ~ 0
-+F1
++SALMIC
 Wire Wire Line
 	12050 2600 10750 2600
 Text GLabel 10750 2950 0    60   Input ~ 0
-+F1
++SUS
 Wire Wire Line
 	12050 2950 10750 2950
 Text GLabel 10750 3100 0    60   Input ~ 0
-+F1
++S
 Wire Wire Line
 	12050 3100 10750 3100
 Text GLabel 10750 3300 0    60   Input ~ 0
-+F1
+-PLI
 Wire Wire Line
 	12050 3300 10750 3300
 Text GLabel 10750 3450 0    60   Input ~ 0
-+F1
+-(PAN.ACN)
 Wire Wire Line
 	12050 3450 10750 3450
 Text GLabel 10750 3600 0    60   Input ~ 0
-+F1
+-(PAZ.ACZ)
 Wire Wire Line
 	12050 3600 10750 3600
@@
 	15950 2350 16150 2350
 Wire Wire Line
-	15950 2200 15950 2350
-Wire Wire Line
-	15950 2350 15950 3350
+	15950 2200 15950 3350
 Wire Wire Line
 	15950 2200 15800 2200
@@
 	14750 1400 10750 1400
 Text GLabel 14100 1600 0    60   Input ~ 0
-+F1
++CE
 Wire Wire Line
 	14100 1600 16300 1600
@@
 	13250 2950 15750 2950
 Wire Wire Line
-	15750 2650 15750 2950
-Wire Wire Line
-	15750 2950 15750 3450
+	15750 2650 15750 3450
 Text GLabel 14100 2750 0    60   Input ~ 0
-+F1
+-(F2.SAESA.S)
 Wire Wire Line
 	16150 2500 15450 2500
@@
 	15450 2750 14100 2750
 $Comp
-L 7402 U?
-U 1 1 579EC2D3
+L 7402 1F_P13
+U 4 1 579EC2D3
 P 14050 3900
-F 0 "U?" H 14050 3950 60  0000 C CNN
+F 0 "1F_P13" H 14050 3950 60  0000 C CNN
 F 1 "7402" H 14100 3850 60  0000 C CNN
 F 2 "~" H 14050 3900 60  0000 C CNN
 F 3 "~" H 14050 3900 60  0000 C CNN
-	1    14050 3900
-	1    0    0    -1
-$EndComp
-$Comp
-L 7402 U?
+	4    14050 3900
+	1    0    0    -1
+$EndComp
+$Comp
+L 7402 3E_P13
 U 1 1 579EC2D9
 P 15850 3800
-F 0 "U?" H 15850 3850 60  0000 C CNN
+F 0 "3E_P13" H 15850 3850 60  0000 C CNN
 F 1 "7402" H 15900 3750 60  0000 C CNN
 F 2 "~" H 15850 3800 60  0000 C CNN
@@
 $EndComp
 $Comp
-L 74HC04 U?
-U 1 1 579EC2DF
+L 74HC04 3F_P13
+U 2 1 579EC2DF
 P 17250 3800
-F 0 "U?" H 17400 3900 40  0000 C CNN
+F 0 "3F_P13" H 17400 3900 40  0000 C CNN
 F 1 "74HC04" H 17450 3700 40  0000 C CNN
 F 2 "~" H 17250 3800 60  0000 C CNN
 F 3 "~" H 17250 3800 60  0000 C CNN
-	1    17250 3800
-	1    0    0    -1
-$EndComp
-$Comp
-L 74HC04 U?
-U 1 1 579EC2EB
+	2    17250 3800
+	1    0    0    -1
+$EndComp
+$Comp
+L 74HC04 4A_P13
+U 5 1 579EC2EB
 P 12550 4250
-F 0 "U?" H 12700 4350 40  0000 C CNN
+F 0 "4A_P13" H 12700 4350 40  0000 C CNN
 F 1 "74HC04" H 12750 4150 40  0000 C CNN
 F 2 "~" H 12550 4250 60  0000 C CNN
 F 3 "~" H 12550 4250 60  0000 C CNN
-	1    12550 4250
-	1    0    0    -1
-$EndComp
-$Comp
-L 74HC04 U?
-U 1 1 579EC2F1
+	5    12550 4250
+	1    0    0    -1
+$EndComp
+$Comp
+L 74HC04 3F_P13
+U 3 1 579EC2F1
 P 17250 4500
-F 0 "U?" H 17400 4600 40  0000 C CNN
+F 0 "3F_P13" H 17400 4600 40  0000 C CNN
 F 1 "74HC04" H 17450 4400 40  0000 C CNN
 F 2 "~" H 17250 4500 60  0000 C CNN
 F 3 "~" H 17250 4500 60  0000 C CNN
-	1    17250 4500
+	3    17250 4500
 	1    0    0    -1
 $EndComp
@@
 	13350 4000 13450 4000
 Text GLabel 10750 4250 0    60   Input ~ 0
-+F1
+-(F2.SAESA.S)
 Wire Wire Line
 	12100 4250 10750 4250
 Text GLabel 14400 3500 0    60   Input ~ 0
-+F1
+-F2
 Wire Wire Line
 	15250 3900 14650 3900
@@
 Wire Wire Line
 	16800 3800 16450 3800
-$Comp
-L 74LS10 U?
-U 1 1 579EC456
-P 15850 4500
-F 0 "U?" H 15850 4550 60  0000 C CNN
-F 1 "74LS10" H 15850 4450 60  0000 C CNN
-F 2 "~" H 15850 4500 60  0000 C CNN
-F 3 "~" H 15850 4500 60  0000 C CNN
-	1    15850 4500
-	1    0    0    -1
-$EndComp
 Wire Wire Line
 	16450 4500 16800 4500
 Text GLabel 14350 4350 0    60   Input ~ 0
-+F1
+-(F4.PUG)
 Wire Wire Line
 	15250 4350 14350 4350
@@
 $EndComp
 Wire Wire Line
-	15250 4500 14950 4500
-Wire Wire Line
-	14950 4500 14950 4800
-Wire Wire Line
 	14950 4800 14700 4800
 Text GLabel 10750 4700 0    60   Input ~ 0
-+F1
++F5
 Text GLabel 10750 4900 0    60   Input ~ 0
-+F1
++PLI
 Wire Wire Line
 	10750 4700 13500 4700
@@
 $EndComp
 Wire Wire Line
-	15250 4650 15100 4650
-Wire Wire Line
-	15100 4650 15100 5450
+	15100 4550 15100 5450
 Wire Wire Line
 	15100 5450 15000 5450
@@
 $EndComp
 Text GLabel 10750 6150 0    60   Input ~ 0
-+F1
++CP
 Text GLabel 10750 5950 0    60   Input ~ 0
-+F1
++MP
 Text GLabel 10750 5700 0    60   Input ~ 0
-+F1
+-(PARTIDA.(-RODA))
 Wire Wire Line
 	10750 5700 12400 5700
@@
 	13800 5550 13700 5550
 Wire Wire Line
-	13700 5550 13700 5800
-Wire Wire Line
-	13700 5800 13700 6200
+	13700 5550 13700 6200
 Wire Wire Line
 	13700 5800 13600 5800
 Text GLabel 10750 5350 0    60   Input ~ 0
-+F1
++PM1
 Wire Wire Line
 	10750 5350 13800 5350
 Text GLabel 13900 6200 2    60   Input ~ 0
-aaa
+PAROP
 Wire Wire Line
 	13700 6200 13900 6200
@@
 $EndComp
 Text GLabel 16900 2900 0    60   Input ~ 0
-+F1
+-F1
 Text GLabel 16900 3100 0    60   Input ~ 0
-+F1
+-F2
 Wire Wire Line
 	16900 3100 17500 3100
@@
 	17500 2900 16900 2900
 $Comp
-L 74LS13 U?
+L 74LS13 4D_P13
 U 1 1 579ECBE3
 P 18900 4100
-F 0 "U?" H 18900 4150 60  0000 C CNN
+F 0 "4D_P13" H 18900 4150 60  0000 C CNN
 F 1 "74LS13" H 18900 4050 60  0000 C CNN
 F 2 "~" H 18900 4100 60  0000 C CNN
@@
 	20550 2100 20550 4100
 Wire Wire Line
-	19500 4100 20550 4100
-Wire Wire Line
-	20550 4100 20650 4100
-Wire Wire Line
-	20100 4000 20500 4000
-Wire Wire Line
-	20500 4000 20650 4000
+	19500 4100 20650 4100
+Wire Wire Line
+	20100 4000 20650 4000
 Wire Wire Line
 	20500 4000 20500 2000
@@
 	20500 2000 20650 2000
 Wire Wire Line
-	19850 3900 20450 3900
-Wire Wire Line
-	20450 3900 20650 3900
+	19850 3900 20650 3900
 Wire Wire Line
 	20450 3900 20450 1900
@@
 	20400 1800 20400 3800
 Wire Wire Line
-	19850 3700 20350 3700
-Wire Wire Line
-	20350 3700 20650 3700
+	19850 3700 20650 3700
 Wire Wire Line
 	20350 3700 20350 1700
@@
 	20300 1600 20300 3600
 Wire Wire Line
-	19050 3600 20300 3600
-Wire Wire Line
-	20300 3600 20650 3600
-Wire Wire Line
-	19850 3500 20250 3500
-Wire Wire Line
-	20250 3500 20650 3500
+	19050 3600 20650 3600
+Wire Wire Line
+	19850 3500 20650 3500
 Wire Wire Line
 	20250 3500 20250 1500
@@
 	20650 1400 20100 1400
 Wire Wire Line
-	20100 1400 20100 1500
-Wire Wire Line
-	20100 1500 20100 3400
+	20100 1400 20100 3400
 Wire Wire Line
 	20100 3400 20650 3400
@@
 Connection ~ 20500 4000
 Text GLabel 19850 3900 0    60   Input ~ 0
-+T6
++T1
 Connection ~ 20450 3900
 Connection ~ 20400 3800
 Text GLabel 19850 3700 0    60   Input ~ 0
-+T6
++T4
 Connection ~ 20350 3700
 Wire Wire Line
-	18900 3800 20400 3800
-Wire Wire Line
-	20400 3800 20650 3800
+	18900 3800 20650 3800
 Text GLabel 19850 3500 0    60   Input ~ 0
-+T6
++T2
 Connection ~ 20250 3500
 Wire Wire Line
@@
 Connection ~ 20100 1500
 Text GLabel 21750 3750 2    60   Input ~ 0
-aaa
+-(C_CI)_2
 Wire Wire Line
 	21750 3750 21550 3750
 Text GLabel 21750 1750 2    60   Input ~ 0
-aaa
+-(C_CI)_1
 Wire Wire Line
 	21550 1750 21750 1750
 Text Notes 16500 5550 0    60   ~ 0
-Este bloco esta com todos lables errados. Falta colocar os nomes certos.
+Este bloco esta com todas referencias de CIs erradas. Falta colocar os numeros certos.
+$Comp
+L 74LS13 2F_P13
+U 1 1 579F9837
+P 15850 4500
+F 0 "2F_P13" H 15850 4550 60  0000 C CNN
+F 1 "74LS13" H 15850 4450 60  0000 C CNN
+F 2 "~" H 15850 4500 60  0000 C CNN
+F 3 "~" H 15850 4500 60  0000 C CNN
+	1    15850 4500
+	1    0    0    -1
+$EndComp
+Wire Wire Line
+	15250 4450 14950 4450
+Wire Wire Line
+	14950 4450 14950 4800
+Wire Wire Line
+	15100 4550 15250 4550
+Wire Wire Line
+	15250 4650 15150 4650
+Wire Wire Line
+	15150 4650 15150 4450
+Connection ~ 15150 4450
 $EndSCHEMATC
