File: prancha-XIII.sch (KiCad schematic (older format))
At the start: 27 parts

Commit message: finalizei a transcrição da prancha 13
Parts:
- added unit 4 of 1E_P13
- added unit 3 of 1E_P13
- added unit 4 of 2A_P13
- added unit 5 of 2A_P13
- added unit 1 of 3B_P13
- added 3C_P13: 74LS54, ~, symbol 74LS54
- added unit 2 of 3D_P13
- added unit 1 of 4A_P13
- added unit 2 of 4D_P13
- added 4E_P13: 7400, ~, symbol 7400
- added unit 1 of 5A_P13
Connections:
- net +F2: now also 1E_P13.12
- net +F3: now also 4E_P13.4
- net +PUG: now also 3D_P13.6
- net +SUS: now also 3D_P13.5
- net +T23: now also 3C_P13.2
- net +T34: now also 3C_P13.4
- net +T56: now also 3C_P13.13
- net -(CAC+SOM): now also 4E_P13.1
- net -(TRO+TRI): now also 4E_P13.2
- net -F2: now also 2A_P13.9
- net -F5: now also 1E_P13.9
- net GND: now also 1E_P13.7 (GND), 1E_P13.7 (GND), 2A_P13.7 (GND), 2A_P13.7 (GND), 3B_P13.7 (GND), 3C_P13.10, 3C_P13.7 (GND), 3C_P13.9, 3D_P13.7 (GND), 4A_P13.7 (GND), 4D_P13.7 (GND), 4E_P13.7 (GND), 4E_P13.7 (GND), 4E_P13.7 (GND), 4E_P13.7 (GND), 5A_P13.7 (GND)
- net VCC: now also 1E_P13.14 (VCC), 1E_P13.14 (VCC), 2A_P13.14 (VCC), 2A_P13.14 (VCC), 3B_P13.14 (VCC), 3C_P13.14 (VCC), 3D_P13.14 (VCC), 4A_P13.14 (VCC), 4D_P13.14 (VCC), 4E_P13.14 (VCC), 4E_P13.14 (VCC), 4E_P13.14 (VCC), 4E_P13.14 (VCC), 5A_P13.14 (VCC)
- net -(CAC+SOM+PLI+ARA): now reaches 3D_P13.3, 4A_P13.4
- net -(CAC+SOM+PLI+ARA): now also 4D_P13.10
- new net: 3D_P13.4, 4D_P13.9
- new net: 1E_P13.10, 1E_P13.11
- new net: 1E_P13.13, 4D_P13.8
- new net: 3C_P13.8, 4A_P13.1
- new net: 2A_P13.8, 4E_P13.13
- new net: 4E_P13.10, 4E_P13.11
- new net: 4E_P13.3, 4E_P13.5
- new net: 4E_P13.6, 4E_P13.9
- new net: 3C_P13.5, 4E_P13.8
- new net: 1E_P13.8, 3C_P13.1
- new net: 3B_P13.3, 4D_P13.12
- new net: 4D_P13.13, 5A_P13.3
- new net: 2A_P13.10, 5A_P13.2
- new net +(F3.SUS.(-RDZ)): 3C_P13.3
- new net +ACN: 3B_P13.2
- new net +IME: 4E_P13.12
- new net +PAN: 3B_P13.1
- new net +PAZ: 5A_P13.1
- new net +RD/Y: 4A_P13.2
- new net -ACZ: 2A_P13.11
Other:
- note removed: "-(CAC+SOM+PLI+ARA)\n"
- moved on the sheet: 1B_P13A, 1B_P13B, 1B_P13C, 1D_P13B, 1D_P13C, 1E_P13B, 1F_P13B, 1F_P13C, 2A_P13C, 2A_P13F, 2B_P13B, 2B_P13C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
