File: prancha-XV.sch (KiCad schematic (older format))
At the start: 0 parts

Commit message: mais um pouco de transcrição, agora na prancha 15
Parts:
- added 1A_P15, 2A_P15, 3A_P15, 3B_P15, 4A_P15: 74LS04, symbol 74LS04
- added 1C_P15, 1D_P15, 5B_P15: 7400, symbol 7400
- added 3D_P15: 74LS15, symbol 74LS15
- added 5A_P15: 74LS20, symbol 74LS20
Connections:
- new net: 1C_P15.10, 1C_P15.6
- new net: 1C_P15.8, 1D_P15.2, 3B_P15.1
- new net: 1C_P15.3, 1C_P15.9
- new net: 1D_P15.4, 3B_P15.2
- new net: 1D_P15.10, 1D_P15.6
- new net: 1D_P15.3, 1D_P15.9
- new net: 5A_P15.6, 5B_P15.5
- new net: 3D_P15.10, 5B_P15.3
- new net: 3D_P15.8, 5B_P15.4
- new net: 3B_P15.13, 5B_P15.8
- new net +(F3+F4): 5B_P15.9
- new net +(PARTIDA.(-RODA)): 3D_P15.11
- new net +1/I: 3B_P15.12
- new net +AC_0: 1A_P15.1
- new net +AC_1: 1A_P15.3
- new net +AC_2: 1A_P15.5
- new net +AC_3: 1A_P15.9
- new net +AC_4: 1A_P15.11
- new net +AC_5: 1A_P15.13
- new net +AC_6: 2A_P15.1
- new net +AC_7: 2A_P15.3
- new net +CASP: 3A_P15.11
- new net +CE: 3B_P15.5
- new net +CP: 2A_P15.13
- new net +F1: 3A_P15.2, 5A_P15.1
- new net +F2: 3A_P15.4
- new net +F3: 3A_P15.6
- new net +F4: 3A_P15.8
- new net +F4.(TRO+TRI): 3B_P15.8
- new net +IME: 4A_P15.11
- new net +MICG1: 5A_P15.5
- new net +MICG2A: 4A_P15.5
- new net +MP: 2A_P15.11
- new net +OVF: 1C_P15.4
- new net +P(4-11)/Y: 5B_P15.6
- new net +RI_4: 5A_P15.4
- new net +RI_5: 1C_P15.2, 2A_P15.5
- new net +RI_6: 1D_P15.1, 2A_P15.9
- new net +RI_7: 3A_P15.13
- new net +SAE: 4A_P15.13
- new net +SALMIC: 1D_P15.8
- new net +SUS: 4A_P15.9
- new net +T: 1C_P15.1
- new net +T12: 3D_P15.9
- new net +T34: 5A_P15.2
- new net +TRI: 4A_P15.3
- new net +TRO: 4A_P15.1, 5B_P15.10
- new net -AC_0: 1A_P15.2
- new net -AC_1: 1A_P15.4
- new net -AC_2: 1A_P15.6
- new net -AC_3: 1A_P15.8
- new net -AC_4: 1A_P15.10
- new net -AC_5: 1A_P15.12
- new net -AC_6: 2A_P15.2
- new net -AC_7: 2A_P15.4
- new net -CASP: 3A_P15.10
- new net -CE: 3B_P15.6, 5B_P15.1
- new net -CP: 2A_P15.12, 5B_P15.2
- new net -F1: 3A_P15.1
- new net -F2: 3A_P15.3
- new net -F3: 3A_P15.5
- new net -F4: 3A_P15.9
- new net -F4.(TRO+TRI): 3B_P15.9
- new net -IME: 4A_P15.10
- new net -MICG2A: 4A_P15.6
- new net -MP: 2A_P15.10
- new net -RI_5: 1C_P15.5, 2A_P15.6
- new net -RI_6: 1D_P15.5, 2A_P15.8
- new net -RI_7: 3A_P15.12
- new net -SAE: 4A_P15.12
- new net -SUS: 4A_P15.8
- new net -TRI: 4A_P15.4
- new net -TRO: 4A_P15.2
- new net GND: 1A_P15.7 (GND), 1A_P15.7 (GND), 1A_P15.7 (GND), 1A_P15.7 (GND), 1A_P15.7 (GND), 1A_P15.7 (GND), 1C_P15.7 (GND), 1C_P15.7 (GND), 1C_P15.7 (GND), 1D_P15.7 (GND), 1D_P15.7 (GND), 1D_P15.7 (GND), 2A_P15.7 (GND), 2A_P15.7 (GND), 2A_P15.7 (GND), 2A_P15.7 (GND), 2A_P15.7 (GND), 2A_P15.7 (GND), 3A_P15.7 (GND), 3A_P15.7 (GND), 3A_P15.7 (GND), 3A_P15.7 (GND), 3A_P15.7 (GND), 3A_P15.7 (GND), 3B_P15.7 (GND), 3B_P15.7 (GND), 3B_P15.7 (GND), 3B_P15.7 (GND), 3D_P15.7 (GND), 4A_P15.7 (GND), 4A_P15.7 (GND), 4A_P15.7 (GND), 4A_P15.7 (GND), 4A_P15.7 (GND), 4A_P15.7 (GND), 5A_P15.7 (GND), 5B_P15.7 (GND), 5B_P15.7 (GND), 5B_P15.7 (GND)
- new net VCC: 1A_P15.14 (VCC), 1A_P15.14 (VCC), 1A_P15.14 (VCC), 1A_P15.14 (VCC), 1A_P15.14 (VCC), 1A_P15.14 (VCC), 1C_P15.14 (VCC), 1C_P15.14 (VCC), 1C_P15.14 (VCC), 1D_P15.14 (VCC), 1D_P15.14 (VCC), 1D_P15.14 (VCC), 2A_P15.14 (VCC), 2A_P15.14 (VCC), 2A_P15.14 (VCC), 2A_P15.14 (VCC), 2A_P15.14 (VCC), 2A_P15.14 (VCC), 3A_P15.14 (VCC), 3A_P15.14 (VCC), 3A_P15.14 (VCC), 3A_P15.14 (VCC), 3A_P15.14 (VCC), 3A_P15.14 (VCC), 3B_P15.14 (VCC), 3B_P15.14 (VCC), 3B_P15.14 (VCC), 3B_P15.14 (VCC), 3D_P15.14 (VCC), 4A_P15.14 (VCC), 4A_P15.14 (VCC), 4A_P15.14 (VCC), 4A_P15.14 (VCC), 4A_P15.14 (VCC), 4A_P15.14 (VCC), 5A_P15.14 (VCC), 5B_P15.14 (VCC), 5B_P15.14 (VCC), 5B_P15.14 (VCC)
Other:
- note added: "O esquemático original \nnão identifica qual CI\nnem quais pinos são usados\npara essa porta NOT."

Commit message: mais um pequeno trecho da prancha 15
Parts:
- added 5C_P15: 7400, symbol 7400
- added 5D_P15: 74LS15, symbol 74LS15
Connections:
- net +(F3+F4): now also 5C_P15.1
- net GND: now also 5C_P15.7 (GND), 5C_P15.7 (GND), 5D_P15.7 (GND)
- net VCC: now also 5C_P15.14 (VCC), 5C_P15.14 (VCC), 5D_P15.14 (VCC)
- new net: 5C_P15.3, 5C_P15.4
- new net: 5C_P15.6, 5D_P15.3, 5D_P15.4, 5D_P15.5
- new net +(TRO+TRI): 5C_P15.2
- new net +RE/I: 5D_P15.6
- new net -F5: 5C_P15.5
Changed lines of the file:
@@
 $EndComp
 Wire Wire Line
-	3950 1550 4250 1550
+	3950 1550 4100 1550
+Wire Wire Line
+	4100 1550 4250 1550
 $Comp
 L 7400 1D_P15
@@
 Wire Wire Line
 	12050 7350 11900 7350
+$Comp
+L 7400 5C_P15
+U 1 1 58727F1C
+P 11700 5200
+F 0 "5C_P15" H 11700 5628 60  0000 C CNN
+F 1 "7400" H 11700 5522 60  0000 C CNN
+F 2 "" H 11700 5200 60  0000 C CNN
+F 3 "" H 11700 5200 60  0000 C CNN
+	1    11700 5200
+	1    0    0    -1
+$EndComp
+Text GLabel 10950 5100 0    60   Input ~ 0
++(F3+F4)
+Text GLabel 10950 5300 0    60   Input ~ 0
++(TRO+TRI)
+Wire Wire Line
+	10950 5100 11100 5100
+Wire Wire Line
+	11100 5300 10950 5300
+$Comp
+L 7400 5C_P15
+U 2 1 5872814E
+P 13050 5300
+F 0 "5C_P15" H 13050 5728 60  0000 C CNN
+F 1 "7400" H 13050 5622 60  0000 C CNN
+F 2 "" H 13050 5300 60  0000 C CNN
+F 3 "" H 13050 5300 60  0000 C CNN
+	2    13050 5300
+	1    0    0    -1
+$EndComp
+Text GLabel 12300 5400 0    60   Input ~ 0
+-F5
+Wire Wire Line
+	12300 5200 12450 5200
+Wire Wire Line
+	12450 5400 12300 5400
+$Comp
+L 74LS15 5D_P15
+U 2 1 5872833B
+P 14500 5300
+F 0 "5D_P15" H 14500 5708 60  0000 C CNN
+F 1 "74LS15" H 14500 5602 60  0000 C CNN
+F 2 "" H 14500 5300 60  0000 C CNN
+F 3 "" H 14500 5300 60  0000 C CNN
+	2    14500 5300
+	1    0    0    -1
+$EndComp
+Text GLabel 15250 5300 2    60   Output ~ 0
++RE/I
+Wire Wire Line
+	15250 5300 15100 5300
+Wire Wire Line
+	13900 5150 13800 5150
+Wire Wire Line
+	13800 5150 13800 5300
+Wire Wire Line
+	13800 5300 13800 5450
+Wire Wire Line
+	13800 5450 13900 5450
+Wire Wire Line
+	13650 5300 13800 5300
+Wire Wire Line
+	13800 5300 13900 5300
+Connection ~ 13800 5300
 $EndSCHEMATC

Commit message: mais um trecho da prancha 15
Parts:
- added 2E_P15, 4D_P15: 7400, symbol 7400
- added 3E_P15, 4E_P15: 7402, ~, symbol 7402
- added 4B_P15: 74LS20, symbol 74LS20
- added 4C_P15: 74LS51, symbol 74LS51
- added unit 1 of 5D_P15
- added 5E_P15: 74LS15, symbol 74LS15
Connections:
- net +RI_5: now also 4E_P15.2, 4E_P15.8
- net +RI_6: now also 4D_P15.2
- net +RI_7: now also 4D_P15.1, 4D_P15.5
- net +T34: now also 4C_P15.4
- net -F1: now also 3E_P15.5
- net -F3: now also 2E_P15.9
- net -F4: now also 2E_P15.10
- net -F5: now also 4D_P15.13
- net -MICG2A: now also 3E_P15.6
- net -RI_5: now also 4E_P15.12, 4E_P15.6
- net -RI_6: now also 4D_P15.4
- net GND: now also 2E_P15.7 (GND), 3E_P15.7 (GND), 4B_P15.7 (GND), 4B_P15.7 (GND), 4C_P15.7 (GND), 4D_P15.7 (GND), 4D_P15.7 (GND), 4D_P15.7 (GND), 4E_P15.7 (GND), 4E_P15.7 (GND), 4E_P15.7 (GND), 4E_P15.7 (GND), 5D_P15.7 (GND), 5E_P15.7 (GND), 5E_P15.7 (GND), 5E_P15.7 (GND)
- net VCC: now also 2E_P15.14 (VCC), 3E_P15.14 (VCC), 4B_P15.14 (VCC), 4B_P15.14 (VCC), 4C_P15.14 (VCC), 4D_P15.14 (VCC), 4D_P15.14 (VCC), 4D_P15.14 (VCC), 4E_P15.14 (VCC), 4E_P15.14 (VCC), 4E_P15.14 (VCC), 4E_P15.14 (VCC), 5D_P15.14 (VCC), 5E_P15.14 (VCC), 5E_P15.14 (VCC), 5E_P15.14 (VCC)
- new net: 4B_P15.1, 4B_P15.2, 4B_P15.4, 4B_P15.5, 4C_P15.6
- new net: 4C_P15.2, 4D_P15.11
- new net: 2E_P15.8, 4B_P15.9
- new net: 4B_P15.8, 4D_P15.12
- new net: 4D_P15.6, 4E_P15.11, 4E_P15.9
- new net: 4E_P15.13, 5D_P15.1
- new net: 3E_P15.4, 5D_P15.13, 5E_P15.11, 5E_P15.13, 5E_P15.5
- new net: 4E_P15.10, 5E_P15.9
- new net: 4E_P15.4, 5E_P15.3
- new net: 4D_P15.3, 4E_P15.3, 4E_P15.5
- new net: 4E_P15.1, 5E_P15.1
- new net +(F4.(TRO+TRI)): 4C_P15.5
- new net +PUG: 4B_P15.10
- new net +RE/X,M: 4B_P15.6
- new net +T56: 4C_P15.3
- new net +T7: 5D_P15.2, 5E_P15.10, 5E_P15.2, 5E_P15.4
- new net -CLEAR_OVF: 5E_P15.12
- new net -CLEAR_T: 5E_P15.6
- new net -SET_OVF: 5E_P15.8
- new net -SET_T: 5D_P15.12
Other:
- moved on the sheet: 3B_P15F, 3D_P15C, 5A_P15A, 5B_P15A, 5B_P15B, 5B_P15C, 5C_P15A, 5C_P15B, 5D_P15B
