File: prancha-III.sch (KiCad schematic (older format))
At the start: 0 parts

Commit message: conector de 70 pinos para a interconexão das placas e término do desenho da prancha 5.
Parts:
- added P?: CONN_35X2, symbol CONN_35X2
Connections:
- new net ?: P?.1 (P1), P?.10 (P10), P?.11 (P11), P?.12 (P12), P?.13 (P13), P?.14 (P14), P?.15 (P15), P?.16 (P16), P?.17 (P17), P?.18 (P18), P?.19 (P19), P?.2 (P2)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
