File: prancha-XII.sch (KiCad schematic (older format))
At the start: 0 parts

Commit message: atualizando com Aurelio Heckert
Parts:
- added U? (x2): 7402, ~, symbol 7402
- added U? (x4): 74HC04, ~, symbol 74HC04
- added U? (x4): 74LS10, ~, symbol 74LS10
Connections:
- new net: U?.1, U?.2
- new net: U?.2, U?.2
- new net: U?.1, U?.1
- new net: U?.2, U?.3
- new net: U?.1, U?.12
- new net: U?.12, U?.13
- new net +F1: U?.1, U?.1, U?.1, U?.13, U?.13, U?.13, U?.2, U?.2, U?.2
- new net +PUL: U?.1
- new net -F1: U?.3
- new net GND: U?.7 (GND), U?.7 (GND), U?.7 (GND), U?.7 (GND), U?.7 (GND), U?.7 (GND), U?.7 (GND), U?.7 (GND), U?.7 (GND), U?.7 (GND)
- new net VCC: U?.14 (VCC), U?.14 (VCC), U?.14 (VCC), U?.14 (VCC), U?.14 (VCC), U?.14 (VCC), U?.14 (VCC), U?.14 (VCC), U?.14 (VCC), U?.14 (VCC)
Changed lines of the file:
@@
 $Descr A4 11693 8268
 encoding utf-8
-Sheet 1 17
+Sheet 4 17
 Title ""
-Date "28 jun 2016"
+Date "15 jul 2016"
 Rev ""
 Comp ""
@@
 Comment4 ""
 $EndDescr
+$Comp
+L 7402 U?
+U 1 1 5772BFAE
+P 3700 3100
+F 0 "U?" H 3700 3150 60  0000 C CNN
+F 1 "7402" H 3750 3050 60  0000 C CNN
+F 2 "~" H 3700 3100 60  0000 C CNN
+F 3 "~" H 3700 3100 60  0000 C CNN
+	1    3700 3100
+	1    0    0    -1
+$EndComp
+$Comp
+L 7402 U?
+U 1 1 5772BFBB
+P 6250 3300
+F 0 "U?" H 6250 3350 60  0000 C CNN
+F 1 "7402" H 6300 3250 60  0000 C CNN
+F 2 "~" H 6250 3300 60  0000 C CNN
+F 3 "~" H 6250 3300 60  0000 C CNN
+	1    6250 3300
+	1    0    0    -1
+$EndComp
+$Comp
+L 74HC04 U?
+U 1 1 5772BFC3
+P 2450 2700
+F 0 "U?" H 2600 2800 40  0000 C CNN
+F 1 "74HC04" H 2650 2600 40  0000 C CNN
+F 2 "~" H 2450 2700 60  0000 C CNN
+F 3 "~" H 2450 2700 60  0000 C CNN
+	1    2450 2700
+	1    0    0    -1
+$EndComp
+$Comp
+L 74HC04 U?
+U 1 1 5772BFD0
+P 4950 3650
+F 0 "U?" H 5100 3750 40  0000 C CNN
+F 1 "74HC04" H 5150 3550 40  0000 C CNN
+F 2 "~" H 4950 3650 60  0000 C CNN
+F 3 "~" H 4950 3650 60  0000 C CNN
+	1    4950 3650
+	1    0    0    -1
+$EndComp
+$Comp
+L 74HC04 U?
+U 1 1 5772BFD6
+P 6150 1900
+F 0 "U?" H 6300 2000 40  0000 C CNN
+F 1 "74HC04" H 6350 1800 40  0000 C CNN
+F 2 "~" H 6150 1900 60  0000 C CNN
+F 3 "~" H 6150 1900 60  0000 C CNN
+	1    6150 1900
+	1    0    0    -1
+$EndComp
+$Comp
+L 74HC04 U?
+U 1 1 5772BFDC
+P 8000 2700
+F 0 "U?" H 8150 2800 40  0000 C CNN
+F 1 "74HC04" H 8200 2600 40  0000 C CNN
+F 2 "~" H 8000 2700 60  0000 C CNN
+F 3 "~" H 8000 2700 60  0000 C CNN
+	1    8000 2700
+	1    0    0    -1
+$EndComp
+Text GLabel 1800 2700 0    60   Input ~ 0
++PUL
+Text GLabel 1800 2150 0    60   Input ~ 0
++(PARTIDA.(-RODA))
+Text GLabel 1800 3200 0    60   Input ~ 0
+-F1
+Text GLabel 1800 3500 0    60   Input ~ 0
++F1
+Wire Wire Line
+	1800 2700 2000 2700
+Wire Wire Line
+	1800 3200 3100 3200
+Wire Wire Line
+	2900 2700 3000 2700
+Wire Wire Line
+	3000 2700 3000 3000
+Wire Wire Line
+	3000 3000 3100 3000
+Wire Wire Line
+	3100 3500 1800 3500
+$Comp
+L 74LS10 U?
+U 1 1 5772C019
+P 3700 3650
+F 0 "U?" H 3700 3700 60  0000 C CNN
+F 1 "74LS10" H 3700 3600 60  0000 C CNN
+F 2 "~" H 3700 3650 60  0000 C CNN
+F 3 "~" H 3700 3650 60  0000 C CNN
+	1    3700 3650
+	1    0    0    -1
+$EndComp
+$Comp
+L 74LS10 U?
+U 1 1 5772C030
+P 3700 4200
+F 0 "U?" H 3700 4250 60  0000 C CNN
+F 1 "74LS10" H 3700 4150 60  0000 C CNN
+F 2 "~" H 3700 4200 60  0000 C CNN
+F 3 "~" H 3700 4200 60  0000 C CNN
+	1    3700 4200
+	1    0    0    -1
+$EndComp
+$Comp
+L 74LS10 U?
+U 1 1 5772C036
+P 3700 4750
+F 0 "U?" H 3700 4800 60  0000 C CNN
+F 1 "74LS10" H 3700 4700 60  0000 C CNN
+F 2 "~" H 3700 4750 60  0000 C CNN
+F 3 "~" H 3700 4750 60  0000 C CNN
+	1    3700 4750
+	1    0    0    -1
+$EndComp
+Text GLabel 1800 4050 0    60   Input ~ 0
++F1
+Wire Wire Line
+	3100 4050 1800 4050
+Text GLabel 1800 3650 0    60   Input ~ 0
++F1
+Wire Wire Line
+	3100 3650 1800 3650
+Text GLabel 1800 3800 0    60   Input ~ 0
++F1
+Wire Wire Line
+	3100 3800 1800 3800
+Text GLabel 1800 4200 0    60   Input ~ 0
++F1
+Wire Wire Line
+	3100 4200 1800 4200
+Text GLabel 1800 4350 0    60   Input ~ 0
++F1
+Wire Wire Line
+	3100 4350 1800 4350
+Text GLabel 1800 4600 0    60   Input ~ 0
++F1
+Wire Wire Line
+	3100 4600 1800 4600
+Text GLabel 1800 4750 0    60   Input ~ 0
++F1
+Wire Wire Line
+	3100 4750 1800 4750
+Text GLabel 1800 4900 0    60   Input ~ 0
++F1
+Wire Wire Line
+	3100 4900 1800 4900
+Wire Wire Line
+	4300 3650 4500 3650
+Wire Wire Line
+	5400 3650 5550 3650
+Wire Wire Line
+	5550 3650 5550 3400
+Wire Wire Line
+	5550 3400 5650 3400
+Wire Wire Line
+	4300 3100 5550 3100
+Wire Wire Line
+	5550 3100 5550 3200
+Wire Wire Line
+	5550 3200 5650 3200
+$Comp
+L 74LS10 U?
+U 1 1 5772C080
+P 7800 3700
+F 0 "U?" H 7800 3750 60  0000 C CNN
+F 1 "74LS10" H 7800 3650 60  0000 C CNN
+F 2 "~" H 7800 3700 60  0000 C CNN
+F 3 "~" H 7800 3700 60  0000 C CNN
+	1    7800 3700
+	1    0    0    -1
+$EndComp
+Wire Wire Line
+	7200 3550 7000 3550
+Wire Wire Line
+	7000 3550 7000 3300
+Wire Wire Line
+	7000 3300 6850 3300
+Wire Wire Line
+	7200 3850 7000 3850
+Wire Wire Line
+	7000 3850 7000 4750
+Wire Wire Line
+	7000 4750 4300 4750
 $EndSCHEMATC

Commit message: mais um pedaço de transcrição dos esquematicos
Parts:
- added U? (x5): 7402, ~, symbol 7402
- added U? (x3): 74HC04, ~, symbol 74HC04
- added U?: 74LS10, ~, symbol 74LS10
- added U? (x3): 7400, ~, symbol 7400
- added U?: 74LS13, ~, symbol 74LS13
- added U? (x2): 74LS54, ~, symbol 74LS54
Connections:
- net +(PARTIDA.(-RODA)): now also U?.1
- net +F1: now also U?.1, U?.2, U?.1, U?.1, U?.1, U?.1, U?.1, U?.2, U?.2, U?.2, U?.2, U?.2, U?.3
- net GND: now also U?.7 (GND), U?.7 (GND), U?.7 (GND), U?.7 (GND), U?.7 (GND), U?.7 (GND), U?.7 (GND), U?.7 (GND), U?.7 (GND), U?.7 (GND), U?.7 (GND), U?.7 (GND), U?.7 (GND), U?.7 (GND), U?.7 (GND)
- net VCC: now also U?.14 (VCC), U?.14 (VCC), U?.14 (VCC), U?.14 (VCC), U?.14 (VCC), U?.14 (VCC), U?.14 (VCC), U?.14 (VCC), U?.14 (VCC), U?.14 (VCC), U?.14 (VCC), U?.14 (VCC), U?.14 (VCC), U?.14 (VCC), U?.14 (VCC)
- net at U?.1, U?.1: now also U?.1
- net at U?.2: now also U?.2
- net at U?.2: now also U?.3
- net at U?.12: now also U?.13, U?.2
- net at U?.12: now also U?.2; no longer U?.13
- net at U?.12: now also U?.2, U?.2
- new net: U?.1, U?.1, U?.1
- new net: U?.1, U?.3 (x2)
- new net: U?.2, U?.3 (x2)
- new net: U?.1, U?.1
- new net: U?.2, U?.4
- new net: U?.1, U?.12
- new net: U?.2, U?.5
- new net: U?.13, U?.3
- new net: U?.3, U?.4, U?.4
- new net: U?.10, U?.10, U?.6
- new net +T6: U?.13, U?.13, U?.3, U?.3, U?.5, U?.5, U?.9, U?.9
- new net aaa: U?.1, U?.2, U?.8, U?.8
Other:
- note added: "Este bloco esta com todos lables errados. Falta colocar os nomes certos."
- moved on the sheet: U?A

Commit message: trocando pranchas XII <=> XIII
Parts:
- removed U? (x7): 7402, ~, symbol 7402
- removed U? (x7): 74HC04, ~, symbol 74HC04
- removed U? (x5): 74LS10, ~, symbol 74LS10
- removed U? (x3): 7400, ~, symbol 7400
- removed U?: 74LS13, ~, symbol 74LS13
- removed U? (x2): 74LS54, ~, symbol 74LS54
Other:
- note removed: "Este bloco esta com todos lables errados. Falta colocar os nomes certos."

Commit message: conector de 70 pinos para a interconexão das placas e término do desenho da prancha 5.
Parts:
- added P?: CONN_35X2, symbol CONN_35X2
Connections:
- new net ?: P?.1 (P1), P?.10 (P10), P?.11 (P11), P?.12 (P12), P?.13 (P13), P?.14 (P14), P?.15 (P15), P?.16 (P16), P?.17 (P17), P?.18 (P18), P?.19 (P19), P?.2 (P2), P?.20 (P20), P?.21 (P21), P?.22 (P22), P?.23 (P23), P?.24 (P24), P?.25, P?.26 (P26), P?.27 (P27), P?.28 (P28), P?.29 (P29), P?.3 (P3), P?.30 (P30), P?.31 (P31), P?.32 (P32), P?.33 (P33), P?.34 (P34), P?.35 (P35), P?.36 (P36), P?.37 (P37), P?.38 (P38), P?.39 (P39), P?.4 (P4), P?.40 (P40), P?.41 (P41), P?.42 (P42), P?.43 (P43), P?.44 (P44), P?.45 (P45), P?.46 (P46), P?.47 (P47), P?.48 (P48), P?.49 (P49), P?.5 (P5), P?.50 (P50), P?.51 (P51), P?.52 (P52), P?.53 (P53), P?.54 (P54), P?.55 (P55), P?.56 (P56), P?.57 (P57), P?.58 (P58), P?.59 (P59), P?.6 (P6), P?.60 (P60), P?.61 (P61), P?.62 (P62), P?.63 (P63), P?.64 (P64), P?.65 (P65), P?.66 (P66), P?.67 (P67), P?.68 (P68), P?.69 (P69), P?.7 (P7), P?.70 (P70), P?.8 (P8), P?.9 (P9)
