File: prancha-XIV.sch (KiCad schematic (older format))
At the start: 0 parts

Commit message: wip
Parts:
- added U? (x2): 7402, ~, symbol 7402
- added U?: 74LS10, ~, symbol 74LS10
- added U? (x2): 74LS22, ~, symbol 74LS22
- added U? (x5): 7400, ~, symbol 7400
- added U? (x11): 74HC04, ~, symbol 74HC04
Connections:
- new net: U?.2, U?.6 (x2)
- new net: U?.2, U?.3 (x3)
- new net: U?.1, U?.2 (x6)
- new net: U?.1, U?.12
- new net: U?.1, U?.13
- new net: U?.3, U?.4
- new net: U?.3, U?.5 (x2)
- new net: U?.2, U?.2 (x3)
- new net: U?.2, U?.4
- new net +(PAN+PAZ): U?.1
- new net +CASP: U?.1
- new net +F5: U?.1
- new net +IME: U?.1
- new net +INDICE: U?.1
- new net +MICRO: U?.2
- new net +PLI: U?.1, U?.2
- new net +SAE: U?.1
- new net +SUS: U?.1
- new net +TRI: U?.3
- new net +TRO: U?.2
- new net -CF1: U?.1
- new net -F1: U?.1
- new net -F2: U?.1
- new net -F3: U?.1
- new net -F4: U?.1
- new net GND: U?.7 (GND), U?.7 (GND), U?.7 (GND), U?.7 (GND), U?.7 (GND), U?.7 (GND), U?.7 (GND), U?.7 (GND), U?.7 (GND), U?.7 (GND), U?.7 (GND), U?.7 (GND), U?.7 (GND), U?.7 (GND), U?.7 (GND), U?.7 (GND), U?.7 (GND), U?.7 (GND), U?.7 (GND), U?.7 (GND), U?.7 (GND)
- new net VCC: U?.14 (VCC), U?.14 (VCC), U?.14 (VCC), U?.14 (VCC), U?.14 (VCC), U?.14 (VCC), U?.14 (VCC), U?.14 (VCC), U?.14 (VCC), U?.14 (VCC), U?.14 (VCC), U?.14 (VCC), U?.14 (VCC), U?.14 (VCC), U?.14 (VCC), U?.14 (VCC), U?.14 (VCC), U?.14 (VCC), U?.14 (VCC), U?.14 (VCC), U?.14 (VCC)

Commit message: wip
Parts:
- gave numbers to parts that had none: 8
Connections:
- net +(PAN+PAZ): now also 1A_P14.9; no longer 1A_P14.1
- net +CASP: now also 1A_P14.11; no longer 1A_P14.1
- net +INDICE: now also 1A_P14.3; no longer 1A_P14.1
- net +MICRO: now also 4C_P14.4; no longer 4C_P14.2
- net +PLI: now also 1B_P14.9, 2B_P14.13; no longer 1B_P14.2, 2B_P14.1
- net +SAE: now also 3A_P14.11; no longer 3A_P14.1
- net +SUS: now also 3A_P14.9; no longer 3A_P14.1
- net -CF1: now also 2C_P14.13; no longer 2C_P14.1
- net -F1: now also 1A_P14.13; no longer 1A_P14.1
- net -F2: now also 3A_P14.3; no longer 3A_P14.1
- net -F3: now also 3A_P14.13; no longer 3A_P14.1
- net -F4: now also 3A_P14.5; no longer 3A_P14.1
- net at 2A_P14.1: now also 4C_P14.5; no longer 4C_P14.13
- net at 1B_P14.3: now also 3C_P14.10; no longer 3C_P14.2
- net at 1B_P14.1: now also 3A_P14.12; no longer 3A_P14.2
- net at 1B_P14.2: now also 1B_P14.11; no longer 1B_P14.3
- net at 3C_P14.6: now also 1B_P14.5; no longer 1B_P14.2
- net at 3C_P14.1: now also 2B_P14.11; no longer 1A_P14.2
- net at 3C_P14.2: now also 3A_P14.10; no longer 1A_P14.2
- net at 3C_P14.4: now also 1A_P14.2; no longer 3A_P14.2
- net at 3C_P14.5: now also 1A_P14.8; no longer 2B_P14.3
- net at 3A_P14.2: now also 1B_P14.10; no longer 1B_P14.1
- net +F5 renamed -F5
- new net: 2C_P14.11, 3A_P14.6
- new net: 2C_P14.12, 3C_P14.8
- new net: 1A_P14.12, 4C_P14.3
- new net: 3C_P14.9, 4C_P14.6
- new net: 1B_P14.8, 3C_P14.12
- new net: 1B_P14.6, 3C_P14.13
- new net: 1B_P14.4, 3A_P14.4
- new net: 1A_P14.4, 2B_P14.12
- new net: 1B_P14.13, 3A_P14.8
- new net: 1A_P14.10, 1B_P14.12
Changed lines of the file:
@@
 LIBS:7451
 LIBS:patinhofeio-cache
-EELAYER 27 0
+EELAYER 25 0
 EELAYER END
 $Descr A2 23386 16535
@@
 $EndDescr
 $Comp
-L 7402 U?
-U 1 1 57A0DCE3
+L 7402 2C_P14
+U 4 1 57A0DCE3
 P 20950 3050
-F 0 "U?" H 20950 3100 60  0000 C CNN
+F 0 "2C_P14" H 20950 3100 60  0000 C CNN
 F 1 "7402" H 21000 3000 60  0000 C CNN
 F 2 "~" H 20950 3050 60  0000 C CNN
 F 3 "~" H 20950 3050 60  0000 C CNN
-	1    20950 3050
-	1    0    0    -1
-$EndComp
-$Comp
-L 74LS10 U?
-U 1 1 57A0DD01
+	4    20950 3050
+	1    0    0    1
+$EndComp
+$Comp
+L 74LS10 4C_P14
+U 2 1 57A0DD01
 P 17750 1650
-F 0 "U?" H 17750 1700 60  0000 C CNN
+F 0 "4C_P14" H 17750 1700 60  0000 C CNN
 F 1 "74LS10" H 17750 1600 60  0000 C CNN
 F 2 "~" H 17750 1650 60  0000 C CNN
 F 3 "~" H 17750 1650 60  0000 C CNN
-	1    17750 1650
-	1    0    0    -1
-$EndComp
-$Comp
-L 74LS22 U?
-U 1 1 57A0DD10
+	2    17750 1650
+	1    0    0    -1
+$EndComp
+$Comp
+L 74LS22 3C_P14
+U 2 1 57A0DD10
 P 19450 2950
-F 0 "U?" H 19450 3050 60  0000 C CNN
+F 0 "3C_P14" H 19450 3050 60  0000 C CNN
 F 1 "74LS22" H 19450 2850 60  0000 C CNN
 F 2 "~" H 19450 2950 60  0000 C CNN
 F 3 "~" H 19450 2950 60  0000 C CNN
-	1    19450 2950
-	1    0    0    -1
-$EndComp
-$Comp
-L 7402 U?
+	2    19450 2950
+	1    0    0    -1
+$EndComp
+$Comp
+L 7402 2A_P14
 U 1 1 57A0DD31
 P 16200 1950
-F 0 "U?" H 16200 2000 60  0000 C CNN
+F 0 "2A_P14" H 16200 2000 60  0000 C CNN
 F 1 "7402" H 16250 1900 60  0000 C CNN
 F 2 "~" H 16200 1950 60  0000 C CNN
@@
 $EndComp
 $Comp
-L 7400 U?
+L 7400 1B_P14
 U 1 1 57A0DD37
 P 17750 2550
-F 0 "U?" H 17750 2600 60  0000 C CNN
+F 0 "1B_P14" H 17750 2600 60  0000 C CNN
 F 1 "7400" H 17750 2450 60  0000 C CNN
 F 2 "~" H 17750 2550 60  0000 C CNN
@@
 $EndComp
 $Comp
-L 7400 U?
-U 1 1 57A0DD5B
+L 7400 1B_P14
+U 2 1 57A0DD5B
 P 17750 4000
-F 0 "U?" H 17750 4050 60  0000 C CNN
+F 0 "1B_P14" H 17750 4050 60  0000 C CNN
 F 1 "7400" H 17750 3900 60  0000 C CNN
 F 2 "~" H 17750 4000 60  0000 C CNN
 F 3 "~" H 17750 4000 60  0000 C CNN
-	1    17750 4000
-	1    0    0    -1
-$EndComp
-$Comp
-L 74LS22 U?
+	2    17750 4000
+	1    0    0    -1
+$EndComp
+$Comp
+L 74LS22 3C_P14
 U 1 1 57A0DD6B
 P 16150 4600
-F 0 "U?" H 16150 4700 60  0000 C CNN
+F 0 "3C_P14" H 16150 4700 60  0000 C CNN
 F 1 "74LS22" H 16150 4500 60  0000 C CNN
 F 2 "~" H 16150 4600 60  0000 C CNN
 F 3 "~" H 16150 4600 60  0000 C CNN
 	1    16150 4600
-	1    0    0    -1
-$EndComp
-$Comp
-L 7400 U?
-U 1 1 57A0DD71
+	1    0    0    1
+$EndComp
+$Comp
+L 7400 2B_P14
+U 4 1 57A0DD71
 P 14650 5150
-F 0 "U?" H 14650 5200 60  0000 C CNN
+F 0 "2B_P14" H 14650 5200 60  0000 C CNN
 F 1 "7400" H 14650 5050 60  0000 C CNN
 F 2 "~" H 14650 5150 60  0000 C CNN
 F 3 "~" H 14650 5150 60  0000 C CNN
-	1    14650 5150
-	1    0    0    -1
-$EndComp
-$Comp
-L 74HC04 U?
-U 1 1 57A0DD77
+	4    14650 5150
+	1    0    0    1
+$EndComp
+$Comp
+L 74HC04 3A_P14
+U 5 1 57A0DD77
 P 14600 4650
-F 0 "U?" H 14750 4750 40  0000 C CNN
+F 0 "3A_P14" H 14750 4750 40  0000 C CNN
 F 1 "74HC04" H 14800 4550 40  0000 C CNN
 F 2 "~" H 14600 4650 60  0000 C CNN
 F 3 "~" H 14600 4650 60  0000 C CNN
-	1    14600 4650
-	1    0    0    -1
-$EndComp
-$Comp
-L 74HC04 U?
-U 1 1 57A0DD7D
+	5    14600 4650
+	1    0    0    -1
+$EndComp
+$Comp
+L 74HC04 1A_P14
+U 4 1 57A0DD7D
 P 14600 4150
-F 0 "U?" H 14750 4250 40  0000 C CNN
+F 0 "1A_P14" H 14750 4250 40  0000 C CNN
 F 1 "74HC04" H 14800 4050 40  0000 C CNN
 F 2 "~" H 14600 4150 60  0000 C CNN
 F 3 "~" H 14600 4150 60  0000 C CNN
-	1    14600 4150
-	1    0    0    -1
-$EndComp
-$Comp
-L 74HC04 U?
+	4    14600 4150
+	1    0    0    -1
+$EndComp
+$Comp
+L 74HC04 1A_P14
 U 1 1 57A0DD83
 P 13400 4400
-F 0 "U?" H 13550 4500 40  0000 C CNN
+F 0 "1A_P14" H 13550 4500 40  0000 C CNN
 F 1 "74HC04" H 13600 4300 40  0000 C CNN
 F 2 "~" H 13400 4400 60  0000 C CNN
@@
 $EndComp
 $Comp
-L 74HC04 U?
-U 1 1 57A0DD89
-P 13100 5350
-F 0 "U?" H 13250 5450 40  0000 C CNN
-F 1 "74HC04" H 13300 5250 40  0000 C CNN
-F 2 "~" H 13100 5350 60  0000 C CNN
-F 3 "~" H 13100 5350 60  0000 C CNN
-	1    13100 5350
+L 74HC04 1A_P14
+U 2 1 57A0DD89
+P 13400 5350
+F 0 "1A_P14" H 13550 5450 40  0000 C CNN
+F 1 "74HC04" H 13600 5250 40  0000 C CNN
+F 2 "~" H 13400 5350 60  0000 C CNN
+F 3 "~" H 13400 5350 60  0000 C CNN
+	2    13400 5350
 	1    0    0    -1
 $EndComp
@@
 +INDICE
 Wire Wire Line
-	12650 5350 12450 5350
+	12950 5350 12450 5350
 Text GLabel 12450 5050 0    60   Input ~ 0
 +PLI
@@
 -F4
 Wire Wire Line
-	13550 5350 13800 5350
+	13850 5350 13950 5350
 Wire Wire Line
 	12450 5050 14050 5050
 Wire Wire Line
-	14050 5250 13800 5250
-Wire Wire Line
-	13800 5250 13800 5350
+	14050 5250 13950 5250
+Wire Wire Line
+	13950 5250 13950 5350
 Wire Wire Line
 	15050 4650 15550 4650
@@
 	15400 5150 15250 5150
 $Comp
-L 74HC04 U?
-U 1 1 57A0DDC4
-P 16400 5700
-F 0 "U?" H 16550 5800 40  0000 C CNN
-F 1 "74HC04" H 16600 5600 40  0000 C CNN
-F 2 "~" H 16400 5700 60  0000 C CNN
-F 3 "~" H 16400 5700 60  0000 C CNN
-	1    16400 5700
-	1    0    0    -1
-$EndComp
-Wire Wire Line
-	15950 5700 12450 5700
+L 74HC04 3A_P14
+U 3 1 57A0DDC4
+P 19200 5700
+F 0 "3A_P14" H 19350 5800 40  0000 C CNN
+F 1 "74HC04" H 19400 5600 40  0000 C CNN
+F 2 "~" H 19200 5700 60  0000 C CNN
+F 3 "~" H 19200 5700 60  0000 C CNN
+	3    19200 5700
+	1    0    0    -1
+$EndComp
+Wire Wire Line
+	18750 5700 12450 5700
 Wire Wire Line
 	15550 4550 15150 4550
@@
 	12450 4150 14150 4150
 $Comp
-L 74HC04 U?
-U 1 1 57A0DE33
+L 74HC04 3A_P14
+U 2 1 57A0DE33
 P 13400 3900
-F 0 "U?" H 13550 4000 40  0000 C CNN
+F 0 "3A_P14" H 13550 4000 40  0000 C CNN
 F 1 "74HC04" H 13600 3800 40  0000 C CNN
 F 2 "~" H 13400 3900 60  0000 C CNN
 F 3 "~" H 13400 3900 60  0000 C CNN
-	1    13400 3900
+	2    13400 3900
 	1    0    0    -1
 $EndComp
@@
 +PLI
 $Comp
-L 74HC04 U?
+L 74HC04 3A_P14
 U 1 1 57A0DE74
 P 13400 3300
-F 0 "U?" H 13550 3400 40  0000 C CNN
+F 0 "3A_P14" H 13550 3400 40  0000 C CNN
 F 1 "74HC04" H 13600 3200 40  0000 C CNN
 F 2 "~" H 13400 3300 60  0000 C CNN
@@
 $EndComp
 Text GLabel 12450 3300 0    60   Input ~ 0
-+F5
+-F5
 Wire Wire Line
 	12450 3300 12950 3300
 $Comp
-L 7400 U?
-U 1 1 57A0DE7E
+L 7400 1B_P14
+U 3 1 57A0DE7E
 P 17750 3400
-F 0 "U?" H 17750 3450 60  0000 C CNN
+F 0 "1B_P14" H 17750 3450 60  0000 C CNN
 F 1 "7400" H 17750 3300 60  0000 C CNN
 F 2 "~" H 17750 3400 60  0000 C CNN
 F 3 "~" H 17750 3400 60  0000 C CNN
-	1    17750 3400
-	1    0    0    -1
+	3    17750 3400
+	1    0    0    1
 $EndComp
 Wire Wire Line
@@
 	18600 3400 18350 3400
 Wire Wire Line
-	18350 2550 18600 2700
-Wire Wire Line
-	18600 2700 18600 2900
-Wire Wire Line
 	18600 2900 18850 2900
 Wire Wire Line
@@
 	19800 3150 19800 5700
 Wire Wire Line
-	19800 5700 16850 5700
+	19800 5700 19650 5700
 Text GLabel 21900 3050 2    60   Output ~ 0
 -CF1
@@
 +CASP
 $Comp
-L 74HC04 U?
-U 1 1 57A0E1AB
+L 74HC04 3A_P14
+U 4 1 57A0E1AB
 P 13400 2700
-F 0 "U?" H 13550 2800 40  0000 C CNN
+F 0 "3A_P14" H 13550 2800 40  0000 C CNN
 F 1 "74HC04" H 13600 2600 40  0000 C CNN
 F 2 "~" H 13400 2700 60  0000 C CNN
 F 3 "~" H 13400 2700 60  0000 C CNN
-	1    13400 2700
+	4    13400 2700
 	1    0    0    -1
 $EndComp
@@
 	13850 2700 15650 2700
 $Comp
-L 7400 U?
-U 1 1 57A0E1B5
+L 7400 1B_P14
+U 4 1 57A0E1B5
 P 16250 2800
-F 0 "U?" H 16250 2850 60  0000 C CNN
+F 0 "1B_P14" H 16250 2850 60  0000 C CNN
 F 1 "7400" H 16250 2700 60  0000 C CNN
 F 2 "~" H 16250 2800 60  0000 C CNN
 F 3 "~" H 16250 2800 60  0000 C CNN
-	1    16250 2800
-	1    0    0    -1
-$EndComp
-$Comp
-L 74HC04 U?
-U 1 1 57A0E1BD
+	4    16250 2800
+	1    0    0    1
+$EndComp
+$Comp
+L 74HC04 1A_P14
+U 5 1 57A0E1BD
 P 14600 2900
-F 0 "U?" H 14750 3000 40  0000 C CNN
+F 0 "1A_P14" H 14750 3000 40  0000 C CNN
 F 1 "74HC04" H 14800 2800 40  0000 C CNN
 F 2 "~" H 14600 2900 60  0000 C CNN
 F 3 "~" H 14600 2900 60  0000 C CNN
-	1    14600 2900
+	5    14600 2900
 	1    0    0    -1
 $EndComp
@@
 -F3
 $Comp
-L 74HC04 U?
-U 1 1 57A0E40B
-P 14600 1400
-F 0 "U?" H 14750 1500 40  0000 C CNN
-F 1 "74HC04" H 14800 1300 40  0000 C CNN
-F 2 "~" H 14600 1400 60  0000 C CNN
-F 3 "~" H 14600 1400 60  0000 C CNN
-	1    14600 1400
+L 74HC04 1A_P14
+U 6 1 57A0E40B
+P 13400 1400
+F 0 "1A_P14" H 13550 1500 40  0000 C CNN
+F 1 "74HC04" H 13600 1300 40  0000 C CNN
+F 2 "~" H 13400 1400 60  0000 C CNN
+F 3 "~" H 13400 1400 60  0000 C CNN
+	6    13400 1400
 	1    0    0    -1
 $EndComp
@@
 	12450 2450 14150 2450
 $Comp
-L 74HC04 U?
-U 1 1 57A0E412
+L 74HC04 3A_P14
+U 6 1 57A0E412
 P 14600 2450
-F 0 "U?" H 14750 2550 40  0000 C CNN
+F 0 "3A_P14" H 14750 2550 40  0000 C CNN
 F 1 "74HC04" H 14800 2350 40  0000 C CNN
 F 2 "~" H 14600 2450 60  0000 C CNN
 F 3 "~" H 14600 2450 60  0000 C CNN
-	1    14600 2450
+	6    14600 2450
 	1    0    0    -1
 $EndComp
@@
 +TRI
 Wire Wire Line
-	12450 2050 14550 2050
+	12450 2050 15600 2050
 Text GLabel 12450 1850 0    60   Input ~ 0
 +TRO
@@
 -F1
 Wire Wire Line
-	12450 1400 14150 1400
-Wire Wire Line
-	15600 2050 14550 2050
+	12450 1400 12950 1400
 Wire Wire Line
 	14550 2050 14550 2050
@@
 	17000 1950 16800 1950
 Wire Wire Line
-	15050 1400 16200 1400
+	13850 1400 16200 1400
 Wire Wire Line
 	16200 1400 16200 1500
@@
 Wire Wire Line
 	18700 1650 18350 1650
+Wire Wire Line
+	18600 2900 18600 2550
+Wire Wire Line
+	18600 2550 18350 2550
 $EndSCHEMATC

Commit message: mais um trecho do esquemático
Parts:
- added unit 3 of 1A_P14
- added 1C_P14: 74LS22, ~, symbol 74LS22
- added unit 2 of 2A_P14
- added unit 4 of 2A_P14
- added unit 3 of 2A_P14
- added unit 1 of 2B_P14
- added unit 2 of 2C_P14
- added unit 3 of 2C_P14
- added unit 1 of 2C_P14
- added 3D_P14, 4B_P14: 7400, ~, symbol 7400
- added 4A_P14: 74HC04, ~, symbol 74HC04
Connections:
- net +SUS: now also 2A_P14.8
- net -F3: now also 2C_P14.3
- net -F5: now also 1C_P14.13
- net GND: now also 1A_P14.7 (GND), 1C_P14.7 (GND), 2A_P14.7 (GND), 2A_P14.7 (GND), 2A_P14.7 (GND), 2B_P14.7 (GND), 2C_P14.7 (GND), 2C_P14.7 (GND), 2C_P14.7 (GND), 3D_P14.7 (GND), 4A_P14.7 (GND), 4B_P14.7 (GND)
- net VCC: now also 1A_P14.14 (VCC), 1C_P14.14 (VCC), 2A_P14.14 (VCC), 2A_P14.14 (VCC), 2A_P14.14 (VCC), 2B_P14.14 (VCC), 2C_P14.14 (VCC), 2C_P14.14 (VCC), 2C_P14.14 (VCC), 3D_P14.14 (VCC), 4A_P14.14 (VCC), 4B_P14.14 (VCC)
- new net: 1C_P14.12, 2B_P14.3
- new net: 1C_P14.8, 2C_P14.5, 3D_P14.13
- new net: 1C_P14.9, 2A_P14.4
- new net: 2A_P14.13, 2B_P14.2
- new net: 2C_P14.4, 2C_P14.9
- new net: 2C_P14.1, 2C_P14.6
- new net: 2A_P14.10, 2C_P14.2
- new net: 1A_P14.6, 2A_P14.9
- new net +(CAC+SOM): 4B_P14.13
- new net +F3: 4B_P14.12
- new net +L/R: 2C_P14.10
- new net +MP: 2B_P14.1
- new net +RODA: 2A_P14.11
- new net +T0123: 3D_P14.12
- new net -M4: 3D_P14.11
- new net -PARTIDA: 2A_P14.12
- new net -T12: 2C_P14.8
- new net 1A_P14_12: 2A_P14.5
- new net 2A_P14_1: 1A_P14.5
- new net 3A_P14_4: 2A_P14.6
- new net 4B_P14_11: 1C_P14.10, 4A_P14.9, 4B_P14.11

Commit message: mais um pedação do esquemático (prancha XIV)
Parts:
- added unit 1 of 1C_P14
- added unit 2 of 2B_P14
- added 2E_P14: 74LS10, ~, symbol 74LS10
- added 3B_P14: 7400, ~, symbol 7400
- added 3E_P14: 7460, symbol 7460
- added unit 6 of 4A_P14
- added unit 5 of 4A_P14
- added unit 2 of 4A_P14
- added unit 2 of 4B_P14
- added unit 1 of 4B_P14
- added 4E_P14: 7453, symbol 7453
Connections:
- net 1A_P14_12 is gone; now on net +F1: 2A_P14.5
- net 2A_P14_1 is gone; now on net -(TRO+TRI): 1A_P14.5
- net 3A_P14_4 is gone; now on net +F2: 2A_P14.6
- net +F3: now also 1B_P14.1, 3A_P14.12, 3B_P14.10, 4B_P14.4
- net -F2: now also 1C_P14.2
- net -F4: now also 2E_P14.1
- net -F5: now also 1C_P14.4
- net GND: now also 1C_P14.7 (GND), 2B_P14.7 (GND), 2E_P14.7 (GND), 3B_P14.7 (GND), 3B_P14.7 (GND), 3B_P14.7 (GND), 3E_P14.7 (GND), 4A_P14.7 (GND), 4A_P14.7 (GND), 4A_P14.7 (GND), 4B_P14.7 (GND), 4B_P14.7 (GND), 4E_P14.2, 4E_P14.3, 4E_P14.4, 4E_P14.5, 4E_P14.7 (GND)
- net VCC: now also 1C_P14.14 (VCC), 2B_P14.14 (VCC), 2E_P14.14 (VCC), 3B_P14.14 (VCC), 3B_P14.14 (VCC), 3B_P14.14 (VCC), 3E_P14.14 (VCC), 3E_P14.8, 4A_P14.14 (VCC), 4A_P14.14 (VCC), 4A_P14.14 (VCC), 4B_P14.14 (VCC), 4B_P14.14 (VCC), 4E_P14.14 (VCC)
- net +F1: now reaches 1A_P14.12, 4C_P14.3
- net -(TRO+TRI): now reaches 2A_P14.1, 4C_P14.5
- net +F2: now reaches 1B_P14.4, 3A_P14.4
- net at 4A_P14.8: now also 3B_P14.2
- net -(PARTIDA+RODA): now reaches 2A_P14.13, 2B_P14.2
- net -(PARTIDA+RODA): now also 2B_P14.4
- net +(F3.(TRO+TRI+SUS)): now reaches 2C_P14.1, 2C_P14.6
- net +(F3.(TRO+TRI+SUS)): now also 3B_P14.3
- net -PARTIDA renamed +PARTIDA
- net 4B_P14_11 renamed -(F3.(CAC+SOM))
- new net: 1C_P14.1, 3B_P14.1
- new net: 1C_P14.6, 4E_P14.13
- new net: 3B_P14.6, 3B_P14.8
- new net: 3B_P14.5, 4A_P14.12
- new net: 3E_P14.10, 4E_P14.11 (Ve)
- new net: 3E_P14.9, 4E_P14.12 (Vc)
- new net: 2E_P14.12, 4E_P14.9
- new net: 3B_P14.4, 3E_P14.6
- new net: 2B_P14.6, 2E_P14.13
- new net: 2E_P14.2, 4B_P14.6
- new net: 4B_P14.3, 4B_P14.5
- new net: 4A_P14.10, 4B_P14.1
- new net: 4A_P14.4, 4B_P14.2
- new net +ARA: 4A_P14.3
- new net +CP: 2B_P14.5
- new net +PUG: 4A_P14.11
- new net +T1: 4E_P14.1
- new net +T2: 4E_P14.10
- new net +T3: 3E_P14.5
- new net -C_RD: 4E_P14.8
- new net -RDZ: 4A_P14.13
- new net -SUS: 3B_P14.9
- new net -T(1/2)34: 3E_P14.4
- new net 2B3: 1C_P14.5
Other:
- note added: "-(TRO+TRI+SUS)"
- moved on the sheet: 1A_P14A, 1A_P14B, 1A_P14D, 1A_P14E, 1A_P14F, 1B_P14A, 1B_P14B, 1B_P14C, 1B_P14D, 2A_P14A, 2B_P14D, 2C_P14D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

Commit message: transcricao de mais um pouco do esquematico (prancha XIV)
Parts:
- added 1D_P14: 74LS51, symbol 74LS51
- added 1E_P14: 7400, ~, symbol 7400
- added unit 3 of 2B_P14
- added unit 1 of 3D_P14
- added unit 3 of 3D_P14
- added 4D_P14: 74LS10, ~, symbol 74LS10
- renumbered 3B_P14 to 4B_P14
Connections:
- net +(CAC+SOM): now also 1E_P14.13
- net +F3: now also 1E_P14.10, 3D_P14.9
- net -F4: now also 4D_P14.11
- net GND: now also 1D_P14.7 (GND), 1E_P14.7 (GND), 1E_P14.7 (GND), 1E_P14.7 (GND), 1E_P14.7 (GND), 2B_P14.7 (GND), 3D_P14.7 (GND), 3D_P14.7 (GND), 4D_P14.7 (GND)
- net VCC: now also 1D_P14.14 (VCC), 1E_P14.12, 1E_P14.14 (VCC), 1E_P14.14 (VCC), 1E_P14.14 (VCC), 1E_P14.14 (VCC), 2B_P14.14 (VCC), 3D_P14.14 (VCC), 3D_P14.14 (VCC), 4D_P14.14 (VCC)
- net +(TRO+TRI): now reaches 1A_P14.6, 2A_P14.9
- net +(TRO+TRI): now also 1E_P14.9
- net (-F3)+SUS: now reaches 3B_P14.6, 4B_P14.8
- net (-F3)+SUS: now also 2B_P14.10, 2B_P14.9
- net 2E_P14_12: now reaches 2E_P14.12, 4E_P14.9
- net 2E_P14_12: now also 1E_P14.1
- net PARTIDA+RODA+(-CP): now reaches 2B_P14.6, 2E_P14.13
- net PARTIDA+RODA+(-CP): now also 4D_P14.10
- new net: 1E_P14.11, 3D_P14.10
- new net: 3D_P14.2, 4D_P14.8
- new net: 3D_P14.8, 4D_P14.9
- new net: 1E_P14.5, 1E_P14.8
- new net: 1E_P14.3, 1E_P14.4
- new net: 1D_P14.2, 1E_P14.6
- new net: 1D_P14.4, 2B_P14.8
- new net +T(1/2)34: 1D_P14.5
- new net +T012: 3D_P14.1
- new net +T34: 1D_P14.3
- new net -M1: 3D_P14.3
- new net -M3: 1D_P14.6
Other:
- note added: "PUG+ARA"
- moved on the sheet: 1A_P14C, 1C_P14B, 2A_P14B, 2A_P14C, 2A_P14D, 2B_P14A, 2C_P14A, 2C_P14B, 2C_P14C, 3D_P14D, 3E_P14B, 4B_P14D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

Commit message: finalizei a transcrição da prancha XIV! E gerei um PDF dos esquemáticos (incompletos).
Parts:
- added 2D_P14, 5B_P14: 7400, ~, symbol 7400
- added unit 3 of 2E_P14
- added unit 2 of 2E_P14
- added unit 4 of 3B_P14
- added unit 3 of 3B_P14
- added unit 2 of 3D_P14
- added unit 1 of 4A_P14
- added unit 3 of 4A_P14
- added unit 1 of 4C_P14
- added unit 3 of 4C_P14
- added unit 1 of 4D_P14
- added unit 2 of 4D_P14
- added 5A_P14: 74LS10, ~, symbol 74LS10
- added 5C_P14, 5D_P14, 5E_P14: 74LS22, ~, symbol 74LS22
Connections:
- net +F2: now also 4C_P14.13, 5A_P14.13, 5A_P14.3
- net +SAE: now also 5A_P14.4
- net +T3: now also 2E_P14.3, 5A_P14.2
- net -F2: now also 3B_P14.12
- net -T(1/2)34: now also 2E_P14.5
- net GND: now also 2D_P14.7 (GND), 2D_P14.7 (GND), 2D_P14.7 (GND), 2D_P14.7 (GND), 2E_P14.7 (GND), 2E_P14.7 (GND), 3B_P14.7 (GND), 3B_P14.7 (GND), 3D_P14.7 (GND), 4A_P14.7 (GND), 4A_P14.7 (GND), 4C_P14.7 (GND), 4C_P14.7 (GND), 4D_P14.7 (GND), 4D_P14.7 (GND), 5A_P14.7 (GND), 5A_P14.7 (GND), 5A_P14.7 (GND), 5B_P14.7 (GND), 5B_P14.7 (GND), 5B_P14.7 (GND), 5B_P14.7 (GND), 5C_P14.7 (GND), 5C_P14.7 (GND), 5D_P14.7 (GND), 5D_P14.7 (GND), 5E_P14.7 (GND), 5E_P14.7 (GND)
- net VCC: now also 1E_P14.2, 2D_P14.14 (VCC), 2D_P14.14 (VCC), 2D_P14.14 (VCC), 2D_P14.14 (VCC), 2E_P14.10, 2E_P14.11, 2E_P14.14 (VCC), 2E_P14.14 (VCC), 3B_P14.14 (VCC), 3B_P14.14 (VCC), 3D_P14.14 (VCC), 4A_P14.14 (VCC), 4A_P14.14 (VCC), 4C_P14.14 (VCC), 4C_P14.14 (VCC), 4D_P14.14 (VCC), 4D_P14.14 (VCC), 5A_P14.11, 5A_P14.14 (VCC), 5A_P14.14 (VCC), 5A_P14.14 (VCC), 5B_P14.14 (VCC), 5B_P14.14 (VCC), 5B_P14.14 (VCC), 5B_P14.14 (VCC), 5C_P14.14 (VCC), 5C_P14.14 (VCC), 5D_P14.14 (VCC), 5D_P14.14 (VCC), 5E_P14.1, 5E_P14.10, 5E_P14.12, 5E_P14.14 (VCC), 5E_P14.14 (VCC), 5E_P14.2
- net +RDZ: now reaches 3B_P14.5, 4A_P14.12
- net +RDZ: now also 5B_P14.13
- net +(F3.(-SUS)): now reaches 1D_P14.4, 2B_P14.8
- net +(F3.(-SUS)): now also 5B_P14.12
- new net: 2E_P14.8, 4C_P14.2
- new net: 4C_P14.12, 5B_P14.9
- new net: 5B_P14.10, 5B_P14.11
- new net: 2E_P14.4, 5B_P14.8
- new net: 2E_P14.6, 5A_P14.10
- new net: 5A_P14.9, 5B_P14.6
- new net: 5A_P14.12, 5B_P14.2
- new net: 5B_P14.3, 5E_P14.9
- new net: 5A_P14.6, 5E_P14.4
- new net: 3D_P14.6, 5E_P14.5
- new net: 2D_P14.13, 2D_P14.3, 2D_P14.4, 4C_P14.11, 4D_P14.13, 4D_P14.3
- new net: 2D_P14.2, 2D_P14.6
- new net: 2D_P14.11, 3B_P14.8, 3B_P14.9
- new net: 2D_P14.12, 3B_P14.13, 4C_P14.9, 4D_P14.2, 4D_P14.5
- new net: 4D_P14.12, 5C_P14.1, 5C_P14.2, 5C_P14.4, 5C_P14.5
- new net: 2D_P14.8, 4D_P14.4
- new net: 4D_P14.6, 5D_P14.10, 5D_P14.12, 5D_P14.13, 5D_P14.9
- new net: 4C_P14.8, 5D_P14.1, 5D_P14.2, 5D_P14.4, 5D_P14.5
- new net: 2D_P14.9, 4A_P14.2
- new net: 3B_P14.11, 4A_P14.6
- new net: 3B_P14.10, 5C_P14.10, 5C_P14.12, 5C_P14.13, 5C_P14.9
- new net +5: 5A_P14.8, 5B_P14.4
- new net +DUPL_SINAL: 5D_P14.6
- new net +RD_0: 4A_P14.1, 4C_P14.10
- new net +RD_1: 2D_P14.10, 4D_P14.1
- new net +SAEFU: 5A_P14.1
- new net +SAESA: 4C_P14.1
- new net +SHIFT: 4A_P14.5
- new net +SHIFT_LEFT: 5C_P14.6
- new net +SHIFT_RIGHT: 5D_P14.8
- new net +T0: 5A_P14.5
- new net -FUNÇÃO: 5B_P14.1, 5E_P14.8
- new net -SENTIDO: 2E_P14.9
- new net -SHIAC: 5C_P14.8
- new net -T70: 2D_P14.5, 3D_P14.5, 5B_P14.5, 5E_P14.13
- new net =T2: 2D_P14.1
- new net MANEN: 3D_P14.4, 5E_P14.6
Other:
- note added: "+SENTIDO"
- moved on the sheet: 1A_P14A, 1A_P14B, 1A_P14C, 1A_P14D, 1A_P14E, 1A_P14F, 1B_P14A, 1B_P14B, 1B_P14C, 1B_P14D, 1C_P14A, 1C_P14B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

Commit message: conector de 70 pinos para a interconexão das placas e término do desenho da prancha 5.
Parts:
- added P?: CONN_35X2, symbol CONN_35X2
- added U?: 74LS54, symbol 74LS54
Connections:
- net GND: now also U?.7 (GND)
- net VCC: now also U?.14 (VCC)
- new net ?: P?.1 (P1), P?.10 (P10), P?.11 (P11), P?.12 (P12), P?.13 (P13), P?.14 (P14), P?.15 (P15), P?.16 (P16), P?.17 (P17), P?.18 (P18), P?.19 (P19), P?.2 (P2), P?.20 (P20), P?.21 (P21), P?.22 (P22), P?.23 (P23), P?.24 (P24), P?.25, P?.26 (P26), P?.27 (P27), P?.28 (P28), P?.29 (P29), P?.3 (P3), P?.30 (P30), P?.31 (P31), P?.32 (P32), P?.33 (P33), P?.34 (P34), P?.35 (P35), P?.36 (P36), P?.37 (P37), P?.38 (P38), P?.39 (P39), P?.4 (P4), P?.40 (P40), P?.41 (P41), P?.42 (P42), P?.43 (P43), P?.44 (P44), P?.45 (P45), P?.46 (P46), P?.47 (P47), P?.48 (P48), P?.49 (P49), P?.5 (P5), P?.50 (P50), P?.51 (P51), P?.52 (P52), P?.53 (P53), P?.54 (P54), P?.55 (P55), P?.56 (P56), P?.57 (P57), P?.58 (P58), P?.59 (P59), P?.6 (P6), P?.60 (P60), P?.61 (P61), P?.62 (P62), P?.63 (P63), P?.64 (P64), P?.65 (P65), P?.66 (P66), P?.67 (P67), P?.68 (P68), P?.69 (P69), P?.7 (P7), P?.70 (P70), P?.8 (P8), P?.9 (P9)
Other:
- moved on the sheet: 1A_P14A, 1A_P14B, 1A_P14C, 1A_P14D, 1A_P14E, 1A_P14F, 1B_P14A, 1B_P14B, 1B_P14C, 1B_P14D, 1C_P14A, 1C_P14B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
