File: prancha-V.sch (KiCad schematic (older format))
At the start: 0 parts

Commit message: conector de 70 pinos para a interconexão das placas e término do desenho da prancha 5.
Parts:
- added 3A_P5, 3B_P5, 4B_P5: 74LS04, symbol 74LS04
- added 4C_P5, 5A_P5: 74LS11, symbol 74LS11
- added 5B_P5: 7400, symbol 7400
- added 5C_P5: 74LS08, symbol 74LS08
- added CONECTOR_P5: CONN_35X2, symbol CONN_35X2
- added R10_P5, R11_P5, R3_P5, R4_P5, R5_P5, R6_P5, R8_P5, R9_P5: R, symbol R
Connections:
- new net: 4B_P5.2, 4C_P5.9
- new net: 3B_P5.12, 4C_P5.4
- new net: 3B_P5.10, 4C_P5.5
- new net: 4C_P5.2, 4C_P5.6
- new net: 4C_P5.13, 4C_P5.8
- new net: 4B_P5.12, 4C_P5.11
- new net: 5A_P5.1, 5B_P5.3
- new net: 5A_P5.13, 5B_P5.8
- new net: 4B_P5.10, 5A_P5.5
- new net: 4B_P5.8, 5A_P5.4
- new net: 5A_P5.3, 5A_P5.9, 5C_P5.8
- new net: 5A_P5.10, 5A_P5.11, 5A_P5.12
- new net -I_0: 3B_P5.5, CONECTOR_P5.57 (P57)
- new net -I_1: 4B_P5.3, CONECTOR_P5.24 (P24)
- new net -I_2: 3B_P5.13, CONECTOR_P5.58 (P58)
- new net -I_3: 3B_P5.11, CONECTOR_P5.23 (P23)
- new net -I_4: 4B_P5.1, CONECTOR_P5.59 (P59)
- new net -LAL1: 5C_P5.9, CONECTOR_P5.68 (P68)
- new net -LCL: 5A_P5.2, 5B_P5.11, CONECTOR_P5.32 (P32)
- new net -LHC: 5B_P5.6, CONECTOR_P5.29 (P29)
- new net -M1: 5B_P5.13, CONECTOR_P5.67 (P67)
- new net -M3: 4B_P5.9, CONECTOR_P5.64 (P64)
- new net -M4: 5B_P5.10, 5B_P5.12, 5B_P5.2, 5B_P5.4, 5B_P5.5, CONECTOR_P5.66 (P66)
- new net -T70: 5B_P5.9, CONECTOR_P5.65 (P65)
- new net FN: 5C_P5.10, CONECTOR_P5.69 (P69)
- new net GND: 3A_P5.7 (GND), 3A_P5.7 (GND), 3A_P5.7 (GND), 3A_P5.7 (GND), 3A_P5.7 (GND), 3A_P5.7 (GND), 3B_P5.7 (GND), 3B_P5.7 (GND), 3B_P5.7 (GND), 3B_P5.7 (GND), 3B_P5.7 (GND), 4B_P5.7 (GND), 4B_P5.7 (GND), 4B_P5.7 (GND), 4B_P5.7 (GND), 4B_P5.7 (GND), 4C_P5.7 (GND), 4C_P5.7 (GND), 4C_P5.7 (GND), 5A_P5.7 (GND), 5A_P5.7 (GND), 5A_P5.7 (GND), 5B_P5.7 (GND), 5B_P5.7 (GND), 5B_P5.7 (GND), 5B_P5.7 (GND), 5C_P5.7 (GND), CONECTOR_P5.2 (P2), CONECTOR_P5.3 (P3), CONECTOR_P5.31 (P31), CONECTOR_P5.33 (P33), CONECTOR_P5.4 (P4), CONECTOR_P5.5 (P5), CONECTOR_P5.6 (P6), CONECTOR_P5.7 (P7), CONECTOR_P5.8 (P8), CONECTOR_P5.9 (P9)
- new net LSB1-12: 3B_P5.6, 4C_P5.3, CONECTOR_P5.22 (P22)
- new net LSB2-13: 4B_P5.4, 4C_P5.10, CONECTOR_P5.60 (P60)
- new net LWBI_0: 3B_P5.2, CONECTOR_P5.14 (P14)
- new net LWBI_1: 3B_P5.4, CONECTOR_P5.15 (P15)
- new net LWBI_2: 3A_P5.4, CONECTOR_P5.51 (P51)
- new net LWBI_3: 3A_P5.6, CONECTOR_P5.52 (P52)
- new net LWBI_4: 3A_P5.2, CONECTOR_P5.18 (P18)
- new net LWBI_5: 3A_P5.8, CONECTOR_P5.54 (P54)
- new net LWBI_6: 3A_P5.10, CONECTOR_P5.55 (P55)
- new net LWBI_7: 3A_P5.12, CONECTOR_P5.56 (P56)
- new net LWBO_0: CONECTOR_P5.13 (P13), CONECTOR_P5.37 (P37), R3_P5.2
- new net LWBO_1: CONECTOR_P5.12 (P12), R4_P5.2
- new net LWBO_2: CONECTOR_P5.11 (P11), R5_P5.2
- new net LWBO_3: CONECTOR_P5.10 (P10), R6_P5.2
- new net LWBO_4: CONECTOR_P5.48 (P48), R11_P5.2
- new net LWBO_5: CONECTOR_P5.47 (P47), R10_P5.2
- new net LWBO_6: CONECTOR_P5.46 (P46), R9_P5.2
- new net LWBO_7: CONECTOR_P5.45 (P45), R8_P5.2
- new net PROT: 4C_P5.1, CONECTOR_P5.25
- new net PST: 5A_P5.8, CONECTOR_P5.34 (P34)
- new net PUP: 4B_P5.11, 4C_P5.12, 5B_P5.1
- new net PW: 5A_P5.6, CONECTOR_P5.30 (P30)
- new net RD_0: 3B_P5.1, CONECTOR_P5.49 (P49)
- new net RD_1: 3B_P5.3, CONECTOR_P5.50 (P50)
- new net RD_2: 3A_P5.3, CONECTOR_P5.16 (P16)
- new net RD_3: 3A_P5.5, CONECTOR_P5.17 (P17)
- new net RD_4: 3A_P5.1, CONECTOR_P5.53 (P53)
- new net RD_5: 3A_P5.9, CONECTOR_P5.19 (P19)
- new net RD_6: 3A_P5.11, CONECTOR_P5.20 (P20)
- new net RD_7: 3A_P5.13, CONECTOR_P5.21 (P21)
- new net TERRA: 4B_P5.13, CONECTOR_P5.61 (P61)
- new net VCC: 3A_P5.14 (VCC), 3A_P5.14 (VCC), 3A_P5.14 (VCC), 3A_P5.14 (VCC), 3A_P5.14 (VCC), 3A_P5.14 (VCC), 3B_P5.14 (VCC), 3B_P5.14 (VCC), 3B_P5.14 (VCC), 3B_P5.14 (VCC), 3B_P5.14 (VCC), 4B_P5.14 (VCC), 4B_P5.14 (VCC), 4B_P5.14 (VCC), 4B_P5.14 (VCC), 4B_P5.14 (VCC), 4C_P5.14 (VCC), 4C_P5.14 (VCC), 4C_P5.14 (VCC), 5A_P5.14 (VCC), 5A_P5.14 (VCC), 5A_P5.14 (VCC), 5B_P5.14 (VCC), 5B_P5.14 (VCC), 5B_P5.14 (VCC), 5B_P5.14 (VCC), 5C_P5.14 (VCC), R10_P5.1, R11_P5.1, R3_P5.1, R4_P5.1, R5_P5.1, R6_P5.1, R8_P5.1, R9_P5.1
- no-connect marks 0 -> 16
Other:
- note added: "LSB1-34"
- note added: "LSB2-24"
