File: patinhofeio.kicad_sch (KiCad schematic)
At the start: 0 parts

Commit message: FS1-3 + FS2-4
Changed lines of the file:
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@@
+	(text "OK"
+		(exclude_from_sim no)
+		(at 64.77 54.102 0)
+		(effects
+			(font
+				(size 2.9972 2.9972)
+			)
+			(justify left bottom)
+		)
+	)
 	(text "OK"
 		(exclude_from_sim no)
@@
 			)
 			(justify left bottom)
-		)
-	)
-	(text "WIP"
-		(exclude_from_sim no)
-		(at 65.278 53.34 0)
-		(effects
-			(font
-				(size 1.524 1.524)
-			)
-			(justify left bottom)

Commit message: FR1/FR2 + FS1/FS2
Other:
- note removed: "TO-DO!"
Changed lines of the file:
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@@
 		)
 	)
-	(text "TO-DO!"
+	(text "OK"
 		(exclude_from_sim no)
-		(at 63.5 36.83 0)
+		(at 66.294 36.068 0)
 		(effects
 			(font
