File: patinhofeio.kicad_sch (KiCad schematic)
At the start: 0 parts

Commit message: FAC-5
Other:
- note removed: "WIP"
Changed lines of the file:
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@@
 		)
 	)
-	(text "WIP"
+	(text "OK"
 		(exclude_from_sim no)
 		(at 65.786 68.834 0)

Commit message: cleaning up references
Other:
- note removed: "OK"
Changed lines of the file:
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@@
 		(comment 4 "Re-desenho: Felipe Sanches")
-	)
-	(text "OK"
-		(exclude_from_sim no)
-		(at 176.53 100.33 0)
-		(effects
-			(font
-				(size 2.9972 2.9972)
-			)
-			(justify left bottom)
-		)
 	)
 	(text "Placa:\n* CT3-6"
@@
 			(font
 				(size 1.524 1.524)
-			)
-			(justify left bottom)
-		)
-	)
-	(text "OK"
-		(exclude_from_sim no)
-		(at 177.038 87.376 0)
-		(effects
-			(font
-				(size 2.9972 2.9972)
 			)
 			(justify left bottom)
@@
 		)
 	)
-	(text "OK"
-		(exclude_from_sim no)
-		(at 64.77 54.102 0)
-		(effects
-			(font
-				(size 2.9972 2.9972)
-			)
-			(justify left bottom)
-		)
-	)
-	(text "OK"
-		(exclude_from_sim no)
-		(at 64.77 83.82 0)
-		(effects
-			(font
-				(size 2.9972 2.9972)
-			)
-			(justify left bottom)
-		)
-	)
 	(text "Placa:\n* FM1-6 (mais-um e porta de seleção 6)"
 		(exclude_from_sim no)
@@
 			(font
 				(size 1.524 1.524)
-			)
-			(justify left bottom)
-		)
-	)
-	(text "OK"
-		(exclude_from_sim no)
-		(at 176.53 34.29 0)
-		(effects
-			(font
-				(size 2.9972 2.9972)
-			)
-			(justify left bottom)
-		)
-	)
-	(text "OK"
-		(exclude_from_sim no)
-		(at 176.53 133.35 0)
-		(effects
-			(font
-				(size 2.9972 2.9972)
 			)
 			(justify left bottom)
@@
 		)
 	)
-	(text "OK"
-		(exclude_from_sim no)
-		(at 65.786 68.834 0)
-		(effects
-			(font
-				(size 1.524 1.524)
-			)
-			(justify left bottom)
-		)
-	)
 	(text "Placa:\n* CT2-5"
 		(exclude_from_sim no)
 		(at 191.77 100.33 0)
-		(effects
-			(font
-				(size 1.524 1.524)
-			)
-			(justify left bottom)
-		)
-	)
-	(text "OK"
-		(exclude_from_sim no)
-		(at 176.53 50.8 0)
-		(effects
-			(font
-				(size 2.9972 2.9972)
-			)
-			(justify left bottom)
-		)
-	)
-	(text "OK"
-		(exclude_from_sim no)
-		(at 63.5 175.26 0)
 		(effects
 			(font
@@
 		)
 	)
-	(text "OK"
-		(exclude_from_sim no)
-		(at 176.53 149.86 0)
-		(effects
-			(font
-				(size 2.9972 2.9972)
-			)
-			(justify left bottom)
-		)
-	)
 	(text "Placa:\n* CRC-1"
 		(exclude_from_sim no)
@@
 			(font
 				(size 1.524 1.524)
-			)
-			(justify left bottom)
-		)
-	)
-	(text "OK"
-		(exclude_from_sim no)
-		(at 176.53 116.84 0)
-		(effects
-			(font
-				(size 2.9972 2.9972)
 			)
 			(justify left bottom)
@@
 			(font
 				(size 1.524 1.524)
-			)
-			(justify left bottom)
-		)
-	)
-	(text "OK"
-		(exclude_from_sim no)
-		(at 64.77 120.65 0)
-		(effects
-			(font
-				(size 2.9972 2.9972)
 			)
 			(justify left bottom)
@@
 		)
 	)
-	(text "OK"
-		(exclude_from_sim no)
-		(at 63.5 160.02 0)
-		(effects
-			(font
-				(size 1.524 1.524)
-			)
-			(justify left bottom)
-		)
-	)
-	(text "OK"
-		(exclude_from_sim no)
-		(at 64.77 101.6 0)
-		(effects
-			(font
-				(size 2.9972 2.9972)
-			)
-			(justify left bottom)
-		)
-	)
 	(text "Placa:\n* FIN-8 (sinais para cartões de interface)"
 		(exclude_from_sim no)
@@
 		(effects
 			(font
-				(size 1.524 1.524)
-			)
-			(justify left bottom)
-		)
-	)
-	(text "OK"
-		(exclude_from_sim no)
-		(at 66.294 36.068 0)
-		(effects
-			(font

Commit message: wip + PDF plot
Changed lines of the file:
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@@
+		)
+	)
+	(text "W.I.P."
+		(exclude_from_sim no)
+		(at 61.722 86.614 0)
+		(effects
+			(font
+				(size 2.9972 2.9972)
+			)
+			(justify left bottom)
 		)
 	)
@@
 		)
 	)
+	(text "W.I.P."
+		(exclude_from_sim no)
+		(at 60.96 103.632 0)
+		(effects
+			(font
+				(size 2.9972 2.9972)
+			)
+			(justify left bottom)
+		)
+	)
 	(text "Placa:\n* CT2-5"
 		(exclude_from_sim no)
@@
 		)
 	)
+	(text "W.I.P."
+		(exclude_from_sim no)
+		(at 171.958 66.802 0)
+		(effects
+			(font
+				(size 3.302 3.302)
+				(thickness 0.6604)
+				(bold yes)
+			)
+			(justify left bottom)
+		)
+	)
 	(text "UNIDADE DE CONTROLE"
 		(exclude_from_sim no)
@@
 	(text "W.I.P."
 		(exclude_from_sim no)
-		(at 173.99 66.04 0)
+		(at 173.99 100.838 0)
 		(effects
 			(font
@@
 			)
 			(justify left bottom)
+		)
+	)
+	(text "W.I.P."
+		(exclude_from_sim no)
+		(at 174.498 118.364 0)
+		(effects
+			(font
+				(size 2.9972 2.9972)
+			)
+			(justify left bottom)

Commit message: wip + PDF plot
Changed lines of the file:
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@@
-		)
-	)
-	(text "W.I.P."
-		(exclude_from_sim no)
-		(at 60.96 103.632 0)
-		(effects
-			(font
-				(size 2.9972 2.9972)
-			)
-			(justify left bottom)
 		)
 	)
