File: CCE-2/CCE-2.sch (KiCad schematic (older format))
At the start: 44 parts, among them Q1_P11 BC168, T1_P11 BRY39

Commit message: Migrando esquemático (incompleto) da prancha 11 (placa CCE-2 - Controle de Estado) para um projeto novo.
Parts:
- removed DUVIDA1_P11, DUVIDA2_P11: 74LS51, symbol 74LS51
- removed DUVIDA3_P11: 74LS55, symbol 74LS55
Connections:
- net labels removed: ESP, INT
- wire segments 357 -> 402
- no-connect marks 56 -> 60
Other:
- note removed: "+INT"
- note removed: "-ATIVO"
- note removed: "-RODA1"
- moved on the sheet: 1B_P11A, 1B_P11B, 1B_P11C, 1B_P11E, 1B_P11F, 1C_P11B, 1C_P11C, 1C_P11D, 1D_P11D, 1E_P11A, 1E_P11B, 2A_P11A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
