File: CCE-2/CCE-2.kicad_sch (KiCad schematic)
At the start: 41 parts, among them Q1_P11 BC168, T1_P11 BRY39

Commit message: These are updated files after I loaded the project on a new version of KICAD
Parts:
- 3F_P11, 4C_P11: footprint ~ -> (none)
