File: CCE-2/CCE-2.kicad_sch (KiCad schematic)
At the start: 41 parts, among them Q1_P11 BC168, T1_P11 BRY39

Commit message: Some initial fixing of ERC errors.
Changed lines of the file:
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@@
 	)
 	(junction
-		(at 99.06 66.04)
-		(diameter 0)
-		(color 0 0 0 0)
-	)
-	(junction
 		(at 210.82 351.79)
 		(diameter 0)
@@
 	)
 	(junction
-		(at 167.64 152.4)
-		(diameter 0)
-		(color 0 0 0 0)
-	)
-	(junction
 		(at 632.46 422.91)
 		(diameter 0)
@@
 	(wire
 		(pts
-			(xy 99.06 63.5) (xy 99.06 66.04)
-		)
-		(stroke
-			(width 0)
-			(type default)
-		)
-	)
-	(wire
-		(pts
 			(xy 525.78 483.87) (xy 525.78 491.49)
 		)
@@
 	(wire
 		(pts
-			(xy 99.06 66.04) (xy 101.6 66.04)
+			(xy 92.71 66.04) (xy 101.6 66.04)
 		)
 		(stroke
@@
 	(wire
 		(pts
-			(xy 167.64 151.13) (xy 167.64 152.4)
-		)
-		(stroke
-			(width 0)
-			(type default)
-		)
-	)
-	(wire
-		(pts
 			(xy 92.71 63.5) (xy 92.71 66.04)
 		)
@@
 	(wire
 		(pts
-			(xy 92.71 66.04) (xy 99.06 66.04)
-		)
-		(stroke
-			(width 0)
-			(type default)
-		)
-	)
-	(wire
-		(pts
 			(xy 697.23 160.02) (xy 697.23 193.04)
 		)
@@
 				)
 			)
-		)
-	)
-	(symbol
-		(lib_id "CCE-2-rescue:PWR_FLAG-power")
-		(at 167.64 151.13 0)
-		(unit 1)
-		(body_style 1)
-		(exclude_from_sim no)
-		(in_bom yes)
-		(on_board yes)
-		(in_pos_files yes)
-		(dnp no)
-		(property "Reference" "#FLG011"
-			(at 167.64 148.717 0)
-			(hide yes)
-			(show_name no)
-			(do_not_autoplace no)
-			(effects
-				(font
-					(size 0.762 0.762)
-				)
-			)
-		)
-		(property "Value" "PWR_FLAG"
-			(at 167.64 145.8468 0)
-			(show_name no)
-			(do_not_autoplace no)
-			(effects
-				(font
-					(size 0.762 0.762)
-				)
-			)
-		)
-		(property "Footprint" ""
-			(at 167.64 151.13 0)
-			(hide yes)
-			(show_name no)
-			(do_not_autoplace no)
-			(effects
-				(font
-					(size 1.524 1.524)
-				)
-			)
-		)
-		(property "Datasheet" ""
-			(at 167.64 151.13 0)
-			(hide yes)
-			(show_name no)
-			(do_not_autoplace no)
-			(effects
-				(font
-					(size 1.524 1.524)
-				)
-			)
-		)
-		(property "Description" ""
-			(at 167.64 151.13 0)
-			(show_name no)
-			(do_not_autoplace no)
-			(effects
-				(font
-					(size 1.27 1.27)
-				)
-			)
-		)
-		(pin "1"
-		)
-		(instances
-			(project "patinhofeio"
-				(path "/aca06203-542d-4682-a7e3-8839e24cce95/bba15d3c-50cc-4e33-8f05-e25d292c5848"
-					(reference "#FLG011")
-					(unit 1)
-				)
-			)
-			(project ""
-				(path "/cbc7ab26-f296-43b4-80b6-f46d8a4d52c1"
-					(reference "#FLG011")
-					(unit 1)
-				)
-			)
-		)
-	)
-	(symbol
-		(lib_id "CCE-2-rescue:PWR_FLAG-power")
-		(at 99.06 63.5 0)
-		(unit 1)
-		(body_style 1)
-		(exclude_from_sim no)
-		(in_bom yes)
-		(on_board yes)
-		(in_pos_files yes)
-		(dnp no)
-		(property "Reference" "#FLG013"
-			(at 99.06 61.087 0)
-			(hide yes)
-			(show_name no)
-			(do_not_autoplace no)
-			(effects
-				(font
-					(size 0.762 0.762)
-				)
-			)
-		)
-		(property "Value" "PWR_FLAG"
-			(at 99.06 58.2168 0)
-			(show_name no)
-			(do_not_autoplace no)
-			(effects
-				(font
-					(size 0.762 0.762)
-				)
-			)
-		)
-		(property "Footprint" ""
-			(at 99.06 63.5 0)
-			(hide yes)
-			(show_name no)
-			(do_not_autoplace no)
-			(effects
-				(font
-					(size 1.524 1.524)
-				)
-			)
-		)
-		(property "Datasheet" ""
-			(at 99.06 63.5 0)
-			(hide yes)
-			(show_name no)
-			(do_not_autoplace no)
-			(effects
-				(font
-					(size 1.524 1.524)
-				)
-			)
-		)
-		(property "Description" ""
-			(at 99.06 63.5 0)
-			(show_name no)
-			(do_not_autoplace no)
-			(effects
-				(font
-					(size 1.27 1.27)
-				)
-			)
-		)
-		(pin "1"
-		)
-		(instances
-			(project "patinhofeio"
-				(path "/aca06203-542d-4682-a7e3-8839e24cce95/bba15d3c-50cc-4e33-8f05-e25d292c5848"
-					(reference "#FLG013")
-					(unit 1)
-				)
-			)
-			(project ""
-				(path "/cbc7ab26-f296-43b4-80b6-f46d8a4d52c1"
-					(reference "#FLG013")
-					(unit 1)
-				)
-			)

Commit message: fixing a whole bunch more ERC errors
Parts:
- removed 1B_P11, 3E_P11, 4F_P11, 5F_P11: 74LS04, symbol CCE-2-rescue:74LS04
- removed 1C_P11, 2E_P11, 3B_P11, 3C_P11, 4A_P11, 5C_P11: 7400, symbol CCE-2-rescue:7400
- removed 1D_P11, 5A_P11: 7402, symbol CCE-2-rescue:7402
- removed 2C_P11, 5B_P11, 5D_P11: 74LS20, symbol CCE-2-rescue:74LS20
- added 1B_P11, 3E_P11, 4F_P11, 5F_P11: 74LS04, symbol 74xx:74LS04
- added 1C_P11, 2E_P11, 3B_P11, 3C_P11, 4A_P11, 5C_P11: 7400, symbol 74xx:7400
- added 1D_P11, 5A_P11: 74LS02, symbol 74xx:74LS02
- added 2C_P11, 5B_P11, 5D_P11: 74LS20, symbol 74xx:74LS20
Connections:
- net +ATIVO: now also 5F_P11.3
- net +CF1: now also 4A_P11.5
- net +CLOCK: now also 5A_P11.9
- net +CS: now also 4A_P11.10
- net +ESP: now also 1C_P11.1
- net +FN: now also 3C_P11.2
- net +INI: now also 2E_P11.4
- net +INT: now also 3C_P11.8, 5B_P11.12, 5C_P11.5
- net +IS: now also 4A_P11.2
- net +PARTIDA: now also 3E_P11.9, 4A_P11.1, 4A_P11.9, 5A_P11.4
- net +PER: now also 2E_P11.1
- net +PUL: now also 3C_P11.12
- net +RODA: now also 1B_P11.10, 2C_P11.10, 2C_P11.4, 5B_P11.4, 5D_P11.10, 5D_P11.4
- net +T0: now also 5C_P11.4
- net +T4: now also 2E_P11.2, 2E_P11.5
- net +T5: now also 1C_P11.5
- net +T6: now also 3C_P11.13, 3C_P11.5
- net +T7: now also 5B_P11.10
- net -(BOT-ESP-A): now also 3B_P11.4
- net -(BOT-ESP-N): now also 3B_P11.10
- net -(BOT-PART-A): now also 3B_P11.2
- net -(BOT-PART-N): now also 3B_P11.12
- net -(ESP.FORÇA_PUG): now also 1C_P11.3
- net -ATIVO: now also 4A_P11.4, 5A_P11.12, 5F_P11.4
- net -CF1: now also 1D_P11.9, 5F_P11.1
- net -CF2: now also 3E_P11.13
- net -CF3: now also 2E_P11.13
- net -CF4: now also 3E_P11.3
- net -CF5: now also 3E_P11.5
- net -F1: now also 5D_P11.6
- net -F2: now also 5D_P11.8
- net -F3: now also 2C_P11.6
- net -F4: now also 2C_P11.8
- net -F5: now also 5B_P11.6
- net -FORÇA_PUG: now also 1B_P11.9, 5B_P11.8
- net -IMPEDE: now also 1D_P11.4, 4A_P11.13, 5F_P11.5
- net -INT: now also 3C_P11.10, 5C_P11.13
- net -LAL: now also 4F_P11.12
- net -LAL1: now also 4F_P11.4
- net -LAL2: now also 4F_P11.6
- net -LAL3: now also 4F_P11.10
- net -LAL4: now also 4F_P11.8
- net -PARTIDA: now also 3E_P11.8
- net -PARTIDA2: now also 2E_P11.8
- net -PEDIDO_INTERRUPÇÃO: now also 1D_P11.2
- net -RODA: now also 1B_P11.11, 1C_P11.4
- net -T1: now also 1C_P11.10
- net -T7: now also 1D_P11.12, 5A_P11.8
- net CLOCK: now also 1D_P11.13
- net GND: now also 1B_P11.7 (GND), 1C_P11.7 (GND), 1D_P11.7 (GND), 1D_P11.8, 2C_P11.7 (GND), 2E_P11.7 (GND), 3B_P11.7 (GND), 3C_P11.7 (GND), 3E_P11.7 (GND), 4A_P11.7 (GND), 4F_P11.7 (GND), 5A_P11.7 (GND), 5B_P11.7 (GND), 5C_P11.7 (GND), 5D_P11.7 (GND), 5F_P11.7 (GND)
- net VCC: now also 1B_P11.14 (VCC), 1C_P11.14 (VCC), 1D_P11.14 (VCC), 2C_P11.14 (VCC), 2E_P11.12, 2E_P11.14 (VCC), 3B_P11.14 (VCC), 3C_P11.14 (VCC), 3E_P11.14 (VCC), 4A_P11.14 (VCC), 4F_P11.14 (VCC), 5A_P11.14 (VCC), 5B_P11.14 (VCC), 5C_P11.14 (VCC), 5D_P11.14 (VCC), 5F_P11.14 (VCC)
- net pcb_15: now also 5C_P11.12
- net at DUVIDA4_P11.8: now also 1B_P11.1
- net at 3A_P11.2, 3A_P11.4, 3A_P11.9: now also 5F_P11.2
- net at 3A_P11.8: now also 1B_P11.3
- net at 2B_P11.1 (J): now also 1B_P11.4
- net at 2B_P11.4 (K): now also 1B_P11.2
- net at 4C_P11.6: now also 5B_P11.13, 5C_P11.9
- net at 3F_P11.10: now also 4A_P11.8
- net at 2A_P11.2: now also 3B_P11.6, 3B_P11.9
- net at 4B_P11.2 (D), D1_P11.1 (A): now also 3B_P11.13, 3B_P11.3
- net at 4C_P11.12: now also 5C_P11.1
- net at 4C_P11.13: now also 1D_P11.6, 5C_P11.3
- net at 4C_P11.3: now also 1D_P11.5, 5C_P11.8
- net at 4C_P11.5: now also 5C_P11.11
- net at 2D_P11.5 (Q): now also 5D_P11.2
- net at 2D_P11.12 (D): now also 3E_P11.12
- net at 2D_P11.9 (Q): now also 5D_P11.12
- net at 2D_P11.2 (D): now also 1D_P11.10
- net at 3D_P11.2 (D): now also 2E_P11.11
- net at 3D_P11.5 (Q): now also 2C_P11.2
- net at 4C_P11.2: now also 2E_P11.3
- net at 3D_P11.12 (D): now also 3E_P11.4
- net at 3D_P11.9 (Q): now also 2C_P11.12
- net at 4D_P11.2 (D): now also 3E_P11.6
- net at 4D_P11.5 (Q): now also 5B_P11.2
- net at 4C_P11.10: now also 3C_P11.11
- net at 4B_P11.12 (D), 4B_P11.5 (Q): now also 2E_P11.9
- net at 4B_P11.6 (~{Q}), 4E_P11.12, 4E_P11.13: now also 5A_P11.5
- net at 4B_P11.11 (Cp): now also 5A_P11.10
- net at 4B_P11.8 (~{Q}): now also 2E_P11.10
- net at 4B_P11.9 (Q), 4E_P11.1, 4E_P11.10: now also 5A_P11.6
- net at 2B_P11.11 (K): now also 1B_P11.12
- net at 2B_P11.8 (J): now also 1B_P11.6
- net at 4D_P11.9 (Q): now also 4A_P11.12, 5A_P11.11
- net at 1E_P11.4 (K): now also 4A_P11.11
- net at 1E_P11.11 (K): now also 5A_P11.13
- net at 2A_P11.6: now also 3E_P11.11
- net at 1E_P11.1 (J): now also 3E_P11.10
- net at Q1_P11.1 (C), R6_P11.1: now also 4F_P11.1
- new net: 1B_P11.13, 4A_P11.6
- new net: 4F_P11.11, 4F_P11.13, 4F_P11.2, 4F_P11.3, 4F_P11.5, 4F_P11.9
- new net: 1C_P11.11, 1C_P11.9
- new net: 1C_P11.12, 1C_P11.8, 3C_P11.1
- new net: 1C_P11.13, 1C_P11.6
- new net: 3B_P11.5, 3B_P11.8
- new net: 3C_P11.6, 3C_P11.9
- new net: 1B_P11.8, 1C_P11.2
- new net: 1D_P11.3, 5F_P11.6
- new net: 1D_P11.11, 3C_P11.3
- new net: 3B_P11.1, 3B_P11.11
- new net: 2E_P11.6, 5C_P11.2
- new net: 3C_P11.4, 3E_P11.2
- new net: 1B_P11.5, 4A_P11.3
- new net: 5C_P11.10, 5C_P11.6

Commit message: melhorias dessa semana
Parts:
- removed 2D_P11, 3D_P11, 4D_P11: 74HC74, symbol CCE-2-rescue:74HC74
- added 2D_P11, 3D_P11, 4D_P11: 74LS74, symbol 74xx:74LS74
Connections:
- net +T6: now also 4D_P11.11 (C)
- net -F1-D: now also 2D_P11.6 (~{Q})
- net -F2-D: now also 2D_P11.8 (~{Q})
- net -F3-D: now also 3D_P11.6 (~{Q})
- net -F4-D: now also 3D_P11.8 (~{Q})
- net -F5-D: now also 4D_P11.6 (~{Q})
- net -FORÇA_PUG: now also 2D_P11.1 (~{R}), 3D_P11.4 (~{S})
- net -LAL3: now also 2D_P11.13 (~{R}), 2D_P11.4 (~{S}), 3D_P11.1 (~{R}), 3D_P11.13 (~{R}), 4D_P11.1 (~{R})
- net -PARTIDA: now also 4D_P11.12 (D)
- net CLOCK: now also 2D_P11.11 (C), 2D_P11.3 (C), 3D_P11.11 (C), 3D_P11.3 (C), 4D_P11.3 (C)
- net GND: now also 2D_P11.7 (GND), 3D_P11.7 (GND), 4D_P11.7 (GND)
- net VCC: now also 2D_P11.14 (VCC), 3D_P11.14 (VCC), 4D_P11.14 (VCC)
- net at 3E_P11.12: now also 2D_P11.12 (D)
- net at 5D_P11.12: now also 2D_P11.9 (Q)
- net at 1D_P11.10: now also 2D_P11.2 (D)
- net at 5D_P11.2: now also 2D_P11.5 (Q)
- net at 2E_P11.11: now also 3D_P11.2 (D)
- net at 2C_P11.2: now also 3D_P11.5 (Q)
- net at 3E_P11.4: now also 3D_P11.12 (D)
- net at 2C_P11.12: now also 3D_P11.9 (Q)
- net at 3E_P11.6: now also 4D_P11.2 (D)
- net at 5B_P11.2: now also 4D_P11.5 (Q)
- net at 4A_P11.12, 5A_P11.11: now also 4D_P11.9 (Q)

Commit message: wip
Parts:
- added U1: 74LS51, symbol 74xx:74LS51
- added U2: 7451, symbol 74xx_IEEE:7451
Changed lines of the file:
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@@
 	)
 	(symbol
+		(lib_id "74xx:74LS51")
+		(at 240.03 327.66 0)
+		(unit 1)
+		(body_style 1)
+		(exclude_from_sim no)
+		(in_bom yes)
+		(on_board yes)
+		(in_pos_files yes)
+		(dnp no)
+		(fields_autoplaced yes)
+		(property "Reference" "U1"
+			(at 240.03 314.96 0)
+			(show_name no)
+			(do_not_autoplace no)
+			(effects
+				(font
+					(size 1.27 1.27)
+				)
+			)
+		)
+		(property "Value" "74LS51"
+			(at 240.03 317.5 0)
+			(show_name no)
+			(do_not_autoplace no)
+			(effects
+				(font
+					(size 1.27 1.27)
+				)
+			)
+		)
+		(property "Footprint" ""
+			(at 240.03 327.66 0)
+			(hide yes)
+			(show_name no)
+			(do_not_autoplace no)
+			(effects
+				(font
+					(size 1.27 1.27)
+				)
+			)
+		)
+		(property "Datasheet" "http://www.ti.com/lit/ds/symlink/sn74ls51.pdf"
+			(at 240.03 327.66 0)
+			(hide yes)
+			(show_name no)
+			(do_not_autoplace no)
+			(effects
+				(font
+					(size 1.27 1.27)
+				)
+			)
+		)
+		(property "Description" "Dual 3- and 2-input AND-NOR ( S = /(AB[C] + DE[F]) )"
+			(at 240.03 327.66 0)
+			(hide yes)
+			(show_name no)
+			(do_not_autoplace no)
+			(effects
+				(font
+					(size 1.27 1.27)
+				)
+			)
+		)
+		(pin "13"
+		)
+		(pin "14"
+		)
+		(pin "1"
+		)
+		(pin "4"
+		)
+		(pin "6"
+		)
+		(pin "5"
+		)
+		(pin "7"
+		)
+		(pin "2"
+		)
+		(pin "3"
+		)
+		(pin "12"
+		)
+		(pin "11"
+		)
+		(pin "10"
+		)
+		(pin "9"
+		)
+		(pin "8"
+		)
+		(instances
+			(project "patinhofeio"
+				(path "/aca06203-542d-4682-a7e3-8839e24cce95/bba15d3c-50cc-4e33-8f05-e25d292c5848"
+					(reference "U1")
+					(unit 1)
+				)
+			)
+		)
+	)
+	(symbol
 		(lib_id "74xx:7400")
 		(at 81.28 391.16 0)
@@
 					(unit 1)
 				)
+			)
+		)
+	)
+	(symbol
+		(lib_id "74xx_IEEE:7451")
+		(at 281.94 328.93 0)
+		(unit 1)
+		(body_style 1)
+		(exclude_from_sim no)
+		(in_bom yes)
+		(on_board yes)
+		(in_pos_files yes)
+		(dnp no)
+		(fields_autoplaced yes)
+		(property "Reference" "U2"
+			(at 295.91 322.5098 0)
+			(show_name no)
+			(do_not_autoplace no)
+			(effects
+				(font
+					(size 1.27 1.27)
+				)
+			)
+		)
+		(property "Value" "7451"
+			(at 295.91 325.0498 0)
+			(show_name no)
+			(do_not_autoplace no)
+			(effects
+				(font
+					(size 1.27 1.27)
+				)
+			)
+		)
+		(property "Footprint" ""
+			(at 281.94 328.93 0)
+			(hide yes)
+			(show_name no)
+			(do_not_autoplace no)
+			(effects
+				(font
+					(size 1.27 1.27)
+				)
+			)
+		)
+		(property "Datasheet" ""
+			(at 281.94 328.93 0)
+			(hide yes)
+			(show_name no)
+			(do_not_autoplace no)
+			(effects
+				(font
+					(size 1.27 1.27)
+				)
+			)
+		)
+		(property "Description" ""
+			(at 281.94 328.93 0)
+			(hide yes)
+			(show_name no)
+			(do_not_autoplace no)
+			(effects
+				(font
+					(size 1.27 1.27)
+				)
+			)
+		)
+		(pin "3"
+		)
+		(pin "6"
+		)
+		(pin "4"
+		)
+		(pin "5"
+		)
+		(pin "2"
+		)
+		(pin "13"
+		)
+		(pin "10"
+		)
+		(pin "9"
+		)
+		(pin "8"
+		)
+		(pin "2"
+		)
+		(pin "14"
+		)
+		(pin "7"
+		)
+		(instances
+			(project "patinhofeio"
+				(path "/aca06203-542d-4682-a7e3-8839e24cce95/bba15d3c-50cc-4e33-8f05-e25d292c5848"
+					(reference "U2")
+					(unit 1)
+				)

Commit message: wip
Parts:
- removed 1E_P11, 2B_P11: 74LS107, symbol CCE-2-rescue:74LS107
- removed 3F_P11, 4C_P11: 74LS10, symbol CCE-2-rescue:74LS10
- removed 4B_P11: 74HC74, symbol CCE-2-rescue:74HC74
- removed U1: 74LS51, symbol 74xx:74LS51
- removed U2: 7451, symbol 74xx_IEEE:7451
- added 1E_P11, 2B_P11: 74LS107, symbol 74xx:74LS107
- added 3F_P11, 4C_P11: 74LS10, symbol 74xx:74LS10
- added 4B_P11: 74LS74, symbol 74xx:74LS74
Connections:
- net +ESP: now also 1E_P11.3 (Q)
- net +INT: now also 4C_P11.9
- net +PAR: now also 1E_P11.5 (Q)
- net +PAR-D: now also 1E_P11.8 (J)
- net +RODA1: now also 2B_P11.2 (~{Q})
- net +T0: now also 4B_P11.3 (C)
- net +T4: now also 1E_P11.9 (C)
- net +T6: now also 2B_P11.12 (C), 2B_P11.9 (C)
- net -(ESP.FORÇA_PUG): now also 2B_P11.13 (~{R})
- net -ESP: now also 1E_P11.2 (~{Q})
- net -INT: now also 4C_P11.8
- net -LAL: now also 2B_P11.10 (~{R}), 3F_P11.4, 4C_P11.1, 4C_P11.11, 4C_P11.4
- net -PAR: now also 1E_P11.6 (~{Q})
- net -RODA: now also 3F_P11.6
- net -RODA1: now also 2B_P11.3 (Q), 3F_P11.11
- net -T3: now also 1E_P11.12 (C)
- net GND: now also 1E_P11.7 (GND), 2B_P11.7 (GND), 3F_P11.7 (GND), 4B_P11.7 (GND), 4C_P11.7 (GND)
- net VCC: now also 1E_P11.14 (VCC), 2B_P11.14 (VCC), 3F_P11.14 (VCC), 4B_P11.14 (VCC), 4C_P11.14 (VCC)
- net at 1B_P11.4: now also 2B_P11.1 (J)
- net at 1B_P11.2: now also 2B_P11.4 (K)
- net at 4A_P11.8: now also 3F_P11.10
- net at 1D_P11.5, 5C_P11.8: now also 4C_P11.3
- net at 5C_P11.11: now also 4C_P11.5
- net at 5B_P11.13, 5C_P11.9: now also 4C_P11.6
- net at 5C_P11.1: now also 4C_P11.12
- net at 1D_P11.6, 5C_P11.3: now also 4C_P11.13
- net at 2E_P11.3: now also 4C_P11.2
- net at 3C_P11.11: now also 4C_P11.10
- net at 3B_P11.13, 3B_P11.3, D1_P11.1 (A): now also 4B_P11.2 (D)
- net at 2E_P11.9: now also 4B_P11.12 (D), 4B_P11.5 (Q)
- net at 4E_P11.12, 4E_P11.13, 5A_P11.5: now also 4B_P11.6 (~{Q})
- net at 5A_P11.10: now also 4B_P11.11 (C)
- net at 2E_P11.10: now also 4B_P11.8 (~{Q})
- net at 4E_P11.1, 4E_P11.10, 5A_P11.6: now also 4B_P11.9 (Q)
- net at 1B_P11.12: now also 2B_P11.11 (K)
- net at 1B_P11.6: now also 2B_P11.8 (J)
- net at 3E_P11.10: now also 1E_P11.1 (J)
- net at 4A_P11.11: now also 1E_P11.4 (K)
- net at 5A_P11.13: now also 1E_P11.11 (K)
- new net: 3F_P11.5, 3F_P11.8
- new net: 2B_P11.6 (~{Q}), 3F_P11.9
Other:
- moved on the sheet: 1B_P11G, 1D_P11E, 2C_P11C, 2D_P11C, 3C_P11B, 3D_P11C, 3E_P11G, 4D_P11C, 4F_P11G, 5A_P11E, 5B_P11C, 5D_P11C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

Commit message: wip + PDF plot
Other:
- moved on the sheet: 1B_P11D, 1B_P11G, 1C_P11A, 1C_P11E, 1D_P11A, 1D_P11B, 1D_P11E, 1E_P11C, 2B_P11C, 2C_P11C, 2D_P11C, 2E_P11A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
