File: FCM-7/FCM-7.sch (KiCad schematic (older format))
At the start: 16 parts

Commit message: criando novos projetos individuais para todas as outras pranchas que ainda faltavam serem migradas.
Connections:
- net GND: now also CONECTOR_P5.70 (P70)
- net LWBO_1: now also CONECTOR_P5.38 (P38)
- net LWBO_2: now also CONECTOR_P5.39 (P39)
- net LWBO_3: now also CONECTOR_P5.40 (P40)
- net LWBO_4: now also CONECTOR_P5.41 (P41)
- net LWBO_5: now also CONECTOR_P5.42 (P42)
- net LWBO_6: now also CONECTOR_P5.43 (P43)
- net LWBO_7: now also CONECTOR_P5.44 (P44)
- net VCC: now also CONECTOR_P5.1 (P1)
- no-connect marks 16 -> 7
Changed lines of the file:
@@
 LIBS:memory
 LIBS:xilinx
-LIBS:special
 LIBS:microcontrollers
 LIBS:dsp
@@
 LIBS:contrib
 LIBS:valves
-LIBS:7451
-LIBS:7454
-LIBS:7460
 LIBS:conn_35x2
-LIBS:patinhofeio-cache
 EELAYER 25 0
 EELAYER END
 $Descr A2 23386 16535
 encoding utf-8
-Sheet 12 17
+Sheet 1 1
 Title ""
 Date "2 aug 2016"
@@
 Text Notes 4050 2400 0    60   ~ 0
 LSB2-24
-NoConn ~ 2750 1250
 NoConn ~ 3550 2550
 NoConn ~ 2750 2550
 NoConn ~ 2750 2950
-NoConn ~ 2750 3150
-NoConn ~ 2750 3350
-NoConn ~ 2750 3250
 NoConn ~ 3550 2950
-NoConn ~ 3550 3150
-NoConn ~ 3550 3050
-NoConn ~ 3550 3250
-NoConn ~ 3550 3350
 NoConn ~ 3550 2450
-NoConn ~ 3550 4650
 NoConn ~ 3550 4250
 NoConn ~ 2750 4350
@@
 PST-
 $Comp
-L GND #PWR037
+L GND #PWR01
 U 1 1 587C2945
 P 13150 6550
-F 0 "#PWR037" H 13150 6550 30  0001 C CNN
+F 0 "#PWR01" H 13150 6550 30  0001 C CNN
 F 1 "GND" H 13150 6480 30  0001 C CNN
 F 2 "" H 13150 6550 60  0001 C CNN
@@
 PW-
 $Comp
-L GND #PWR038
+L GND #PWR02
 U 1 1 587C2A21
 P 11450 7250
-F 0 "#PWR038" H 11450 7250 30  0001 C CNN
+F 0 "#PWR02" H 11450 7250 30  0001 C CNN
 F 1 "GND" H 11450 7180 30  0001 C CNN
 F 2 "" H 11450 7250 60  0001 C CNN
@@
 $EndComp
 $Comp
-L VCC #PWR039
+L VCC #PWR03
 U 1 1 587C2C3B
 P 18350 1250
-F 0 "#PWR039" H 18350 1350 30  0001 C CNN
+F 0 "#PWR03" H 18350 1350 30  0001 C CNN
 F 1 "VCC" H 18353 1378 30  0000 C CNN
 F 2 "" H 18350 1250 60  0001 C CNN
@@
 Connection ~ 18350 1950
 $Comp
-L GND #PWR040
+L GND #PWR04
 U 1 1 587C2F2D
 P 18850 2500
-F 0 "#PWR040" H 18850 2500 30  0001 C CNN
+F 0 "#PWR04" H 18850 2500 30  0001 C CNN
 F 1 "GND" H 18850 2430 30  0001 C CNN
 F 2 "" H 18850 2500 60  0001 C CNN
@@
 $EndComp
 $Comp
-L VCC #PWR041
+L VCC #PWR05
 U 1 1 587C3220
 P 18350 2800
-F 0 "#PWR041" H 18350 2900 30  0001 C CNN
+F 0 "#PWR05" H 18350 2900 30  0001 C CNN
 F 1 "VCC" H 18353 2928 30  0000 C CNN
 F 2 "" H 18350 2800 60  0001 C CNN
@@
 Connection ~ 18350 3500
 $Comp
-L GND #PWR042
+L GND #PWR06
 U 1 1 587C3229
 P 18850 4050
-F 0 "#PWR042" H 18850 4050 30  0001 C CNN
+F 0 "#PWR06" H 18850 4050 30  0001 C CNN
 F 1 "GND" H 18850 3980 30  0001 C CNN
 F 2 "" H 18850 4050 60  0001 C CNN
@@
 $EndComp
 $Comp
-L VCC #PWR043
+L VCC #PWR07
 U 1 1 587C35E0
 P 18350 4450
-F 0 "#PWR043" H 18350 4550 30  0001 C CNN
+F 0 "#PWR07" H 18350 4550 30  0001 C CNN
 F 1 "VCC" H 18353 4578 30  0000 C CNN
 F 2 "" H 18350 4450 60  0001 C CNN
@@
 Connection ~ 18350 5150
 $Comp
-L GND #PWR044
+L GND #PWR08
 U 1 1 587C35E9
 P 18850 5700
-F 0 "#PWR044" H 18850 5700 30  0001 C CNN
+F 0 "#PWR08" H 18850 5700 30  0001 C CNN
 F 1 "GND" H 18850 5630 30  0001 C CNN
 F 2 "" H 18850 5700 60  0001 C CNN
@@
 $EndComp
 $Comp
-L VCC #PWR045
+L VCC #PWR09
 U 1 1 587C35FC
 P 18350 6000
-F 0 "#PWR045" H 18350 6100 30  0001 C CNN
+F 0 "#PWR09" H 18350 6100 30  0001 C CNN
 F 1 "VCC" H 18353 6128 30  0000 C CNN
 F 2 "" H 18350 6000 60  0001 C CNN
@@
 Connection ~ 18350 6700
 $Comp
-L GND #PWR046
+L GND #PWR010
 U 1 1 587C3605
 P 18850 7250
-F 0 "#PWR046" H 18850 7250 30  0001 C CNN
+F 0 "#PWR010" H 18850 7250 30  0001 C CNN
 F 1 "GND" H 18850 7180 30  0001 C CNN
 F 2 "" H 18850 7250 60  0001 C CNN
@@
 $EndComp
 $Comp
-L VCC #PWR047
+L VCC #PWR011
 U 1 1 587C3A4C
 P 18350 7900
-F 0 "#PWR047" H 18350 8000 30  0001 C CNN
+F 0 "#PWR011" H 18350 8000 30  0001 C CNN
 F 1 "VCC" H 18353 8028 30  0000 C CNN
 F 2 "" H 18350 7900 60  0001 C CNN
@@
 Connection ~ 18350 8600
 $Comp
-L GND #PWR048
+L GND #PWR012
 U 1 1 587C3A55
 P 18850 9150
-F 0 "#PWR048" H 18850 9150 30  0001 C CNN
+F 0 "#PWR012" H 18850 9150 30  0001 C CNN
 F 1 "GND" H 18850 9080 30  0001 C CNN
 F 2 "" H 18850 9150 60  0001 C CNN
@@
 $EndComp
 $Comp
-L VCC #PWR049
+L VCC #PWR013
 U 1 1 587C3A68
 P 18350 9450
-F 0 "#PWR049" H 18350 9550 30  0001 C CNN
+F 0 "#PWR013" H 18350 9550 30  0001 C CNN
 F 1 "VCC" H 18353 9578 30  0000 C CNN
 F 2 "" H 18350 9450 60  0001 C CNN
@@
 Connection ~ 18350 10150
 $Comp
-L GND #PWR050
+L GND #PWR014
 U 1 1 587C3A71
 P 18850 10700
-F 0 "#PWR050" H 18850 10700 30  0001 C CNN
+F 0 "#PWR014" H 18850 10700 30  0001 C CNN
 F 1 "GND" H 18850 10630 30  0001 C CNN
 F 2 "" H 18850 10700 60  0001 C CNN
@@
 $EndComp
 $Comp
-L VCC #PWR051
+L VCC #PWR015
 U 1 1 587C3A84
 P 18350 11100
-F 0 "#PWR051" H 18350 11200 30  0001 C CNN
+F 0 "#PWR015" H 18350 11200 30  0001 C CNN
 F 1 "VCC" H 18353 11228 30  0000 C CNN
 F 2 "" H 18350 11100 60  0001 C CNN
@@
 Connection ~ 18350 11800
 $Comp
-L GND #PWR052
+L GND #PWR016
 U 1 1 587C3A8D
 P 18850 12350
-F 0 "#PWR052" H 18850 12350 30  0001 C CNN
+F 0 "#PWR016" H 18850 12350 30  0001 C CNN
 F 1 "GND" H 18850 12280 30  0001 C CNN
 F 2 "" H 18850 12350 60  0001 C CNN
@@
 $EndComp
 $Comp
-L VCC #PWR053
+L VCC #PWR017
 U 1 1 587C3AA0
 P 18350 12650
-F 0 "#PWR053" H 18350 12750 30  0001 C CNN
+F 0 "#PWR017" H 18350 12750 30  0001 C CNN
 F 1 "VCC" H 18353 12778 30  0000 C CNN
 F 2 "" H 18350 12650 60  0001 C CNN
@@
 Connection ~ 18350 13350
 $Comp
-L GND #PWR054
+L GND #PWR018
 U 1 1 587C3AA9
 P 18850 13900
-F 0 "#PWR054" H 18850 13900 30  0001 C CNN
+F 0 "#PWR018" H 18850 13900 30  0001 C CNN
 F 1 "GND" H 18850 13830 30  0001 C CNN
 F 2 "" H 18850 13900 60  0001 C CNN
@@
 	9450 11300 9450 11900
 Connection ~ 9450 11900
+$Comp
+L PWR_FLAG #FLG019
+U 1 1 587EA3FA
+P 5300 4550
+F 0 "#FLG019" H 5300 4645 30  0001 C CNN
+F 1 "PWR_FLAG" H 5300 4758 30  0000 C CNN
+F 2 "" H 5300 4550 60  0001 C CNN
+F 3 "" H 5300 4550 60  0001 C CNN
+	1    5300 4550
+	1    0    0    -1
+$EndComp
+$Comp
+L GND #PWR020
+U 1 1 587EA47A
+P 5300 4800
+F 0 "#PWR020" H 5300 4800 30  0001 C CNN
+F 1 "GND" H 5300 4730 30  0001 C CNN
+F 2 "" H 5300 4800 60  0001 C CNN
+F 3 "" H 5300 4800 60  0001 C CNN
+	1    5300 4800
+	1    0    0    -1
+$EndComp
+Wire Wire Line
+	5300 4550 5300 4800
+Wire Wire Line
+	3550 4650 5300 4650
+Connection ~ 5300 4650
+$Comp
+L PWR_FLAG #FLG021
+U 1 1 587EA773
+P 2600 1100
+F 0 "#FLG021" H 2600 1195 30  0001 C CNN
+F 1 "PWR_FLAG" H 2600 1308 30  0000 C CNN
+F 2 "" H 2600 1100 60  0001 C CNN
+F 3 "" H 2600 1100 60  0001 C CNN
+	1    2600 1100
+	1    0    0    -1
+$EndComp
+$Comp
+L VCC #PWR022
+U 1 1 587EA9C1
+P 2400 1100
+F 0 "#PWR022" H 2400 1200 30  0001 C CNN
+F 1 "VCC" H 2403 1228 30  0000 C CNN
+F 2 "" H 2400 1100 60  0001 C CNN
+F 3 "" H 2400 1100 60  0001 C CNN
+	1    2400 1100
+	1    0    0    -1
+$EndComp
+Wire Wire Line
+	2400 1250 2750 1250
+Wire Wire Line
+	2600 1250 2600 1100
+Wire Wire Line
+	2400 1250 2400 1100
+Connection ~ 2600 1250
+Text GLabel 4800 3050 2    60   Input ~ 0
+LWBO_1
+Wire Wire Line
+	3550 3050 4800 3050
+Text GLabel 4800 3250 2    60   Input ~ 0
+LWBO_5
+Text GLabel 3750 3150 2    60   Input ~ 0
+LWBO_3
+Text GLabel 3750 3350 2    60   Input ~ 0
+LWBO_7
+Wire Wire Line
+	3750 3150 3550 3150
+Wire Wire Line
+	3550 3250 4800 3250
+Wire Wire Line
+	3750 3350 3550 3350
+Text GLabel 2600 3150 0    60   Input ~ 0
+LWBO_2
+Text GLabel 2600 3350 0    60   Input ~ 0
+LWBO_6
+Text GLabel 1500 3250 0    60   Input ~ 0
+LWBO_4
+Wire Wire Line
+	2600 3350 2750 3350
+Wire Wire Line
+	2750 3250 1500 3250
+Wire Wire Line
+	2600 3150 2750 3150
 $EndSCHEMATC
