File: CT5-8/CT5-8.sch (KiCad schematic (older format))
At the start: 12 parts

Commit message: terminando de corrigir todos os error do DRC no esquemático CT5-8
Connections:
- net -(F2.5AE5A) is gone; now on net -(F2.SAESA): 1D_P16.6
- net +F1: now also 1A_P16.12, 3B_P16.13
- net +MICG2A: now also CONECTOR_P16.10 (P10)
- net +PUG: now also CONECTOR_P16.12 (P12)
- net +PUL: now also CONECTOR_P16.9 (P9)
- net +RI_7: now also CONECTOR_P16.43 (P43)
- net +S: now also CONECTOR_P16.48 (P48)
- net +SAESA: now also CONECTOR_P16.5 (P5)
- net +SALMIC: now also CONECTOR_P16.11 (P11)
- net +SUS: now also CONECTOR_P16.15 (P15)
- net +T01: now also CONECTOR_P16.45 (P45)
- net +T23: now also CONECTOR_P16.7 (P7)
- net +T34: now also CONECTOR_P16.42 (P42)
- net +T56: now also CONECTOR_P16.47 (P47)
- net +VUQ: now also CONECTOR_P16.41 (P41)
- net -F1: now also CONECTOR_P16.44 (P44)
- net -F2: now also CONECTOR_P16.6 (P6)
- net -F3: now also CONECTOR_P16.14 (P14)
- net -F4: now also CONECTOR_P16.46 (P46)
- net -SINTA: now also CONECTOR_P16.40 (P40)
- net GND: now also CONECTOR_P16.70 (P70)
- net VCC: now also CONECTOR_P16.1 (P1)
- net +(PARTIDA+RODA).(MP+CP) renamed +(PARTIDA.(-RODA).(MP+CP))
- net +(PARTIDA.(-RODA).(MP+CP)): now also CONECTOR_P16.13 (P13)
- net +MIC01 renamed +MICG1
- net +MICG1: now also CONECTOR_P16.8 (P8)
- removed net ?: CONECTOR_P16.1 (P1), CONECTOR_P16.10 (P10), CONECTOR_P16.11 (P11), CONECTOR_P16.12 (P12), CONECTOR_P16.13 (P13), CONECTOR_P16.14 (P14), CONECTOR_P16.15 (P15), CONECTOR_P16.16 (P16), CONECTOR_P16.17 (P17), CONECTOR_P16.18 (P18), CONECTOR_P16.19 (P19), CONECTOR_P16.2 (P2), CONECTOR_P16.20 (P20), CONECTOR_P16.21 (P21), CONECTOR_P16.22 (P22), CONECTOR_P16.23 (P23), CONECTOR_P16.24 (P24), CONECTOR_P16.25, CONECTOR_P16.26 (P26), CONECTOR_P16.27 (P27), CONECTOR_P16.28 (P28), CONECTOR_P16.29 (P29), CONECTOR_P16.3 (P3), CONECTOR_P16.30 (P30), CONECTOR_P16.31 (P31), CONECTOR_P16.32 (P32), CONECTOR_P16.33 (P33), CONECTOR_P16.34 (P34), CONECTOR_P16.35 (P35), CONECTOR_P16.36 (P36), CONECTOR_P16.37 (P37), CONECTOR_P16.38 (P38), CONECTOR_P16.39 (P39), CONECTOR_P16.4 (P4), CONECTOR_P16.40 (P40), CONECTOR_P16.41 (P41), CONECTOR_P16.42 (P42), CONECTOR_P16.43 (P43), CONECTOR_P16.44 (P44), CONECTOR_P16.45 (P45), CONECTOR_P16.46 (P46), CONECTOR_P16.47 (P47), CONECTOR_P16.48 (P48), CONECTOR_P16.49 (P49), CONECTOR_P16.5 (P5), CONECTOR_P16.50 (P50), CONECTOR_P16.51 (P51), CONECTOR_P16.52 (P52), CONECTOR_P16.53 (P53), CONECTOR_P16.54 (P54), CONECTOR_P16.55 (P55), CONECTOR_P16.56 (P56), CONECTOR_P16.57 (P57), CONECTOR_P16.58 (P58), CONECTOR_P16.59 (P59), CONECTOR_P16.6 (P6), CONECTOR_P16.60 (P60), CONECTOR_P16.61 (P61), CONECTOR_P16.62 (P62), CONECTOR_P16.63 (P63), CONECTOR_P16.64 (P64), CONECTOR_P16.65 (P65), CONECTOR_P16.66 (P66), CONECTOR_P16.67 (P67), CONECTOR_P16.68 (P68), CONECTOR_P16.69 (P69), CONECTOR_P16.7 (P7), CONECTOR_P16.70 (P70), CONECTOR_P16.8 (P8), CONECTOR_P16.9 (P9)
- no-connect marks 0 -> 48
