File: CT5-8/CT5-8.kicad_sch (KiCad schematic)
At the start: 12 parts

Commit message: These are updated files after I loaded the project on a new version of KICAD
Parts:
- 1A_P16, 1B_P16, 1C_P16, 1D_P16, 2A_P16, 2B_P16, 2C_P16, 2D_P16, 3A_P16, 3B_P16, 3C_P16: footprint ~ -> (none)
