File: CT5-8/CT5-8.kicad_sch (KiCad schematic)
At the start: 12 parts

Commit message: cleaning up references
Changed lines of the file:
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@@
 	(wire
 		(pts
-			(xy 127 167.64) (xy 127 170.18)
+			(xy 123.19 167.64) (xy 123.19 170.18)
 		)
 		(stroke
@@
 	(wire
 		(pts
-			(xy 127 170.18) (xy 130.81 170.18)
+			(xy 123.19 170.18) (xy 130.81 170.18)
 		)
 		(stroke
@@
 	(symbol
 		(lib_id "CT5-8-rescue:PWR_FLAG-power")
-		(at 130.81 167.64 0)
+		(at 161.29 255.27 0)
 		(unit 1)
 		(body_style 1)
@@
 		(in_pos_files yes)
 		(dnp no)
-		(property "Reference" "#FLG01"
-			(at 130.81 165.227 0)
+		(property "Reference" "#FLG03"
+			(at 161.29 252.857 0)
 			(hide yes)
 			(show_name no)
@@
 		)
 		(property "Value" "PWR_FLAG"
-			(at 130.81 162.3568 0)
+			(at 161.29 249.9868 0)
 			(show_name no)
 			(do_not_autoplace no)
@@
 		)
 		(property "Footprint" ""
-			(at 130.81 167.64 0)
+			(at 161.29 255.27 0)
 			(hide yes)
 			(show_name no)
@@
 		)
 		(property "Datasheet" ""
-			(at 130.81 167.64 0)
+			(at 161.29 255.27 0)
 			(hide yes)
 			(show_name no)
@@
 		)
 		(property "Description" ""
-			(at 130.81 167.64 0)
+			(at 161.29 255.27 0)
 			(show_name no)
 			(do_not_autoplace no)
@@
 			(project ""
 				(path "/8dd0d409-5aaf-4e71-90f1-464fc883daa9"
-					(reference "#FLG01")
+					(reference "#FLG03")
 					(unit 1)
 				)
@@
 			(project "patinhofeio"
 				(path "/aca06203-542d-4682-a7e3-8839e24cce95/a95f568a-1ac6-4cdd-a7e9-88a5e8192029"
-					(reference "#FLG01")
+					(reference "#FLG03")
 					(unit 1)
 				)
@@
 	)
 	(symbol
-		(lib_id "CT5-8-rescue:VCC-power")
-		(at 127 167.64 0)
+		(lib_id "power:PWR_FLAG")
+		(at 130.81 167.64 0)
 		(unit 1)
 		(body_style 1)
@@
 		(in_pos_files yes)
 		(dnp no)
-		(property "Reference" "#PWR02"
-			(at 127 165.1 0)
+		(fields_autoplaced yes)
+		(property "Reference" "#FLG041"
+			(at 130.81 165.735 0)
 			(hide yes)
 			(show_name no)
@@
 			(effects
 				(font
-					(size 0.762 0.762)
+					(size 1.27 1.27)
 				)
 			)
 		)
-		(property "Value" "VCC"
-			(at 127.0762 164.3888 0)
+		(property "Value" "PWR_FLAG"
+			(at 130.81 162.56 0)
 			(show_name no)
 			(do_not_autoplace no)
 			(effects
 				(font
-					(size 0.762 0.762)
+					(size 1.27 1.27)
 				)
 			)
 		)
 		(property "Footprint" ""
-			(at 127 167.64 0)
+			(at 130.81 167.64 0)
 			(hide yes)
 			(show_name no)
@@
 			(effects
 				(font
-					(size 1.524 1.524)
+					(size 1.27 1.27)
 				)
 			)
 		)
 		(property "Datasheet" ""
-			(at 127 167.64 0)
+			(at 130.81 167.64 0)
 			(hide yes)
 			(show_name no)
@@
 			(effects
 				(font
-					(size 1.524 1.524)
+					(size 1.27 1.27)
 				)
 			)
 		)
-		(property "Description" ""
-			(at 127 167.64 0)
+		(property "Description" "Special symbol for telling ERC where power comes from"
+			(at 130.81 167.64 0)
+			(hide yes)
 			(show_name no)
 			(do_not_autoplace no)
@@
 		)
 		(instances
-			(project ""
-				(path "/8dd0d409-5aaf-4e71-90f1-464fc883daa9"
-					(reference "#PWR02")
-					(unit 1)
-				)
-			)
 			(project "patinhofeio"
 				(path "/aca06203-542d-4682-a7e3-8839e24cce95/a95f568a-1ac6-4cdd-a7e9-88a5e8192029"
-					(reference "#PWR02")
+					(reference "#FLG041")
 					(unit 1)
 				)
@@
 	)
 	(symbol
-		(lib_id "CT5-8-rescue:PWR_FLAG-power")
-		(at 161.29 255.27 0)
+		(lib_id "power:VCC")
+		(at 123.19 167.64 0)
 		(unit 1)
 		(body_style 1)
@@
 		(in_pos_files yes)
 		(dnp no)
-		(property "Reference" "#FLG03"
-			(at 161.29 252.857 0)
+		(fields_autoplaced yes)
+		(property "Reference" "#PWR0136"
+			(at 123.19 171.45 0)
 			(hide yes)
 			(show_name no)
@@
 			(effects
 				(font
-					(size 0.762 0.762)
+					(size 1.27 1.27)
 				)
 			)
 		)
-		(property "Value" "PWR_FLAG"
-			(at 161.29 249.9868 0)
+		(property "Value" "VCC"
+			(at 123.19 162.56 0)
 			(show_name no)
 			(do_not_autoplace no)
 			(effects
 				(font
-					(size 0.762 0.762)
+					(size 1.27 1.27)
 				)
 			)
 		)
 		(property "Footprint" ""
-			(at 161.29 255.27 0)
+			(at 123.19 167.64 0)
 			(hide yes)
 			(show_name no)
@@
 			(effects
 				(font
-					(size 1.524 1.524)
+					(size 1.27 1.27)
 				)
 			)
 		)
 		(property "Datasheet" ""
-			(at 161.29 255.27 0)
+			(at 123.19 167.64 0)
 			(hide yes)
 			(show_name no)
@@
 			(effects
 				(font
-					(size 1.524 1.524)
+					(size 1.27 1.27)
 				)
 			)
 		)
-		(property "Description" ""
-			(at 161.29 255.27 0)
+		(property "Description" "Power symbol creates a global label with name \"VCC\""
+			(at 123.19 167.64 0)
+			(hide yes)
 			(show_name no)
 			(do_not_autoplace no)
@@
 		)
 		(instances
-			(project ""
-				(path "/8dd0d409-5aaf-4e71-90f1-464fc883daa9"
-					(reference "#FLG03")
-					(unit 1)
-				)
-			)
 			(project "patinhofeio"
 				(path "/aca06203-542d-4682-a7e3-8839e24cce95/a95f568a-1ac6-4cdd-a7e9-88a5e8192029"
-					(reference "#FLG03")
+					(reference "#PWR0136")
 					(unit 1)
 				)
@@
 	)
 	(symbol
-		(lib_id "CT5-8-rescue:GND")
+		(lib_id "power:GND")
 		(at 161.29 259.08 0)
 		(unit 1)
@@
 		(in_pos_files yes)
 		(dnp no)
-		(property "Reference" "#PWR04"
-			(at 161.29 259.08 0)
+		(fields_autoplaced yes)
+		(property "Reference" "#PWR0138"
+			(at 161.29 265.43 0)
 			(hide yes)
 			(show_name no)
@@
 			(effects
 				(font
-					(size 0.762 0.762)
+					(size 1.27 1.27)
 				)
 			)
 		)
 		(property "Value" "GND"
-			(at 161.29 260.858 0)
-			(hide yes)
+			(at 161.29 264.16 0)
 			(show_name no)
 			(do_not_autoplace no)
 			(effects
 				(font
-					(size 0.762 0.762)
+					(size 1.27 1.27)
 				)
 			)
@@
 			(effects
 				(font
-					(size 1.524 1.524)
+					(size 1.27 1.27)
 				)
 			)
@@
 			(effects
 				(font
-					(size 1.524 1.524)
+					(size 1.27 1.27)
 				)
 			)
 		)
-		(property "Description" ""
+		(property "Description" "Power symbol creates a global label with name \"GND\" , ground"
 			(at 161.29 259.08 0)
+			(hide yes)
 			(show_name no)
 			(do_not_autoplace no)
@@
 		)
 		(instances
-			(project ""
-				(path "/8dd0d409-5aaf-4e71-90f1-464fc883daa9"
-					(reference "#PWR04")
-					(unit 1)
-				)
-			)
 			(project "patinhofeio"
 				(path "/aca06203-542d-4682-a7e3-8839e24cce95/a95f568a-1ac6-4cdd-a7e9-88a5e8192029"
-					(reference "#PWR04")
+					(reference "#PWR0138")
 					(unit 1)
 				)

Commit message: Some initial fixing of ERC errors.
Changed lines of the file:
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@@
 	)
 	(junction
-		(at 130.81 170.18)
-		(diameter 0)
-		(color 0 0 0 0)
-	)
-	(junction
 		(at 350.52 172.72)
 		(diameter 0)
@@
 	)
 	(junction
-		(at 161.29 256.54)
-		(diameter 0)
-		(color 0 0 0 0)
-	)
-	(junction
 		(at 407.67 171.45)
 		(diameter 0)
@@
 	(wire
 		(pts
-			(xy 123.19 170.18) (xy 130.81 170.18)
-		)
-		(stroke
-			(width 0)
-			(type default)
-		)
-	)
-	(wire
-		(pts
 			(xy 266.7 250.19) (xy 271.78 250.19)
 		)
@@
 	(wire
 		(pts
-			(xy 130.81 167.64) (xy 130.81 170.18)
-		)
-		(stroke
-			(width 0)
-			(type default)
-		)
-	)
-	(wire
-		(pts
 			(xy 339.09 439.42) (xy 335.28 439.42)
 		)
@@
 	(wire
 		(pts
-			(xy 130.81 170.18) (xy 133.35 170.18)
+			(xy 123.19 170.18) (xy 133.35 170.18)
 		)
 		(stroke
@@
 	(wire
 		(pts
-			(xy 161.29 255.27) (xy 161.29 256.54)
-		)
-		(stroke
-			(width 0)
-			(type default)
-		)
-	)
-	(wire
-		(pts
 			(xy 486.41 261.62) (xy 483.87 261.62)
 		)
@@
 					(unit 1)
 				)
-			)
-		)
-	)
-	(symbol
-		(lib_id "CT5-8-rescue:PWR_FLAG-power")
-		(at 161.29 255.27 0)
-		(unit 1)
-		(body_style 1)
-		(exclude_from_sim no)
-		(in_bom yes)
-		(on_board yes)
-		(in_pos_files yes)
-		(dnp no)
-		(property "Reference" "#FLG03"
-			(at 161.29 252.857 0)
-			(hide yes)
-			(show_name no)
-			(do_not_autoplace no)
-			(effects
-				(font
-					(size 0.762 0.762)
-				)
-			)
-		)
-		(property "Value" "PWR_FLAG"
-			(at 161.29 249.9868 0)
-			(show_name no)
-			(do_not_autoplace no)
-			(effects
-				(font
-					(size 0.762 0.762)
-				)
-			)
-		)
-		(property "Footprint" ""
-			(at 161.29 255.27 0)
-			(hide yes)
-			(show_name no)
-			(do_not_autoplace no)
-			(effects
-				(font
-					(size 1.524 1.524)
-				)
-			)
-		)
-		(property "Datasheet" ""
-			(at 161.29 255.27 0)
-			(hide yes)
-			(show_name no)
-			(do_not_autoplace no)
-			(effects
-				(font
-					(size 1.524 1.524)
-				)
-			)
-		)
-		(property "Description" ""
-			(at 161.29 255.27 0)
-			(show_name no)
-			(do_not_autoplace no)
-			(effects
-				(font
-					(size 1.27 1.27)
-				)
-			)
-		)
-		(pin "1"
-		)
-		(instances
-			(project ""
-				(path "/8dd0d409-5aaf-4e71-90f1-464fc883daa9"
-					(reference "#FLG03")
-					(unit 1)
-				)
-			)
-			(project "patinhofeio"
-				(path "/aca06203-542d-4682-a7e3-8839e24cce95/a95f568a-1ac6-4cdd-a7e9-88a5e8192029"
-					(reference "#FLG03")
-					(unit 1)
-				)
-			)
-		)
-	)
-	(symbol
-		(lib_id "power:PWR_FLAG")
-		(at 130.81 167.64 0)
-		(unit 1)
-		(body_style 1)
-		(exclude_from_sim no)
-		(in_bom yes)
-		(on_board yes)
-		(in_pos_files yes)
-		(dnp no)
-		(fields_autoplaced yes)
-		(property "Reference" "#FLG041"
-			(at 130.81 165.735 0)
-			(hide yes)
-			(show_name no)
-			(do_not_autoplace no)
-			(effects
-				(font
-					(size 1.27 1.27)
-				)
-			)
-		)
-		(property "Value" "PWR_FLAG"
-			(at 130.81 162.56 0)
-			(show_name no)
-			(do_not_autoplace no)
-			(effects
-				(font
-					(size 1.27 1.27)
-				)
-			)
-		)
-		(property "Footprint" ""
-			(at 130.81 167.64 0)
-			(hide yes)
-			(show_name no)
-			(do_not_autoplace no)
-			(effects
-				(font
-					(size 1.27 1.27)
-				)
-			)
-		)
-		(property "Datasheet" ""
-			(at 130.81 167.64 0)
-			(hide yes)
-			(show_name no)
-			(do_not_autoplace no)
-			(effects
-				(font
-					(size 1.27 1.27)
-				)
-			)
-		)
-		(property "Description" "Special symbol for telling ERC where power comes from"
-			(at 130.81 167.64 0)
-			(hide yes)
-			(show_name no)
-			(do_not_autoplace no)
-			(effects
-				(font
-					(size 1.27 1.27)
-				)
-			)
-		)
-		(pin "1"
-		)
-		(instances
-			(project "patinhofeio"
-				(path "/aca06203-542d-4682-a7e3-8839e24cce95/a95f568a-1ac6-4cdd-a7e9-88a5e8192029"
-					(reference "#FLG041")
-					(unit 1)
-				)

Commit message: fixing a whole bunch more ERC errors
Connections:
- net +F3: no longer names the net of 1A_P16.8, 2D_P16.2
- net -PUG: no longer names the net of 1A_P16.10, 3B_P16.9
Other:
- moved on the sheet: 1A_P16D, 1A_P16E
Changed lines of the file:
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@@
 	(wire
 		(pts
-			(xy 332.74 245.11) (xy 332.74 264.16)
-		)
-		(stroke
-			(width 0)
-			(type default)
-		)
-	)
-	(wire
-		(pts
-			(xy 256.54 254) (xy 271.78 254)
+			(xy 271.78 275.59) (xy 283.21 275.59)
 		)
 		(stroke
@@
 	(wire
 		(pts
-			(xy 255.27 361.95) (xy 273.05 361.95)
+			(xy 332.74 245.11) (xy 332.74 264.16)
 		)
 		(stroke
@@
 	(wire
 		(pts
-			(xy 676.91 358.14) (xy 701.04 358.14)
+			(xy 256.54 254) (xy 271.78 254)
 		)
 		(stroke
@@
 	(wire
 		(pts
-			(xy 256.54 285.75) (xy 312.42 285.75)
+			(xy 255.27 361.95) (xy 273.05 361.95)
 		)
 		(stroke
@@
 	(wire
 		(pts
-			(xy 283.21 280.67) (xy 256.54 280.67)
+			(xy 256.54 280.67) (xy 283.21 280.67)
 		)
 		(stroke
@@
 	(wire
 		(pts
-			(xy 676.91 386.08) (xy 701.04 386.08)
+			(xy 287.02 285.75) (xy 312.42 285.75)
 		)
 		(stroke
@@
 	(wire
 		(pts
-			(xy 632.46 358.14) (xy 654.05 358.14)
-		)
-		(stroke
-			(width 0)
-			(type default)
-		)
-	)
-	(wire
-		(pts
 			(xy 379.73 447.04) (xy 406.4 447.04)
 		)
@@
 	(wire
 		(pts
+			(xy 229.87 280.67) (xy 233.68 280.67)
+		)
+		(stroke
+			(width 0)
+			(type default)
+		)
+	)
+	(wire
+		(pts
 			(xy 110.49 226.06) (xy 133.35 226.06)
 		)
@@
 	(wire
 		(pts
-			(xy 283.21 275.59) (xy 256.54 275.59)
-		)
-		(stroke
-			(width 0)
-			(type default)
-		)
-	)
-	(wire
-		(pts
 			(xy 407.67 168.91) (xy 407.67 171.45)
 		)
@@
 	(wire
 		(pts
-			(xy 632.46 386.08) (xy 654.05 386.08)
+			(xy 261.62 285.75) (xy 264.16 285.75)
 		)
 		(stroke
@@
 	(global_label "+PUG"
 		(shape input)
-		(at 632.46 358.14 180)
+		(at 229.87 280.67 180)
 		(effects
 			(font
@@
 		)
 		(property "Intersheetrefs" "${INTERSHEET_REFS}"
-			(at 632.46 358.14 0)
+			(at 229.87 280.67 0)
 			(hide yes)
 			(show_name no)
@@
 		)
 	)
-	(global_label "+F3"
-		(shape output)
-		(at 701.04 386.08 0)
-		(effects
-			(font
-				(size 1.524 1.524)
-			)
-			(justify left)
-		)
-		(property "Intersheetrefs" "${INTERSHEET_REFS}"
-			(at 701.04 386.08 0)
-			(hide yes)
-			(show_name no)
-			(do_not_autoplace no)
-			(effects
-				(font
-					(size 1.27 1.27)
-				)
-			)
-		)
-	)
 	(global_label "-F4"
 		(shape output)
@@
 		)
 	)
-	(global_label "-PUG"
-		(shape output)
-		(at 701.04 358.14 0)
-		(effects
-			(font
-				(size 1.524 1.524)
-			)
-			(justify left)
-		)
-		(property "Intersheetrefs" "${INTERSHEET_REFS}"
-			(at 701.04 358.14 0)
-			(hide yes)
-			(show_name no)
-			(do_not_autoplace no)
-			(effects
-				(font
-					(size 1.27 1.27)
-				)
-			)
-		)
-	)
 	(global_label "+SAESA"
 		(shape input)
@@
 		)
 	)
-	(global_label "-PUG"
-		(shape input)
-		(at 256.54 280.67 180)
-		(effects
-			(font
-				(size 1.524 1.524)
-			)
-			(justify right)
-		)
-		(property "Intersheetrefs" "${INTERSHEET_REFS}"
-			(at 256.54 280.67 0)
-			(hide yes)
-			(show_name no)
-			(do_not_autoplace no)
-			(effects
-				(font
-					(size 1.27 1.27)
-				)
-			)
-		)
-	)
 	(global_label "+S"
 		(shape output)
@@
 	(global_label "-F3"
 		(shape input)
-		(at 632.46 386.08 180)
-		(effects
-			(font
-				(size 1.524 1.524)
-			)
-			(justify right)
-		)
-		(property "Intersheetrefs" "${INTERSHEET_REFS}"
-			(at 632.46 386.08 0)
-			(hide yes)
-			(show_name no)
-			(do_not_autoplace no)
-			(effects
-				(font
-					(size 1.27 1.27)
-				)
-			)
-		)
-	)
-	(global_label "+F3"
-		(shape input)
-		(at 256.54 285.75 180)
+		(at 261.62 285.75 180)
 		(effects
 			(font
@@
 		)
 		(property "Intersheetrefs" "${INTERSHEET_REFS}"
-			(at 256.54 285.75 0)
+			(at 261.62 285.75 0)
 			(hide yes)
 			(show_name no)
@@
 	(global_label "-(F3.SUS.S)"
 		(shape input)
-		(at 256.54 275.59 180)
+		(at 271.78 275.59 180)
 		(effects
 			(font
@@
 		)
 		(property "Intersheetrefs" "${INTERSHEET_REFS}"
-			(at 256.54 275.59 0)
+			(at 271.78 275.59 0)
 			(hide yes)
 			(show_name no)
@@
 	(symbol
 		(lib_id "CT5-8-rescue:74HC04")
-		(at 665.48 358.14 0)
+		(at 245.11 280.67 0)
 		(unit 5)
 		(body_style 1)
@@
 		(dnp no)
 		(property "Reference" "1A_P16"
-			(at 669.29 355.6 0)
+			(at 248.92 278.13 0)
 			(show_name no)
 			(do_not_autoplace no)
@@
 		)
 		(property "Value" "74HC04"
-			(at 670.56 360.68 0)
+			(at 250.19 283.21 0)
 			(show_name no)
 			(do_not_autoplace no)
@@
 		)
 		(property "Footprint" ""
-			(at 665.48 358.14 0)
+			(at 245.11 280.67 0)
 			(show_name no)
 			(do_not_autoplace no)
@@
 		)
 		(property "Datasheet" ""
-			(at 665.48 358.14 0)
+			(at 245.11 280.67 0)
 			(show_name no)
 			(do_not_autoplace no)
@@
 		)
 		(property "Description" ""
-			(at 665.48 358.14 0)
+			(at 245.11 280.67 0)
 			(show_name no)
 			(do_not_autoplace no)
@@
 	(symbol
 		(lib_id "CT5-8-rescue:74HC04")
-		(at 665.48 386.08 0)
+		(at 275.59 285.75 0)
 		(unit 4)
 		(body_style 1)
@@
 		(dnp no)
 		(property "Reference" "1A_P16"
-			(at 669.29 383.54 0)
+			(at 279.4 283.21 0)
 			(show_name no)
 			(do_not_autoplace no)
@@
 		)
 		(property "Value" "74HC04"
-			(at 670.56 388.62 0)
+			(at 280.67 288.29 0)
 			(show_name no)
 			(do_not_autoplace no)
@@
 		)
 		(property "Footprint" ""
-			(at 665.48 386.08 0)
+			(at 275.59 285.75 0)
 			(show_name no)
 			(do_not_autoplace no)
@@
 		)
 		(property "Datasheet" ""
-			(at 665.48 386.08 0)
+			(at 275.59 285.75 0)
 			(show_name no)
 			(do_not_autoplace no)
@@
 		)
 		(property "Description" ""
-			(at 665.48 386.08 0)
+			(at 275.59 285.75 0)
 			(show_name no)
 			(do_not_autoplace no)

Commit message: wip
Parts:
- removed 1A_P16, 1D_P16: 74HC04, symbol CT5-8-rescue:74HC04
- removed 1B_P16, 3C_P16: 74LS40, symbol CT5-8-rescue:74LS40
- removed 1C_P16: 74HC02, symbol CT5-8-rescue:74HC02
- removed 2A_P16, 2D_P16, 3B_P16: 7400, symbol CT5-8-rescue:7400
- removed 3A_P16: 74LS10, symbol CT5-8-rescue:74LS10
- added 1A_P16, 1D_P16: 74LS04, symbol 74xx:74LS04
- added 1B_P16, 3C_P16: 74LS40, symbol 74xx:74LS40
- added 1C_P16: 74LS02, symbol 74xx:74LS02
- added 2A_P16, 2D_P16, 3B_P16: 74LS00, symbol 74xx:74LS00
- added 3A_P16: 74LS10, symbol 74xx:74LS10
Connections:
- net +(F1+F2): now also 2A_P16.6
- net +(F2.SAESA): now also 1C_P16.1, 1D_P16.5, 3B_P16.1
- net +F1: now also 1A_P16.12, 2D_P16.5, 3A_P16.1, 3B_P16.13
- net +MICG1: now also 2A_P16.1
- net +MICG2A: now also 2A_P16.10, 3A_P16.2
- net +PUG: now also 1A_P16.11, 2A_P16.13
- net +PUL: now also 1A_P16.3
- net +RI_7: now also 2A_P16.2
- net +S: now also 1D_P16.13, 3B_P16.2
- net +SAESA: now also 1A_P16.1
- net +SALMIC: now also 2A_P16.9, 3A_P16.13
- net +SUS: now also 2D_P16.9
- net +VUQ: now also 1D_P16.2
- net -(F1.(MICG2A.SALMIC+PUL)): now also 1B_P16.1, 3B_P16.11
- net -(F2.SAESA): now also 1D_P16.6, 3A_P16.10
- net -(F2.SAESA.S): now also 1B_P16.2, 3B_P16.3
- net -(F3.SUS.S): now also 2D_P16.8, 3A_P16.9, 3B_P16.10
- net -(MICG2A.SALMIC.F1): now also 3A_P16.12, 3A_P16.5
- net -F1: now also 1A_P16.13, 2A_P16.4
- net -F2: now also 1C_P16.2, 2A_P16.5
- net -F3: now also 1A_P16.9, 1C_P16.5
- net -F4: now also 1A_P16.5
- net -PUL: now also 1A_P16.4, 3A_P16.4, 3B_P16.5
- net -SAESA: now also 1A_P16.2, 1C_P16.3
- net -SINTA: now also 3C_P16.6
- net GND: now also 1A_P16.7 (GND), 1B_P16.7 (GND), 1C_P16.7 (GND), 1D_P16.7 (GND), 2A_P16.7 (GND), 2D_P16.7 (GND), 3A_P16.7 (GND), 3B_P16.14 (VCC), 3C_P16.7 (GND)
- net VCC: now also 1A_P16.14 (VCC), 1B_P16.14 (VCC), 1C_P16.14 (VCC), 1D_P16.14 (VCC), 2A_P16.14 (VCC), 2D_P16.14 (VCC), 3A_P16.14 (VCC), 3B_P16.7 (GND), 3C_P16.14 (VCC)
- net at 2B_P16.13: now also 3A_P16.8
- net at 2B_P16.4: now also 1B_P16.6
- net at 2B_P16.8: now also 1D_P16.1
- net at 2C_P16.6: now also 1D_P16.3
- new net: 1A_P16.10, 3B_P16.9
- new net: 2D_P16.1, 3B_P16.8
- new net: 1C_P16.4, 2D_P16.10
- new net: 1C_P16.6, 1D_P16.12
- new net: 2A_P16.8, 3B_P16.4
- new net: 3B_P16.12, 3B_P16.6
- new net: 1A_P16.6, 2A_P16.12
- new net: 1D_P16.4, 3C_P16.1, 3C_P16.2, 3C_P16.4, 3C_P16.5
- new net: 2D_P16.6, 3A_P16.11
- new net: 2A_P16.3, 3A_P16.3
- new net: 2D_P16.4, 3A_P16.6
- new net: 1B_P16.4, 2D_P16.3
- new net: 1B_P16.5, 2A_P16.11
- new net: 1A_P16.8, 2D_P16.2
- no-connect marks 48 -> 71
Other:
- moved on the sheet: 2B_P16, 2C_P16A

Commit message: wip + PDF plot
Other:
- moved on the sheet: 1A_P16G, 1B_P16B, 1B_P16C, 1C_P16C, 1C_P16D, 1C_P16E, 1D_P16D, 1D_P16E, 1D_P16G, 2A_P16E, 2D_P16D, 2D_P16E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
