File: CT3-6/CT3-6.sch (KiCad schematic (older format))
At the start: 26 parts

Commit message: terminei a transcrição do esquema da placa CT3-6
Connections:
- net +F2_(P14) is gone; now on net +F2: 1B_P14.4, 2A_P14.6, 3A_P14.4
- net +F3_(P14) is gone; now on net +F3: 1B_P14.1, 1E_P14.10, 3A_P14.12, 4B_P14.12
- net -SUS is gone; now on net +SUS: 4B_P14.9
- net 2B3 is gone; now on net +(PARTIDA+RODA+(-MP)): 1C_P14.5
- net +(CAC+SOM): now also CONECTOR_P14.25
- net +(PAN+PAZ): now also CONECTOR_P14.41 (P41)
- net +ARA: now also CONECTOR_P14.62 (P62)
- net +CASP: now also CONECTOR_P14.6 (P6)
- net +CP: now also CONECTOR_P14.9 (P9)
- net +DUPL_SINAL: now also CONECTOR_P14.69 (P69)
- net +IME: now also CONECTOR_P14.42 (P42)
- net +INDICE: now also CONECTOR_P14.7 (P7)
- net +L/R: now also CONECTOR_P14.10 (P10)
- net +MICRO: now also CONECTOR_P14.3 (P3)
- net +MP: now also CONECTOR_P14.8 (P8)
- net +PLI: now also CONECTOR_P14.40 (P40)
- net +PUG: now also CONECTOR_P14.63 (P63)
- net +RD_0: now also CONECTOR_P14.65 (P65)
- net +RD_1: now also CONECTOR_P14.64 (P64)
- net +RODA: now also CONECTOR_P14.44 (P44)
- net +S: now also CONECTOR_P14.32 (P32)
- net +SAE: now also CONECTOR_P14.59 (P59)
- net +SAEFU: now also CONECTOR_P14.28 (P28)
- net +SAESA: now also CONECTOR_P14.30 (P30)
- net +SHIFT: now also CONECTOR_P14.15 (P15)
- net +SHIFT_LEFT: now also CONECTOR_P14.67 (P67)
- net +SHIFT_RIGHT: now also CONECTOR_P14.68 (P68)
- net +SUS: now also CONECTOR_P14.19 (P19)
- net +T(1/2)34: now also CONECTOR_P14.37 (P37)
- net +T0: now also CONECTOR_P14.56 (P56)
- net +T012: now also CONECTOR_P14.58 (P58)
- net +T0123: now also CONECTOR_P14.55 (P55)
- net +T1: now also CONECTOR_P14.20 (P20)
- net +T2: now also CONECTOR_P14.27 (P27)
- net +T3: now also CONECTOR_P14.22 (P22)
- net +T34: now also CONECTOR_P14.38 (P38)
- net +TRI: now also CONECTOR_P14.5 (P5)
- net +TRO: now also CONECTOR_P14.4 (P4)
- net -CF1: now also CONECTOR_P14.11 (P11)
- net -C_RD: now also CONECTOR_P14.61 (P61)
- net -F1: now also CONECTOR_P14.2 (P2)
- net -F2: now also CONECTOR_P14.46 (P46)
- net -F3: now also CONECTOR_P14.18 (P18)
- net -F4: now also CONECTOR_P14.23 (P23)
- net -F5: now also CONECTOR_P14.14 (P14)
- net -FUNÇÃO: now also CONECTOR_P14.26 (P26)
- net -M1: now also CONECTOR_P14.54 (P54)
- net -M3: now also CONECTOR_P14.39 (P39)
- net -M4: now also CONECTOR_P14.24 (P24)
- net -RDZ: now also CONECTOR_P14.29 (P29)
- net -SENTIDO: now also CONECTOR_P14.31 (P31)
- net -SHIAC: now also CONECTOR_P14.66 (P66)
- net -T(1/2)34: now also CONECTOR_P14.33 (P33)
- net -T12: now also CONECTOR_P14.12 (P12)
- net -T70: now also CONECTOR_P14.34 (P34)
- net GND: now also CONECTOR_P14.70 (P70)
- net MANEN: now also CONECTOR_P14.57 (P57)
- net VCC: now also CONECTOR_P14.1 (P1)
- net +(PARTIDA+RODA+(-MP)): now reaches 1C_P14.12, 2B_P14.3
- net +(TRO+TRI)_(P14) renamed +(TRO+TRI)
- net +F1_(P14) renamed +F1
- net +PARTIDA renamed -PARTIDA
- net -PARTIDA: now also CONECTOR_P14.43 (P43)
- net -(TRO+TRI)_(P14) renamed -(TRO+TRI)
- net =T2 renamed -T2
- net -T2: now also CONECTOR_P14.60 (P60)
- removed net ?: CONECTOR_P14.1 (P1), CONECTOR_P14.10 (P10), CONECTOR_P14.11 (P11), CONECTOR_P14.12 (P12), CONECTOR_P14.13 (P13), CONECTOR_P14.14 (P14), CONECTOR_P14.15 (P15), CONECTOR_P14.16 (P16), CONECTOR_P14.17 (P17), CONECTOR_P14.18 (P18), CONECTOR_P14.19 (P19), CONECTOR_P14.2 (P2), CONECTOR_P14.20 (P20), CONECTOR_P14.21 (P21), CONECTOR_P14.22 (P22), CONECTOR_P14.23 (P23), CONECTOR_P14.24 (P24), CONECTOR_P14.25, CONECTOR_P14.26 (P26), CONECTOR_P14.27 (P27), CONECTOR_P14.28 (P28), CONECTOR_P14.29 (P29), CONECTOR_P14.3 (P3), CONECTOR_P14.30 (P30), CONECTOR_P14.31 (P31), CONECTOR_P14.32 (P32), CONECTOR_P14.33 (P33), CONECTOR_P14.34 (P34), CONECTOR_P14.35 (P35), CONECTOR_P14.36 (P36), CONECTOR_P14.37 (P37), CONECTOR_P14.38 (P38), CONECTOR_P14.39 (P39), CONECTOR_P14.4 (P4), CONECTOR_P14.40 (P40), CONECTOR_P14.41 (P41), CONECTOR_P14.42 (P42), CONECTOR_P14.43 (P43), CONECTOR_P14.44 (P44), CONECTOR_P14.45 (P45), CONECTOR_P14.46 (P46), CONECTOR_P14.47 (P47), CONECTOR_P14.48 (P48), CONECTOR_P14.49 (P49), CONECTOR_P14.5 (P5), CONECTOR_P14.50 (P50), CONECTOR_P14.51 (P51), CONECTOR_P14.52 (P52), CONECTOR_P14.53 (P53), CONECTOR_P14.54 (P54), CONECTOR_P14.55 (P55), CONECTOR_P14.56 (P56), CONECTOR_P14.57 (P57), CONECTOR_P14.58 (P58), CONECTOR_P14.59 (P59), CONECTOR_P14.6 (P6), CONECTOR_P14.60 (P60), CONECTOR_P14.61 (P61), CONECTOR_P14.62 (P62), CONECTOR_P14.63 (P63), CONECTOR_P14.64 (P64), CONECTOR_P14.65 (P65), CONECTOR_P14.66 (P66), CONECTOR_P14.67 (P67), CONECTOR_P14.68 (P68), CONECTOR_P14.69 (P69), CONECTOR_P14.7 (P7), CONECTOR_P14.70 (P70), CONECTOR_P14.8 (P8), CONECTOR_P14.9 (P9)
- no-connect marks 0 -> 14
