File: CT3-6/CT3-6.kicad_sch (KiCad schematic)
At the start: 26 parts

Commit message: These are updated files after I loaded the project on a new version of KICAD
Parts:
- 1A_P14, 1B_P14, 1C_P14, 1E_P14, 2A_P14, 2B_P14, 2C_P14, 2D_P14, 2E_P14, 3A_P14, 3B_P14, 3C_P14, 3D_P14, 4A_P14, 4B_P14, 4C_P14, 4D_P14, 5A_P14, 5B_P14, 5C_P14, 5D_P14, 5E_P14: footprint ~ -> (none)
