File: FIN-8/FIN-8.sch (KiCad schematic (older format))
At the start: 1 part

Commit message: esquematico da placa FIN-8
Parts:
- added 1A_P6, 5E_P6, 5F_P6: 74LS04, symbol 74LS04
- added 1B_P6: 74LS10, symbol 74LS10
- added 1C_P6: 74LS02, symbol 74LS02
- added 1E_P6, 1F_P6, 2E_P6, 2F_P6, 3A_P6, 3B_P6, 3C_P6, 3D_P6, 3E_P6, 3F_P6, 4E_P6, 4F_P6, 5A_P6, 5B_P6, 5C_P6: 74LS13, symbol 74LS13
- added R1, R2, R3, R4, R5, R6, R7: R, symbol R
Connections:
- removed net ?: CONECTOR_P6.1 (P1), CONECTOR_P6.10 (P10), CONECTOR_P6.11 (P11), CONECTOR_P6.12 (P12), CONECTOR_P6.13 (P13), CONECTOR_P6.14 (P14), CONECTOR_P6.15 (P15), CONECTOR_P6.16 (P16), CONECTOR_P6.17 (P17), CONECTOR_P6.18 (P18), CONECTOR_P6.19 (P19), CONECTOR_P6.2 (P2), CONECTOR_P6.20 (P20), CONECTOR_P6.21 (P21), CONECTOR_P6.22 (P22), CONECTOR_P6.23 (P23), CONECTOR_P6.24 (P24), CONECTOR_P6.25, CONECTOR_P6.26 (P26), CONECTOR_P6.27 (P27), CONECTOR_P6.28 (P28), CONECTOR_P6.29 (P29), CONECTOR_P6.3 (P3), CONECTOR_P6.30 (P30), CONECTOR_P6.31 (P31), CONECTOR_P6.32 (P32), CONECTOR_P6.33 (P33), CONECTOR_P6.34 (P34), CONECTOR_P6.35 (P35), CONECTOR_P6.36 (P36), CONECTOR_P6.37 (P37), CONECTOR_P6.38 (P38), CONECTOR_P6.39 (P39), CONECTOR_P6.4 (P4), CONECTOR_P6.40 (P40), CONECTOR_P6.41 (P41), CONECTOR_P6.42 (P42), CONECTOR_P6.43 (P43), CONECTOR_P6.44 (P44), CONECTOR_P6.45 (P45), CONECTOR_P6.46 (P46), CONECTOR_P6.47 (P47), CONECTOR_P6.48 (P48), CONECTOR_P6.49 (P49), CONECTOR_P6.5 (P5), CONECTOR_P6.50 (P50), CONECTOR_P6.51 (P51), CONECTOR_P6.52 (P52), CONECTOR_P6.53 (P53), CONECTOR_P6.54 (P54), CONECTOR_P6.55 (P55), CONECTOR_P6.56 (P56), CONECTOR_P6.57 (P57), CONECTOR_P6.58 (P58), CONECTOR_P6.59 (P59), CONECTOR_P6.6 (P6), CONECTOR_P6.60 (P60), CONECTOR_P6.61 (P61), CONECTOR_P6.62 (P62), CONECTOR_P6.63 (P63), CONECTOR_P6.64 (P64), CONECTOR_P6.65 (P65), CONECTOR_P6.66 (P66), CONECTOR_P6.67 (P67), CONECTOR_P6.68 (P68), CONECTOR_P6.69 (P69), CONECTOR_P6.7 (P7), CONECTOR_P6.70 (P70), CONECTOR_P6.8 (P8), CONECTOR_P6.9 (P9)
- new net: 5B_P6.1, 5B_P6.12, 5B_P6.13, 5B_P6.2, R6.2
- new net: 5C_P6.1, 5C_P6.12, 5C_P6.13, 5C_P6.2, R7.2
- new net: 1A_P6.1, 1B_P6.6
- new net: 1A_P6.13, 1B_P6.8
- new net: 1B_P6.12, 1B_P6.3, 1B_P6.4, 1B_P6.5
- new net: 1B_P6.1, 1C_P6.13
- new net: 1B_P6.13, 1C_P6.10
- new net: 1B_P6.2, 1C_P6.1
- new net: 5A_P6.1, 5A_P6.10, 5A_P6.12, 5A_P6.13, 5A_P6.2, 5A_P6.4, R5.2
- new net: 3D_P6.1, 3D_P6.12, 3D_P6.13, 3D_P6.2, R4.2
- new net: 3A_P6.1, 3A_P6.12, 3A_P6.13, 3A_P6.2, R3.2
- new net: 3B_P6.1, 3B_P6.12, 3B_P6.13, 3B_P6.2, R2.2
- new net: 3C_P6.1, 3C_P6.12, 3C_P6.13, 3C_P6.2, R1.2
- new net +AC_0: 3C_P6.4, CONECTOR_P6.49 (P49)
- new net +AC_1: 3C_P6.9, CONECTOR_P6.50 (P50)
- new net +AC_2: 3B_P6.4, CONECTOR_P6.51 (P51)
- new net +AC_3: 3B_P6.9, CONECTOR_P6.52 (P52)
- new net +AC_4: 3A_P6.5, CONECTOR_P6.53 (P53)
- new net +AC_5: 3A_P6.9, CONECTOR_P6.54 (P54)
- new net +AC_6: 3D_P6.5, CONECTOR_P6.55 (P55)
- new net +AC_7: 3D_P6.9, CONECTOR_P6.56 (P56)
- new net +RD_4: 5F_P6.9, CONECTOR_P6.69 (P69)
- new net +RD_4*: 1F_P6.13, 1F_P6.2, 2F_P6.13, 2F_P6.2, 3F_P6.13, 3F_P6.2, 4F_P6.13, 4F_P6.2, 5F_P6.4
- new net +RD_5: 5E_P6.13, CONECTOR_P6.34 (P34)
- new net +RD_5*: 1E_P6.10, 1E_P6.5, 1F_P6.10, 1F_P6.5, 2E_P6.10, 2E_P6.5, 2F_P6.10, 2F_P6.5, 5E_P6.4
- new net +RD_6: 5F_P6.13, CONECTOR_P6.68 (P68)
- new net +RD_6*: 1E_P6.12, 1E_P6.4, 1F_P6.12, 1F_P6.4, 3E_P6.12, 3E_P6.4, 3F_P6.12, 3F_P6.4, 5F_P6.2
- new net +RD_7: 5E_P6.11, CONECTOR_P6.33 (P33)
- new net +RD_7*: 1E_P6.1, 1F_P6.1, 2E_P6.1, 2F_P6.1, 3E_P6.1, 3F_P6.1, 4E_P6.1, 4F_P6.1, 5E_P6.2
- new net +RI_4: 5B_P6.9, CONECTOR_P6.31 (P31)
- new net +RI_5: 5B_P6.5, CONECTOR_P6.66 (P66)
- new net +RI_6: 5C_P6.10, CONECTOR_P6.32 (P32)
- new net +RI_7: 5C_P6.4, CONECTOR_P6.67 (P67)
- new net +T4: 5A_P6.5, CONECTOR_P6.28 (P28)
- new net +T6: 5A_P6.9, CONECTOR_P6.29 (P29)
- new net +TUBE: 1B_P6.10, 1B_P6.9, CONECTOR_P6.8 (P8)
- new net -COM_0: 4E_P6.8, CONECTOR_P6.60 (P60)
- new net -COM_1: 4E_P6.6, CONECTOR_P6.25
- new net -COM_10: 3F_P6.8, CONECTOR_P6.39 (P39)
- new net -COM_11: 3F_P6.6, CONECTOR_P6.4 (P4)
- new net -COM_12: 2F_P6.8, CONECTOR_P6.38 (P38)
- new net -COM_13: 2F_P6.6, CONECTOR_P6.3 (P3)
- new net -COM_14: 1F_P6.8, CONECTOR_P6.37 (P37)
- new net -COM_15: 1C_P6.8, 1F_P6.6, CONECTOR_P6.2 (P2)
- new net -COM_2: 3E_P6.8, CONECTOR_P6.59 (P59)
- new net -COM_3: 3E_P6.6, CONECTOR_P6.24 (P24)
- new net -COM_4: 2E_P6.8, CONECTOR_P6.58 (P58)
- new net -COM_5: 2E_P6.6, CONECTOR_P6.23 (P23)
- new net -COM_6: 1E_P6.8, CONECTOR_P6.57 (P57)
- new net -COM_7: 1E_P6.6, CONECTOR_P6.22 (P22)
- new net -COM_8: 4F_P6.8, CONECTOR_P6.40 (P40)
- new net -COM_9: 4F_P6.6, CONECTOR_P6.5 (P5)
- new net -END_0: 1C_P6.11, 5B_P6.8, CONECTOR_P6.62 (P62)
- new net -END_1: 1C_P6.12, 5B_P6.6, CONECTOR_P6.27 (P27)
- new net -END_2: 1C_P6.3, 5C_P6.8, CONECTOR_P6.61 (P61)
- new net -END_3: 1C_P6.2, 5C_P6.6, CONECTOR_P6.26 (P26)
- new net -PED_INT: 1A_P6.12, CONECTOR_P6.7 (P7)
- new net -PED_INT_PAINEL: 1B_P6.11, CONECTOR_P6.9 (P9)
- new net -RD_4: 1E_P6.13, 1E_P6.2, 2E_P6.13, 2E_P6.2, 3E_P6.13, 3E_P6.2, 4E_P6.13, 4E_P6.2, 5F_P6.3, 5F_P6.8
- new net -RD_5: 3E_P6.10, 3E_P6.5, 3F_P6.10, 3F_P6.5, 4E_P6.10, 4E_P6.5, 4F_P6.10, 4F_P6.5, 5E_P6.12, 5E_P6.3
- new net -RD_6: 2E_P6.12, 2E_P6.4, 2F_P6.12, 2F_P6.4, 4E_P6.12, 4E_P6.4, 4F_P6.12, 4F_P6.4, 5F_P6.1, 5F_P6.12
- new net -RD_7: 1E_P6.9, 1F_P6.9, 2E_P6.9, 2F_P6.9, 3E_P6.9, 3F_P6.9, 4E_P6.9, 4F_P6.9, 5E_P6.1, 5E_P6.10
- new net -SENTIDO: 1A_P6.2, CONECTOR_P6.6 (P6)
- new net -SINTA: 1C_P6.9, CONECTOR_P6.10 (P10)
- new net -T4*: 5A_P6.6, CONECTOR_P6.63 (P63)
- new net -T6*: 5A_P6.8, CONECTOR_P6.64 (P64)
- new net DAD_0: 3C_P6.6, CONECTOR_P6.14 (P14)
- new net DAD_1: 3C_P6.8, CONECTOR_P6.15 (P15)
- new net DAD_2: 3B_P6.6, CONECTOR_P6.16 (P16)
- new net DAD_3: 3B_P6.8, CONECTOR_P6.17 (P17)
- new net DAD_4: 3A_P6.6, CONECTOR_P6.18 (P18)
- new net DAD_5: 3A_P6.8, CONECTOR_P6.19 (P19)
- new net DAD_6: 3D_P6.6, CONECTOR_P6.20 (P20)
- new net DAD_7: 3D_P6.8, CONECTOR_P6.21 (P21)
- new net GND: 1A_P6.7 (GND), 1A_P6.7 (GND), 1B_P6.7 (GND), 1B_P6.7 (GND), 1B_P6.7 (GND), 1C_P6.7 (GND), 1C_P6.7 (GND), 1C_P6.7 (GND), 1E_P6.7 (GND), 1E_P6.7 (GND), 1F_P6.7 (GND), 1F_P6.7 (GND), 2E_P6.7 (GND), 2E_P6.7 (GND), 2F_P6.7 (GND), 2F_P6.7 (GND), 3A_P6.7 (GND), 3A_P6.7 (GND), 3B_P6.7 (GND), 3B_P6.7 (GND), 3C_P6.7 (GND), 3C_P6.7 (GND), 3D_P6.7 (GND), 3D_P6.7 (GND), 3E_P6.7 (GND), 3E_P6.7 (GND), 3F_P6.7 (GND), 3F_P6.7 (GND), 4E_P6.7 (GND), 4E_P6.7 (GND), 4F_P6.7 (GND), 4F_P6.7 (GND), 5A_P6.7 (GND), 5A_P6.7 (GND), 5B_P6.7 (GND), 5B_P6.7 (GND), 5C_P6.7 (GND), 5C_P6.7 (GND), 5E_P6.7 (GND), 5E_P6.7 (GND), 5E_P6.7 (GND), 5E_P6.7 (GND), 5F_P6.7 (GND), 5F_P6.7 (GND), 5F_P6.7 (GND), 5F_P6.7 (GND), CONECTOR_P6.70 (P70)
- new net MANDA: 3A_P6.10, 3A_P6.4, 3B_P6.10, 3B_P6.5, 3C_P6.10, 3C_P6.5, 3D_P6.10, 3D_P6.4, CONECTOR_P6.48 (P48)
- new net MANEN: 5B_P6.10, 5B_P6.4, 5C_P6.5, 5C_P6.9, CONECTOR_P6.65 (P65)
- new net VCC: 1A_P6.14 (VCC), 1A_P6.14 (VCC), 1B_P6.14 (VCC), 1B_P6.14 (VCC), 1B_P6.14 (VCC), 1C_P6.14 (VCC), 1C_P6.14 (VCC), 1C_P6.14 (VCC), 1E_P6.14 (VCC), 1E_P6.14 (VCC), 1F_P6.14 (VCC), 1F_P6.14 (VCC), 2E_P6.14 (VCC), 2E_P6.14 (VCC), 2F_P6.14 (VCC), 2F_P6.14 (VCC), 3A_P6.14 (VCC), 3A_P6.14 (VCC), 3B_P6.14 (VCC), 3B_P6.14 (VCC), 3C_P6.14 (VCC), 3C_P6.14 (VCC), 3D_P6.14 (VCC), 3D_P6.14 (VCC), 3E_P6.14 (VCC), 3E_P6.14 (VCC), 3F_P6.14 (VCC), 3F_P6.14 (VCC), 4E_P6.14 (VCC), 4E_P6.14 (VCC), 4F_P6.14 (VCC), 4F_P6.14 (VCC), 5A_P6.14 (VCC), 5A_P6.14 (VCC), 5B_P6.14 (VCC), 5B_P6.14 (VCC), 5C_P6.14 (VCC), 5C_P6.14 (VCC), 5E_P6.14 (VCC), 5E_P6.14 (VCC), 5E_P6.14 (VCC), 5E_P6.14 (VCC), 5F_P6.14 (VCC), 5F_P6.14 (VCC), 5F_P6.14 (VCC), 5F_P6.14 (VCC), CONECTOR_P6.1 (P1), R1.1, R2.1, R3.1, R4.1, R5.1, R6.1, R7.1
- no-connect marks 0 -> 13
Other:
- moved on the sheet: CONECTOR_P6
