File: FIN-8/FIN-8.kicad_sch (KiCad schematic)
At the start: 28 parts

Commit message: cleaning up references
Parts:
- renumbered R1 to R1_P6, R2 to R2_P6, R3 to R3_P6, R4 to R4_P6, R5 to R5_P6, R6 to R6_P6, R7 to R7_P6

Commit message: Some initial fixing of ERC errors.
Changed lines of the file:
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@@
 	)
 	(junction
-		(at 58.42 36.83)
-		(diameter 0)
-		(color 0 0 0 0)
-	)
-	(junction
 		(at 260.35 134.62)
 		(diameter 0)
@@
 	)
 	(junction
-		(at 129.54 123.19)
-		(diameter 0)
-		(color 0 0 0 0)
-	)
-	(junction
 		(at 468.63 299.72)
 		(diameter 0)
@@
 	(wire
 		(pts
-			(xy 129.54 119.38) (xy 129.54 123.19)
-		)
-		(stroke
-			(width 0)
-			(type default)
-		)
-	)
-	(wire
-		(pts
 			(xy 66.04 293.37) (xy 50.8 293.37)
 		)
@@
 	(wire
 		(pts
-			(xy 58.42 31.75) (xy 58.42 36.83)
-		)
-		(stroke
-			(width 0)
-			(type default)
-		)
-	)
-	(wire
-		(pts
 			(xy 355.6 297.18) (xy 360.68 297.18)
 		)
@@
 	(wire
 		(pts
-			(xy 50.8 36.83) (xy 58.42 36.83)
-		)
-		(stroke
-			(width 0)
-			(type default)
-		)
-	)
-	(wire
-		(pts
 			(xy 100.33 283.21) (xy 96.52 283.21)
 		)
@@
 	(wire
 		(pts
-			(xy 58.42 36.83) (xy 63.5 36.83)
+			(xy 50.8 36.83) (xy 63.5 36.83)
 		)
 		(stroke
@@
 				)
 			)
-		)
-	)
-	(symbol
-		(lib_id "FIN-8-rescue:PWR_FLAG-power")
-		(at 129.54 119.38 0)
-		(unit 1)
-		(body_style 1)
-		(exclude_from_sim no)
-		(in_bom yes)
-		(on_board yes)
-		(in_pos_files yes)
-		(dnp no)
-		(property "Reference" "#FLG09"
-			(at 129.54 116.967 0)
-			(hide yes)
-			(show_name no)
-			(do_not_autoplace no)
-			(effects
-				(font
-					(size 0.762 0.762)
-				)
-			)
-		)
-		(property "Value" "PWR_FLAG"
-			(at 129.54 114.0968 0)
-			(show_name no)
-			(do_not_autoplace no)
-			(effects
-				(font
-					(size 0.762 0.762)
-				)
-			)
-		)
-		(property "Footprint" ""
-			(at 129.54 119.38 0)
-			(hide yes)
-			(show_name no)
-			(do_not_autoplace no)
-			(effects
-				(font
-					(size 1.524 1.524)
-				)
-			)
-		)
-		(property "Datasheet" ""
-			(at 129.54 119.38 0)
-			(hide yes)
-			(show_name no)
-			(do_not_autoplace no)
-			(effects
-				(font
-					(size 1.524 1.524)
-				)
-			)
-		)
-		(property "Description" ""
-			(at 129.54 119.38 0)
-			(show_name no)
-			(do_not_autoplace no)
-			(effects
-				(font
-					(size 1.27 1.27)
-				)
-			)
-		)
-		(pin "1"
-		)
-		(instances
-			(project ""
-				(path "/8b6e24fe-0a10-4897-8420-99aac79caa8b"
-					(reference "#FLG09")
-					(unit 1)
-				)
-			)
-			(project "patinhofeio"
-				(path "/aca06203-542d-4682-a7e3-8839e24cce95/8431fe73-c409-4911-974c-c727a5dc461e"
-					(reference "#FLG09")
-					(unit 1)
-				)
-			)
-		)
-	)
-	(symbol
-		(lib_id "FIN-8-rescue:PWR_FLAG-power")
-		(at 58.42 31.75 0)
-		(unit 1)
-		(body_style 1)
-		(exclude_from_sim no)
-		(in_bom yes)
-		(on_board yes)
-		(in_pos_files yes)
-		(dnp no)
-		(property "Reference" "#FLG010"
-			(at 58.42 29.337 0)
-			(hide yes)
-			(show_name no)
-			(do_not_autoplace no)
-			(effects
-				(font
-					(size 0.762 0.762)
-				)
-			)
-		)
-		(property "Value" "PWR_FLAG"
-			(at 58.42 26.4668 0)
-			(show_name no)
-			(do_not_autoplace no)
-			(effects
-				(font
-					(size 0.762 0.762)
-				)
-			)
-		)
-		(property "Footprint" ""
-			(at 58.42 31.75 0)
-			(hide yes)
-			(show_name no)
-			(do_not_autoplace no)
-			(effects
-				(font
-					(size 1.524 1.524)
-				)
-			)
-		)
-		(property "Datasheet" ""
-			(at 58.42 31.75 0)
-			(hide yes)
-			(show_name no)
-			(do_not_autoplace no)
-			(effects
-				(font
-					(size 1.524 1.524)
-				)
-			)
-		)
-		(property "Description" ""
-			(at 58.42 31.75 0)
-			(show_name no)
-			(do_not_autoplace no)
-			(effects
-				(font
-					(size 1.27 1.27)
-				)
-			)
-		)
-		(pin "1"
-		)
-		(instances
-			(project ""
-				(path "/8b6e24fe-0a10-4897-8420-99aac79caa8b"
-					(reference "#FLG010")
-					(unit 1)
-				)
-			)
-			(project "patinhofeio"
-				(path "/aca06203-542d-4682-a7e3-8839e24cce95/8431fe73-c409-4911-974c-c727a5dc461e"
-					(reference "#FLG010")
-					(unit 1)
-				)
-			)

Commit message: fix a whole bunch of errors
Parts:
- removed 1A_P6, 5E_P6, 5F_P6: 74LS04, symbol FIN-8-rescue:74LS04
- removed 1B_P6: 74LS10, symbol FIN-8-rescue:74LS10
- removed 1C_P6: 74LS02, symbol FIN-8-rescue:74LS02
- removed 1E_P6, 1F_P6, 2E_P6, 2F_P6, 3A_P6, 3B_P6, 3C_P6, 3D_P6, 3E_P6, 3F_P6, 4E_P6, 4F_P6, 5A_P6, 5B_P6, 5C_P6: 74LS13, symbol FIN-8-rescue:74LS13
- added 1A_P6, 5E_P6, 5F_P6: 74HC04, symbol 74xx:74HC04
- added 1B_P6: 74LS10, symbol 74xx:74LS10
- added 1C_P6: 74HC02, symbol 74xx:74HC02
- added 1E_P6, 1F_P6, 2E_P6, 2F_P6, 3A_P6, 3B_P6, 3C_P6, 3D_P6, 3E_P6, 3F_P6, 4E_P6, 4F_P6, 5A_P6, 5B_P6, 5C_P6: 74LS13, symbol 74xx:74LS13
Connections:
- net MANDA is gone; now on net +AC_7: CONECTOR_P6.48 (P48)
- net +AC_0: now also 3C_P6.4
- net +AC_1: now also 3C_P6.9
- net +AC_2: now also 3B_P6.4
- net +AC_3: now also 3B_P6.9
- net +AC_4: now also 3A_P6.5
- net +AC_5: now also 3A_P6.9
- net +AC_6: now also 3D_P6.5
- net +AC_7: now also 3A_P6.10, 3A_P6.4, 3B_P6.10, 3B_P6.5, 3C_P6.10, 3C_P6.5, 3D_P6.10, 3D_P6.4, 3D_P6.9
- net +RD_4: now also 5F_P6.9
- net +RD_4*: now also 1F_P6.13, 1F_P6.2, 2F_P6.13, 2F_P6.2, 3F_P6.13, 3F_P6.2, 4F_P6.13, 4F_P6.2, 5F_P6.4
- net +RD_5: now also 5E_P6.13
- net +RD_5*: now also 1E_P6.10, 1E_P6.5, 1F_P6.10, 1F_P6.5, 2E_P6.10, 2E_P6.5, 2F_P6.10, 2F_P6.5, 5E_P6.4
- net +RD_6: now also 5F_P6.13
- net +RD_6*: now also 1E_P6.12, 1E_P6.4, 1F_P6.12, 1F_P6.4, 3E_P6.12, 3E_P6.4, 3F_P6.12, 3F_P6.4, 5F_P6.2
- net +RD_7: now also 5E_P6.11
- net +RD_7*: now also 1E_P6.1, 1F_P6.1, 2E_P6.1, 2F_P6.1, 3E_P6.1, 3F_P6.1, 4E_P6.1, 4F_P6.1, 5E_P6.2
- net +RI_4: now also 5B_P6.9
- net +RI_5: now also 5B_P6.5
- net +RI_6: now also 5C_P6.10
- net +RI_7: now also 5C_P6.4
- net +T4: now also 5A_P6.5
- net +T6: now also 5A_P6.9
- net +TUBE: now also 1B_P6.10, 1B_P6.9
- net -COM_0: now also 4E_P6.8
- net -COM_1: now also 4E_P6.6
- net -COM_10: now also 3F_P6.8
- net -COM_11: now also 3F_P6.6
- net -COM_12: now also 2F_P6.8
- net -COM_13: now also 2F_P6.6
- net -COM_14: now also 1F_P6.8
- net -COM_15: now also 1C_P6.8, 1F_P6.6
- net -COM_2: now also 3E_P6.8
- net -COM_3: now also 3E_P6.6
- net -COM_4: now also 2E_P6.8
- net -COM_5: now also 2E_P6.6
- net -COM_6: now also 1E_P6.8
- net -COM_7: now also 1E_P6.6
- net -COM_8: now also 4F_P6.8
- net -COM_9: now also 4F_P6.6
- net -END_0: now also 1C_P6.11, 5B_P6.8
- net -END_1: now also 1C_P6.12, 5B_P6.6
- net -END_2: now also 1C_P6.3, 5C_P6.8
- net -END_3: now also 1C_P6.2, 5C_P6.6
- net -PED_INT: now also 1A_P6.12
- net -PED_INT_PAINEL: now also 1B_P6.11
- net -RD_4: now also 1E_P6.13, 1E_P6.2, 2E_P6.13, 2E_P6.2, 3E_P6.13, 3E_P6.2, 4E_P6.13, 4E_P6.2, 5F_P6.3, 5F_P6.8
- net -RD_5: now also 3E_P6.10, 3E_P6.5, 3F_P6.10, 3F_P6.5, 4E_P6.10, 4E_P6.5, 4F_P6.10, 4F_P6.5, 5E_P6.12, 5E_P6.3
- net -RD_6: now also 2E_P6.12, 2E_P6.4, 2F_P6.12, 2F_P6.4, 4E_P6.12, 4E_P6.4, 4F_P6.12, 4F_P6.4, 5F_P6.1, 5F_P6.12
- net -RD_7: now also 1E_P6.9, 1F_P6.9, 2E_P6.9, 2F_P6.9, 3E_P6.9, 3F_P6.9, 4E_P6.9, 4F_P6.9, 5E_P6.1, 5E_P6.10
- net -SENTIDO: now also 1A_P6.2
- net -SINTA: now also 1C_P6.9
- net -T4*: now also 5A_P6.6
- net -T6*: now also 5A_P6.8
- net DAD_0: now also 3C_P6.6
- net DAD_1: now also 3C_P6.8
- net DAD_2: now also 3B_P6.6
- net DAD_3: now also 3B_P6.8
- net DAD_4: now also 3A_P6.6
- net DAD_5: now also 3A_P6.8
- net DAD_6: now also 3D_P6.6
- net DAD_7: now also 3D_P6.8
- net GND: now also 1A_P6.7 (GND), 1B_P6.7 (GND), 1C_P6.7 (GND), 1E_P6.7 (GND), 1F_P6.7 (GND), 2E_P6.7 (GND), 2F_P6.7 (GND), 3A_P6.7 (GND), 3B_P6.7 (GND), 3C_P6.7 (GND), 3D_P6.7 (GND), 3E_P6.7 (GND), 3F_P6.7 (GND), 4E_P6.7 (GND), 4F_P6.7 (GND), 5A_P6.7 (GND), 5B_P6.7 (GND), 5C_P6.7 (GND), 5E_P6.7 (GND), 5F_P6.7 (GND)
- net MANEN: now also 5B_P6.10, 5B_P6.4, 5C_P6.5, 5C_P6.9
- net VCC: now also 1A_P6.14 (VCC), 1B_P6.14 (VCC), 1C_P6.14 (VCC), 1E_P6.14 (VCC), 1F_P6.14 (VCC), 2E_P6.14 (VCC), 2F_P6.14 (VCC), 3A_P6.14 (VCC), 3B_P6.14 (VCC), 3C_P6.14 (VCC), 3D_P6.14 (VCC), 3E_P6.14 (VCC), 3F_P6.14 (VCC), 4E_P6.14 (VCC), 4F_P6.14 (VCC), 5A_P6.14 (VCC), 5B_P6.14 (VCC), 5C_P6.14 (VCC), 5E_P6.14 (VCC), 5F_P6.14 (VCC)
- net at R6_P6.2: now also 5B_P6.1, 5B_P6.12, 5B_P6.13, 5B_P6.2
- net at R7_P6.2: now also 5C_P6.1, 5C_P6.12, 5C_P6.13, 5C_P6.2
- net at R5_P6.2: now also 5A_P6.1, 5A_P6.10, 5A_P6.12, 5A_P6.13, 5A_P6.2, 5A_P6.4
- net at R4_P6.2: now also 3D_P6.1, 3D_P6.12, 3D_P6.13, 3D_P6.2
- net at R3_P6.2: now also 3A_P6.1, 3A_P6.12, 3A_P6.13, 3A_P6.2
- net at R2_P6.2: now also 3B_P6.1, 3B_P6.12, 3B_P6.13, 3B_P6.2
- net at R1_P6.2: now also 3C_P6.1, 3C_P6.12, 3C_P6.13, 3C_P6.2
- new net: 1A_P6.1, 1B_P6.6
- new net: 1B_P6.1, 1C_P6.13
- new net: 1A_P6.13, 1B_P6.8
- new net: 1B_P6.2, 1C_P6.1
- new net: 1B_P6.13, 1C_P6.10
- new net: 1B_P6.12, 1B_P6.3, 1B_P6.4, 1B_P6.5

Commit message: fixing a whole bunch more ERC errors
Changed lines of the file:
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@@
+		)
+	)
+	(label "-RD_6"
+		(at 49.53 368.3 180)
+		(effects
+			(font
+				(size 1.524 1.524)
+			)
+			(justify right bottom)
+		)
+	)
+	(label "-RD_6"
+		(at 140.97 298.45 180)
+		(effects
+			(font
+				(size 1.524 1.524)
+			)
+			(justify right bottom)
+		)
+	)
+	(label "-RD_6"
+		(at 110.49 204.47 0)
+		(effects
+			(font
+				(size 1.524 1.524)
+			)
+			(justify left bottom)
+		)
+	)
+	(label "-RD_6"
+		(at 49.53 312.42 180)
+		(effects
+			(font
+				(size 1.524 1.524)
+			)
+			(justify right bottom)
+		)
+	)
+	(label "-RD_6"
+		(at 49.53 298.45 180)
+		(effects
+			(font
+				(size 1.524 1.524)
+			)
+			(justify right bottom)
+		)
+	)
+	(label "-RD_6"
+		(at 140.97 368.3 180)
+		(effects
+			(font
+				(size 1.524 1.524)
+			)
+			(justify right bottom)
+		)
+	)
+	(label "-RD_6"
+		(at 49.53 354.33 180)
+		(effects
+			(font
+				(size 1.524 1.524)
+			)
+			(justify right bottom)
+		)
+	)
+	(label "-RD_6"
+		(at 140.97 354.33 180)
+		(effects
+			(font
+				(size 1.524 1.524)
+			)
+			(justify right bottom)
+		)
+	)
+	(label "-RD_6"
+		(at 140.97 312.42 180)
+		(effects
+			(font
+				(size 1.524 1.524)
+			)
+			(justify right bottom)
 		)
 	)
@@
 		)
 	)
-	(global_label "-RD_6"
-		(shape input)
-		(at 140.97 312.42 180)
-		(effects
-			(font
-				(size 1.524 1.524)
-			)
-			(justify right)
-		)
-		(property "Intersheetrefs" "${INTERSHEET_REFS}"
-			(at 140.97 312.42 0)
-			(hide yes)
-			(show_name no)
-			(do_not_autoplace no)
-			(effects
-				(font
-					(size 1.27 1.27)
-				)
-			)
-		)
-	)
 	(global_label "+AC_7"
 		(shape output)
@@
 		)
 	)
-	(global_label "-RD_6"
-		(shape input)
-		(at 49.53 312.42 180)
-		(effects
-			(font
-				(size 1.524 1.524)
-			)
-			(justify right)
-		)
-		(property "Intersheetrefs" "${INTERSHEET_REFS}"
-			(at 49.53 312.42 0)
-			(hide yes)
-			(show_name no)
-			(do_not_autoplace no)
-			(effects
-				(font
-					(size 1.27 1.27)
-				)
-			)
-		)
-	)
 	(global_label "DAD_3"
 		(shape output)
@@
 		)
 	)
-	(global_label "-RD_6"
-		(shape input)
-		(at 140.97 298.45 180)
-		(effects
-			(font
-				(size 1.524 1.524)
-			)
-			(justify right)
-		)
-		(property "Intersheetrefs" "${INTERSHEET_REFS}"
-			(at 140.97 298.45 0)
-			(hide yes)
-			(show_name no)
-			(do_not_autoplace no)
-			(effects
-				(font
-					(size 1.27 1.27)
-				)
-			)
-		)
-	)
 	(global_label "+RD_5*"
 		(shape input)
@@
 		)
 	)
-	(global_label "-RD_6"
-		(shape input)
-		(at 49.53 368.3 180)
-		(effects
-			(font
-				(size 1.524 1.524)
-			)
-			(justify right)
-		)
-		(property "Intersheetrefs" "${INTERSHEET_REFS}"
-			(at 49.53 368.3 0)
-			(hide yes)
-			(show_name no)
-			(do_not_autoplace no)
-			(effects
-				(font
-					(size 1.27 1.27)
-				)
-			)
-		)
-	)
-	(global_label "-RD_6"
-		(shape input)
-		(at 49.53 354.33 180)
-		(effects
-			(font
-				(size 1.524 1.524)
-			)
-			(justify right)
-		)
-		(property "Intersheetrefs" "${INTERSHEET_REFS}"
-			(at 49.53 354.33 0)
-			(hide yes)
-			(show_name no)
-			(do_not_autoplace no)
-			(effects
-				(font
-					(size 1.27 1.27)
-				)
-			)
-		)
-	)
 	(global_label "-RD_7"
 		(shape input)
@@
 		)
 	)
-	(global_label "-RD_6"
-		(shape input)
-		(at 140.97 354.33 180)
-		(effects
-			(font
-				(size 1.524 1.524)
-			)
-			(justify right)
-		)
-		(property "Intersheetrefs" "${INTERSHEET_REFS}"
-			(at 140.97 354.33 0)
-			(hide yes)
-			(show_name no)
-			(do_not_autoplace no)
-			(effects
-				(font
-					(size 1.27 1.27)
-				)
-			)
-		)
-	)
-	(global_label "-RD_6"
-		(shape input)
-		(at 140.97 368.3 180)
-		(effects
-			(font
-				(size 1.524 1.524)
-			)
-			(justify right)
-		)
-		(property "Intersheetrefs" "${INTERSHEET_REFS}"
-			(at 140.97 368.3 0)
-			(hide yes)
-			(show_name no)
-			(do_not_autoplace no)
-			(effects
-				(font
-					(size 1.27 1.27)
-				)
-			)
-		)
-	)
 	(global_label "+RD_6*"
 		(shape output)
@@
 		)
 	)
-	(global_label "-RD_6"
-		(shape output)
-		(at 110.49 204.47 0)
-		(effects
-			(font
-				(size 1.524 1.524)
-			)
-			(justify left)
-		)
-		(property "Intersheetrefs" "${INTERSHEET_REFS}"
-			(at 110.49 204.47 0)
-			(hide yes)
-			(show_name no)
-			(do_not_autoplace no)
-			(effects
-				(font
-					(size 1.27 1.27)
-				)
-			)
-		)
-	)
 	(global_label "+RD_6*"
 		(shape input)
@@
 			(hide yes)
 			(show_name no)
-			(do_not_autoplace no)
-			(effects
-				(font
-					(size 1.27 1.27)
-				)
-			)
-		)
-	)
-	(global_label "-RD_6"
-		(shape input)
-		(at 49.53 298.45 180)
-		(effects
-			(font
-				(size 1.524 1.524)
-			)
-			(justify right)
-		)
-		(property "Intersheetrefs" "${INTERSHEET_REFS}"
-			(at 49.53 298.45 0)
-			(hide yes)
-			(show_name no)

Commit message: wip + PDF plot
Other:
- moved on the sheet: 1A_P6A, 1A_P6F, 1A_P6G, 1B_P6A, 1B_P6B, 1B_P6C, 1B_P6D, 1C_P6A, 1C_P6C, 1C_P6D, 1C_P6E, 1E_P6C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
