File: CRC-1/CRC-1.sch (KiCad schematic (older format))
At the start: 33 parts, among them Q1_P9 BF185, Q2_P9 BF185, Q3_P9 BF185

Commit message: placa CRC-1: remapping de símbolos após atualização para versao mais nova do KICAD
Parts:
- 1A_P9, 1B_P9, 1C_P9, 1D_P9, 1F_P9: symbol 74HC74 -> CRC-1-rescue:74HC74
- 1E_P9, 3A_P9, 3B_P9, 3C_P9, 3D_P9, 5A_P9, 5C_P9, 5E_P9: symbol 74LS04 -> CRC-1-rescue:74LS04
- 3E_P9: symbol 74LS15 -> CRC-1-rescue:74LS15
- 5B_P9, 5D_P9: symbol 7400 -> CRC-1-rescue:7400
- C1_P9, C2_P9, C3_P9, C4_P9, C5_P9: symbol C -> CRC-1-rescue:C
- CONECTOR_P9: symbol CONN_35X2 -> CRC-1-rescue:CONN_35X2
- L1_P9: symbol INDUCTOR -> CRC-1-rescue:INDUCTOR
- Q1_P9, Q2_P9, Q3_P9: symbol BC413B -> CRC-1-rescue:BC413B
- R1_P9, R2_P9, R3_P9, R4_P9, R5_P9, R6_P9: symbol R -> CRC-1-rescue:R
- XTAL1_P9: symbol CRYSTAL -> CRC-1-rescue:CRYSTAL
Connections:
- net at 1A_P9.1 (Cd), 1A_P9.13 (Cd), 1B_P9.1 (Cd)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: no longer 1C_P9.13 (Cd)
