File: CRC-1/CRC-1.kicad_sch (KiCad schematic)
At the start: 33 parts, among them Q1_P9 BF185, Q2_P9 BF185, Q3_P9 BF185

Commit message: Some initial fixing of ERC errors.
Changed lines of the file:
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@@
 	)
 	(junction
-		(at 106.68 177.8)
-		(diameter 0)
-		(color 0 0 0 0)
-	)
-	(junction
 		(at 262.89 306.07)
 		(diameter 0)
@@
 	)
 	(junction
-		(at 168.91 264.16)
-		(diameter 0)
-		(color 0 0 0 0)
-	)
-	(junction
 		(at 770.89 186.69)
 		(diameter 0)
@@
 	(wire
 		(pts
-			(xy 168.91 262.89) (xy 168.91 264.16)
-		)
-		(stroke
-			(width 0)
-			(type default)
-		)
-	)
-	(wire
-		(pts
 			(xy 727.71 186.69) (xy 732.79 186.69)
 		)
@@
 	(wire
 		(pts
-			(xy 106.68 172.72) (xy 106.68 177.8)
-		)
-		(stroke
-			(width 0)
-			(type default)
-		)
-	)
-	(wire
-		(pts
 			(xy 318.77 213.36) (xy 321.31 213.36)
 		)
@@
 	(wire
 		(pts
-			(xy 106.68 177.8) (xy 110.49 177.8)
-		)
-		(stroke
-			(width 0)
-			(type default)
-		)
-	)
-	(wire
-		(pts
 			(xy 135.89 251.46) (xy 130.81 251.46)
 		)
@@
 	(wire
 		(pts
-			(xy 101.6 177.8) (xy 106.68 177.8)
+			(xy 101.6 177.8) (xy 110.49 177.8)
 		)
 		(stroke
@@
 					(unit 1)
 				)
-			)
-		)
-	)
-	(symbol
-		(lib_id "CRC-1-rescue:PWR_FLAG-power")
-		(at 168.91 262.89 0)
-		(unit 1)
-		(body_style 1)
-		(exclude_from_sim no)
-		(in_bom yes)
-		(on_board yes)
-		(in_pos_files yes)
-		(dnp no)
-		(property "Reference" "#FLG017"
-			(at 168.91 260.477 0)
-			(hide yes)
-			(show_name no)
-			(do_not_autoplace no)
-			(effects
-				(font
-					(size 0.762 0.762)
-				)
-			)
-		)
-		(property "Value" "PWR_FLAG"
-			(at 168.91 257.6068 0)
-			(show_name no)
-			(do_not_autoplace no)
-			(effects
-				(font
-					(size 0.762 0.762)
-				)
-			)
-		)
-		(property "Footprint" ""
-			(at 168.91 262.89 0)
-			(hide yes)
-			(show_name no)
-			(do_not_autoplace no)
-			(effects
-				(font
-					(size 1.524 1.524)
-				)
-			)
-		)
-		(property "Datasheet" ""
-			(at 168.91 262.89 0)
-			(hide yes)
-			(show_name no)
-			(do_not_autoplace no)
-			(effects
-				(font
-					(size 1.524 1.524)
-				)
-			)
-		)
-		(property "Description" ""
-			(at 168.91 262.89 0)
-			(show_name no)
-			(do_not_autoplace no)
-			(effects
-				(font
-					(size 1.27 1.27)
-				)
-			)
-		)
-		(pin "1"
-		)
-		(instances
-			(project ""
-				(path "/8a862d08-4b2a-44ae-a055-3e87830c3c62"
-					(reference "#FLG017")
-					(unit 1)
-				)
-			)
-			(project "patinhofeio"
-				(path "/aca06203-542d-4682-a7e3-8839e24cce95/953025c0-c249-406a-b635-15d71cc54afc"
-					(reference "#FLG017")
-					(unit 1)
-				)
-			)
-		)
-	)
-	(symbol
-		(lib_id "CRC-1-rescue:PWR_FLAG-power")
-		(at 106.68 172.72 0)
-		(unit 1)
-		(body_style 1)
-		(exclude_from_sim no)
-		(in_bom yes)
-		(on_board yes)
-		(in_pos_files yes)
-		(dnp no)
-		(property "Reference" "#FLG018"
-			(at 106.68 170.307 0)
-			(hide yes)
-			(show_name no)
-			(do_not_autoplace no)
-			(effects
-				(font
-					(size 0.762 0.762)
-				)
-			)
-		)
-		(property "Value" "PWR_FLAG"
-			(at 106.68 167.4368 0)
-			(show_name no)
-			(do_not_autoplace no)
-			(effects
-				(font
-					(size 0.762 0.762)
-				)
-			)
-		)
-		(property "Footprint" ""
-			(at 106.68 172.72 0)
-			(hide yes)
-			(show_name no)
-			(do_not_autoplace no)
-			(effects
-				(font
-					(size 1.524 1.524)
-				)
-			)
-		)
-		(property "Datasheet" ""
-			(at 106.68 172.72 0)
-			(hide yes)
-			(show_name no)
-			(do_not_autoplace no)
-			(effects
-				(font
-					(size 1.524 1.524)
-				)
-			)
-		)
-		(property "Description" ""
-			(at 106.68 172.72 0)
-			(show_name no)
-			(do_not_autoplace no)
-			(effects
-				(font
-					(size 1.27 1.27)
-				)
-			)
-		)
-		(pin "1"
-		)
-		(instances
-			(project ""
-				(path "/8a862d08-4b2a-44ae-a055-3e87830c3c62"
-					(reference "#FLG018")
-					(unit 1)
-				)
-			)
-			(project "patinhofeio"
-				(path "/aca06203-542d-4682-a7e3-8839e24cce95/953025c0-c249-406a-b635-15d71cc54afc"
-					(reference "#FLG018")
-					(unit 1)
-				)

Commit message: wip
Parts:
- removed 1E_P9, 3A_P9, 3B_P9, 3C_P9, 3D_P9, 5A_P9, 5C_P9, 5E_P9: 74LS04, symbol CRC-1-rescue:74LS04
- added 1E_P9, 3A_P9, 3B_P9, 3C_P9, 3D_P9, 5A_P9, 5C_P9, 5E_P9: 74LS04, symbol 74xx:74LS04
Connections:
- net +CLOCK: now also 1E_P9.2
- net +T0-1: now also 5E_P9.4
- net +T0-2: now also 5E_P9.6
- net +T01-1: now also 3D_P9.4
- net +T01-2: now also 3D_P9.6
- net +T012: now also 5E_P9.1
- net +T0123: now also 5E_P9.13
- net +T1-1: now also 5E_P9.8
- net +T1-2: now also 5E_P9.10
- net +T12-1: now also 3D_P9.8
- net +T12-2: now also 3D_P9.10
- net +T2-1: now also 5C_P9.4
- net +T2-2: now also 5C_P9.6
- net +T23-1: now also 3C_P9.8
- net +T23-2: now also 3C_P9.10
- net +T3-1: now also 5C_P9.12
- net +T3-2: now also 5C_P9.2
- net +T34: now also 3C_P9.5
- net +T34-1: now also 3C_P9.2
- net +T34-2: now also 3C_P9.4
- net +T4-1: now also 5C_P9.8
- net +T4-2: now also 5C_P9.10
- net +T45-1: now also 3B_P9.4
- net +T45-2: now also 3B_P9.6
- net +T5-1: now also 5A_P9.2
- net +T5-2: now also 5A_P9.12
- net +T56-1: now also 3B_P9.8
- net +T56-2: now also 3B_P9.10
- net +T6-1: now also 5A_P9.4
- net +T6-2: now also 5A_P9.6
- net +T67-1: now also 3A_P9.8
- net +T67-2: now also 3A_P9.10
- net +T7-1: now also 5A_P9.8
- net +T7-2: now also 5A_P9.10
- net +T70-1: now also 3A_P9.2
- net +T70-2: now also 3A_P9.4
- net -CLOCK: now also 1E_P9.10
- net -LAL: now also 1E_P9.3
- net -T0: now also 5E_P9.3, 5E_P9.5
- net -T01: now also 3D_P9.2
- net -T01*: now also 3D_P9.3, 3D_P9.5
- net -T012: now also 5E_P9.2
- net -T0123: now also 5E_P9.12
- net -T1: now also 5E_P9.11, 5E_P9.9
- net -T12*: now also 3D_P9.11, 3D_P9.9
- net -T2: now also 5C_P9.3, 5C_P9.5
- net -T23: now also 3C_P9.12
- net -T23*: now also 3C_P9.11, 3C_P9.9
- net -T3: now also 5C_P9.1, 5C_P9.13
- net -T34: now also 3C_P9.6
- net -T34*: now also 3C_P9.1, 3C_P9.3
- net -T4: now also 5C_P9.11, 5C_P9.9
- net -T45: now also 3B_P9.2
- net -T45*: now also 3B_P9.3, 3B_P9.5
- net -T5: now also 5A_P9.1, 5A_P9.13
- net -T56: now also 3B_P9.12
- net -T56*: now also 3B_P9.11, 3B_P9.9
- net -T6: now also 5A_P9.3, 5A_P9.5
- net -T67: now also 3A_P9.12
- net -T67*: now also 3A_P9.11, 3A_P9.9
- net -T7: now also 5A_P9.11, 5A_P9.9
- net -T70: now also 3A_P9.6
- net -T70*: now also 3A_P9.1, 3A_P9.3
- net GND: now also 1E_P9.7 (GND), 3A_P9.7 (GND), 3B_P9.7 (GND), 3C_P9.7 (GND), 3D_P9.7 (GND), 5A_P9.7 (GND), 5C_P9.7 (GND), 5E_P9.7 (GND)
- net VCC: now also 1E_P9.14 (VCC), 3A_P9.14 (VCC), 3B_P9.14 (VCC), 3C_P9.14 (VCC), 3D_P9.14 (VCC), 5A_P9.14 (VCC), 5C_P9.14 (VCC), 5E_P9.14 (VCC)
- net at 1A_P9.11 (Cp), 1A_P9.3 (Cp), 1B_P9.11 (Cp)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: now also 1E_P9.6
- net at 3E_P9.13, 3E_P9.2: now also 1E_P9.4
- net at 1A_P9.5 (Q), 1D_P9.2 (D), 5B_P9.9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: now also 3A_P9.5
- net at 1D_P9.12 (D), 1D_P9.5 (Q), 5D_P9.13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: now also 3D_P9.1
- net at 1C_P9.12 (D), 1D_P9.9 (Q), 5D_P9.12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: now also 3D_P9.13
- net at 1C_P9.2 (D), 1C_P9.9 (Q), 5D_P9.10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: now also 3C_P9.13
- net at 1B_P9.12 (D), 1B_P9.5 (Q), 5B_P9.13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: now also 3B_P9.1
- net at 1A_P9.12 (D), 1B_P9.9 (Q), 5B_P9.12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: now also 3B_P9.13
- net at 1A_P9.2 (D), 1A_P9.9 (Q), 5B_P9.10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: now also 3A_P9.13
- net at 1F_P9.11 (Cp): now also 1E_P9.12
- net at 1F_P9.12 (D), 1F_P9.8 (~{Q}): now also 1E_P9.11, 1E_P9.9
- net at 1F_P9.9 (Q): now also 1E_P9.1, 1E_P9.5
- net at 1F_P9.3 (Cp): now also 1E_P9.8
- net at Q1_P9.3 (E), R1_P9.1: now also 1E_P9.13

Commit message: a lot more work on the circuit transcription
Parts:
- removed 1A_P9, 1B_P9, 1C_P9, 1D_P9, 1F_P9: 74HC74, symbol CRC-1-rescue:74HC74
- removed 3E_P9: 74LS15, symbol CRC-1-rescue:74LS15
- removed 5B_P9, 5D_P9: 7400, symbol CRC-1-rescue:7400
- added 1A_P9, 1B_P9, 1C_P9, 1D_P9, 1F_P9: 74LS74, symbol 74xx:74LS74
- added 3E_P9: 74LS15, symbol 74xx:74LS15
- added 5B_P9, 5D_P9: 74LS00, symbol 74xx:74LS00
- added C1, C10, C11, C12, C13, C14, C15, C2, C3, C4, C5, C6, C7, C8, C9: C, symbol Device:C
Connections:
- net +T(3/4)2: now also 1F_P9.5 (Q)
- net +T012: now also 3E_P9.6
- net +T0123: now also 3E_P9.8
- net +T34: now also 1B_P9.2 (D), 1C_P9.5 (Q), 1F_P9.2 (D), 5B_P9.1, 5D_P9.9
- net -T(3/4)2: now also 1F_P9.6 (~{Q})
- net -T0: now also 5D_P9.3
- net -T01*: now also 1D_P9.6 (~{Q}), 3E_P9.11, 3E_P9.4
- net -T1: now also 5D_P9.11
- net -T12: now also 3D_P9.12
- net -T12*: now also 1D_P9.8 (~{Q}), 3E_P9.10, 3E_P9.5
- net -T2: now also 5D_P9.6
- net -T23*: now also 1C_P9.8 (~{Q}), 3E_P9.9
- net -T3: now also 5D_P9.8
- net -T34*: now also 1C_P9.6 (~{Q})
- net -T4: now also 5B_P9.3
- net -T45*: now also 1B_P9.6 (~{Q})
- net -T5: now also 1F_P9.1 (~{R}), 5B_P9.11
- net -T56*: now also 1B_P9.8 (~{Q})
- net -T6: now also 5B_P9.6
- net -T67*: now also 1A_P9.8 (~{Q})
- net -T7: now also 5B_P9.8
- net -T70*: now also 1A_P9.6 (~{Q})
- net GND: now also 1A_P9.7 (GND), 1B_P9.7 (GND), 1C_P9.7 (GND), 1D_P9.7 (GND), 3E_P9.7 (GND), 5B_P9.7 (GND), 5D_P9.7 (GND), C1.2, C10.2, C11.2, C12.2, C13.2, C14.2, C15.2, C2.2, C3.2, C4.2, C5.2, C6.2, C7.2, C8.2, C9.2
- net VCC: now also 1A_P9.10 (~{S}), 1A_P9.14 (VCC), 1A_P9.4 (~{S}), 1B_P9.10 (~{S}), 1B_P9.14 (VCC), 1B_P9.4 (~{S}), 1C_P9.10 (~{S}), 1C_P9.14 (VCC), 1C_P9.4 (~{S}), 1D_P9.1 (~{R}), 1D_P9.13 (~{R}), 1D_P9.14 (VCC), 1F_P9.10 (~{S}), 1F_P9.13 (~{R}), 1F_P9.4 (~{S}), 3E_P9.14 (VCC), 3E_P9.3, 5B_P9.14 (VCC), 5D_P9.14 (VCC), C1.1, C10.1, C11.1, C12.1, C13.1, C14.1, C15.1, C2.1, C3.1, C4.1, C5.1, C6.1, C7.1, C8.1, C9.1
- net at 1E_P9.6: now also 1A_P9.11 (C), 1A_P9.3 (C), 1B_P9.11 (C), 1B_P9.3 (C), 1C_P9.11 (C), 1C_P9.3 (C), 1D_P9.11 (C), 1D_P9.3 (C), 3E_P9.1
- net at 1E_P9.4: now also 3E_P9.13, 3E_P9.2
- net at 3A_P9.5: now also 1A_P9.5 (Q), 1D_P9.2 (D), 5B_P9.9, 5D_P9.1
- net at 3D_P9.1: now also 1D_P9.12 (D), 1D_P9.5 (Q), 5D_P9.13, 5D_P9.2
- net at 3D_P9.13: now also 1C_P9.12 (D), 1D_P9.9 (Q), 5D_P9.12, 5D_P9.4
- net at 3C_P9.13: now also 1C_P9.2 (D), 1C_P9.9 (Q), 5D_P9.10, 5D_P9.5
- net at 3B_P9.1: now also 1B_P9.12 (D), 1B_P9.5 (Q), 5B_P9.13, 5B_P9.2
- net at 3B_P9.13: now also 1A_P9.12 (D), 1B_P9.9 (Q), 5B_P9.12, 5B_P9.4
- net at 3A_P9.13: now also 1A_P9.2 (D), 1A_P9.9 (Q), 5B_P9.10, 5B_P9.5
- net at 1E_P9.12: now also 1F_P9.11 (C)
- net at 1E_P9.11, 1E_P9.9: now also 1F_P9.12 (D), 1F_P9.8 (~{Q})
- net at 1E_P9.1, 1E_P9.5: now also 1F_P9.9 (Q)
- net at 1E_P9.8: now also 1F_P9.3 (C)
- new net: 1A_P9.1 (~{R}), 1A_P9.13 (~{R}), 1B_P9.1 (~{R}), 1B_P9.13 (~{R}), 1C_P9.1 (~{R}), 1C_P9.13 (~{R}), 1D_P9.10 (~{S}), 1D_P9.4 (~{S}), 3E_P9.12
Other:
- moved on the sheet: 1E_P9F, 1E_P9G, 3A_P9G, 3B_P9G, 3C_P9G, 3D_P9G, 5A_P9G, 5C_P9G, 5E_P9G
