File: CDE-3-debug/CDE-3-debug.sch (KiCad schematic (older format))
At the start: 79 parts

Commit message: preparando PCB CDE-3-debug
Parts:
- D1, D10, D11, D12, D13, D14, D15, D16, D17, D18, D19, D2, D20, D21, D22, D23, D24, D25, D26, D27, D28, D29, D3, D30, D31, D32, D33, D34, D35, D36, D37, D38, D39, D4, D40, D41, D42, D43, D44, D45, D46, D47, D48, D49, D5, D50, D51, D52, D6, D7, D8, D9: footprint (none) -> LEDs:LED_D3.0mm
- JP1, JP10, JP11, JP12, JP13, JP14, JP15, JP16, JP2, JP3, JP4, JP5, JP6, JP7, JP8, JP9: footprint (none) -> Pin_Headers:Pin_Header_Straight_1x02_Pitch2.54mm
- RR1, RR2, RR3, RR4, RR5, RR6, RR7, RR8, RR9: footprint (none) -> Resistors_ThroughHole:R_Array_SIP9
- renumbered CONECTOR_debug_P10 to CONECTOR_FEMEA_DEBUG_CDE3, CONECTOR_P10 to CONECTOR_MACHO_DEBUG_CDE3

Commit message: placa CDE-3-debug: symbol remap
Parts:
- CONECTOR_FEMEA_DEBUG_CDE3, CONECTOR_MACHO_DEBUG_CDE3: symbol CONN_35X2 -> CDE-3-debug-rescue:CONN_35X2
- D1, D10, D11, D12, D13, D14, D15, D16, D17, D18, D19, D2, D20, D21, D22, D23, D24, D25, D26, D27, D28, D29, D3, D30, D31, D32, D33, D34, D35, D36, D37, D38, D39, D4, D40, D41, D42, D43, D44, D45, D46, D47, D48, D49, D5, D50, D51, D52, D6, D7, D8, D9: symbol LED -> CDE-3-debug-rescue:LED
- JP1, JP10, JP11, JP12, JP13, JP14, JP15, JP16, JP2, JP3, JP4, JP5, JP6, JP7, JP8, JP9: symbol JUMPER -> CDE-3-debug-rescue:JUMPER
- RR1, RR2, RR3, RR4, RR5, RR6, RR7, RR8, RR9: symbol RR8 -> CDE-3-debug-rescue:RR8
