File: CT1-4/CT1-4.sch (KiCad schematic (older format))
At the start: 1 part

Commit message: wip: esquema da placa CT1-4
Parts:
- added 1A_P12, 1E_P12, 3B_P12, 4A_P12: 74LS04, symbol 74LS04
- added 1B_P12, 1D_P12, 2A_P12, 3D_P12, 4B_P12, 4C_P12, 5A_P12, 5C_P12: 7400, symbol 7400
- added 1C_P12, 3A_P12, 4E_P12: 74LS10, symbol 74LS10
- added 2B_P12, 5B_P12: 7402, symbol 7402
- added 2C_P12: 7453, symbol 7453
- added 2D_P12, 2E_P12: 7460, symbol 7460
- added 3C_P12: 74LS54, symbol 74LS54
- added 3E_P12, 5D_P12: 74LS13, symbol 74LS13
- added _2C_P12: 74LS51, symbol 74LS51
Connections:
- net ?: no longer CONECTOR_P12.1 (P1), CONECTOR_P12.10 (P10), CONECTOR_P12.11 (P11), CONECTOR_P12.12 (P12), CONECTOR_P12.13 (P13), CONECTOR_P12.15 (P15), CONECTOR_P12.16 (P16), CONECTOR_P12.17 (P17), CONECTOR_P12.18 (P18), CONECTOR_P12.19 (P19), CONECTOR_P12.2 (P2), CONECTOR_P12.20 (P20), CONECTOR_P12.21 (P21), CONECTOR_P12.22 (P22), CONECTOR_P12.23 (P23), CONECTOR_P12.24 (P24), CONECTOR_P12.25, CONECTOR_P12.26 (P26), CONECTOR_P12.27 (P27), CONECTOR_P12.28 (P28), CONECTOR_P12.3 (P3), CONECTOR_P12.37 (P37), CONECTOR_P12.38 (P38), CONECTOR_P12.39 (P39), CONECTOR_P12.4 (P4), CONECTOR_P12.40 (P40), CONECTOR_P12.41 (P41), CONECTOR_P12.42 (P42), CONECTOR_P12.43 (P43), CONECTOR_P12.44 (P44), CONECTOR_P12.45 (P45), CONECTOR_P12.46 (P46), CONECTOR_P12.5 (P5), CONECTOR_P12.50 (P50), CONECTOR_P12.51 (P51), CONECTOR_P12.52 (P52), CONECTOR_P12.53 (P53), CONECTOR_P12.54 (P54), CONECTOR_P12.55 (P55), CONECTOR_P12.56 (P56), CONECTOR_P12.57 (P57), CONECTOR_P12.58 (P58), CONECTOR_P12.59 (P59), CONECTOR_P12.6 (P6), CONECTOR_P12.60 (P60), CONECTOR_P12.61 (P61), CONECTOR_P12.62 (P62), CONECTOR_P12.68 (P68), CONECTOR_P12.69 (P69), CONECTOR_P12.7 (P7), CONECTOR_P12.70 (P70), CONECTOR_P12.8 (P8), CONECTOR_P12.9 (P9)
- new net: 1B_P12.3, 1C_P12.1
- new net: 1A_P12.10, 1B_P12.4
- new net: 1A_P12.11, 2B_P12.10
- new net: 1A_P12.13, 1C_P12.12
- new net: 1D_P12.2, 1D_P12.6
- new net: 1D_P12.3, 1E_P12.1
- new net: 5B_P12.1, 5C_P12.2
- new net: 5C_P12.3, 5C_P12.4
- new net: 5C_P12.5, 5C_P12.8, 5D_P12.10, 5D_P12.12, 5D_P12.13, 5D_P12.9
- new net: 5C_P12.6, 5C_P12.9, 5D_P12.1, 5D_P12.2, 5D_P12.4, 5D_P12.5
- new net: 3D_P12.5, 3D_P12.8
- new net: 3D_P12.6, 3D_P12.9, 3E_P12.10, 3E_P12.12, 3E_P12.13, 3E_P12.9
- new net: 1D_P12.11, 1E_P12.9
- new net: 1C_P12.4, 1D_P12.8
- new net: 1D_P12.9, 5B_P12.13
- new net: 2A_P12.8, 3A_P12.5
- new net: 3A_P12.8, 3C_P12.1
- new net: 2A_P12.6, 3A_P12.9
- new net: 3C_P12.4, 3D_P12.11
- new net: 3B_P12.3, 3C_P12.8
- new net: 3A_P12.12, 3B_P12.1
- new net: 2A_P12.3, 3D_P12.13
- new net: 4B_P12.3, 5A_P12.12, 5A_P12.13
- new net: 1E_P12.5, _2C_P12.6
- new net: 2B_P12.13, _2C_P12.2
- new net: 2C_P12.8, 3E_P12.1, 3E_P12.2, 3E_P12.4, 3E_P12.5
- new net: 2C_P12.11 (Ve), 2D_P12.11, 2D_P12.9, 2E_P12.11, 2E_P12.9
- new net: 2C_P12.12 (Vc), 2D_P12.10, 2D_P12.12, 2E_P12.10, 2E_P12.12
- new net: 2B_P12.1, 2D_P12.13, 2D_P12.8, 2E_P12.13, 2E_P12.6
- new net: 2C_P12.10, 4C_P12.11
- new net: 4C_P12.12, 4C_P12.8
- new net +(CAC+SOM): 1B_P12.2, CONECTOR_P12.4 (P4)
- new net +(F1.MICG1): 2A_P12.4, 3B_P12.6
- new net +(F2.IME): 3A_P12.3, 3B_P12.8, 4C_P12.9
- new net +(F2.SAEDE): 2B_P12.4, 2C_P12.13, 5A_P12.1
- new net +AC/X: 3B_P12.4, CONECTOR_P12.13 (P13)
- new net +ARA: 2A_P12.2, CONECTOR_P12.43 (P43)
- new net +C_AC: 3E_P12.6, CONECTOR_P12.21 (P21)
- new net +E/A: 1E_P12.12, CONECTOR_P12.55 (P55)
- new net +F1: 1A_P12.2, 1B_P12.9, 5A_P12.4
- new net +F2: 1A_P12.4, 1B_P12.12, 1C_P12.9, 4E_P12.2
- new net +F3: 1A_P12.6, 1B_P12.1, 2A_P12.1, 2A_P12.12, 3A_P12.1
- new net +F4: 1A_P12.8, 1B_P12.5
- new net +IME: 1B_P12.13, CONECTOR_P12.6 (P6)
- new net +IMEADD: 1D_P12.10, 2A_P12.9, CONECTOR_P12.41 (P41)
- new net +IMENAND: 1C_P12.11, CONECTOR_P12.25
- new net +IMEXOR: 2A_P12.10, 4E_P12.13, CONECTOR_P12.44 (P44)
- new net +MANDA: 5D_P12.8, CONECTOR_P12.61 (P61)
- new net +MICG1: 1B_P12.10, CONECTOR_P12.39 (P39)
- new net +MICRO: 4A_P12.5, CONECTOR_P12.22 (P22)
- new net +NAND: 1E_P12.10, CONECTOR_P12.26 (P26)
- new net +RD_4: 2D_P12.2, CONECTOR_P12.52 (P52)
- new net +RD_5: 2D_P12.5, CONECTOR_P12.19 (P19)
- new net +RD_6: 2E_P12.2, CONECTOR_P12.53 (P53)
- new net +RD_7: 2E_P12.5, CONECTOR_P12.20 (P20)
- new net +RI_5: 2A_P12.5, CONECTOR_P12.10 (P10)
- new net +RI_6: 4A_P12.9, CONECTOR_P12.23 (P23)
- new net +SAEDE: 4A_P12.3, CONECTOR_P12.54 (P54)
- new net +SAEDS: 4A_P12.11, CONECTOR_P12.60 (P60)
- new net +SHIFT: 3B_P12.11, CONECTOR_P12.42 (P42)
- new net +SOM: 2A_P12.13, CONECTOR_P12.11 (P11)
- new net +SOXOR: 1C_P12.8, 1E_P12.11, CONECTOR_P12.59 (P59)
- new net +SUS: 3A_P12.2, CONECTOR_P12.45 (P45)
- new net +T12: 3C_P12.5, CONECTOR_P12.12 (P12)
- new net +T23: 3C_P12.10, CONECTOR_P12.46 (P46), _2C_P12.4
- new net +T3: 2D_P12.1, 5A_P12.2, CONECTOR_P12.50 (P50)
- new net +T34: 1C_P12.10, 3C_P12.13, 4E_P12.1, 5C_P12.1, CONECTOR_P12.40 (P40), _2C_P12.3
- new net +T4: 2C_P12.1, 2D_P12.4, 5A_P12.9, CONECTOR_P12.17 (P17)
- new net +T45: 1D_P12.1, 1D_P12.12, CONECTOR_P12.69 (P69)
- new net +T5: 2C_P12.9, 2E_P12.1, CONECTOR_P12.51 (P51)
- new net +T6: 2E_P12.4, CONECTOR_P12.18 (P18)
- new net +T70: 4A_P12.13, CONECTOR_P12.15 (P15)
- new net +TR/T: 1E_P12.8, CONECTOR_P12.8 (P8)
- new net +TRI: 2B_P12.9, CONECTOR_P12.5 (P5)
- new net +TRO: 2B_P12.8, CONECTOR_P12.62 (P62)
- new net +X: 1C_P12.6, 1D_P12.13, 4A_P12.1, 5A_P12.10
- new net +X1: 1E_P12.13, 3D_P12.4, 5A_P12.3
- new net +Z: 3B_P12.2, 3C_P12.9, _2C_P12.5
- new net +Z/A: 1E_P12.2, CONECTOR_P12.7 (P7)
- new net +~AC/X: 1E_P12.6, CONECTOR_P12.57 (P57)
- new net -(F1.MICG1): 1B_P12.8, 1C_P12.13, 1C_P12.5, 2B_P12.11, 3B_P12.5
- new net -(F2.IME): 1B_P12.11, 1D_P12.5, 3B_P12.9
- new net -(F3.SOM): 1C_P12.3, 2A_P12.11, 3A_P12.11
- new net -(F4.(TRO+TRI)): 1B_P12.6, 1C_P12.2, 3D_P12.12
- new net -CF2: 5A_P12.6, CONECTOR_P12.56 (P56)
- new net -CLOCK: 2D_P12.3, 2D_P12.6, 2E_P12.3, 2E_P12.8, CONECTOR_P12.16 (P16)
- new net -C_OVF: 5A_P12.8, CONECTOR_P12.24 (P24)
- new net -DADEN: 3E_P12.8, CONECTOR_P12.28 (P28)
- new net -DADSA: 5D_P12.6, CONECTOR_P12.27 (P27)
- new net -F1: 1A_P12.1, CONECTOR_P12.2 (P2)
- new net -F2: 1A_P12.3, 2B_P12.3, 2B_P12.5, 5B_P12.2, CONECTOR_P12.37 (P37)
- new net -F3: 1A_P12.5, CONECTOR_P12.3 (P3)
- new net -F4: 1A_P12.9, CONECTOR_P12.38 (P38)
- new net -MICRO: 4A_P12.6, 5A_P12.5
- new net -RDZ: 3A_P12.13, CONECTOR_P12.9 (P9)
- new net -RI_6: 2B_P12.12, 4A_P12.8
- new net -SAEDE: 2B_P12.6, 4A_P12.4
- new net -SAEDS: 4A_P12.10, 5B_P12.3
- new net -SHIFT: 2B_P12.2, 3A_P12.4, 3B_P12.10, 4B_P12.1, 4C_P12.10
- new net -T70: 3D_P12.10, 4A_P12.12, 5C_P12.10
- new net -X: 4A_P12.2, 4B_P12.2
- new net -XOR: 4E_P12.12, CONECTOR_P12.58 (P58)
- new net -Y: 1A_P12.12, 1D_P12.4, 4C_P12.13
- new net GND: 1A_P12.7 (GND), 1A_P12.7 (GND), 1A_P12.7 (GND), 1A_P12.7 (GND), 1A_P12.7 (GND), 1A_P12.7 (GND), 1B_P12.7 (GND), 1B_P12.7 (GND), 1B_P12.7 (GND), 1B_P12.7 (GND), 1C_P12.7 (GND), 1C_P12.7 (GND), 1C_P12.7 (GND), 1D_P12.7 (GND), 1D_P12.7 (GND), 1D_P12.7 (GND), 1D_P12.7 (GND), 1E_P12.7 (GND), 1E_P12.7 (GND), 1E_P12.7 (GND), 1E_P12.7 (GND), 1E_P12.7 (GND), 2A_P12.7 (GND), 2A_P12.7 (GND), 2A_P12.7 (GND), 2A_P12.7 (GND), 2B_P12.7 (GND), 2B_P12.7 (GND), 2B_P12.7 (GND), 2B_P12.7 (GND), 2C_P12.2, 2C_P12.3, 2C_P12.4, 2C_P12.5, 2C_P12.7 (GND), 2D_P12.7 (GND), 2D_P12.7 (GND), 2E_P12.7 (GND), 2E_P12.7 (GND), 3A_P12.7 (GND), 3A_P12.7 (GND), 3A_P12.7 (GND), 3B_P12.7 (GND), 3B_P12.7 (GND), 3B_P12.7 (GND), 3B_P12.7 (GND), 3B_P12.7 (GND), 3C_P12.2, 3C_P12.3, 3C_P12.7 (GND), 3D_P12.7 (GND), 3D_P12.7 (GND), 3D_P12.7 (GND), 3E_P12.7 (GND), 3E_P12.7 (GND), 4A_P12.7 (GND), 4A_P12.7 (GND), 4A_P12.7 (GND), 4A_P12.7 (GND), 4A_P12.7 (GND), 4A_P12.7 (GND), 4B_P12.7 (GND), 4C_P12.7 (GND), 4C_P12.7 (GND), 4E_P12.7 (GND), 5A_P12.7 (GND), 5A_P12.7 (GND), 5A_P12.7 (GND), 5A_P12.7 (GND), 5B_P12.7 (GND), 5B_P12.7 (GND), 5C_P12.7 (GND), 5C_P12.7 (GND), 5C_P12.7 (GND), 5D_P12.7 (GND), 5D_P12.7 (GND), CONECTOR_P12.70 (P70), _2C_P12.7 (GND)
- new net P12_3A6: 3A_P12.10, 3A_P12.6, 5B_P12.11, 5B_P12.12
- new net T/T: 5A_P12.11, CONECTOR_P12.68 (P68)
- new net VCC: 1A_P12.14 (VCC), 1A_P12.14 (VCC), 1A_P12.14 (VCC), 1A_P12.14 (VCC), 1A_P12.14 (VCC), 1A_P12.14 (VCC), 1B_P12.14 (VCC), 1B_P12.14 (VCC), 1B_P12.14 (VCC), 1B_P12.14 (VCC), 1C_P12.14 (VCC), 1C_P12.14 (VCC), 1C_P12.14 (VCC), 1D_P12.14 (VCC), 1D_P12.14 (VCC), 1D_P12.14 (VCC), 1D_P12.14 (VCC), 1E_P12.14 (VCC), 1E_P12.14 (VCC), 1E_P12.14 (VCC), 1E_P12.14 (VCC), 1E_P12.14 (VCC), 2A_P12.14 (VCC), 2A_P12.14 (VCC), 2A_P12.14 (VCC), 2A_P12.14 (VCC), 2B_P12.14 (VCC), 2B_P12.14 (VCC), 2B_P12.14 (VCC), 2B_P12.14 (VCC), 2C_P12.14 (VCC), 2D_P12.14 (VCC), 2D_P12.14 (VCC), 2E_P12.14 (VCC), 2E_P12.14 (VCC), 3A_P12.14 (VCC), 3A_P12.14 (VCC), 3A_P12.14 (VCC), 3B_P12.14 (VCC), 3B_P12.14 (VCC), 3B_P12.14 (VCC), 3B_P12.14 (VCC), 3B_P12.14 (VCC), 3C_P12.14 (VCC), 3D_P12.14 (VCC), 3D_P12.14 (VCC), 3D_P12.14 (VCC), 3E_P12.14 (VCC), 3E_P12.14 (VCC), 4A_P12.14 (VCC), 4A_P12.14 (VCC), 4A_P12.14 (VCC), 4A_P12.14 (VCC), 4A_P12.14 (VCC), 4A_P12.14 (VCC), 4B_P12.14 (VCC), 4C_P12.14 (VCC), 4C_P12.14 (VCC), 4E_P12.14 (VCC), 5A_P12.14 (VCC), 5A_P12.14 (VCC), 5A_P12.14 (VCC), 5A_P12.14 (VCC), 5B_P12.14 (VCC), 5B_P12.14 (VCC), 5C_P12.14 (VCC), 5C_P12.14 (VCC), 5C_P12.14 (VCC), 5D_P12.14 (VCC), 5D_P12.14 (VCC), CONECTOR_P12.1 (P1), _2C_P12.14 (VCC)
Other:
- note added: "-(F3.(CAC+SOM))"
- note added: "Precisamos revisar essa parte\nHá alguns chutes aqui sobre qual é a\nforma correta de se interligar esses\nchips expansores."

Commit message: placa CT1-4: symbol remap
Parts:
- 1A_P12, 1E_P12, 3B_P12, 4A_P12: symbol 74LS04 -> CT1-4-rescue:74LS04
- 1B_P12, 1D_P12, 2A_P12, 3D_P12, 4B_P12, 4C_P12, 5A_P12, 5C_P12: symbol 7400 -> CT1-4-rescue:7400
- 1C_P12, 3A_P12, 4E_P12: symbol 74LS10 -> CT1-4-rescue:74LS10
- 2B_P12, 5B_P12: symbol 7402 -> CT1-4-rescue:7402
- 2C_P12: symbol 7453 -> CT1-4-rescue:7453
- 2D_P12, 2E_P12: symbol 7460 -> CT1-4-rescue:7460
- 3C_P12: symbol 74LS54 -> CT1-4-rescue:74LS54
- 3E_P12, 5D_P12: symbol 74LS13 -> CT1-4-rescue:74LS13
- CONECTOR_P12: symbol CONN_35X2 -> CT1-4-rescue:CONN_35X2
- _2C_P12: symbol 74LS51 -> CT1-4-rescue:74LS51
