File: CT1-4/CT1-4.kicad_sch (KiCad schematic)
At the start: 25 parts

Commit message: wip: backplane connectors
Connections:
- removed net ?: CONECTOR_P12.14 (P14), CONECTOR_P12.29 (P29), CONECTOR_P12.30 (P30), CONECTOR_P12.31 (P31), CONECTOR_P12.32 (P32), CONECTOR_P12.33 (P33), CONECTOR_P12.34 (P34), CONECTOR_P12.35 (P35), CONECTOR_P12.36 (P36), CONECTOR_P12.47 (P47), CONECTOR_P12.48 (P48), CONECTOR_P12.49 (P49)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
- no-connect marks 0 -> 17
