File: CT1-4/CT1-4.kicad_sch (KiCad schematic)
At the start: 25 parts

Commit message: wip
Parts:
- removed 1B_P12, 1D_P12, 2A_P12, 3D_P12, 4B_P12, 4C_P12, 5A_P12, 5C_P12: 7400, symbol CT1-4-rescue:7400
- removed 1C_P12, 3A_P12, 4E_P12: 74LS10, symbol CT1-4-rescue:74LS10
- removed 1E_P12, 3B_P12: 74LS04, symbol CT1-4-rescue:74LS04
- removed unit 4 of 2B_P12
- removed 3E_P12, 5D_P12: 74LS13, symbol CT1-4-rescue:74LS13
- added 1B_P12, 1D_P12, 2A_P12, 3D_P12, 4B_P12, 4C_P12, 5A_P12, 5C_P12: 74LS00, symbol 74xx:74LS00
- added 1C_P12, 3A_P12, 4E_P12: 74LS10, symbol 74xx:74LS10
- added 1E_P12: 74LS04, symbol 74xx:74LS04
- added unit 4 of 2B_P12
- added 3E_P12, 5D_P12: 74LS13, symbol 74xx:74LS13
Connections:
- net +(CAC+SOM): now also 1B_P12.2
- net +(F1.MICG1): now also 2A_P12.4
- net +(F2.IME): now also 3A_P12.3, 4C_P12.9
- net +(F2.SAEDE): now also 5A_P12.1
- net +AC/X: now also 3B_P12.4
- net +ARA: now also 2A_P12.2
- net +C_AC: now also 3E_P12.6
- net +E/A: now also 1E_P12.12
- net +F1: now also 1B_P12.9, 5A_P12.4
- net +F2: now also 1B_P12.12, 1C_P12.9, 4E_P12.2
- net +F3: now also 1B_P12.1, 2A_P12.1, 2A_P12.12, 3A_P12.1
- net +F4: now also 1B_P12.5
- net +IME: now also 1B_P12.13
- net +IMEADD: now also 1D_P12.10, 2A_P12.9
- net +IMENAND: now also 1C_P12.11
- net +IMEXOR: now also 2A_P12.10, 4E_P12.13
- net +MANDA: now also 5D_P12.8
- net +MICG1: now also 1B_P12.10
- net +NAND: now also 1E_P12.10
- net +RI_5: now also 2A_P12.5
- net +SOM: now also 2A_P12.13
- net +SOXOR: now also 1C_P12.8, 1E_P12.11
- net +SUS: now also 3A_P12.2
- net +T3: now also 5A_P12.2
- net +T34: now also 1C_P12.10, 4E_P12.1, 5C_P12.1
- net +T4: now also 5A_P12.9
- net +T45: now also 1D_P12.1, 1D_P12.12
- net +TR/T: now also 1E_P12.8
- net +X: now also 1C_P12.6, 1D_P12.13, 5A_P12.10
- net +X1: now also 1E_P12.13, 3D_P12.4, 5A_P12.3
- net +Z/A: now also 1E_P12.2
- net +~{AC/X}: now also 1E_P12.6
- net -(F1.MICG1): now also 1B_P12.8, 1C_P12.13, 1C_P12.5, 2B_P12.11
- net -(F2.IME): now also 1B_P12.11, 1D_P12.5
- net -(F3.SOM): now also 1C_P12.3, 2A_P12.11, 3A_P12.11
- net -(F4.(TRO+TRI)): now also 1B_P12.6, 1C_P12.2, 3D_P12.12
- net -CF2: now also 5A_P12.6
- net -C_OVF: now also 5A_P12.8
- net -DADEN: now also 3E_P12.8
- net -DADSA: now also 5D_P12.6
- net -MICRO: now also 5A_P12.5
- net -RDZ: now also 3A_P12.13
- net -RI_6: now also 2B_P12.12
- net -SHIFT: now also 3A_P12.4, 4B_P12.1, 4C_P12.10
- net -X: now also 4B_P12.2
- net -XOR: now also 4E_P12.12
- net -Y: now also 1D_P12.4, 4C_P12.13
- net GND: now also 1B_P12.7 (GND), 1C_P12.7 (GND), 1D_P12.7 (GND), 1E_P12.7 (GND), 2A_P12.7 (GND), 3A_P12.7 (GND), 3D_P12.7 (GND), 3E_P12.7 (GND), 4B_P12.7 (GND), 4C_P12.7 (GND), 4E_P12.7 (GND), 5A_P12.7 (GND), 5C_P12.7 (GND), 5D_P12.7 (GND)
- net P12_3A6: now also 3A_P12.10, 3A_P12.6
- net T/T: now also 5A_P12.11
- net VCC: now also 1B_P12.14 (VCC), 1C_P12.14 (VCC), 1D_P12.14 (VCC), 1E_P12.14 (VCC), 2A_P12.14 (VCC), 3A_P12.14 (VCC), 3D_P12.14 (VCC), 3E_P12.14 (VCC), 4B_P12.14 (VCC), 4C_P12.14 (VCC), 4E_P12.14 (VCC), 5A_P12.14 (VCC), 5C_P12.14 (VCC), 5D_P12.14 (VCC)
- net at 1A_P12.10: now also 1B_P12.4
- net at 1A_P12.13: now also 1C_P12.12
- net at 5B_P12.1: now also 5C_P12.2
- net at 4A_P12.12: now also 3D_P12.10, 5C_P12.10
- net at 5B_P12.13: now also 1D_P12.9
- net at 3C_P12.1: now also 3A_P12.8
- net at 3C_P12.4: now also 3D_P12.11
- net at 3C_P12.8: now also 3B_P12.3
- net at 3B_P12.1: now also 3A_P12.12
- net at _2C_P12.6: now also 1E_P12.5
- net at _2C_P12.2: now also 2B_P12.13
- net at 2C_P12.8: now also 3E_P12.1, 3E_P12.2, 3E_P12.4, 3E_P12.5
- net at 2C_P12.10: now also 4C_P12.11
- new net: 1C_P12.4, 1D_P12.8
- new net: 5C_P12.3, 5C_P12.4
- new net: 5C_P12.5, 5C_P12.8, 5D_P12.10, 5D_P12.12, 5D_P12.13, 5D_P12.9
- new net: 5C_P12.6, 5C_P12.9, 5D_P12.1, 5D_P12.2, 5D_P12.4, 5D_P12.5
- new net: 1D_P12.2, 1D_P12.6
- new net: 1D_P12.3, 1E_P12.1
- new net: 3D_P12.5, 3D_P12.8
- new net: 3D_P12.6, 3D_P12.9, 3E_P12.10, 3E_P12.12, 3E_P12.13, 3E_P12.9
- new net: 4C_P12.12, 4C_P12.8
- new net: 4B_P12.3, 5A_P12.12, 5A_P12.13
- new net: 2A_P12.8, 3A_P12.5
- new net: 2A_P12.6, 3A_P12.9
- new net: 1B_P12.3, 1C_P12.1
- new net: 2A_P12.3, 3D_P12.13
- new net: 1D_P12.11, 1E_P12.9
Other:
- moved on the sheet: 1A_P12E, 1A_P12F, 1A_P12G, 2B_P12C, 2B_P12E, 3B_P12A, 3B_P12B, 3B_P12F, 3B_P12G, 4A_P12E, 4A_P12F, 4A_P12G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
