File: CT2-5/CT2-5.sch (KiCad schematic (older format))
At the start: 29 parts

Commit message: finalizado o desenho do esquematico da placa CT2-5
Connections:
- net +(PARTIDA(-RODA)) is gone; now on net +(PARTIDA.(-RODA)): 3A_P13.11
- net -(F2.SAESA.5) is gone; now on net -(F2.SAESA.S): 5C_P13.8
- net 3E13 is gone; now on net +(PARTIDA.CE.(-RODA)): 5D_P13.2, 5E_P13.2
- net +(CAC+SOM): now also CONECTOR_P13.39 (P39)
- net +(F1+F2): now also 3B_P13.6, 4B_P13.5, 4C_P13.5
- net +(F3.SUS.(-RDZ)): now also 2B_P13.8, 2D_P13.4
- net +(PARTIDA.(-RODA)): now also 1B_P13.5, 3D_P13.13
- net +(TRO+TRI): now also 1C_P13.11, 1C_P13.9
- net +ACN: now also CONECTOR_P13.48 (P48)
- net +ARA: now also CONECTOR_P13.4 (P4)
- net +CE: now also CONECTOR_P13.51 (P51)
- net +CP: now also CONECTOR_P13.41 (P41)
- net +F1: now also 1A_P13.6, 1C_P13.10
- net +F2: now also 2A_P13.8, 4E_P13.13
- net +F4: now also 3F_P13.12, 5C_P13.1
- net +F5: now also 2A_P13.2, 2C_P13.1
- net +IME: now also CONECTOR_P13.56 (P56)
- net +INDICE: now also CONECTOR_P13.3 (P3)
- net +MICG2A: now also CONECTOR_P13.61 (P61)
- net +MP: now also CONECTOR_P13.28 (P28)
- net +P(0-3)/M: now also CONECTOR_P13.46 (P46)
- net +PAN: now also CONECTOR_P13.12 (P12)
- net +PAZ: now also CONECTOR_P13.21 (P21)
- net +PLI: now also CONECTOR_P13.7 (P7)
- net +PM1: now also CONECTOR_P13.57 (P57)
- net +PUG: now also CONECTOR_P13.5 (P5)
- net +PUL: now also CONECTOR_P13.23 (P23)
- net +RD/Y: now also CONECTOR_P13.17 (P17)
- net +RI_(4-7)/M: now also CONECTOR_P13.60 (P60)
- net +RODA: now also CONECTOR_P13.50 (P50)
- net +S: now also CONECTOR_P13.59 (P59)
- net +SAESA: now also CONECTOR_P13.24 (P24)
- net +SALMIC: now also CONECTOR_P13.26 (P26)
- net +SUS: now also CONECTOR_P13.40 (P40)
- net +T1: now also CONECTOR_P13.54 (P54)
- net +T12: now also CONECTOR_P13.6 (P6)
- net +T2: now also CONECTOR_P13.53 (P53)
- net +T23: now also CONECTOR_P13.49 (P49)
- net +T34: now also CONECTOR_P13.52 (P52)
- net +T4: now also CONECTOR_P13.18 (P18)
- net +T56: now also CONECTOR_P13.16 (P16)
- net +T6: now also CONECTOR_P13.19 (P19)
- net +TRI: now also CONECTOR_P13.37 (P37)
- net +TRO: now also CONECTOR_P13.2 (P2)
- net +U/R: now also CONECTOR_P13.45 (P45)
- net +Z/R: now also CONECTOR_P13.10 (P10)
- net -(CAC+SOM): now also 1A_P13.10, 1C_P13.1
- net -(C_CI)_1: now also CONECTOR_P13.55 (P55)
- net -(C_CI)_2: now also CONECTOR_P13.20 (P20)
- net -(C_RE)_1: now also CONECTOR_P13.62 (P62)
- net -(C_RE)_2: now also CONECTOR_P13.27 (P27)
- net -(C_RI): now also CONECTOR_P13.58 (P58)
- net -(PAN.ACN): now also 3B_P13.3, 4D_P13.12
- net -(PARTIDA.(-RODA)): now also 3E_P13.12, 3F_P13.10
- net -(PAZ.ACZ): now also 4D_P13.13, 5A_P13.3
- net -(TRO+TRI): now also 2B_P13.10, 2C_P13.5
- net -ACZ: now also CONECTOR_P13.8 (P8)
- net -ARA: now also 1A_P13.8, 1C_P13.2
- net -CF3: now also CONECTOR_P13.9 (P9)
- net -CF4: now also CONECTOR_P13.47 (P47)
- net -CF5: now also CONECTOR_P13.11 (P11)
- net -F1: now also CONECTOR_P13.38 (P38)
- net -F2: now also CONECTOR_P13.44 (P44)
- net -F3: now also CONECTOR_P13.43 (P43)
- net -F4: now also CONECTOR_P13.13 (P13)
- net -F5: now also CONECTOR_P13.42 (P42)
- net -INDICE: now also 1A_P13.12, 1C_P13.4
- net -PARTIDA: now also CONECTOR_P13.14 (P14)
- net -PLI: now also 2A_P13.4, 2C_P13.2
- net -PUG: now also 2A_P13.12, 2C_P13.4
- net -RDZ: now also CONECTOR_P13.15 (P15)
- net GND: now also CONECTOR_P13.70 (P70)
- net PAROP: now also CONECTOR_P13.22 (P22)
- net VCC: now also CONECTOR_P13.1 (P1)
- net +(PARTIDA.CE.(-RODA)): now reaches 3E_P13.13, 4B_P13.13, 4C_P13.13
- net -(PAROP.PMI) renamed -(PAROP.PM1)
- removed net ?: CONECTOR_P13.1 (P1), CONECTOR_P13.10 (P10), CONECTOR_P13.11 (P11), CONECTOR_P13.12 (P12), CONECTOR_P13.13 (P13), CONECTOR_P13.14 (P14), CONECTOR_P13.15 (P15), CONECTOR_P13.16 (P16), CONECTOR_P13.17 (P17), CONECTOR_P13.18 (P18), CONECTOR_P13.19 (P19), CONECTOR_P13.2 (P2), CONECTOR_P13.20 (P20), CONECTOR_P13.21 (P21), CONECTOR_P13.22 (P22), CONECTOR_P13.23 (P23), CONECTOR_P13.24 (P24), CONECTOR_P13.25, CONECTOR_P13.26 (P26), CONECTOR_P13.27 (P27), CONECTOR_P13.28 (P28), CONECTOR_P13.29 (P29), CONECTOR_P13.3 (P3), CONECTOR_P13.30 (P30), CONECTOR_P13.31 (P31), CONECTOR_P13.32 (P32), CONECTOR_P13.33 (P33), CONECTOR_P13.34 (P34), CONECTOR_P13.35 (P35), CONECTOR_P13.36 (P36), CONECTOR_P13.37 (P37), CONECTOR_P13.38 (P38), CONECTOR_P13.39 (P39), CONECTOR_P13.4 (P4), CONECTOR_P13.40 (P40), CONECTOR_P13.41 (P41), CONECTOR_P13.42 (P42), CONECTOR_P13.43 (P43), CONECTOR_P13.44 (P44), CONECTOR_P13.45 (P45), CONECTOR_P13.46 (P46), CONECTOR_P13.47 (P47), CONECTOR_P13.48 (P48), CONECTOR_P13.49 (P49), CONECTOR_P13.5 (P5), CONECTOR_P13.50 (P50), CONECTOR_P13.51 (P51), CONECTOR_P13.52 (P52), CONECTOR_P13.53 (P53), CONECTOR_P13.54 (P54), CONECTOR_P13.55 (P55), CONECTOR_P13.56 (P56), CONECTOR_P13.57 (P57), CONECTOR_P13.58 (P58), CONECTOR_P13.59 (P59), CONECTOR_P13.6 (P6), CONECTOR_P13.60 (P60), CONECTOR_P13.61 (P61), CONECTOR_P13.62 (P62), CONECTOR_P13.63 (P63), CONECTOR_P13.64 (P64), CONECTOR_P13.65 (P65), CONECTOR_P13.66 (P66), CONECTOR_P13.67 (P67), CONECTOR_P13.68 (P68), CONECTOR_P13.69 (P69), CONECTOR_P13.7 (P7), CONECTOR_P13.70 (P70), CONECTOR_P13.8 (P8), CONECTOR_P13.9 (P9)
- no-connect marks 0 -> 16
Other:
- moved on the sheet: 2A_P13B, 2B_P13D, 5B_P13A

Commit message: placa CT2-5: symbol remap
Parts:
- 1A_P13, 2A_P13, 2B_P13, 3F_P13, 4A_P13: symbol 74HC04 -> CT2-5-rescue:74HC04
- 1B_P13, 1C_P13, 1E_P13, 2C_P13, 3B_P13, 4E_P13, 5A_P13, 5C_P13: symbol 7400 -> CT2-5-rescue:7400
- 1D_P13, 2E_P13, 3A_P13: symbol 74LS10 -> CT2-5-rescue:74LS10
- 1F_P13, 3D_P13, 3E_P13, 5B_P13: symbol 7402 -> CT2-5-rescue:7402
- 2D_P13: symbol 74LS51 -> CT2-5-rescue:74LS51
- 2F_P13, 4D_P13: symbol 74LS13 -> CT2-5-rescue:74LS13
- 3C_P13, 4B_P13, 4C_P13, 5D_P13, 5E_P13: symbol 74LS54 -> CT2-5-rescue:74LS54
- CONECTOR_P13: symbol CONN_35X2 -> CT2-5-rescue:CONN_35X2
