File: CT2-5/CT2-5.kicad_sch (KiCad schematic)
At the start: 29 parts

Commit message: These are updated files after I loaded the project on a new version of KICAD
Parts:
- 1A_P13, 1B_P13, 1C_P13, 1D_P13, 1E_P13, 1F_P13, 2A_P13, 2B_P13, 2C_P13, 2E_P13, 2F_P13, 3A_P13, 3B_P13, 3C_P13, 3D_P13, 3E_P13, 3F_P13, 4A_P13, 4B_P13, 4C_P13, 4D_P13, 4E_P13, 5A_P13, 5B_P13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: footprint ~ -> (none)
