File: CT4-7/CT4-7.sch (KiCad schematic (older format))
At the start: 26 parts

Commit message: terminei a transcrição do esquema da placa CT4-7
Connections:
- net +F4.(TRO+TRI) is gone; now on net +(F4.(TRO+TRI)): 3B_P15.8
- net -ACN is gone; now on net -AC_0: 2B_P15.5
- net -F4.(TRO+TRI) is gone; now on net -(F4.(TRO+TRI)): 3B_P15.9
- net +(F3+F4): now also 2E_P15.8, 4D_P15.9
- net +(PARTIDA.(-RODA)): now also 2E_P15.12, 3E_P15.1
- net +(TRO+TRI): now also 2B_P15.11, 3C_P15.10
- net +1/I: now also CONECTOR_P15.24 (P24)
- net +AC_0: now also CONECTOR_P15.2 (P2)
- net +AC_1: now also CONECTOR_P15.37 (P37)
- net +AC_2: now also CONECTOR_P15.3 (P3)
- net +AC_3: now also CONECTOR_P15.38 (P38)
- net +AC_4: now also CONECTOR_P15.4 (P4)
- net +AC_5: now also CONECTOR_P15.39 (P39)
- net +AC_6: now also CONECTOR_P15.5 (P5)
- net +AC_7: now also CONECTOR_P15.40 (P40)
- net +CASP: now also CONECTOR_P15.11 (P11)
- net +CE: now also CONECTOR_P15.56 (P56)
- net +CI(4-11)/X: now also CONECTOR_P15.55 (P55)
- net +CP: now also CONECTOR_P15.42 (P42)
- net +IME: now also CONECTOR_P15.14 (P14)
- net +MICG1: now also CONECTOR_P15.57 (P57)
- net +MICG2A: now also CONECTOR_P15.13 (P13)
- net +MP: now also CONECTOR_P15.7 (P7)
- net +OVF: now also CONECTOR_P15.15 (P15)
- net +P(4-11)/Y: now also CONECTOR_P15.23 (P23)
- net +PAN: now also CONECTOR_P15.43 (P43)
- net +PAZ: now also CONECTOR_P15.8 (P8)
- net +PUG: now also CONECTOR_P15.52 (P52)
- net +RE/I: now also CONECTOR_P15.26 (P26)
- net +RE/X,M: now also CONECTOR_P15.60 (P60)
- net +RI_4: now also CONECTOR_P15.22 (P22)
- net +RI_5: now also CONECTOR_P15.6 (P6)
- net +RI_6: now also CONECTOR_P15.41 (P41)
- net +RI_7: now also CONECTOR_P15.46 (P46)
- net +RODA: now also CONECTOR_P15.53 (P53)
- net +S: now also CONECTOR_P15.51 (P51)
- net +SAE: now also CONECTOR_P15.49 (P49)
- net +SAESA: now also CONECTOR_P15.16 (P16)
- net +SALMIC: now also CONECTOR_P15.29 (P29)
- net +SUS: now also CONECTOR_P15.48 (P48)
- net +T: now also CONECTOR_P15.50 (P50)
- net +T01: now also CONECTOR_P15.19 (P19)
- net +T12: now also CONECTOR_P15.17 (P17)
- net +T34: now also CONECTOR_P15.54 (P54)
- net +T56: now also CONECTOR_P15.20 (P20)
- net +T7: now also CONECTOR_P15.64 (P64)
- net +TRI: now also CONECTOR_P15.47 (P47)
- net +TRO: now also CONECTOR_P15.12 (P12)
- net -ACZ: now also CONECTOR_P15.63 (P63)
- net -CLEAR_OVF: now also CONECTOR_P15.61 (P61)
- net -CLEAR_T: now also CONECTOR_P15.27 (P27)
- net -F1: now also CONECTOR_P15.9 (P9)
- net -F2: now also CONECTOR_P15.44 (P44)
- net -F3: now also CONECTOR_P15.10 (P10)
- net -F4: now also CONECTOR_P15.45 (P45)
- net -F5: now also CONECTOR_P15.25
- net -PARTIDA: now also CONECTOR_P15.18 (P18)
- net -SET_OVF: now also CONECTOR_P15.62 (P62)
- net -SET_T: now also CONECTOR_P15.28 (P28)
- net ?: no longer CONECTOR_P15.1 (P1), CONECTOR_P15.10 (P10), CONECTOR_P15.11 (P11), CONECTOR_P15.12 (P12), CONECTOR_P15.13 (P13), CONECTOR_P15.14 (P14), CONECTOR_P15.15 (P15), CONECTOR_P15.16 (P16), CONECTOR_P15.17 (P17), CONECTOR_P15.18 (P18), CONECTOR_P15.19 (P19), CONECTOR_P15.2 (P2), CONECTOR_P15.20 (P20), CONECTOR_P15.21 (P21), CONECTOR_P15.22 (P22), CONECTOR_P15.23 (P23), CONECTOR_P15.24 (P24), CONECTOR_P15.25, CONECTOR_P15.26 (P26), CONECTOR_P15.27 (P27), CONECTOR_P15.28 (P28), CONECTOR_P15.29 (P29), CONECTOR_P15.3 (P3), CONECTOR_P15.37 (P37), CONECTOR_P15.38 (P38), CONECTOR_P15.39 (P39), CONECTOR_P15.4 (P4), CONECTOR_P15.40 (P40), CONECTOR_P15.41 (P41), CONECTOR_P15.42 (P42), CONECTOR_P15.43 (P43), CONECTOR_P15.44 (P44), CONECTOR_P15.45 (P45), CONECTOR_P15.46 (P46), CONECTOR_P15.47 (P47), CONECTOR_P15.48 (P48), CONECTOR_P15.49 (P49), CONECTOR_P15.5 (P5), CONECTOR_P15.50 (P50), CONECTOR_P15.51 (P51), CONECTOR_P15.52 (P52), CONECTOR_P15.53 (P53), CONECTOR_P15.54 (P54), CONECTOR_P15.55 (P55), CONECTOR_P15.56 (P56), CONECTOR_P15.57 (P57), CONECTOR_P15.6 (P6), CONECTOR_P15.60 (P60), CONECTOR_P15.61 (P61), CONECTOR_P15.62 (P62), CONECTOR_P15.63 (P63), CONECTOR_P15.64 (P64), CONECTOR_P15.7 (P7), CONECTOR_P15.70 (P70), CONECTOR_P15.8 (P8), CONECTOR_P15.9 (P9)
- net GND: now also CONECTOR_P15.70 (P70)
- net VCC: now also CONECTOR_P15.1 (P1)
- net -(F4.(TRO+TRI)): now reaches 2D_P15.13, 3C_P15.8
- net +CI(0-3)/X renamed +CI(0-3)/M
- net +CI(0-3)/M: now also CONECTOR_P15.21 (P21)
- net -RI_7: no longer names the net of 3A_P15.12
- no-connect marks 0 -> 1
Other:
- note added: "(!) Essa porta gera o sinal -RI_7.\nEntretanto esse sinal não é usado nesta placa.\nPortanto, a porta NOT da unidade F da\npastilha 3A não é realmente necessária."
- note added: "(!) O esquema original indica 1A2\n(que corresponde a -AC_0),\nmas ao mesmo tempo\nchama esse sinal de -ACN"
- note added: "-RI_7"
- moved on the sheet: 2E_P15C

Commit message: placa CT4-7: symbol remap
Parts:
- 1A_P15, 2A_P15, 3A_P15, 3B_P15, 4A_P15: symbol 74LS04 -> CT4-7-rescue:74LS04
- 1B_P15: symbol 74LS30 -> CT4-7-rescue:74LS30
- 1C_P15, 1D_P15, 2B_P15, 2E_P15, 3C_P15, 4D_P15, 5B_P15, 5C_P15: symbol 7400 -> CT4-7-rescue:7400
- 1E_P15: symbol 74LS54 -> CT4-7-rescue:74LS54
- 2C_P15, 3D_P15, 5D_P15, 5E_P15: symbol 74LS15 -> CT4-7-rescue:74LS15
- 2D_P15, 4B_P15, 5A_P15: symbol 74LS20 -> CT4-7-rescue:74LS20
- 3E_P15, 4E_P15: symbol 7402 -> CT4-7-rescue:7402
- 4C_P15: symbol 74LS51 -> CT4-7-rescue:74LS51
- CONECTOR_P15: symbol CONN_35X2 -> CT4-7-rescue:CONN_35X2
