File: CT4-7/CT4-7.kicad_sch (KiCad schematic)
At the start: 26 parts

Commit message: These are updated files after I loaded the project on a new version of KICAD
Parts:
- 3E_P15, 4E_P15: footprint ~ -> (none)
