File: CT4-7/CT4-7.kicad_sch (KiCad schematic)
At the start: 26 parts

Commit message: a lot more work on the circuit transcription
Parts:
- removed 1A_P15, 2A_P15, 3A_P15, 3B_P15, 4A_P15: 74LS04, symbol CT4-7-rescue:74LS04
- removed 1B_P15: 74LS30, symbol CT4-7-rescue:74LS30
- removed 1E_P15: 74LS54, symbol CT4-7-rescue:74LS54
- removed 2C_P15, 3D_P15, 5D_P15, 5E_P15: 74LS15, symbol CT4-7-rescue:74LS15
- removed 2D_P15, 4B_P15, 5A_P15: 74LS20, symbol CT4-7-rescue:74LS20
- removed 3E_P15, 4E_P15: 7402, symbol CT4-7-rescue:7402
- added 1A_P15, 2A_P15, 3A_P15, 3B_P15, 4A_P15: 74LS04, symbol 74xx:74LS04
- added 1B_P15: 74LS30, symbol 74xx:74LS30
- added 1E_P15: 7454, symbol 74xx_IEEE:7454
- added 2C_P15, 3D_P15, 5D_P15, 5E_P15: 74LS15, symbol 74xx:74LS15
- added 2D_P15, 4B_P15, 5A_P15: 74LS20, symbol 74xx:74LS20
- added 3E_P15, 4E_P15: 74LS02, symbol 74xx:74LS02
Connections:
- net +(F4.(TRO+TRI)): now also 3B_P15.8
- net +(PARTIDA.(-RODA)): now also 3D_P15.11, 3E_P15.1
- net +1/I: now also 3B_P15.12
- net +AC_0: now also 1A_P15.1
- net +AC_1: now also 1A_P15.3
- net +AC_2: now also 1A_P15.5
- net +AC_3: now also 1A_P15.9
- net +AC_4: now also 1A_P15.11
- net +AC_5: now also 1A_P15.13
- net +AC_6: now also 2A_P15.1
- net +AC_7: now also 2A_P15.3
- net +CASP: now also 3A_P15.11
- net +CE: now also 3B_P15.5
- net +CP: now also 2A_P15.13
- net +F1: now also 2C_P15.13, 3A_P15.2, 5A_P15.1
- net +F2: now also 3A_P15.4
- net +F3: now also 2C_P15.9, 3A_P15.6, 3D_P15.4
- net +F4: now also 3A_P15.8, 3D_P15.2
- net +IME: now also 4A_P15.11
- net +MICG1: now also 5A_P15.5
- net +MICG2A: now also 2C_P15.1, 4A_P15.5
- net +MP: now also 2A_P15.11
- net +PUG: now also 3D_P15.13, 3D_P15.5
- net +RE/I: now also 5D_P15.6
- net +RE/X,M: now also 4B_P15.6
- net +RI_4: now also 5A_P15.4
- net +RI_5: now also 2A_P15.5, 4E_P15.2, 4E_P15.8
- net +RI_6: now also 2A_P15.9
- net +RI_7: now also 3A_P15.13
- net +RODA: now also 3E_P15.3
- net +S: now also 2C_P15.11
- net +SAE: now also 4A_P15.13
- net +SALMIC: now also 2C_P15.2
- net +SUS: now also 2C_P15.10, 4A_P15.9
- net +T01: now also 1E_P15.13
- net +T12: now also 3D_P15.1, 3D_P15.3, 3D_P15.9
- net +T34: now also 1E_P15.2, 5A_P15.2
- net +T56: now also 1E_P15.4, 1E_P15.9
- net +T7: now also 5D_P15.2, 5E_P15.10, 5E_P15.2, 5E_P15.4
- net +TRI: now also 4A_P15.3
- net +TRO: now also 4A_P15.1
- net -(F4.(TRO+TRI)): now also 2D_P15.13, 3B_P15.9
- net -ACZ: now also 1B_P15.8
- net -AC_0: now also 1A_P15.2, 1B_P15.1
- net -AC_1: now also 1A_P15.4, 1B_P15.2
- net -AC_2: now also 1A_P15.6, 1B_P15.3
- net -AC_3: now also 1A_P15.8, 1B_P15.4
- net -AC_4: now also 1A_P15.10, 1B_P15.5
- net -AC_5: now also 1A_P15.12, 1B_P15.6
- net -AC_6: now also 1B_P15.11, 2A_P15.2
- net -AC_7: now also 1B_P15.12, 2A_P15.4
- net -CASP: now also 3A_P15.10
- net -CE: now also 3B_P15.6
- net -CLEAR_OVF: now also 5E_P15.12
- net -CLEAR_T: now also 5E_P15.6
- net -CP: now also 2A_P15.12
- net -F1: now also 2D_P15.9, 3A_P15.1, 3E_P15.5
- net -F2: now also 3A_P15.3
- net -F3: now also 3A_P15.5
- net -F4: now also 3A_P15.9
- net -IME: now also 2D_P15.2, 4A_P15.10
- net -MICG2A: now also 3E_P15.6, 4A_P15.6
- net -MP: now also 2A_P15.10
- net -PARTIDA: now also 3E_P15.2
- net -RD_5: now also 2A_P15.6, 4E_P15.6
- net -RI_5: now also 4E_P15.12
- net -RI_6: now also 2A_P15.8
- net -SAE: now also 2D_P15.5, 4A_P15.12
- net -SET_OVF: now also 5E_P15.8
- net -SET_T: now also 5D_P15.12
- net -SUS: now also 4A_P15.8
- net -TRI: now also 4A_P15.4
- net -TRO: now also 4A_P15.2
- net GND: now also 1A_P15.7 (GND), 1B_P15.7 (GND), 1E_P15.7 (GND), 2A_P15.7 (GND), 2C_P15.7 (GND), 2D_P15.7 (GND), 3A_P15.7 (GND), 3B_P15.7 (GND), 3D_P15.7 (GND), 3E_P15.7 (GND), 4A_P15.7 (GND), 4B_P15.7 (GND), 4E_P15.7 (GND), 5A_P15.7 (GND), 5D_P15.7 (GND), 5E_P15.7 (GND)
- net VCC: now also 1A_P15.14 (VCC), 1B_P15.14 (VCC), 1E_P15.14 (VCC), 2A_P15.14 (VCC), 2C_P15.14 (VCC), 2D_P15.14 (VCC), 3A_P15.14 (VCC), 3B_P15.14 (VCC), 3D_P15.14 (VCC), 3E_P15.14 (VCC), 4A_P15.14 (VCC), 4B_P15.14 (VCC), 4E_P15.14 (VCC), 5A_P15.14 (VCC), 5D_P15.14 (VCC), 5E_P15.14 (VCC)
- net at 5C_P15.6: now also 5D_P15.3, 5D_P15.4, 5D_P15.5
- net at 1C_P15.8, 1D_P15.2: now also 3B_P15.1
- net at 1D_P15.4: now also 3B_P15.2
- net at 5B_P15.5: now also 5A_P15.6
- net at 5B_P15.3: now also 3D_P15.10
- net at 5B_P15.4: now also 3D_P15.8
- net at 5B_P15.8: now also 3B_P15.13
- net at 4C_P15.6: now also 4B_P15.1, 4B_P15.2, 4B_P15.4, 4B_P15.5
- net at 4D_P15.6: now also 4E_P15.11, 4E_P15.9
- net at 4D_P15.3: now also 4E_P15.3, 4E_P15.5
- net at 2E_P15.5: now also 3D_P15.6
- net at 2E_P15.1, 2E_P15.4: now also 1E_P15.8; no longer 2E_P15.2
- net at 1D_P15.11: now also 1E_P15.1
- net at 1C_P15.11: now also 2C_P15.4
- net at 2E_P15.11: now also 3B_P15.3
- net at 2B_P15.3: now also 2D_P15.1
- net at 2B_P15.6: now also 2D_P15.4
- net at 3C_P15.1: now also 2D_P15.6
- net at 3C_P15.3: now also 2D_P15.10
- net at 3C_P15.6: now also 2D_P15.12
- new net: 1E_P15.5, 3B_P15.4
- new net: 1E_P15.10, 2D_P15.8
- new net: 1E_P15.3, 2C_P15.6
- new net: 4E_P15.4, 5E_P15.3
- new net: 4E_P15.13, 5D_P15.1
- new net: 3E_P15.4, 5D_P15.13, 5E_P15.11, 5E_P15.13, 5E_P15.5
- new net: 2C_P15.5, 2C_P15.8
- new net: 2E_P15.2, 3D_P15.12
- new net: 4E_P15.10, 5E_P15.9
- new net: 4E_P15.1, 5E_P15.1
- new net: 2C_P15.12, 2C_P15.3
Other:
- moved on the sheet: 1C_P15A, 1C_P15B, 1C_P15C, 1C_P15D, 1D_P15A, 1D_P15B, 1D_P15C, 1D_P15D, 2B_P15A, 2B_P15B, 2B_P15C, 2B_P15D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

Commit message: wip + PDF plot
Other:
- moved on the sheet: 1A_P15G, 1B_P15B, 1C_P15E, 1D_P15E, 2A_P15G, 2B_P15E, 2C_P15D, 2D_P15C, 2E_P15E, 3A_P15G, 3B_P15G, 3C_P15E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
