File: PCP-2/PCP-2.sch (KiCad schematic (older format))
At the start: 1 part

Commit message: finalizado o desenho da placa PCP-2
Parts:
- added 2A_P8, 4B_P8, 4C_P8: 7400, symbol 7400
- added 3A_P8, 3B_P8, 4D_P8: 74LS04, symbol 74LS04
- added 4E_P8, 5B_P8, 5C_P8, 5D_P8: 74LS10, symbol 74LS10
- added 5E_P8, U1: 74LS08, symbol 74LS08
- added CONECTOR_T_P8: CONN_35X2, symbol CONN_35X2
- added D1, D2, D3, D4, D5, D6: BAX13, symbol DIODE
- added Q10_P8, Q11_P8, Q12_P8, Q13_P8, Q14_P8, Q15_P8, Q1_P8, Q2_P8, Q3_P8, Q4_P8, Q5_P8, Q6_P8, Q7_P8, Q8_P8, Q9_P8: BC237, TO92, symbol BC414
- added R1, R10, R11, R12, R13, R14, R15, R16, R17, R18, R2, R22, R23, R3, R4, R5, R6, R7, R8, R9: 3,9k 1/8W, symbol R
- added R19, R20, R21, R24, R25, R26, R37, R38, R39: 5,6k 1/8W, symbol R
- added R27, R28, R29, R30, R31, R32, R33, R34, R35, R36, R40, R41, R42, R43, R44, R45, R46, R47: R, symbol R
- renumbered CONECTOR_P8 to CONECTOR_F_P8
Connections:
- removed net ?: CONECTOR_F_P8.1 (P1), CONECTOR_F_P8.10 (P10), CONECTOR_F_P8.11 (P11), CONECTOR_F_P8.12 (P12), CONECTOR_F_P8.13 (P13), CONECTOR_F_P8.14 (P14), CONECTOR_F_P8.15 (P15), CONECTOR_F_P8.16 (P16), CONECTOR_F_P8.17 (P17), CONECTOR_F_P8.18 (P18), CONECTOR_F_P8.19 (P19), CONECTOR_F_P8.2 (P2), CONECTOR_F_P8.20 (P20), CONECTOR_F_P8.21 (P21), CONECTOR_F_P8.22 (P22), CONECTOR_F_P8.23 (P23), CONECTOR_F_P8.24 (P24), CONECTOR_F_P8.25, CONECTOR_F_P8.26 (P26), CONECTOR_F_P8.27 (P27), CONECTOR_F_P8.28 (P28), CONECTOR_F_P8.29 (P29), CONECTOR_F_P8.3 (P3), CONECTOR_F_P8.30 (P30), CONECTOR_F_P8.31 (P31), CONECTOR_F_P8.32 (P32), CONECTOR_F_P8.33 (P33), CONECTOR_F_P8.34 (P34), CONECTOR_F_P8.35 (P35), CONECTOR_F_P8.36 (P36), CONECTOR_F_P8.37 (P37), CONECTOR_F_P8.38 (P38), CONECTOR_F_P8.39 (P39), CONECTOR_F_P8.4 (P4), CONECTOR_F_P8.40 (P40), CONECTOR_F_P8.41 (P41), CONECTOR_F_P8.42 (P42), CONECTOR_F_P8.43 (P43), CONECTOR_F_P8.44 (P44), CONECTOR_F_P8.45 (P45), CONECTOR_F_P8.46 (P46), CONECTOR_F_P8.47 (P47), CONECTOR_F_P8.48 (P48), CONECTOR_F_P8.49 (P49), CONECTOR_F_P8.5 (P5), CONECTOR_F_P8.50 (P50), CONECTOR_F_P8.51 (P51), CONECTOR_F_P8.52 (P52), CONECTOR_F_P8.53 (P53), CONECTOR_F_P8.54 (P54), CONECTOR_F_P8.55 (P55), CONECTOR_F_P8.56 (P56), CONECTOR_F_P8.57 (P57), CONECTOR_F_P8.58 (P58), CONECTOR_F_P8.59 (P59), CONECTOR_F_P8.6 (P6), CONECTOR_F_P8.60 (P60), CONECTOR_F_P8.61 (P61), CONECTOR_F_P8.62 (P62), CONECTOR_F_P8.63 (P63), CONECTOR_F_P8.64 (P64), CONECTOR_F_P8.65 (P65), CONECTOR_F_P8.66 (P66), CONECTOR_F_P8.67 (P67), CONECTOR_F_P8.68 (P68), CONECTOR_F_P8.69 (P69), CONECTOR_F_P8.7 (P7), CONECTOR_F_P8.70 (P70), CONECTOR_F_P8.8 (P8), CONECTOR_F_P8.9 (P9)
- new net: D1.1 (A), R7.1, R8.1
- new net: Q1_P8.2 (B), R8.2
- new net: 4E_P8.9, 5D_P8.11, 5D_P8.13, 5D_P8.3, 5E_P8.8
- new net: 4D_P8.3, 4E_P8.12
- new net: 4D_P8.4, 5B_P8.1
- new net: 4E_P8.11, 4E_P8.13, 4E_P8.4, 5D_P8.4, 5E_P8.6
- new net: 4E_P8.2, 4E_P8.5, 5D_P8.1, 5D_P8.9, U1.3
- new net: 4C_P8.2, 5B_P8.12
- new net: D2.1 (A), R10.1, R9.1
- new net: Q2_P8.2 (B), R10.2
- new net: 4D_P8.1, 4E_P8.6
- new net: 4D_P8.2, 5B_P8.5
- new net: 4C_P8.5, 5B_P8.6
- new net: D3.1 (A), R11.1, R12.1
- new net: Q3_P8.2 (B), R12.2
- new net: 4D_P8.12, 5C_P8.11
- new net: 4D_P8.13, 5D_P8.12
- new net: 4C_P8.9, 5C_P8.8
- new net: D4.1 (A), R13.1, R14.1
- new net: Q4_P8.2 (B), R14.2
- new net: 4B_P8.1, 4D_P8.10
- new net: 4D_P8.11, 5D_P8.8
- new net: 4B_P8.3, 5B_P8.9
- new net: D5.1 (A), R15.1, R16.1
- new net: Q5_P8.2 (B), R16.2
- new net: 4D_P8.8, 5C_P8.1
- new net: 4D_P8.9, 5D_P8.6
- new net: 4B_P8.12, 5C_P8.12
- new net: D6.1 (A), R17.1, R18.1
- new net: Q6_P8.2 (B), R18.2
- new net: 4D_P8.5, 4E_P8.8
- new net: 4D_P8.6, 5C_P8.3
- new net: 4C_P8.12, 5C_P8.6
- new net: 2A_P8.12, 2A_P8.8
- new net: 3B_P8.10, Q10_P8.2 (B), R24.1
- new net: 3B_P8.2, Q9_P8.2 (B), R21.1
- new net: 3B_P8.4, Q8_P8.2 (B), R20.1
- new net: 3B_P8.6, Q7_P8.2 (B), R19.1
- new net: 3A_P8.8, Q12_P8.2 (B), R26.1
- new net: 3B_P8.12, Q11_P8.2 (B), R25.1
- new net: 3A_P8.10, Q13_P8.2 (B), R37.1
- new net: 3A_P8.12, Q15_P8.2 (B), R39.1
- new net: 3B_P8.8, Q14_P8.2 (B), R38.1
- new net +24V: CONECTOR_F_P8.34 (P34), CONECTOR_F_P8.69 (P69), CONECTOR_T_P8.2 (P2), CONECTOR_T_P8.35 (P35)
- new net +ATIVO: 4C_P8.3, 5B_P8.13, CONECTOR_T_P8.66 (P66), D1.2 (K)
- new net +CE: 4B_P8.2, 5B_P8.8, CONECTOR_T_P8.67 (P67), D4.2 (K)
- new net +CP: 4B_P8.11, 5C_P8.2, CONECTOR_T_P8.63 (P63), D5.2 (K)
- new net +CS: 4C_P8.6, 5B_P8.3, CONECTOR_T_P8.64 (P64), D2.2 (K)
- new net +IS: 4C_P8.8, 5C_P8.9, CONECTOR_T_P8.59 (P59), D3.2 (K)
- new net +MP: 4C_P8.11, 5C_P8.5, CONECTOR_T_P8.61 (P61), D6.2 (K)
- new net +PROTEÇÃO: CONECTOR_F_P8.27 (P27), CONECTOR_T_P8.46 (P46), R31.2
- new net +P_(+1): CONECTOR_F_P8.22 (P22), CONECTOR_T_P8.11 (P11), R32.2
- new net +P_0: CONECTOR_F_P8.33 (P33), CONECTOR_T_P8.3 (P3), R47.2
- new net +P_1: CONECTOR_F_P8.68 (P68), CONECTOR_T_P8.4 (P4), R46.2
- new net +P_10: CONECTOR_F_P8.23 (P23), CONECTOR_T_P8.10 (P10), R34.2
- new net +P_11: CONECTOR_F_P8.28 (P28), CONECTOR_T_P8.45 (P45), R33.2
- new net +P_2: CONECTOR_F_P8.32 (P32), CONECTOR_T_P8.5 (P5), R45.2
- new net +P_3: CONECTOR_F_P8.31 (P31), CONECTOR_T_P8.6 (P6), R44.2
- new net +P_4: CONECTOR_F_P8.26 (P26), CONECTOR_T_P8.7 (P7), R43.2
- new net +P_5: CONECTOR_F_P8.30 (P30), CONECTOR_T_P8.42 (P42), R42.2
- new net +P_6: CONECTOR_F_P8.25, CONECTOR_T_P8.8 (P8), R41.2
- new net +P_7: CONECTOR_F_P8.29 (P29), CONECTOR_T_P8.43 (P43), R40.2
- new net +P_8: CONECTOR_F_P8.24 (P24), CONECTOR_T_P8.9 (P9), R36.2
- new net +P_9: CONECTOR_F_P8.63 (P63), CONECTOR_T_P8.44 (P44), R35.2
- new net -BOT-ESP-A: CONECTOR_F_P8.19 (P19), CONECTOR_T_P8.14 (P14), R28.2
- new net -BOT-ESP-N: CONECTOR_F_P8.18 (P18), CONECTOR_T_P8.15 (P15), R27.2
- new net -BOT-INT-A: 2A_P8.9, CONECTOR_F_P8.16 (P16), R23.1
- new net -BOT-INT-N: 2A_P8.13, CONECTOR_F_P8.15 (P15), R22.1
- new net -BOT-PART-A: CONECTOR_F_P8.21 (P21), CONECTOR_T_P8.12 (P12), R30.2
- new net -BOT-PART-N: CONECTOR_F_P8.20 (P20), CONECTOR_T_P8.13 (P13), R29.2
- new net -ES: 3B_P8.9, CONECTOR_T_P8.56 (P56)
- new net -FASE1: 3B_P8.5, CONECTOR_T_P8.20 (P20)
- new net -FASE2: 3B_P8.3, CONECTOR_T_P8.19 (P19)
- new net -FASE3: 3B_P8.1, CONECTOR_T_P8.18 (P18)
- new net -FASE4: 3B_P8.11, CONECTOR_T_P8.57 (P57)
- new net -FASE5: 3B_P8.13, CONECTOR_T_P8.58 (P58)
- new net -INT: 3A_P8.13, CONECTOR_T_P8.21 (P21)
- new net -LAL: 5B_P8.11, 5B_P8.2, 5B_P8.4, 5C_P8.10, 5C_P8.13, 5C_P8.4, CONECTOR_T_P8.65 (P65)
- new net -PAR: 3A_P8.9, CONECTOR_T_P8.23 (P23)
- new net -PEDIDO_DE_INTERRUPÇÃO: 2A_P8.10, 2A_P8.11, CONECTOR_T_P8.17 (P17)
- new net -RODA: 3A_P8.11, CONECTOR_T_P8.22 (P22)
- new net AT: 4C_P8.1, 4E_P8.3, 5E_P8.9, CONECTOR_F_P8.5 (P5), R3.1
- new net CE: 5B_P8.10, 5D_P8.2, 5E_P8.4, CONECTOR_F_P8.7 (P7), R5.1
- new net CP: 4B_P8.13, 4E_P8.10, CONECTOR_F_P8.6 (P6), U1.1
- new net CS: 4C_P8.4, 5E_P8.10, CONECTOR_F_P8.40 (P40), R4.1
- new net GND: 2A_P8.7 (GND), 2A_P8.7 (GND), 3A_P8.7 (GND), 3A_P8.7 (GND), 3A_P8.7 (GND), 3B_P8.7 (GND), 3B_P8.7 (GND), 3B_P8.7 (GND), 3B_P8.7 (GND), 3B_P8.7 (GND), 3B_P8.7 (GND), 4B_P8.7 (GND), 4B_P8.7 (GND), 4C_P8.7 (GND), 4C_P8.7 (GND), 4C_P8.7 (GND), 4C_P8.7 (GND), 4D_P8.7 (GND), 4D_P8.7 (GND), 4D_P8.7 (GND), 4D_P8.7 (GND), 4D_P8.7 (GND), 4D_P8.7 (GND), 4E_P8.7 (GND), 4E_P8.7 (GND), 4E_P8.7 (GND), 5B_P8.7 (GND), 5B_P8.7 (GND), 5B_P8.7 (GND), 5C_P8.7 (GND), 5C_P8.7 (GND), 5C_P8.7 (GND), 5D_P8.7 (GND), 5D_P8.7 (GND), 5D_P8.7 (GND), 5E_P8.7 (GND), 5E_P8.7 (GND), CONECTOR_F_P8.70 (P70), CONECTOR_T_P8.70 (P70), Q10_P8.3 (E), Q11_P8.3 (E), Q12_P8.3 (E), Q13_P8.3 (E), Q14_P8.3 (E), Q15_P8.3 (E), Q1_P8.3 (E), Q2_P8.3 (E), Q3_P8.3 (E), Q4_P8.3 (E), Q5_P8.3 (E), Q6_P8.3 (E), Q7_P8.3 (E), Q8_P8.3 (E), Q9_P8.3 (E), U1.7 (GND)
- new net IS: 4C_P8.10, 5D_P8.10, 5E_P8.5, CONECTOR_F_P8.8 (P8)
- new net MP: 4C_P8.13, 5D_P8.5, CONECTOR_F_P8.41 (P41), R6.1, U1.2
- new net PAT: 4E_P8.1, CONECTOR_F_P8.4 (P4), Q1_P8.1 (C)
- new net PCE: CONECTOR_F_P8.38 (P38), Q4_P8.1 (C), R1.1
- new net PCP: CONECTOR_F_P8.2 (P2), Q5_P8.1 (C)
- new net PCS: CONECTOR_F_P8.39 (P39), Q2_P8.1 (C), R2.1
- new net PESP: CONECTOR_F_P8.14 (P14), Q14_P8.1 (C)
- new net PF1: CONECTOR_F_P8.10 (P10), Q7_P8.1 (C)
- new net PF2: CONECTOR_F_P8.45 (P45), Q8_P8.1 (C)
- new net PF3: CONECTOR_F_P8.11 (P11), Q9_P8.1 (C)
- new net PF4: CONECTOR_F_P8.12 (P12), Q10_P8.1 (C)
- new net PF5: CONECTOR_F_P8.47 (P47), Q11_P8.1 (C)
- new net PIS: CONECTOR_F_P8.3 (P3), Q3_P8.1 (C)
- new net PMP: CONECTOR_F_P8.37 (P37), Q6_P8.1 (C)
- new net PNT: CONECTOR_F_P8.49 (P49), Q15_P8.1 (C)
- new net POP: CONECTOR_F_P8.13 (P13), Q13_P8.1 (C)
- new net PPAR: CONECTOR_F_P8.48 (P48), Q12_P8.1 (C)
- new net VCC: 2A_P8.14 (VCC), 2A_P8.14 (VCC), 3A_P8.14 (VCC), 3A_P8.14 (VCC), 3A_P8.14 (VCC), 3B_P8.14 (VCC), 3B_P8.14 (VCC), 3B_P8.14 (VCC), 3B_P8.14 (VCC), 3B_P8.14 (VCC), 3B_P8.14 (VCC), 4B_P8.14 (VCC), 4B_P8.14 (VCC), 4C_P8.14 (VCC), 4C_P8.14 (VCC), 4C_P8.14 (VCC), 4C_P8.14 (VCC), 4D_P8.14 (VCC), 4D_P8.14 (VCC), 4D_P8.14 (VCC), 4D_P8.14 (VCC), 4D_P8.14 (VCC), 4D_P8.14 (VCC), 4E_P8.14 (VCC), 4E_P8.14 (VCC), 4E_P8.14 (VCC), 5B_P8.14 (VCC), 5B_P8.14 (VCC), 5B_P8.14 (VCC), 5C_P8.14 (VCC), 5C_P8.14 (VCC), 5C_P8.14 (VCC), 5D_P8.14 (VCC), 5D_P8.14 (VCC), 5D_P8.14 (VCC), 5E_P8.14 (VCC), 5E_P8.14 (VCC), CONECTOR_F_P8.1 (P1), CONECTOR_T_P8.1 (P1), R1.2, R11.2, R13.2, R15.2, R17.2, R19.2, R2.2, R20.2, R21.2, R22.2, R23.2, R24.2, R25.2, R26.2, R27.1, R28.1, R29.1, R3.2, R30.1, R31.1, R32.1, R33.1, R34.1, R35.1, R36.1, R37.2, R38.2, R39.2, R4.2, R40.1, R41.1, R42.1, R43.1, R44.1, R45.1, R46.1, R47.1, R5.2, R6.2, R7.2, R9.2, U1.14 (VCC)
- no-connect marks 0 -> 56
Other:
- note added: "(!) Isso aparenta estar errado.\nHá ainda 2 unidades disponíveis na pastilha 4B.\nPor que não usá-las aqui?"
- note added: "CONECTOR\nFRONTAL"
- note added: "CONECTOR\nTRASEIRO"
- moved on the sheet: CONECTOR_F_P8

Commit message: placa PCP-2: symbol remap
Parts:
- 2A_P8, 4B_P8, 4C_P8: symbol 7400 -> PCP-2-rescue:7400
- 3A_P8, 3B_P8, 4D_P8: symbol 74LS04 -> PCP-2-rescue:74LS04
- 4E_P8, 5B_P8, 5C_P8, 5D_P8: symbol 74LS10 -> PCP-2-rescue:74LS10
- 5E_P8, U1: symbol 74LS08 -> PCP-2-rescue:74LS08
- CONECTOR_F_P8, CONECTOR_T_P8: symbol CONN_35X2 -> PCP-2-rescue:CONN_35X2
- D1, D2, D3, D4, D5, D6: symbol DIODE -> PCP-2-rescue:DIODE
- Q10_P8, Q11_P8, Q12_P8, Q13_P8, Q14_P8, Q15_P8, Q1_P8, Q2_P8, Q3_P8, Q4_P8, Q5_P8, Q6_P8, Q7_P8, Q8_P8, Q9_P8: symbol BC414 -> PCP-2-rescue:BC414
- R1, R10, R11, R12, R13, R14, R15, R16, R17, R18, R19, R2, R20, R21, R22, R23, R24, R25, R26, R27, R28, R29, R3, R30, R31, R32, R33, R34, R35, R36, R37, R38, R39, R4, R40, R41, R42, R43, R44, R45, R46, R47, R5, R6, R7, R8, R9: symbol R -> PCP-2-rescue:R
