File: PCP-2/PCP-2.kicad_sch (KiCad schematic)
At the start: 82 parts, among them Q10_P8 BC237, Q11_P8 BC237, Q12_P8 BC237, Q13_P8 BC237, Q14_P8 BC237, Q15_P8 BC237, Q1_P8 BC237, Q2_P8 BC237, Q3_P8 BC237, Q4_P8 BC237, Q5_P8 BC237, Q6_P8 BC237, Q7_P8 BC237, Q8_P8 BC237, Q9_P8 BC237, U1 74LS08

Commit message: cleaning up references
Parts:
- renumbered R1 to R1_P8, R2 to R2_P8, R3 to R3_P8, R4 to R4_P8, R5 to R5_P8, R6 to R6_P8, R7 to R7_P8

Commit message: Some initial fixing of ERC errors.
Changed lines of the file:
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@@
 	)
 	(junction
-		(at 632.46 321.31)
-		(diameter 0)
-		(color 0 0 0 0)
-	)
-	(junction
 		(at 687.07 44.45)
 		(diameter 0)
@@
 	)
 	(junction
-		(at 571.5 234.95)
-		(diameter 0)
-		(color 0 0 0 0)
-	)
-	(junction
 		(at 82.55 58.42)
 		(diameter 0)
@@
 	(wire
 		(pts
-			(xy 571.5 231.14) (xy 571.5 234.95)
-		)
-		(stroke
-			(width 0)
-			(type default)
-		)
-	)
-	(wire
-		(pts
 			(xy 289.56 427.99) (xy 289.56 430.53)
 		)
@@
 	(wire
 		(pts
-			(xy 562.61 234.95) (xy 571.5 234.95)
-		)
-		(stroke
-			(width 0)
-			(type default)
-		)
-	)
-	(wire
-		(pts
 			(xy 214.63 422.91) (xy 214.63 419.1)
 		)
@@
 	(wire
 		(pts
-			(xy 632.46 318.77) (xy 632.46 321.31)
-		)
-		(stroke
-			(width 0)
-			(type default)
-		)
-	)
-	(wire
-		(pts
 			(xy 513.08 515.62) (xy 506.73 515.62)
 		)
@@
 	(wire
 		(pts
-			(xy 571.5 234.95) (xy 575.31 234.95)
+			(xy 562.61 234.95) (xy 575.31 234.95)
 		)
 		(stroke
@@
 	)
 	(symbol
-		(lib_id "power:PWR_FLAG")
-		(at 632.46 318.77 0)
-		(unit 1)
-		(body_style 1)
-		(exclude_from_sim no)
-		(in_bom yes)
-		(on_board yes)
-		(in_pos_files yes)
-		(dnp no)
-		(fields_autoplaced yes)
-		(property "Reference" "#FLG046"
-			(at 632.46 316.865 0)
-			(hide yes)
-			(show_name no)
-			(do_not_autoplace no)
-			(effects
-				(font
-					(size 1.27 1.27)
-				)
-			)
-		)
-		(property "Value" "PWR_FLAG"
-			(at 632.46 313.69 0)
-			(show_name no)
-			(do_not_autoplace no)
-			(effects
-				(font
-					(size 1.27 1.27)
-				)
-			)
-		)
-		(property "Footprint" ""
-			(at 632.46 318.77 0)
-			(hide yes)
-			(show_name no)
-			(do_not_autoplace no)
-			(effects
-				(font
-					(size 1.27 1.27)
-				)
-			)
-		)
-		(property "Datasheet" ""
-			(at 632.46 318.77 0)
-			(hide yes)
-			(show_name no)
-			(do_not_autoplace no)
-			(effects
-				(font
-					(size 1.27 1.27)
-				)
-			)
-		)
-		(property "Description" "Special symbol for telling ERC where power comes from"
-			(at 632.46 318.77 0)
-			(hide yes)
-			(show_name no)
-			(do_not_autoplace no)
-			(effects
-				(font
-					(size 1.27 1.27)
-				)
-			)
-		)
-		(pin "1"
-		)
-		(instances
-			(project "patinhofeio"
-				(path "/aca06203-542d-4682-a7e3-8839e24cce95/053788d3-9bb3-44f4-9df2-cd47e5e806b1"
-					(reference "#FLG046")
-					(unit 1)
-				)
-			)
-		)
-	)
-	(symbol
 		(lib_id "power:+24V")
 		(at 632.46 274.32 0)
@@
 					(unit 1)
 				)
-			)
-		)
-	)
-	(symbol
-		(lib_id "power:PWR_FLAG")
-		(at 571.5 231.14 0)
-		(unit 1)
-		(body_style 1)
-		(exclude_from_sim no)
-		(in_bom yes)
-		(on_board yes)
-		(in_pos_files yes)
-		(dnp no)
-		(fields_autoplaced yes)
-		(property "Reference" "#FLG06"
-			(at 571.5 229.235 0)
-			(hide yes)
-			(show_name no)
-			(do_not_autoplace no)
-			(effects
-				(font
-					(size 1.27 1.27)
-				)
-			)
-		)
-		(property "Value" "PWR_FLAG"
-			(at 571.5 226.06 0)
-			(show_name no)
-			(do_not_autoplace no)
-			(effects
-				(font
-					(size 1.27 1.27)
-				)
-			)
-		)
-		(property "Footprint" ""
-			(at 571.5 231.14 0)
-			(hide yes)
-			(show_name no)
-			(do_not_autoplace no)
-			(effects
-				(font
-					(size 1.27 1.27)
-				)
-			)
-		)
-		(property "Datasheet" ""
-			(at 571.5 231.14 0)
-			(hide yes)
-			(show_name no)
-			(do_not_autoplace no)
-			(effects
-				(font
-					(size 1.27 1.27)
-				)
-			)
-		)
-		(property "Description" "Special symbol for telling ERC where power comes from"
-			(at 571.5 231.14 0)
-			(hide yes)
-			(show_name no)
-			(do_not_autoplace no)
-			(effects
-				(font
-					(size 1.27 1.27)
-				)
-			)
-		)
-		(pin "1"
-		)
-		(instances
-			(project "patinhofeio"
-				(path "/aca06203-542d-4682-a7e3-8839e24cce95/053788d3-9bb3-44f4-9df2-cd47e5e806b1"
-					(reference "#FLG06")
-					(unit 1)
-				)

Commit message: fix a whole bunch of errors
Parts:
- removed 2A_P8, 4B_P8, 4C_P8: 7400, symbol PCP-2-rescue:7400
- removed 3A_P8, 3B_P8, 4D_P8: 74LS04, symbol PCP-2-rescue:74LS04
- removed 4E_P8, 5B_P8, 5C_P8, 5D_P8: 74LS10, symbol PCP-2-rescue:74LS10
- removed 5E_P8, U1: 74LS08, symbol PCP-2-rescue:74LS08
- added 2A_P8, 4B_P8, 4C_P8: 74LS00, symbol 74xx:74LS00
- added 3A_P8, 3B_P8, 4D_P8: 74LS04, symbol 74xx:74LS04
- added 4E_P8, 5B_P8, 5C_P8, 5D_P8: 74LS10, symbol 74xx:74LS10
- added 5E_P8: 74LS08, symbol 74xx:74LS08
Connections:
- net +ATIVO: now also 4C_P8.3, 5B_P8.13
- net +CE: now also 4B_P8.2, 5B_P8.8
- net +CP: now also 4B_P8.11, 5C_P8.2
- net +CS: now also 4C_P8.6, 5B_P8.3
- net +IS: now also 4C_P8.8, 5C_P8.9
- net +MP: now also 4C_P8.11, 5C_P8.5
- net -BOT-INT-A: now also 2A_P8.9
- net -BOT-INT-N: now also 2A_P8.13
- net -ES: now also 3B_P8.9
- net -FASE1: now also 3B_P8.5
- net -FASE2: now also 3B_P8.3
- net -FASE3: now also 3B_P8.1
- net -FASE4: now also 3B_P8.11
- net -FASE5: now also 3B_P8.13
- net -INT: now also 3A_P8.13
- net -LAL: now also 5B_P8.11, 5B_P8.2, 5B_P8.4, 5C_P8.10, 5C_P8.13, 5C_P8.4
- net -PAR: now also 3A_P8.9
- net -PEDIDO_DE_INTERRUPÇÃO: now also 2A_P8.10, 2A_P8.11
- net -RODA: now also 3A_P8.11
- net AT: now also 4C_P8.1, 4E_P8.3, 5E_P8.9
- net CE: now also 5B_P8.10, 5D_P8.2, 5E_P8.4
- net CP: now also 4B_P8.13, 4E_P8.10, 5E_P8.1
- net CS: now also 4C_P8.4, 5E_P8.10
- net GND: now also 2A_P8.14 (VCC), 3A_P8.14 (VCC), 3B_P8.14 (VCC), 4B_P8.14 (VCC), 4C_P8.14 (VCC), 4D_P8.7 (GND), 4E_P8.14 (VCC), 5B_P8.14 (VCC), 5C_P8.14 (VCC), 5D_P8.14 (VCC), 5E_P8.7 (GND)
- net IS: now also 4C_P8.10, 5D_P8.10, 5E_P8.5
- net MP: now also 4C_P8.13, 5D_P8.5, 5E_P8.2
- net PAT: now also 4E_P8.1
- net VCC: now also 2A_P8.7 (GND), 3A_P8.7 (GND), 3B_P8.7 (GND), 4B_P8.7 (GND), 4C_P8.7 (GND), 4D_P8.14 (VCC), 4E_P8.7 (GND), 5B_P8.7 (GND), 5C_P8.7 (GND), 5D_P8.7 (GND), 5E_P8.14 (VCC)
- net at Q10_P8.2 (B), R24.1: now also 3B_P8.10
- net at Q9_P8.2 (B), R21.1: now also 3B_P8.2
- net at Q8_P8.2 (B), R20.1: now also 3B_P8.4
- net at Q7_P8.2 (B), R19.1: now also 3B_P8.6
- net at Q12_P8.2 (B), R26.1: now also 3A_P8.8
- net at Q11_P8.2 (B), R25.1: now also 3B_P8.12
- net at Q13_P8.2 (B), R37.1: now also 3A_P8.10
- net at Q15_P8.2 (B), R39.1: now also 3A_P8.12
- net at Q14_P8.2 (B), R38.1: now also 3B_P8.8
- new net: 4D_P8.8, 5C_P8.1
- new net: 4B_P8.12, 5C_P8.12
- new net: 4E_P8.11, 4E_P8.13, 4E_P8.4, 5D_P8.4, 5E_P8.6
- new net: 4D_P8.5, 4E_P8.8
- new net: 4E_P8.9, 5D_P8.11, 5D_P8.13, 5D_P8.3, 5E_P8.8
- new net: 2A_P8.12, 2A_P8.8
- new net: 4C_P8.12, 5C_P8.6
- new net: 4D_P8.4, 5B_P8.1
- new net: 4C_P8.2, 5B_P8.12
- new net: 4D_P8.6, 5C_P8.3
- new net: 4B_P8.3, 5B_P8.9
- new net: 4B_P8.1, 4D_P8.10
- new net: 4D_P8.1, 4E_P8.6
- new net: 4D_P8.2, 5B_P8.5
- new net: 4D_P8.3, 4E_P8.12
- new net: 4D_P8.12, 5C_P8.11
- new net: 4D_P8.13, 5D_P8.12
- new net: 4E_P8.2, 4E_P8.5, 5D_P8.1, 5D_P8.9, 5E_P8.3
- new net: 4C_P8.5, 5B_P8.6
- new net: 4D_P8.11, 5D_P8.8
- new net: 4C_P8.9, 5C_P8.8
- new net: 4D_P8.9, 5D_P8.6

Commit message: wip + PDF plot
Other:
- moved on the sheet: 2A_P8E, 3A_P8G, 3B_P8G, 4B_P8E, 4C_P8E, 4D_P8G, 4E_P8D, 5B_P8D, 5C_P8D, 5D_P8D, 5E_P8E
