File: PMR-1/PMR-1.sch (KiCad schematic (older format))
At the start: 1 part

Commit message: finalizada transcrição do esquemático PMR-1 (Painel - Mostra Registradores)
Parts:
- added 1A_P7, 1C_P7, 1E_P7, 3A_P7, 3C_P7, 3E_P7, 5A_P7, 5C_P7, 5E_P7: 74HC04, symbol 74HC04
- added CONECTOR_T_P7: CONN_35X2, symbol CONN_35X2
- renumbered CONECTOR_P7 to CONECTOR_F_P7
Connections:
- removed net ?: CONECTOR_F_P7.1 (P1), CONECTOR_F_P7.10 (P10), CONECTOR_F_P7.11 (P11), CONECTOR_F_P7.12 (P12), CONECTOR_F_P7.13 (P13), CONECTOR_F_P7.14 (P14), CONECTOR_F_P7.15 (P15), CONECTOR_F_P7.16 (P16), CONECTOR_F_P7.17 (P17), CONECTOR_F_P7.18 (P18), CONECTOR_F_P7.19 (P19), CONECTOR_F_P7.2 (P2), CONECTOR_F_P7.20 (P20), CONECTOR_F_P7.21 (P21), CONECTOR_F_P7.22 (P22), CONECTOR_F_P7.23 (P23), CONECTOR_F_P7.24 (P24), CONECTOR_F_P7.25, CONECTOR_F_P7.26 (P26), CONECTOR_F_P7.27 (P27), CONECTOR_F_P7.28 (P28), CONECTOR_F_P7.29 (P29), CONECTOR_F_P7.3 (P3), CONECTOR_F_P7.30 (P30), CONECTOR_F_P7.31 (P31), CONECTOR_F_P7.32 (P32), CONECTOR_F_P7.33 (P33), CONECTOR_F_P7.34 (P34), CONECTOR_F_P7.35 (P35), CONECTOR_F_P7.36 (P36), CONECTOR_F_P7.37 (P37), CONECTOR_F_P7.38 (P38), CONECTOR_F_P7.39 (P39), CONECTOR_F_P7.4 (P4), CONECTOR_F_P7.40 (P40), CONECTOR_F_P7.41 (P41), CONECTOR_F_P7.42 (P42), CONECTOR_F_P7.43 (P43), CONECTOR_F_P7.44 (P44), CONECTOR_F_P7.45 (P45), CONECTOR_F_P7.46 (P46), CONECTOR_F_P7.47 (P47), CONECTOR_F_P7.48 (P48), CONECTOR_F_P7.49 (P49), CONECTOR_F_P7.5 (P5), CONECTOR_F_P7.50 (P50), CONECTOR_F_P7.51 (P51), CONECTOR_F_P7.52 (P52), CONECTOR_F_P7.53 (P53), CONECTOR_F_P7.54 (P54), CONECTOR_F_P7.55 (P55), CONECTOR_F_P7.56 (P56), CONECTOR_F_P7.57 (P57), CONECTOR_F_P7.58 (P58), CONECTOR_F_P7.59 (P59), CONECTOR_F_P7.6 (P6), CONECTOR_F_P7.60 (P60), CONECTOR_F_P7.61 (P61), CONECTOR_F_P7.62 (P62), CONECTOR_F_P7.63 (P63), CONECTOR_F_P7.64 (P64), CONECTOR_F_P7.65 (P65), CONECTOR_F_P7.66 (P66), CONECTOR_F_P7.67 (P67), CONECTOR_F_P7.68 (P68), CONECTOR_F_P7.69 (P69), CONECTOR_F_P7.7 (P7), CONECTOR_F_P7.70 (P70), CONECTOR_F_P7.8 (P8), CONECTOR_F_P7.9 (P9)
- new net +AC_0: 1A_P7.1, CONECTOR_T_P7.5 (P5)
- new net +AC_1: 1A_P7.3, CONECTOR_T_P7.40 (P40)
- new net +AC_2: 1A_P7.5, CONECTOR_T_P7.6 (P6)
- new net +AC_3: 1A_P7.9, CONECTOR_T_P7.43 (P43)
- new net +AC_4: 1A_P7.11, CONECTOR_T_P7.8 (P8)
- new net +AC_5: 1A_P7.13, CONECTOR_T_P7.44 (P44)
- new net +AC_6: 3A_P7.1, CONECTOR_T_P7.15 (P15)
- new net +AC_7: 3A_P7.3, CONECTOR_T_P7.51 (P51)
- new net +CI_0: 3E_P7.1, CONECTOR_T_P7.12 (P12)
- new net +CI_1: 3E_P7.3, CONECTOR_T_P7.48 (P48)
- new net +CI_10: 3E_P7.11, CONECTOR_T_P7.58 (P58)
- new net +CI_11: 3E_P7.13, CONECTOR_T_P7.24 (P24)
- new net +CI_2: 3E_P7.5, CONECTOR_T_P7.13 (P13)
- new net +CI_3: 3C_P7.1, CONECTOR_T_P7.49 (P49)
- new net +CI_4: 3C_P7.3, CONECTOR_T_P7.14 (P14)
- new net +CI_5: 3C_P7.5, CONECTOR_T_P7.50 (P50)
- new net +CI_6: 3C_P7.9, CONECTOR_T_P7.56 (P56)
- new net +CI_7: 3C_P7.11, CONECTOR_T_P7.22 (P22)
- new net +CI_8: 3C_P7.13, CONECTOR_T_P7.57 (P57)
- new net +CI_9: 3E_P7.9, CONECTOR_T_P7.23 (P23)
- new net +LA_0: 1A_P7.2, CONECTOR_F_P7.68 (P68)
- new net +LA_1: 1A_P7.4, CONECTOR_F_P7.34 (P34)
- new net +LA_2: 1A_P7.6, CONECTOR_F_P7.69 (P69)
- new net +LA_3: 1A_P7.8, CONECTOR_F_P7.24 (P24)
- new net +LA_4: 1A_P7.10, CONECTOR_F_P7.60 (P60)
- new net +LA_5: 1A_P7.12, CONECTOR_F_P7.25
- new net +LA_6: 3A_P7.2, CONECTOR_F_P7.58 (P58)
- new net +LA_7: 3A_P7.4, CONECTOR_F_P7.23 (P23)
- new net +LD_0: 3A_P7.10, CONECTOR_F_P7.13 (P13)
- new net +LD_1: 3A_P7.12, CONECTOR_F_P7.48 (P48)
- new net +LD_2: 5A_P7.2, CONECTOR_F_P7.11 (P11)
- new net +LD_3: 5A_P7.4, CONECTOR_F_P7.46 (P46)
- new net +LD_4: 5A_P7.6, CONECTOR_F_P7.12 (P12)
- new net +LD_5: 5A_P7.8, CONECTOR_F_P7.37 (P37)
- new net +LD_6: 5A_P7.10, CONECTOR_F_P7.2 (P2)
- new net +LD_7: 5A_P7.12, CONECTOR_F_P7.38 (P38)
- new net +LE_0: 1E_P7.2, CONECTOR_F_P7.65 (P65)
- new net +LE_1: 1E_P7.4, CONECTOR_F_P7.31 (P31)
- new net +LE_10: 1E_P7.10, CONECTOR_F_P7.63 (P63)
- new net +LE_11: 1E_P7.12, CONECTOR_F_P7.28 (P28)
- new net +LE_2: 1E_P7.6, CONECTOR_F_P7.66 (P66)
- new net +LE_3: 1C_P7.2, CONECTOR_F_P7.32 (P32)
- new net +LE_4: 1C_P7.4, CONECTOR_F_P7.67 (P67)
- new net +LE_5: 1C_P7.6, CONECTOR_F_P7.33 (P33)
- new net +LE_6: 1C_P7.8, CONECTOR_F_P7.61 (P61)
- new net +LE_7: 1C_P7.10, CONECTOR_F_P7.26 (P26)
- new net +LE_8: 1C_P7.12, CONECTOR_F_P7.62 (P62)
- new net +LE_9: 1E_P7.8, CONECTOR_F_P7.27 (P27)
- new net +LI_0: 3E_P7.2, CONECTOR_F_P7.55 (P55)
- new net +LI_1: 3E_P7.4, CONECTOR_F_P7.20 (P20)
- new net +LI_10: 3E_P7.10, CONECTOR_F_P7.16 (P16)
- new net +LI_11: 3E_P7.12, CONECTOR_F_P7.51 (P51)
- new net +LI_2: 3E_P7.6, CONECTOR_F_P7.56 (P56)
- new net +LI_3: 3C_P7.2, CONECTOR_F_P7.21 (P21)
- new net +LI_4: 3C_P7.4, CONECTOR_F_P7.57 (P57)
- new net +LI_5: 3C_P7.6, CONECTOR_F_P7.22 (P22)
- new net +LI_6: 3C_P7.8, CONECTOR_F_P7.14 (P14)
- new net +LI_7: 3C_P7.10, CONECTOR_F_P7.49 (P49)
- new net +LI_8: 3C_P7.12, CONECTOR_F_P7.15 (P15)
- new net +LI_9: 3E_P7.8, CONECTOR_F_P7.50 (P50)
- new net +LR_0: 5E_P7.2, CONECTOR_F_P7.8 (P8)
- new net +LR_1: 5E_P7.4, CONECTOR_F_P7.43 (P43)
- new net +LR_2: 5E_P7.6, CONECTOR_F_P7.9 (P9)
- new net +LR_3: 5C_P7.2, CONECTOR_F_P7.44 (P44)
- new net +LR_4: 5C_P7.12, CONECTOR_F_P7.4 (P4)
- new net +LR_5: 5E_P7.8, CONECTOR_F_P7.40 (P40)
- new net +LR_6: 5E_P7.10, CONECTOR_F_P7.5 (P5)
- new net +LR_7: 5E_P7.12, CONECTOR_F_P7.41 (P41)
- new net +OVF: 3A_P7.9, CONECTOR_T_P7.20 (P20)
- new net +RD_0: 3A_P7.11, CONECTOR_T_P7.55 (P55)
- new net +RD_1: 3A_P7.13, CONECTOR_T_P7.21 (P21)
- new net +RD_2: 5A_P7.1, CONECTOR_T_P7.62 (P62)
- new net +RD_3: 5A_P7.3, CONECTOR_T_P7.28 (P28)
- new net +RD_4: 5A_P7.5, CONECTOR_T_P7.63 (P63)
- new net +RD_5: 5A_P7.9, CONECTOR_T_P7.30 (P30)
- new net +RD_6: 5A_P7.11, CONECTOR_T_P7.66 (P66)
- new net +RD_7: 5A_P7.13, CONECTOR_T_P7.31 (P31)
- new net +RE_0: 1E_P7.1, CONECTOR_T_P7.2 (P2)
- new net +RE_1: 1E_P7.3, CONECTOR_T_P7.37 (P37)
- new net +RE_10: 1E_P7.11, CONECTOR_T_P7.11 (P11)
- new net +RE_11: 1E_P7.13, CONECTOR_T_P7.47 (P47)
- new net +RE_2: 1E_P7.5, CONECTOR_T_P7.3 (P3)
- new net +RE_3: 1C_P7.1, CONECTOR_T_P7.38 (P38)
- new net +RE_4: 1C_P7.3, CONECTOR_T_P7.4 (P4)
- new net +RE_5: 1C_P7.5, CONECTOR_T_P7.39 (P39)
- new net +RE_6: 1C_P7.9, CONECTOR_T_P7.9 (P9)
- new net +RE_7: 1C_P7.11, CONECTOR_T_P7.45 (P45)
- new net +RE_8: 1C_P7.13, CONECTOR_T_P7.10 (P10)
- new net +RE_9: 1E_P7.9, CONECTOR_T_P7.46 (P46)
- new net +RI_0: 5E_P7.1, CONECTOR_T_P7.59 (P59)
- new net +RI_1: 5E_P7.3, CONECTOR_T_P7.25
- new net +RI_2: 5E_P7.5, CONECTOR_T_P7.60 (P60)
- new net +RI_3: 5C_P7.1, CONECTOR_T_P7.26 (P26)
- new net +RI_4: 5C_P7.13, CONECTOR_T_P7.68 (P68)
- new net +RI_5: 5E_P7.9, CONECTOR_T_P7.33 (P33)
- new net +RI_6: 5E_P7.11, CONECTOR_T_P7.69 (P69)
- new net +RI_7: 5E_P7.13, CONECTOR_T_P7.34 (P34)
- new net +T: 3A_P7.5, CONECTOR_T_P7.16 (P16)
- new net F10: 5C_P7.4, CONECTOR_F_P7.10 (P10)
- new net F3: 5C_P7.8, CONECTOR_F_P7.3 (P3)
- new net F39: 5C_P7.10, CONECTOR_F_P7.39 (P39)
- new net F45: 5C_P7.6, CONECTOR_F_P7.45 (P45)
- new net GND: 1A_P7.7 (GND), 1A_P7.7 (GND), 1A_P7.7 (GND), 1A_P7.7 (GND), 1A_P7.7 (GND), 1A_P7.7 (GND), 1C_P7.7 (GND), 1C_P7.7 (GND), 1C_P7.7 (GND), 1C_P7.7 (GND), 1C_P7.7 (GND), 1C_P7.7 (GND), 1E_P7.7 (GND), 1E_P7.7 (GND), 1E_P7.7 (GND), 1E_P7.7 (GND), 1E_P7.7 (GND), 1E_P7.7 (GND), 3A_P7.7 (GND), 3A_P7.7 (GND), 3A_P7.7 (GND), 3A_P7.7 (GND), 3A_P7.7 (GND), 3A_P7.7 (GND), 3C_P7.7 (GND), 3C_P7.7 (GND), 3C_P7.7 (GND), 3C_P7.7 (GND), 3C_P7.7 (GND), 3C_P7.7 (GND), 3E_P7.7 (GND), 3E_P7.7 (GND), 3E_P7.7 (GND), 3E_P7.7 (GND), 3E_P7.7 (GND), 3E_P7.7 (GND), 5A_P7.7 (GND), 5A_P7.7 (GND), 5A_P7.7 (GND), 5A_P7.7 (GND), 5A_P7.7 (GND), 5A_P7.7 (GND), 5C_P7.7 (GND), 5C_P7.7 (GND), 5C_P7.7 (GND), 5C_P7.7 (GND), 5C_P7.7 (GND), 5C_P7.7 (GND), 5E_P7.7 (GND), 5E_P7.7 (GND), 5E_P7.7 (GND), 5E_P7.7 (GND), 5E_P7.7 (GND), 5E_P7.7 (GND), CONECTOR_F_P7.70 (P70), CONECTOR_T_P7.70 (P70)
- new net LEX: 3A_P7.8, CONECTOR_F_P7.47 (P47)
- new net LT: 3A_P7.6, CONECTOR_F_P7.59 (P59)
- new net T27: 5C_P7.5, CONECTOR_T_P7.27 (P27)
- new net T32: 5C_P7.11, CONECTOR_T_P7.32 (P32)
- new net T61: 5C_P7.3, CONECTOR_T_P7.61 (P61)
- new net T67: 5C_P7.9, CONECTOR_T_P7.67 (P67)
- new net VCC: 1A_P7.14 (VCC), 1A_P7.14 (VCC), 1A_P7.14 (VCC), 1A_P7.14 (VCC), 1A_P7.14 (VCC), 1A_P7.14 (VCC), 1C_P7.14 (VCC), 1C_P7.14 (VCC), 1C_P7.14 (VCC), 1C_P7.14 (VCC), 1C_P7.14 (VCC), 1C_P7.14 (VCC), 1E_P7.14 (VCC), 1E_P7.14 (VCC), 1E_P7.14 (VCC), 1E_P7.14 (VCC), 1E_P7.14 (VCC), 1E_P7.14 (VCC), 3A_P7.14 (VCC), 3A_P7.14 (VCC), 3A_P7.14 (VCC), 3A_P7.14 (VCC), 3A_P7.14 (VCC), 3A_P7.14 (VCC), 3C_P7.14 (VCC), 3C_P7.14 (VCC), 3C_P7.14 (VCC), 3C_P7.14 (VCC), 3C_P7.14 (VCC), 3C_P7.14 (VCC), 3E_P7.14 (VCC), 3E_P7.14 (VCC), 3E_P7.14 (VCC), 3E_P7.14 (VCC), 3E_P7.14 (VCC), 3E_P7.14 (VCC), 5A_P7.14 (VCC), 5A_P7.14 (VCC), 5A_P7.14 (VCC), 5A_P7.14 (VCC), 5A_P7.14 (VCC), 5A_P7.14 (VCC), 5C_P7.14 (VCC), 5C_P7.14 (VCC), 5C_P7.14 (VCC), 5C_P7.14 (VCC), 5C_P7.14 (VCC), 5C_P7.14 (VCC), 5E_P7.14 (VCC), 5E_P7.14 (VCC), 5E_P7.14 (VCC), 5E_P7.14 (VCC), 5E_P7.14 (VCC), 5E_P7.14 (VCC), CONECTOR_F_P7.1 (P1), CONECTOR_T_P7.1 (P1)
- no-connect marks 0 -> 28
Other:
- note added: "CONECTOR\nFRONTAL"
- note added: "CONECTOR\nTRASEIRO"
- moved on the sheet: CONECTOR_F_P7

Commit message: placa PMR-1: symbol remap
Parts:
- 1A_P7, 1C_P7, 1E_P7, 3A_P7, 3C_P7, 3E_P7, 5A_P7, 5C_P7, 5E_P7: symbol 74HC04 -> PMR-1-rescue:74HC04
- CONECTOR_F_P7, CONECTOR_T_P7: symbol CONN_35X2 -> PMR-1-rescue:CONN_35X2
