File: PMR-1/PMR-1.kicad_sch (KiCad schematic)
At the start: 11 parts

Commit message: Some initial fixing of ERC errors.
Changed lines of the file:
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@@
 		)
 	)
-	(junction
-		(at 133.35 320.04)
-		(diameter 0)
-		(color 0 0 0 0)
-	)
-	(junction
-		(at 72.39 76.2)
-		(diameter 0)
-		(color 0 0 0 0)
-	)
 	(no_connect
 		(at 74.93 99.06)
@@
 	(wire
 		(pts
-			(xy 133.35 318.77) (xy 133.35 320.04)
-		)
-		(stroke
-			(width 0)
-			(type default)
-		)
-	)
-	(wire
-		(pts
 			(xy 355.6 68.58) (xy 344.17 68.58)
 		)
@@
 	(wire
 		(pts
-			(xy 63.5 76.2) (xy 72.39 76.2)
-		)
-		(stroke
-			(width 0)
-			(type default)
-		)
-	)
-	(wire
-		(pts
 			(xy 532.13 203.2) (xy 518.16 203.2)
 		)
@@
 	(wire
 		(pts
-			(xy 72.39 72.39) (xy 72.39 76.2)
-		)
-		(stroke
-			(width 0)
-			(type default)
-		)
-	)
-	(wire
-		(pts
 			(xy 210.82 309.88) (xy 199.39 309.88)
 		)
@@
 	(wire
 		(pts
-			(xy 72.39 76.2) (xy 74.93 76.2)
+			(xy 63.5 76.2) (xy 74.93 76.2)
 		)
 		(stroke
@@
 	)
 	(symbol
-		(lib_id "power:PWR_FLAG")
-		(at 133.35 318.77 0)
-		(unit 1)
-		(body_style 1)
-		(exclude_from_sim no)
-		(in_bom yes)
-		(on_board yes)
-		(in_pos_files yes)
-		(dnp no)
-		(fields_autoplaced yes)
-		(property "Reference" "#FLG045"
-			(at 133.35 316.865 0)
-			(hide yes)
-			(show_name no)
-			(do_not_autoplace no)
-			(effects
-				(font
-					(size 1.27 1.27)
-				)
-			)
-		)
-		(property "Value" "PWR_FLAG"
-			(at 133.35 313.69 0)
-			(show_name no)
-			(do_not_autoplace no)
-			(effects
-				(font
-					(size 1.27 1.27)
-				)
-			)
-		)
-		(property "Footprint" ""
-			(at 133.35 318.77 0)
-			(hide yes)
-			(show_name no)
-			(do_not_autoplace no)
-			(effects
-				(font
-					(size 1.27 1.27)
-				)
-			)
-		)
-		(property "Datasheet" ""
-			(at 133.35 318.77 0)
-			(hide yes)
-			(show_name no)
-			(do_not_autoplace no)
-			(effects
-				(font
-					(size 1.27 1.27)
-				)
-			)
-		)
-		(property "Description" "Special symbol for telling ERC where power comes from"
-			(at 133.35 318.77 0)
-			(hide yes)
-			(show_name no)
-			(do_not_autoplace no)
-			(effects
-				(font
-					(size 1.27 1.27)
-				)
-			)
-		)
-		(pin "1"
-		)
-		(instances
-			(project "patinhofeio"
-				(path "/aca06203-542d-4682-a7e3-8839e24cce95/a4f4823c-2ff3-41ac-bc83-eeeb03b1c1d2"
-					(reference "#FLG045")
-					(unit 1)
-				)
-			)
-		)
-	)
-	(symbol
 		(lib_id "power:VCC")
 		(at 63.5 72.39 0)
@@
 					(unit 1)
 				)
-			)
-		)
-	)
-	(symbol
-		(lib_id "power:PWR_FLAG")
-		(at 72.39 72.39 0)
-		(unit 1)
-		(body_style 1)
-		(exclude_from_sim no)
-		(in_bom yes)
-		(on_board yes)
-		(in_pos_files yes)
-		(dnp no)
-		(fields_autoplaced yes)
-		(property "Reference" "#FLG01"
-			(at 72.39 70.485 0)
-			(hide yes)
-			(show_name no)
-			(do_not_autoplace no)
-			(effects
-				(font
-					(size 1.27 1.27)
-				)
-			)
-		)
-		(property "Value" "PWR_FLAG"
-			(at 72.39 67.31 0)
-			(show_name no)
-			(do_not_autoplace no)
-			(effects
-				(font
-					(size 1.27 1.27)
-				)
-			)
-		)
-		(property "Footprint" ""
-			(at 72.39 72.39 0)
-			(hide yes)
-			(show_name no)
-			(do_not_autoplace no)
-			(effects
-				(font
-					(size 1.27 1.27)
-				)
-			)
-		)
-		(property "Datasheet" ""
-			(at 72.39 72.39 0)
-			(hide yes)
-			(show_name no)
-			(do_not_autoplace no)
-			(effects
-				(font
-					(size 1.27 1.27)
-				)
-			)
-		)
-		(property "Description" "Special symbol for telling ERC where power comes from"
-			(at 72.39 72.39 0)
-			(hide yes)
-			(show_name no)
-			(do_not_autoplace no)
-			(effects
-				(font
-					(size 1.27 1.27)
-				)
-			)
-		)
-		(pin "1"
-		)
-		(instances
-			(project "patinhofeio"
-				(path "/aca06203-542d-4682-a7e3-8839e24cce95/a4f4823c-2ff3-41ac-bc83-eeeb03b1c1d2"
-					(reference "#FLG01")
-					(unit 1)
-				)

Commit message: wip + PDF plot
Parts:
- removed 1A_P7, 1C_P7, 1E_P7, 3A_P7, 3C_P7, 3E_P7, 5A_P7, 5C_P7, 5E_P7: 74HC04, symbol PMR-1-rescue:74HC04
- added 1A_P7, 1C_P7, 1E_P7, 3A_P7, 3C_P7, 3E_P7, 5A_P7, 5C_P7, 5E_P7: 74LS04, symbol 74xx:74LS04
Connections:
- net +AC_0: now also 1A_P7.1
- net +AC_1: now also 1A_P7.3
- net +AC_2: now also 1A_P7.5
- net +AC_3: now also 1A_P7.9
- net +AC_4: now also 1A_P7.11
- net +AC_5: now also 1A_P7.13
- net +AC_6: now also 3A_P7.1
- net +AC_7: now also 3A_P7.3
- net +CI_0: now also 3E_P7.1
- net +CI_1: now also 3E_P7.3
- net +CI_10: now also 3E_P7.11
- net +CI_11: now also 3E_P7.13
- net +CI_2: now also 3E_P7.5
- net +CI_3: now also 3C_P7.1
- net +CI_4: now also 3C_P7.3
- net +CI_5: now also 3C_P7.5
- net +CI_6: now also 3C_P7.9
- net +CI_7: now also 3C_P7.11
- net +CI_8: now also 3C_P7.13
- net +CI_9: now also 3E_P7.9
- net +LA_0: now also 1A_P7.2
- net +LA_1: now also 1A_P7.4
- net +LA_2: now also 1A_P7.6
- net +LA_3: now also 1A_P7.8
- net +LA_4: now also 1A_P7.10
- net +LA_5: now also 1A_P7.12
- net +LA_6: now also 3A_P7.2
- net +LA_7: now also 3A_P7.4
- net +LD_0: now also 3A_P7.10
- net +LD_1: now also 3A_P7.12
- net +LD_2: now also 5A_P7.2
- net +LD_3: now also 5A_P7.4
- net +LD_4: now also 5A_P7.6
- net +LD_5: now also 5A_P7.8
- net +LD_6: now also 5A_P7.10
- net +LD_7: now also 5A_P7.12
- net +LE_0: now also 1E_P7.2
- net +LE_1: now also 1E_P7.4
- net +LE_10: now also 1E_P7.10
- net +LE_11: now also 1E_P7.12
- net +LE_2: now also 1E_P7.6
- net +LE_3: now also 1C_P7.2
- net +LE_4: now also 1C_P7.4
- net +LE_5: now also 1C_P7.6
- net +LE_6: now also 1C_P7.8
- net +LE_7: now also 1C_P7.10
- net +LE_8: now also 1C_P7.12
- net +LE_9: now also 1E_P7.8
- net +LI_0: now also 3E_P7.2
- net +LI_1: now also 3E_P7.4
- net +LI_10: now also 3E_P7.10
- net +LI_11: now also 3E_P7.12
- net +LI_2: now also 3E_P7.6
- net +LI_3: now also 3C_P7.2
- net +LI_4: now also 3C_P7.4
- net +LI_5: now also 3C_P7.6
- net +LI_6: now also 3C_P7.8
- net +LI_7: now also 3C_P7.10
- net +LI_8: now also 3C_P7.12
- net +LI_9: now also 3E_P7.8
- net +LR_0: now also 5E_P7.2
- net +LR_1: now also 5E_P7.4
- net +LR_2: now also 5E_P7.6
- net +LR_3: now also 5C_P7.2
- net +LR_4: now also 5C_P7.12
- net +LR_5: now also 5E_P7.8
- net +LR_6: now also 5E_P7.10
- net +LR_7: now also 5E_P7.12
- net +OVF: now also 3A_P7.9
- net +RD_0: now also 3A_P7.11
- net +RD_1: now also 3A_P7.13
- net +RD_2: now also 5A_P7.1
- net +RD_3: now also 5A_P7.3
- net +RD_4: now also 5A_P7.5
- net +RD_5: now also 5A_P7.9
- net +RD_6: now also 5A_P7.11
- net +RD_7: now also 5A_P7.13
- net +RE_0: now also 1E_P7.1
- net +RE_1: now also 1E_P7.3
- net +RE_10: now also 1E_P7.11
- net +RE_11: now also 1E_P7.13
- net +RE_2: now also 1E_P7.5
- net +RE_3: now also 1C_P7.1
- net +RE_4: now also 1C_P7.3
- net +RE_5: now also 1C_P7.5
- net +RE_6: now also 1C_P7.9
- net +RE_7: now also 1C_P7.11
- net +RE_8: now also 1C_P7.13
- net +RE_9: now also 1E_P7.9
- net +RI_0: now also 5E_P7.1
- net +RI_1: now also 5E_P7.3
- net +RI_2: now also 5E_P7.5
- net +RI_3: now also 5C_P7.1
- net +RI_4: now also 5C_P7.13
- net +RI_5: now also 5E_P7.9
- net +RI_6: now also 5E_P7.11
- net +RI_7: now also 5E_P7.13
- net +T: now also 3A_P7.5
- net F10: now also 5C_P7.4
- net F3: now also 5C_P7.8
- net F39: now also 5C_P7.10
- net F45: now also 5C_P7.6
- net GND: now also 1A_P7.7 (GND), 1C_P7.7 (GND), 1E_P7.7 (GND), 3A_P7.7 (GND), 3C_P7.7 (GND), 3E_P7.7 (GND), 5A_P7.7 (GND), 5C_P7.7 (GND), 5E_P7.7 (GND)
- net LEX: now also 3A_P7.8
- net LT: now also 3A_P7.6
- net T27: now also 5C_P7.5
- net T32: now also 5C_P7.11
- net T61: now also 5C_P7.3
- net T67: now also 5C_P7.9
- net VCC: now also 1A_P7.14 (VCC), 1C_P7.14 (VCC), 1E_P7.14 (VCC), 3A_P7.14 (VCC), 3C_P7.14 (VCC), 3E_P7.14 (VCC), 5A_P7.14 (VCC), 5C_P7.14 (VCC), 5E_P7.14 (VCC)
