File: CDE-3/CDE-3.kicad_sch (KiCad schematic)
At the start: 43 parts

Commit message: I've started modifying the CDE-3 board to use DIN-41612 connectors. This is still wip! I'll get back to it once I receive some sample parts by mail.
Parts:
- CONECTOR_P10: footprint Pin_Headers:Pin_Header_Angled_2x35_Pitch2.54mm -> Connector_DIN:DIN41612_C_3x32_Male_Horizontal_THT
