File: CDE-3/CDE-3.kicad_sch (KiCad schematic)
At the start: 43 parts

Commit message: cleaning up references
Other:
- moved on the sheet: C1A_P10, C1C_P10, C2A_P10, C2C_P10, C3A_P10, C3C_P10, C4A_P10, C4C_P10, C5A_P10, C5C_P10

Commit message: Some initial fixing of ERC errors.
Changed lines of the file:
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@@
 	)
 	(junction
-		(at 90.17 135.89)
-		(diameter 0)
-		(color 0 0 0 0)
-	)
-	(junction
 		(at 703.58 405.13)
 		(diameter 0)
@@
 	)
 	(junction
-		(at 154.94 222.25)
-		(diameter 0)
-		(color 0 0 0 0)
-	)
-	(junction
 		(at 631.19 420.37)
 		(diameter 0)
@@
 	(wire
 		(pts
-			(xy 90.17 135.89) (xy 93.98 135.89)
-		)
-		(stroke
-			(width 0)
-			(type default)
-		)
-	)
-	(wire
-		(pts
 			(xy 631.19 461.01) (xy 647.7 461.01)
 		)
@@
 	(wire
 		(pts
-			(xy 154.94 219.71) (xy 154.94 222.25)
-		)
-		(stroke
-			(width 0)
-			(type default)
-		)
-	)
-	(wire
-		(pts
 			(xy 71.12 146.05) (xy 93.98 146.05)
 		)
@@
 	(wire
 		(pts
-			(xy 90.17 133.35) (xy 90.17 135.89)
-		)
-		(stroke
-			(width 0)
-			(type default)
-		)
-	)
-	(wire
-		(pts
 			(xy 88.9 184.15) (xy 93.98 184.15)
 		)
@@
 	(wire
 		(pts
-			(xy 83.82 135.89) (xy 90.17 135.89)
+			(xy 83.82 135.89) (xy 93.98 135.89)
 		)
 		(stroke
@@
 	)
 	(symbol
-		(lib_id "power:PWR_FLAG")
-		(at 90.17 133.35 0)
-		(unit 1)
-		(body_style 1)
-		(exclude_from_sim no)
-		(in_bom yes)
-		(on_board yes)
-		(in_pos_files yes)
-		(dnp no)
-		(fields_autoplaced yes)
-		(property "Reference" "#FLG048"
-			(at 90.17 131.445 0)
-			(hide yes)
-			(show_name no)
-			(do_not_autoplace no)
-			(effects
-				(font
-					(size 1.27 1.27)
-				)
-			)
-		)
-		(property "Value" "PWR_FLAG"
-			(at 90.17 128.27 0)
-			(show_name no)
-			(do_not_autoplace no)
-			(effects
-				(font
-					(size 1.27 1.27)
-				)
-			)
-		)
-		(property "Footprint" ""
-			(at 90.17 133.35 0)
-			(hide yes)
-			(show_name no)
-			(do_not_autoplace no)
-			(effects
-				(font
-					(size 1.27 1.27)
-				)
-			)
-		)
-		(property "Datasheet" ""
-			(at 90.17 133.35 0)
-			(hide yes)
-			(show_name no)
-			(do_not_autoplace no)
-			(effects
-				(font
-					(size 1.27 1.27)
-				)
-			)
-		)
-		(property "Description" "Special symbol for telling ERC where power comes from"
-			(at 90.17 133.35 0)
-			(hide yes)
-			(show_name no)
-			(do_not_autoplace no)
-			(effects
-				(font
-					(size 1.27 1.27)
-				)
-			)
-		)
-		(pin "1"
-		)
-		(instances
-			(project "patinhofeio"
-				(path "/aca06203-542d-4682-a7e3-8839e24cce95/66c98193-5e9c-4ee0-b18c-21adfe296f8d"
-					(reference "#FLG048")
-					(unit 1)
-				)
-			)
-		)
-	)
-	(symbol
 		(lib_id "power:VCC")
 		(at 687.07 443.23 0)
@@
 					(unit 1)
 				)
-			)
-		)
-	)
-	(symbol
-		(lib_id "power:PWR_FLAG")
-		(at 154.94 219.71 0)
-		(unit 1)
-		(body_style 1)
-		(exclude_from_sim no)
-		(in_bom yes)
-		(on_board yes)
-		(in_pos_files yes)
-		(dnp no)
-		(fields_autoplaced yes)
-		(property "Reference" "#FLG051"
-			(at 154.94 217.805 0)
-			(hide yes)
-			(show_name no)
-			(do_not_autoplace no)
-			(effects
-				(font
-					(size 1.27 1.27)
-				)
-			)
-		)
-		(property "Value" "PWR_FLAG"
-			(at 154.94 214.63 0)
-			(show_name no)
-			(do_not_autoplace no)
-			(effects
-				(font
-					(size 1.27 1.27)
-				)
-			)
-		)
-		(property "Footprint" ""
-			(at 154.94 219.71 0)
-			(hide yes)
-			(show_name no)
-			(do_not_autoplace no)
-			(effects
-				(font
-					(size 1.27 1.27)
-				)
-			)
-		)
-		(property "Datasheet" ""
-			(at 154.94 219.71 0)
-			(hide yes)
-			(show_name no)
-			(do_not_autoplace no)
-			(effects
-				(font
-					(size 1.27 1.27)
-				)
-			)
-		)
-		(property "Description" "Special symbol for telling ERC where power comes from"
-			(at 154.94 219.71 0)
-			(hide yes)
-			(show_name no)
-			(do_not_autoplace no)
-			(effects
-				(font
-					(size 1.27 1.27)
-				)
-			)
-		)
-		(pin "1"
-		)
-		(instances
-			(project "patinhofeio"
-				(path "/aca06203-542d-4682-a7e3-8839e24cce95/66c98193-5e9c-4ee0-b18c-21adfe296f8d"
-					(reference "#FLG051")
-					(unit 1)
-				)

Commit message: fix a whole bunch of errors
Parts:
- removed 2E_P10: 74LS13, Housings_DIP:DIP-14_W7.62mm_Socket_LongPads, symbol CDE-3-rescue:74LS13-RESCUE-CDE-3
- removed 4D_P10: 7400, Housings_DIP:DIP-14_W7.62mm_Socket_LongPads, symbol CDE-3-rescue:7400-RESCUE-CDE-3
- added 2E_P10: 74LS13, symbol 74xx:74LS13
- added 4D_P10: 74LS00, symbol 74xx:74LS00
Connections:
- net (+)RI_0: now also 2E_P10.1, 2E_P10.13
- net (+)RI_1: now also 2E_P10.12, 2E_P10.2, 4D_P10.12
- net (+)RI_3: now also 2E_P10.5, 4D_P10.2
- net -RI_0: now also 4D_P10.1, 4D_P10.13, 4D_P10.5
- net -RI_1: now also 4D_P10.4
- net -RI_2: now also 2E_P10.10, 2E_P10.4
- net -RI_3: now also 2E_P10.9
- net GND: now also 2E_P10.7 (GND), 4D_P10.7 (GND)
- net VCC: now also 2E_P10.14 (VCC), 4D_P10.14 (VCC)
- net at 3B_P10.1, 4B_P10.12, 4B_P10.3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: now also 2E_P10.8
- net at 3A_P10.5, 4C_P10.3, 4C_P10.5: now also 4D_P10.6
- net at 3A_P10.1: now also 4D_P10.3
- net at 3A_P10.3, 4C_P10.12, 4C_P10.8: now also 4D_P10.11
- net at 3A_P10.9, 5B_P10.12, 5B_P10.3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: now also 2E_P10.6

Commit message: fixing more errors
Parts:
- removed 1A_P10, 1B_P10, 2A_P10, 2B_P10, 3A_P10, 3B_P10: 74HC04, Housings_DIP:DIP-14_W7.62mm_Socket_LongPads, symbol CDE-3-rescue:74HC04-RESCUE-CDE-3
- removed 3C_P10, 4A_P10, 4B_P10, 4C_P10, 5A_P10, 5B_P10, 5C_P10: 7402, Housings_DIP:DIP-14_W7.62mm_Socket_LongPads, symbol CDE-3-rescue:7402-RESCUE-CDE-3
- added 1A_P10, 1B_P10, 2A_P10, 2B_P10, 3A_P10, 3B_P10: 74LS04, symbol 74xx:74LS04
- added 3C_P10, 4A_P10, 4B_P10, 4C_P10, 5A_P10, 5B_P10, 5C_P10: 74LS02, symbol 74xx:74LS02
Connections:
- net (+)RI_0: now also 1A_P10.10
- net (+)RI_1: now also 1A_P10.4
- net (+)RI_2: now also 1A_P10.12, 4C_P10.11, 4C_P10.2
- net (+)RI_3: now also 1B_P10.10, 4A_P10.3, 5C_P10.11, 5C_P10.2
- net (+)RI_4: now also 1B_P10.4
- net (+)RI_5: now also 1B_P10.12
- net (+)RI_6: now also 2A_P10.10
- net (+)RI_7: now also 2A_P10.4
- net +(CAC+SOM): now also 3A_P10.4
- net +(PAN+PAZ): now also 3A_P10.10
- net +(PLI+ARA): now also 3A_P10.6
- net +(SUS+PUG): now also 3A_P10.12
- net +ARA: now also 4C_P10.4
- net +CAC: now also 4C_P10.13
- net +ESP-D: now also 5A_P10.4
- net +IME: now also 3A_P10.8
- net +IMEADD: now also 5B_P10.1
- net +IMENAND: now also 5B_P10.4
- net +IMEXOR: now also 5B_P10.13
- net +INDICE: now also 3A_P10.2
- net +INI: now also 4A_P10.10
- net +MIC: now also 3B_P10.4
- net +MICG1: now also 4A_P10.1
- net +MICG2A: now also 3B_P10.12
- net +MICG2B: now also 3B_P10.6
- net +PAN: now also 5C_P10.13
- net +PAR-D: now also 5A_P10.13
- net +PAZ: now also 5C_P10.10
- net +PER: now also 5A_P10.1
- net +PLI: now also 4C_P10.1
- net +PUG: now also 5C_P10.4
- net +PUL: now also 4A_P10.4
- net +RD_0: now also 2A_P10.1
- net +RD_1: now also 2A_P10.13
- net +RD_2: now also 2B_P10.5
- net +RD_3: now also 2B_P10.3
- net +RD_4: now also 2B_P10.1
- net +RD_5: now also 2B_P10.9
- net +RD_6: now also 2B_P10.11
- net +RD_7: now also 2B_P10.13
- net +RESERVADO: now also 3C_P10.1
- net +RI_0: now also 1A_P10.9
- net +RI_1: now also 1A_P10.5
- net +RI_2: now also 1A_P10.1
- net +RI_3: now also 1B_P10.9
- net +RI_4: now also 1B_P10.5
- net +RI_5: now also 1B_P10.1
- net +RI_6: now also 2A_P10.9
- net +RI_7: now also 2A_P10.5
- net +SAE: now also 3B_P10.2
- net +SAEDE: now also 4B_P10.4
- net +SAEDS: now also 4B_P10.1
- net +SAEFU: now also 4B_P10.10
- net +SAESA: now also 4B_P10.13
- net +SHIFT: now also 5B_P10.10
- net +SOM: now also 4C_P10.10
- net +SUS: now also 5C_P10.1
- net +TRI: now also 5A_P10.10
- net +TRO: now also 4A_P10.13
- net -RD_0: now also 2A_P10.2, 4B_P10.2
- net -RD_1: now also 2A_P10.12, 4B_P10.5
- net -RD_2: now also 2B_P10.6, 4B_P10.11
- net -RD_3: now also 2B_P10.4, 4B_P10.8
- net -RD_4: now also 2B_P10.2
- net -RD_5: now also 2B_P10.8
- net -RD_6: now also 2B_P10.10
- net -RD_7: now also 2B_P10.12
- net -RI_0: now also 1A_P10.11, 1A_P10.8
- net -RI_1: now also 1A_P10.3, 1A_P10.6
- net -RI_2: now also 1A_P10.13, 1A_P10.2, 4C_P10.6, 4C_P10.9
- net -RI_3: now also 1B_P10.11, 1B_P10.8, 5C_P10.6, 5C_P10.9
- net -RI_4: now also 1B_P10.3, 1B_P10.6, 5B_P10.2
- net -RI_5: now also 1B_P10.13, 1B_P10.2, 5B_P10.5
- net -RI_6: now also 2A_P10.11, 2A_P10.8, 5B_P10.11
- net -RI_7: now also 2A_P10.3, 2A_P10.6, 5B_P10.8
- net GND: now also 1A_P10.7 (GND), 1B_P10.7 (GND), 2A_P10.7 (GND), 2B_P10.7 (GND), 3A_P10.7 (GND), 3B_P10.7 (GND), 3C_P10.14 (VCC), 4A_P10.14 (VCC), 4B_P10.14 (VCC), 4C_P10.14 (VCC), 5A_P10.14 (VCC), 5B_P10.14 (VCC), 5C_P10.14 (VCC)
- net VCC: now also 1A_P10.14 (VCC), 1B_P10.14 (VCC), 2A_P10.14 (VCC), 2B_P10.14 (VCC), 3A_P10.14 (VCC), 3B_P10.14 (VCC), 3C_P10.7 (GND), 4A_P10.7 (GND), 4B_P10.7 (GND), 4C_P10.7 (GND), 5A_P10.7 (GND), 5B_P10.7 (GND), 5C_P10.7 (GND)
- net at 2E_P10.8: now also 3B_P10.1, 4B_P10.12, 4B_P10.3, 4B_P10.6, 4B_P10.9
- net at 4D_P10.6: now also 3A_P10.5, 4C_P10.3, 4C_P10.5
- net at 4D_P10.3: now also 3A_P10.1
- net at 4D_P10.11: now also 3A_P10.3, 4C_P10.12, 4C_P10.8
- net at 1C_P10.12: now also 3A_P10.11, 5C_P10.3, 5C_P10.5
- net at 1C_P10.6: now also 3A_P10.13, 5C_P10.12, 5C_P10.8
- net at 2E_P10.6: now also 3A_P10.9, 5B_P10.12, 5B_P10.3, 5B_P10.6, 5B_P10.9
- net at 2D_P10.12: now also 5A_P10.5
- net at 1D_P10.12: now also 3B_P10.5, 3C_P10.3, 4A_P10.12, 4A_P10.5, 4A_P10.9, 5A_P10.12, 5A_P10.3, 5A_P10.6, 5A_P10.9
- net at 2D_P10.6: now also 5A_P10.11
- net at 1D_P10.8: now also 5A_P10.8
- net at 1C_P10.8: now also 3C_P10.2
- net at 1D_P10.6: now also 3B_P10.13
- net at 3D_P10.12: now also 4A_P10.6
- net at 3D_P10.6: now also 4A_P10.11
- net at 3D_P10.8: now also 4A_P10.8
- net at 1E_P10.12: now also 5A_P10.2
- net at 2D_P10.8: now also 3B_P10.3, 4A_P10.2
Other:
- moved on the sheet: 2E_P10C, 4D_P10E

Commit message: fixing a whole bunch more ERC errors
Parts:
- removed 1C_P10, 1D_P10, 1E_P10, 2D_P10, 3D_P10: 74LS10, Housings_DIP:DIP-14_W7.62mm_Socket_LongPads, symbol CDE-3-rescue:74LS10-RESCUE-CDE-3
- added 1C_P10, 1D_P10, 1E_P10, 2D_P10, 3D_P10: 74LS10, symbol 74xx:74LS10
Connections:
- net (+)RI_0: now also 1C_P10.1, 1C_P10.3, 2D_P10.11
- net (+)RI_1: now also 1C_P10.2
- net (+)RI_2: now also 1C_P10.13, 1C_P10.5
- net (+)RI_3: now also 1D_P10.2, 1D_P10.4
- net (+)RI_4: now also 1D_P10.13
- net (+)RI_5: now also 1C_P10.11, 1D_P10.11, 2D_P10.1, 2D_P10.3
- net (+)RI_6: now also 1C_P10.10, 1D_P10.10, 1E_P10.2, 3D_P10.10
- net (+)RI_7: now also 1C_P10.9, 1E_P10.13, 2D_P10.5, 3D_P10.5
- net +MIC: now also 1D_P10.1, 1D_P10.3
- net -RI_1: now also 1C_P10.4, 2D_P10.10
- net -RI_2: now also 2D_P10.9
- net -RI_4: now also 1D_P10.5
- net -RI_5: now also 1E_P10.1, 3D_P10.1, 3D_P10.3, 3D_P10.9
- net -RI_6: now also 2D_P10.2, 2D_P10.4, 3D_P10.2, 3D_P10.4
- net -RI_7: now also 1D_P10.9, 2D_P10.13, 3D_P10.11, 3D_P10.13
- net GND: now also 1C_P10.7 (GND), 1D_P10.7 (GND), 1E_P10.7 (GND), 2D_P10.7 (GND), 3D_P10.7 (GND)
- net VCC: now also 1C_P10.14 (VCC), 1D_P10.14 (VCC), 1E_P10.14 (VCC), 2D_P10.14 (VCC), 3D_P10.14 (VCC)
- net at 3A_P10.11, 5C_P10.3, 5C_P10.5: now also 1C_P10.12
- net at 3A_P10.13, 5C_P10.12, 5C_P10.8: now also 1C_P10.6
- net at 4A_P10.6: now also 3D_P10.12
- net at 4A_P10.11: now also 3D_P10.6
- net at 4A_P10.8: now also 3D_P10.8
- net at 5A_P10.2: now also 1E_P10.12
- net at 5A_P10.5: now also 2D_P10.12
- net at 5A_P10.11: now also 2D_P10.6
- net at 5A_P10.8: now also 1D_P10.8
- net at 3C_P10.2: now also 1C_P10.8
- net at 3B_P10.5, 3C_P10.3, 4A_P10.12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: now also 1D_P10.12
- net at 3B_P10.13: now also 1D_P10.6
- net at 3B_P10.3, 4A_P10.2: now also 2D_P10.8
Other:
- moved on the sheet: 1A_P10G, 1B_P10G, 2A_P10G, 2B_P10G, 2E_P10C, 3A_P10G, 3B_P10G, 3C_P10E, 4A_P10E, 4B_P10E, 4C_P10E, 4D_P10E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

Commit message: a lot more work on the circuit transcription
Parts:
- removed 2C_P10: 74LS30, Housings_DIP:DIP-14_W7.62mm_Socket_LongPads, symbol CDE-3-rescue:74LS30-RESCUE-CDE-3
- added 2C_P10: 74LS30, symbol 74xx:74LS30
Connections:
- net -RDZ: now also 2C_P10.8
- net -RD_0: now also 2C_P10.1
- net -RD_1: now also 2C_P10.2
- net -RD_2: now also 2C_P10.3
- net -RD_3: now also 2C_P10.4
- net -RD_4: now also 2C_P10.5
- net -RD_5: now also 2C_P10.6
- net -RD_6: now also 2C_P10.11
- net -RD_7: now also 2C_P10.12
- net GND: now also 2C_P10.7 (GND)
- net VCC: now also 2C_P10.14 (VCC)
Other:
- moved on the sheet: C1A_P10, C1B_P10, C1C_P10, C1D_P10, C1E_P10, C2A_P10, C2B_P10, C2C_P10, C2D_P10, C2E_P10, C3A_P10, C3B_P10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
