File: FM1-6/FM1-6.kicad_sch (KiCad schematic)
At the start: 13 parts

Commit message: These are updated files after I loaded the project on a new version of KICAD
Parts:
- 1A_P4, 1B_P4, 1C_P4, 1D_P4, 3A_P4, 3B_P4, 3C_P4, 3D_P4, 5A_P4, 5B_P4, 5C_P4, 5D_P4: footprint ~ -> (none)
