File: FAC-5/FAC-5.kicad_sch (KiCad schematic)
At the start: 19 parts, among them U1 74AHC04, U10 74LS54, U11 74LS54, U12 74LS74, U13 74LS74, U14 74LS74, U15 74LS74, U16 74LS55, U17 74LS55, U18 74LS54, U2 74LS54, U3 74LS74, U4 74LS10, U5 74LS54, U6 74LS54, U7 74LS54, U8 74LS54, U9 74LS54

Commit message: initial work on schematics for a backplane to which all boards will be attached.
Parts:
- renumbered U1 to U?, U5 to U?, U18 to U?, U8 to U?, U14 to U?, U9 to U?, U12 to U?, U11 to U?, U3 to U?, U16 to U?, U6 to U?, U13 to U?, U10 to U?, U7 to U?, U2 to U?, U4 to U?, U15 to U?, U17 to U?
Connections:
- net +AC0: now also U?.5 (Q); no longer U?.9 (Q)
- net +AC2: now also U?.5 (Q); no longer U?.9 (Q)
- net +AC4: now also U?.5 (Q); no longer U?.9 (Q)
- net +AC6: now also U?.5 (Q); no longer U?.9 (Q)
- net +OVF: now also U?.6 (~{Q}); no longer U?.8 (~{Q})
- net +RD2: now also U?.1; no longer U?.13
- net +RD3: now also U?.1; no longer U?.5
- net +RESET: now also U?.1 (~{R}), U?.1 (~{R}), U?.1 (~{R}), U?.1 (~{R}); no longer U?.13 (~{R}), U?.13 (~{R}), U?.13 (~{R}), U?.13 (~{R})
- net +SET: now also U?.4 (~{S}), U?.4 (~{S}), U?.4 (~{S}), U?.4 (~{S}); no longer U?.10 (~{S}), U?.10 (~{S}), U?.10 (~{S}), U?.10 (~{S})
- net -AC0: now also U?.6 (~{Q}); no longer U?.8 (~{Q})
- net -AC2: now also U?.6 (~{Q}); no longer U?.8 (~{Q})
- net -AC4: now also U?.6 (~{Q}); no longer U?.8 (~{Q})
- net -AC6: now also U?.6 (~{Q}); no longer U?.8 (~{Q})
- net -C-AC: now also U?.3 (C), U?.3 (C), U?.3 (C), U?.3 (C); no longer U?.11 (C), U?.11 (C), U?.11 (C), U?.11 (C)
- net -C-OVF: now also U?.3 (C); no longer U?.11 (C)
- net -CLEAR-OVF: now also U?.4 (~{S}); no longer U?.10 (~{S})
- net -D-OVF: now also U?.2 (D); no longer U?.12 (D)
- net -OVF: now also U?.5 (Q); no longer U?.9 (Q)
- net -SET-OVF: now also U?.1 (~{R}); no longer U?.13 (~{R})
- net DUPLSINAL: now also U?.1; no longer U?.11
- net SEM G: now also U?.1, U?.2; no longer U?.12, U?.3
- net SEM T: now also U?.2, U?.2; no longer U?.4, U?.6
- net at U?.13: now also U?.2; no longer U?.8
- net at U?.8, U?.8: now also U?.2 (D); no longer U?.12 (D)
- net at U?.8: now also U?.2 (D); no longer U?.12 (D) (x3)
- new net: U?.13, U?.2
- new net: U?.1, U?.12

Commit message: wip: preparing to draw all PCBs
Parts:
- gave numbers to parts that had none: 1
Connections:
- net +AC0: now also CONECTOR_P3.41 (P41)
- net +AC1: now also CONECTOR_P3.45 (P45)
- net +AC2: now also CONECTOR_P3.46 (P46)
- net +AC3: now also CONECTOR_P3.52 (P52)
- net +AC4: now also CONECTOR_P3.53 (P53)
- net +AC5: now also CONECTOR_P3.59 (P59)
- net +AC6: now also CONECTOR_P3.25
- net +AC7: now also CONECTOR_P3.28 (P28)
- net +RESET: now also CONECTOR_P3.7 (P7)
- net +SET: now also CONECTOR_P3.6 (P6)
- net -AC0: now also CONECTOR_P3.42 (P42)
- net -AC1: now also CONECTOR_P3.10 (P10)
- net -AC2: now also CONECTOR_P3.47 (P47)
- net -AC3: now also CONECTOR_P3.51 (P51)
- net -AC4: now also CONECTOR_P3.54 (P54)
- net -AC5: now also CONECTOR_P3.58 (P58)
- net -AC6: now also CONECTOR_P3.61 (P61)
- net -AC7: now also CONECTOR_P3.62 (P62)
- net -C-AC: now also CONECTOR_P3.55 (P55)
- net ?: no longer CONECTOR_P3.1 (P1), CONECTOR_P3.10 (P10), CONECTOR_P3.25, CONECTOR_P3.28 (P28), CONECTOR_P3.41 (P41), CONECTOR_P3.42 (P42), CONECTOR_P3.45 (P45), CONECTOR_P3.46 (P46), CONECTOR_P3.47 (P47), CONECTOR_P3.51 (P51), CONECTOR_P3.52 (P52), CONECTOR_P3.53 (P53), CONECTOR_P3.54 (P54), CONECTOR_P3.55 (P55), CONECTOR_P3.58 (P58), CONECTOR_P3.59 (P59), CONECTOR_P3.6 (P6), CONECTOR_P3.61 (P61), CONECTOR_P3.62 (P62), CONECTOR_P3.7 (P7), CONECTOR_P3.70 (P70)
- net GND: now also CONECTOR_P3.70 (P70)
- new net VCC: CONECTOR_P3.1 (P1)
