File: FAC-5/FAC-5.kicad_sch (KiCad schematic)
At the start: 29 parts

Commit message: FAC-5
Parts:
- removed U?: 74AHC04, symbol 74xx:74AHC04
- removed U? (x2): 74LS54, symbol 74xx:74LS54
- removed U? (x2): 74LS55, symbol 74xx:74LS55
- added 1B_P3_, 5C_P3_: 7460, symbol CT1-4-rescue:7460
- added 1C_P3, 5B_P3: 7453, symbol CT1-4-rescue:7453
- gave numbers to parts that had none: 8
Connections:
- net +5V: now also 1B_P3_.13, 5C_P3_.13
- net +AC0: now also 1A_P3_.9 (Q); no longer 1A_P3_.5 (Q)
- net +AC2: now also 2A_P3_.9 (Q); no longer 2A_P3_.5 (Q)
- net +AC4: now also 3A_P3_.9 (Q); no longer 3A_P3_.5 (Q)
- net +AC6: now also 4A_P3_.9 (Q); no longer 4A_P3_.5 (Q)
- net +OVF: now also 5A_P3_.8 (~{Q}); no longer 5A_P3_.6 (~{Q})
- net +RD2: now also 3D_P3_.13, CONECTOR_P3.67 (P67), 1B_P3_.8, 5C_P3_.8; no longer 3D_P3_.1
- net +RD3: now also 3D_P3_.5, CONECTOR_P3.2 (P2), 1B_P3_.3, 5C_P3_.3; no longer 3D_P3_.1
- net +RESET: now also 1A_P3_.13 (~{R}), 2A_P3_.13 (~{R}), 3A_P3_.13 (~{R}), 4A_P3_.13 (~{R}); no longer 1A_P3_.1 (~{R}), 2A_P3_.1 (~{R}), 3A_P3_.1 (~{R}), 4A_P3_.1 (~{R})
- net +SET: now also 1A_P3_.10 (~{S}), 2A_P3_.10 (~{S}), 3A_P3_.10 (~{S}), 4A_P3_.10 (~{S}); no longer 1A_P3_.4 (~{S}), 2A_P3_.4 (~{S}), 3A_P3_.4 (~{S}), 4A_P3_.4 (~{S})
- net +SL: now also 1D_P3_.9, CONECTOR_P3.56 (P56), 1C_P3.10, 5B_P3.9, 5C_P3_.2, 5C_P3_.4; no longer 1D_P3_.3
- net +SR: now also 1D_P3_.5, CONECTOR_P3.17 (P17), 1B_P3_.2, 1B_P3_.4, 1C_P3.1, 5B_P3.2; no longer 1D_P3_.13
- net +T: now also CONECTOR_P3.40 (P40)
- net +TR: now also CONECTOR_P3.68 (P68)
- net -A0: now also CONECTOR_P3.37 (P37), 1C_P3.3
- net -A1: now also CONECTOR_P3.43 (P43)
- net -A2: now also CONECTOR_P3.44 (P44)
- net -A3: now also CONECTOR_P3.48 (P48)
- net -A4: now also CONECTOR_P3.50 (P50)
- net -A5: now also CONECTOR_P3.69 (P69)
- net -A6: now also CONECTOR_P3.57 (P57)
- net -A7: now also CONECTOR_P3.33 (P33), 5B_P3.13
- net -AC0: now also 1A_P3_.8 (~{Q}), 1D_P3_.10, 1C_P3.5, 5C_P3_.5; no longer 1A_P3_.6 (~{Q}), 1D_P3_.2
- net -AC1: now also 1C_P3.9
- net -AC2: now also 2A_P3_.8 (~{Q}); no longer 2A_P3_.6 (~{Q})
- net -AC4: now also 3A_P3_.8 (~{Q}); no longer 3A_P3_.6 (~{Q})
- net -AC6: now also 4A_P3_.8 (~{Q}), 5B_P3.3; no longer 4A_P3_.6 (~{Q})
- net -AC7: now also 1D_P3_.4, 1B_P3_.5; no longer 1D_P3_.1
- net -C-AC: now also 1A_P3_.11 (C), 2A_P3_.11 (C), 3A_P3_.11 (C), 4A_P3_.11 (C); no longer 1A_P3_.3 (C), 2A_P3_.3 (C), 3A_P3_.3 (C), 4A_P3_.3 (C)
- net -C-OVF: now also 5A_P3_.11 (C), CONECTOR_P3.65 (P65); no longer 5A_P3_.3 (C)
- net -CLEAR-OVF: now also 5A_P3_.10 (~{S}), CONECTOR_P3.63 (P63); no longer 5A_P3_.4 (~{S})
- net -CLEAR-T: now also CONECTOR_P3.3 (P3)
- net -D-OVF: now also 5A_P3_.12 (D), CONECTOR_P3.66 (P66); no longer 5A_P3_.2 (D)
- net -OVF: now also 5A_P3_.9 (Q); no longer 5A_P3_.5 (Q)
- net -SET-OVF: now also 5A_P3_.13 (~{R}), CONECTOR_P3.32 (P32); no longer 5A_P3_.1 (~{R})
- net -SET-T: now also CONECTOR_P3.39 (P39)
- net -SHIAC: now also CONECTOR_P3.49 (P49), 1C_P3.2, 5B_P3.1
- net -T: now also 1D_P3_.2, CONECTOR_P3.38 (P38), 1B_P3_.1, 5C_P3_.1; no longer 1D_P3_.5
- net DUPLSINAL: now also 3D_P3_.11, CONECTOR_P3.60 (P60), 1C_P3.4; no longer 3D_P3_.1
- net GND: now also 1B_P3_.7 (GND), 1B_P3_.7 (GND), 1C_P3.7 (GND), 5B_P3.4, 5B_P3.5, 5B_P3.7 (GND), 5C_P3_.7 (GND), 5C_P3_.7 (GND)
- net TR/T: now also 1D_P3_.1, CONECTOR_P3.30 (P30); no longer 1D_P3_.10
- net T/T: now also 1D_P3_.3, CONECTOR_P3.4 (P4); no longer 1D_P3_.4
- net VCC: now also 1B_P3_.14 (VCC), 1B_P3_.14 (VCC), 1C_P3.14 (VCC), 5B_P3.14 (VCC), 5C_P3_.14 (VCC), 5C_P3_.14 (VCC)
- net at 5A_P3_.2 (D): now also 5B_P3.8
- net at U?.8: now also 3A_P3_.12 (D); no longer 3A_P3_.2 (D)
- net at U?.8: now also 4A_P3_.12 (D); no longer 4A_P3_.2 (D)
- net at 3D_P3_.2: now also 1D_P3_.13; no longer 1D_P3_.9
- net at U?.8: now also 2A_P3_.12 (D); no longer 2A_P3_.2 (D)
- removed net ?: CONECTOR_P3.11 (P11), CONECTOR_P3.12 (P12), CONECTOR_P3.13 (P13), CONECTOR_P3.14 (P14), CONECTOR_P3.15 (P15), CONECTOR_P3.16 (P16), CONECTOR_P3.17 (P17), CONECTOR_P3.18 (P18), CONECTOR_P3.19 (P19), CONECTOR_P3.2 (P2), CONECTOR_P3.20 (P20), CONECTOR_P3.21 (P21), CONECTOR_P3.22 (P22), CONECTOR_P3.23 (P23), CONECTOR_P3.24 (P24), CONECTOR_P3.26 (P26), CONECTOR_P3.27 (P27), CONECTOR_P3.29 (P29), CONECTOR_P3.3 (P3), CONECTOR_P3.30 (P30), CONECTOR_P3.31 (P31), CONECTOR_P3.32 (P32), CONECTOR_P3.33 (P33), CONECTOR_P3.34 (P34), CONECTOR_P3.35 (P35), CONECTOR_P3.36 (P36), CONECTOR_P3.37 (P37), CONECTOR_P3.38 (P38), CONECTOR_P3.39 (P39), CONECTOR_P3.4 (P4), CONECTOR_P3.40 (P40), CONECTOR_P3.43 (P43), CONECTOR_P3.44 (P44), CONECTOR_P3.48 (P48), CONECTOR_P3.49 (P49), CONECTOR_P3.5 (P5), CONECTOR_P3.50 (P50), CONECTOR_P3.56 (P56), CONECTOR_P3.57 (P57), CONECTOR_P3.60 (P60), CONECTOR_P3.63 (P63), CONECTOR_P3.64 (P64), CONECTOR_P3.65 (P65), CONECTOR_P3.66 (P66), CONECTOR_P3.67 (P67), CONECTOR_P3.68 (P68), CONECTOR_P3.69 (P69), CONECTOR_P3.8 (P8), CONECTOR_P3.9 (P9)
- removed net SEM G: 3D_P3_.2, 4D_P3_.1
- removed net SEM T: 3D_P3_.2, 4D_P3_.2
- new net: 5B_P3.11 (Ve), 5C_P3_.11, 5C_P3_.9
- new net: 5B_P3.12 (Vc), 5C_P3_.10, 5C_P3_.12
- new net: 1B_P3_.11, 1B_P3_.9, 1C_P3.11 (Ve)
- new net: 1B_P3_.10, 1B_P3_.12, 1C_P3.12 (Vc)
- new net: 1C_P3.13, 3D_P3_.8
- new net: 1A_P3_.12 (D), 1C_P3.8
- new net: 3D_P3_.10, 4D_P3_.5
- new net: 3D_P3_.9, 4D_P3_.6
- new net +OVR: CONECTOR_P3.29 (P29)
- new net +SG: 5B_P3.10
- new net -OVR: CONECTOR_P3.64 (P64)
- new net Sem_G: 3D_P3_.12, 4D_P3_.3
- new net Sem_T: 1B_P3_.6, 3D_P3_.6, 4D_P3_.4, 5C_P3_.6
- no-connect marks 0 -> 22
Other:
- note removed: "Revisar"
- moved on the sheet: 1A_P3_A, 1A_P3_B, 1D_P3_A, 2A_P3_A, 2A_P3_B, 3A_P3_A, 3A_P3_B, 3D_P3_A, 3D_P3_C, 3D_P3_D, 3D_P3_E, 3D_P3_F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

Commit message: cleaning up references
Parts:
- gave numbers to parts that had none: 6
- renumbered 1A_P3_ to 1A_P3, 1B_P3_ to 1B_P3, 1D_P3_ to 1D_P3, 2A_P3_ to 2A_P3, 3A_P3_ to 3A_P3, 3D_P3_ to 3D_P3, 4A_P3_ to 4A_P3, 4D_P3_ to 4D_P3, 5A_P3_ to 5A_P3, 5C_P3_ to 5C_P3

Commit message: Some initial fixing of ERC errors.
Changed lines of the file:
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@@
 	)
 	(junction
-		(at 139.7 156.21)
-		(diameter 0)
-		(color 0 0 0 0)
-	)
-	(junction
 		(at 266.7 273.05)
 		(diameter 0)
@@
 	(wire
 		(pts
-			(xy 139.7 153.67) (xy 139.7 156.21)
-		)
-		(stroke
-			(width 0)
-			(type default)
-		)
-	)
-	(wire
-		(pts
 			(xy 340.36 208.28) (xy 342.9 208.28)
 		)
@@
 					(unit 1)
 				)
-			)
-		)
-	)
-	(symbol
-		(lib_id "FM1-6-rescue:PWR_FLAG-power")
-		(at 139.7 153.67 0)
-		(unit 1)
-		(body_style 1)
-		(exclude_from_sim no)
-		(in_bom yes)
-		(on_board yes)
-		(in_pos_files yes)
-		(dnp no)
-		(property "Reference" "#FLG052"
-			(at 139.7 151.257 0)
-			(hide yes)
-			(show_name no)
-			(do_not_autoplace no)
-			(effects
-				(font
-					(size 0.762 0.762)
-				)
-			)
-		)
-		(property "Value" "PWR_FLAG"
-			(at 139.7 148.3868 0)
-			(show_name no)
-			(do_not_autoplace no)
-			(effects
-				(font
-					(size 0.762 0.762)
-				)
-			)
-		)
-		(property "Footprint" ""
-			(at 139.7 153.67 0)
-			(hide yes)
-			(show_name no)
-			(do_not_autoplace no)
-			(effects
-				(font
-					(size 1.524 1.524)
-				)
-			)
-		)
-		(property "Datasheet" ""
-			(at 139.7 153.67 0)
-			(hide yes)
-			(show_name no)
-			(do_not_autoplace no)
-			(effects
-				(font
-					(size 1.524 1.524)
-				)
-			)
-		)
-		(property "Description" ""
-			(at 139.7 153.67 0)
-			(show_name no)
-			(do_not_autoplace no)
-			(effects
-				(font
-					(size 1.27 1.27)
-				)
-			)
-		)
-		(pin "1"
-		)
-		(instances
-			(project "patinhofeio"
-				(path "/aca06203-542d-4682-a7e3-8839e24cce95/c4fc9564-1c4f-4175-9e51-1a074c56e995"
-					(reference "#FLG052")
-					(unit 1)
-				)

Commit message: addressing a few more ERC errors
Parts:
- added unit 3 of 1A_P3
- added unit 2 of 1D_P3
- added unit 3 of 2A_P3
- added unit 2 of 2B_P3
- added unit 2 of 2C_P3
- added unit 3 of 3A_P3
- added unit 2 of 3B_P3
- added unit 2 of 3C_P3
- added unit 7 of 3D_P3
- added unit 3 of 4A_P3
- added unit 2 of 4B_P3
- added unit 2 of 4C_P3
- added unit 4 of 4D_P3
- added unit 3 of 5A_P3
Connections:
- net +SG is gone; now on net Sem_G: 5B_P3.10
- net GND: now also 1A_P3.7 (GND), 1D_P3.14 (VCC), 2A_P3.7 (GND), 2B_P3.14 (VCC), 2C_P3.14 (VCC), 3A_P3.7 (GND), 3B_P3.14 (VCC), 3C_P3.14 (VCC), 3D_P3.7 (GND), 4A_P3.7 (GND), 4B_P3.14 (VCC), 4C_P3.14 (VCC), 4D_P3.7 (GND), 5A_P3.7 (GND)
- net VCC: now also 1A_P3.14 (VCC), 1D_P3.7 (GND), 2A_P3.14 (VCC), 2B_P3.7 (GND), 2C_P3.7 (GND), 3A_P3.14 (VCC), 3B_P3.7 (GND), 3C_P3.7 (GND), 3D_P3.14 (VCC), 4A_P3.14 (VCC), 4B_P3.7 (GND), 4C_P3.7 (GND), 4D_P3.14 (VCC), 5A_P3.14 (VCC)
