File: FR1-1/FR1-1.kicad_sch (KiCad schematic)
At the start: 1 part

Commit message: FR1/FR2 + FS1/FS2
Parts:
- added 1A_FR1_, 1A_FR2_, 1B_FR1_, 1B_FR2_, 1C_FR1_, 1C_FR2_, 3A_FR1_, 3A_FR2_, 3B_FR1_, 3B_FR2_, 3C_FR1_, 3C_FR2_, 3E_FR1_, 3E_FR2_, 3F_FR1_, 3F_FR2_, 5E_FR1_, 5E_FR2_, 5F_FR1_, 5F_FR2_: 74HC74, symbol CCE-2-rescue:74HC74
- added 1D_FR1_, 1D_FR2_, 5C_FR1_1, 5C_FR2_: 74LS51, symbol 74xx:74LS51
- added 1E_FR1_, 1E_FR2_: 7400, Housings_DIP:DIP-14_W7.62mm_Socket_LongPads, symbol CDE-3-rescue:7400-RESCUE-CDE-3
- added 5A_FR1_1, 5A_FR2_, 5B_FR1_1, 5B_FR2_: 74LS54, symbol 74xx:74LS54
- added CONECTOR_P1_FR1: CONN_35X2, symbol FR1-1-rescue:CONN_35X2-conn_35x2
- gave numbers to parts that had none: 1
Connections:
- removed net ?: CONECTOR_P1_FR2.1 (P1), CONECTOR_P1_FR2.10 (P10), CONECTOR_P1_FR2.11 (P11), CONECTOR_P1_FR2.12 (P12), CONECTOR_P1_FR2.13 (P13), CONECTOR_P1_FR2.14 (P14), CONECTOR_P1_FR2.15 (P15), CONECTOR_P1_FR2.16 (P16), CONECTOR_P1_FR2.17 (P17), CONECTOR_P1_FR2.18 (P18), CONECTOR_P1_FR2.19 (P19), CONECTOR_P1_FR2.2 (P2), CONECTOR_P1_FR2.20 (P20), CONECTOR_P1_FR2.21 (P21), CONECTOR_P1_FR2.22 (P22), CONECTOR_P1_FR2.23 (P23), CONECTOR_P1_FR2.24 (P24), CONECTOR_P1_FR2.25, CONECTOR_P1_FR2.26 (P26), CONECTOR_P1_FR2.27 (P27), CONECTOR_P1_FR2.28 (P28), CONECTOR_P1_FR2.29 (P29), CONECTOR_P1_FR2.3 (P3), CONECTOR_P1_FR2.30 (P30), CONECTOR_P1_FR2.31 (P31), CONECTOR_P1_FR2.32 (P32), CONECTOR_P1_FR2.33 (P33), CONECTOR_P1_FR2.34 (P34), CONECTOR_P1_FR2.35 (P35), CONECTOR_P1_FR2.36 (P36), CONECTOR_P1_FR2.37 (P37), CONECTOR_P1_FR2.38 (P38), CONECTOR_P1_FR2.39 (P39), CONECTOR_P1_FR2.4 (P4), CONECTOR_P1_FR2.40 (P40), CONECTOR_P1_FR2.41 (P41), CONECTOR_P1_FR2.42 (P42), CONECTOR_P1_FR2.43 (P43), CONECTOR_P1_FR2.44 (P44), CONECTOR_P1_FR2.45 (P45), CONECTOR_P1_FR2.46 (P46), CONECTOR_P1_FR2.47 (P47), CONECTOR_P1_FR2.48 (P48), CONECTOR_P1_FR2.49 (P49), CONECTOR_P1_FR2.5 (P5), CONECTOR_P1_FR2.50 (P50), CONECTOR_P1_FR2.51 (P51), CONECTOR_P1_FR2.52 (P52), CONECTOR_P1_FR2.53 (P53), CONECTOR_P1_FR2.54 (P54), CONECTOR_P1_FR2.55 (P55), CONECTOR_P1_FR2.56 (P56), CONECTOR_P1_FR2.57 (P57), CONECTOR_P1_FR2.58 (P58), CONECTOR_P1_FR2.59 (P59), CONECTOR_P1_FR2.6 (P6), CONECTOR_P1_FR2.60 (P60), CONECTOR_P1_FR2.61 (P61), CONECTOR_P1_FR2.62 (P62), CONECTOR_P1_FR2.63 (P63), CONECTOR_P1_FR2.64 (P64), CONECTOR_P1_FR2.65 (P65), CONECTOR_P1_FR2.66 (P66), CONECTOR_P1_FR2.67 (P67), CONECTOR_P1_FR2.68 (P68), CONECTOR_P1_FR2.69 (P69), CONECTOR_P1_FR2.7 (P7), CONECTOR_P1_FR2.70 (P70), CONECTOR_P1_FR2.8 (P8), CONECTOR_P1_FR2.9 (P9)
- new net -I0: 1E_FR1_.3, CONECTOR_P1_FR1.38 (P38)
- new net -I1: 1E_FR2_.3, CONECTOR_P1_FR2.38 (P38)
- new net -I10: 1D_FR1_.8, CONECTOR_P1_FR1.11 (P11)
- new net -I11: 1D_FR2_.8, CONECTOR_P1_FR2.11 (P11)
- new net -I2: 1E_FR1_.6, CONECTOR_P1_FR1.3 (P3)
- new net -I3: 1E_FR2_.6, CONECTOR_P1_FR2.3 (P3)
- new net -I4: 1E_FR1_.11, CONECTOR_P1_FR1.48 (P48)
- new net -I5: 1E_FR2_.11, CONECTOR_P1_FR2.48 (P48)
- new net -I6: 1E_FR1_.8, CONECTOR_P1_FR1.47 (P47)
- new net -I7: 1E_FR2_.8, CONECTOR_P1_FR2.47 (P47)
- new net -I8: 1D_FR1_.6, CONECTOR_P1_FR1.9 (P9)
- new net -I9: 1D_FR2_.6, CONECTOR_P1_FR2.9 (P9)
- new net -R0: 5C_FR1_1.8, CONECTOR_P1_FR1.33 (P33)
- new net -R0b: 3F_FR1_.2 (D), 5F_FR1_.2 (D), CONECTOR_P1_FR1.69 (P69)
- new net -R1: 5C_FR2_.8, CONECTOR_P1_FR2.33 (P33)
- new net -R1b: 3F_FR2_.2 (D), 5F_FR2_.2 (D), CONECTOR_P1_FR2.69 (P69)
- new net -R2: 5C_FR1_1.6, CONECTOR_P1_FR1.62 (P62)
- new net -R2b: 3F_FR1_.12 (D), 5F_FR1_.12 (D), CONECTOR_P1_FR1.68 (P68)
- new net -R3: 5C_FR2_.6, CONECTOR_P1_FR2.62 (P62)
- new net -R3b: 3F_FR2_.12 (D), 5F_FR2_.12 (D), CONECTOR_P1_FR2.68 (P68)
- new net -R4: 5B_FR1_1.8, CONECTOR_P1_FR1.32 (P32)
- new net -R4b: 3E_FR1_.2 (D), 5E_FR1_.2 (D), CONECTOR_P1_FR1.50 (P50)
- new net -R5: 5B_FR2_.8, CONECTOR_P1_FR2.32 (P32)
- new net -R5b: 3E_FR2_.2 (D), 5E_FR2_.2 (D), CONECTOR_P1_FR2.50 (P50)
- new net -R6: 5A_FR1_1.8, CONECTOR_P1_FR1.30 (P30)
- new net -R6b: 3E_FR1_.12 (D), 5E_FR1_.12 (D), CONECTOR_P1_FR1.19 (P19)
- new net -R7: 5A_FR2_.8, CONECTOR_P1_FR2.30 (P30)
- new net -R7b: 3E_FR2_.12 (D), 5E_FR2_.12 (D), CONECTOR_P1_FR2.19 (P19)
- new net -RRE02468: 1A_FR1_.1 (Cd), 1B_FR1_.1 (Cd), 1B_FR1_.13 (Cd), 1C_FR1_.1 (Cd), 1C_FR1_.13 (Cd), CONECTOR_P1_FR1.5 (P5)
- new net -RRE10: 1A_FR1_.13 (Cd), CONECTOR_P1_FR1.44 (P44)
- new net -RRE11: 1A_FR2_.13 (Cd), CONECTOR_P1_FR2.44 (P44)
- new net -RRE13579: 1A_FR2_.1 (Cd), 1B_FR2_.1 (Cd), 1B_FR2_.13 (Cd), 1C_FR2_.1 (Cd), 1C_FR2_.13 (Cd), CONECTOR_P1_FR2.5 (P5)
- new net -SRE10: CONECTOR_P1_FR1.43 (P43)
- new net -SRE11: CONECTOR_P1_FR2.43 (P43)
- new net ??/I: 1D_FR2_.10, 1D_FR2_.9, CONECTOR_P1_FR1.64 (P64), CONECTOR_P1_FR2.64 (P64)
- new net C-CI: 3A_FR1_.11 (Cp), 3A_FR1_.3 (Cp), 3A_FR2_.11 (Cp), 3A_FR2_.3 (Cp), 3B_FR1_.11 (Cp), 3B_FR1_.3 (Cp), 3B_FR2_.11 (Cp), 3B_FR2_.3 (Cp), 3C_FR1_.11 (Cp), 3C_FR1_.3 (Cp), 3C_FR2_.11 (Cp), 3C_FR2_.3 (Cp), CONECTOR_P1_FR1.34 (P34), CONECTOR_P1_FR2.34 (P34)
- new net C-RD: 3E_FR1_.11 (Cp), 3E_FR1_.3 (Cp), 3E_FR2_.11 (Cp), 3E_FR2_.3 (Cp), 3F_FR1_.11 (Cp), 3F_FR1_.3 (Cp), 3F_FR2_.11 (Cp), 3F_FR2_.3 (Cp), CONECTOR_P1_FR1.49 (P49), CONECTOR_P1_FR2.49 (P49)
- new net C-RE: 1A_FR1_.11 (Cp), 1A_FR1_.3 (Cp), 1A_FR2_.11 (Cp), 1A_FR2_.3 (Cp), 1B_FR1_.11 (Cp), 1B_FR1_.3 (Cp), 1B_FR2_.11 (Cp), 1B_FR2_.3 (Cp), 1C_FR1_.11 (Cp), 1C_FR1_.3 (Cp), 1C_FR2_.11 (Cp), 1C_FR2_.3 (Cp), CONECTOR_P1_FR1.40 (P40), CONECTOR_P1_FR2.40 (P40)
- new net C-RI: 5E_FR1_.11 (Cp), 5E_FR1_.3 (Cp), 5E_FR2_.11 (Cp), 5E_FR2_.3 (Cp), 5F_FR1_.11 (Cp), 5F_FR1_.3 (Cp), 5F_FR2_.11 (Cp), 5F_FR2_.3 (Cp), CONECTOR_P1_FR1.53 (P53), CONECTOR_P1_FR2.53 (P53)
- new net CI0: 3C_FR1_.5 (Q), CONECTOR_P1_FR1.51 (P51)
- new net CI1: 3C_FR2_.5 (Q), CONECTOR_P1_FR2.51 (P51)
- new net CI10: 3A_FR1_.9 (Q), CONECTOR_P1_FR1.55 (P55)
- new net CI11: 3A_FR2_.9 (Q), CONECTOR_P1_FR2.55 (P55)
- new net CI2: 3C_FR1_.9 (Q), CONECTOR_P1_FR1.56 (P56)
- new net CI3: 3C_FR2_.9 (Q), CONECTOR_P1_FR2.56 (P56)
- new net CI4: 3B_FR1_.5 (Q), CONECTOR_P1_FR1.52 (P52)
- new net CI5: 3B_FR2_.5 (Q), CONECTOR_P1_FR2.52 (P52)
- new net CI6: 3B_FR1_.9 (Q), CONECTOR_P1_FR1.20 (P20)
- new net CI7: 3B_FR2_.9 (Q), CONECTOR_P1_FR2.20 (P20)
- new net CI8: 3A_FR1_.5 (Q), CONECTOR_P1_FR1.18 (P18)
- new net CI9: 3A_FR2_.5 (Q), CONECTOR_P1_FR2.18 (P18)
- new net CLEAR: 5E_FR1_.1 (Cd), 5E_FR1_.13 (Cd), 5E_FR2_.1 (Cd), 5E_FR2_.13 (Cd), 5F_FR1_.1 (Cd), 5F_FR1_.13 (Cd), 5F_FR2_.1 (Cd), 5F_FR2_.13 (Cd), CONECTOR_P1_FR1.57 (P57), CONECTOR_P1_FR2.57 (P57)
- new net GND: 1A_FR1_.7 (GND), 1A_FR1_.7 (GND), 1A_FR2_.7 (GND), 1A_FR2_.7 (GND), 1B_FR1_.7 (GND), 1B_FR1_.7 (GND), 1B_FR2_.7 (GND), 1B_FR2_.7 (GND), 1C_FR1_.7 (GND), 1C_FR1_.7 (GND), 1C_FR2_.7 (GND), 1C_FR2_.7 (GND), 1D_FR1_.4, 1D_FR1_.5, 1D_FR2_.4, 1D_FR2_.5, 1E_FR1_.7 (GND), 1E_FR1_.7 (GND), 1E_FR1_.7 (GND), 1E_FR1_.7 (GND), 1E_FR2_.7 (GND), 1E_FR2_.7 (GND), 1E_FR2_.7 (GND), 1E_FR2_.7 (GND), 3A_FR1_.7 (GND), 3A_FR1_.7 (GND), 3A_FR2_.7 (GND), 3A_FR2_.7 (GND), 3B_FR1_.7 (GND), 3B_FR1_.7 (GND), 3B_FR2_.7 (GND), 3B_FR2_.7 (GND), 3C_FR1_.7 (GND), 3C_FR1_.7 (GND), 3C_FR2_.7 (GND), 3C_FR2_.7 (GND), 3E_FR1_.7 (GND), 3E_FR1_.7 (GND), 3E_FR2_.7 (GND), 3E_FR2_.7 (GND), 3F_FR1_.7 (GND), 3F_FR1_.7 (GND), 3F_FR2_.7 (GND), 3F_FR2_.7 (GND), 5A_FR1_1.4, 5A_FR1_1.5, 5A_FR2_.4, 5A_FR2_.5, 5B_FR1_1.4, 5B_FR1_1.5, 5B_FR2_.4, 5B_FR2_.5, 5E_FR1_.7 (GND), 5E_FR1_.7 (GND), 5E_FR2_.7 (GND), 5E_FR2_.7 (GND), 5F_FR1_.7 (GND), 5F_FR1_.7 (GND), 5F_FR2_.7 (GND), 5F_FR2_.7 (GND), CONECTOR_P1_FR1.70 (P70), CONECTOR_P1_FR2.70 (P70)
- new net L0: 5C_FR1_1.1, CONECTOR_P1_FR1.24 (P24)
- new net L1: 5C_FR2_.1, CONECTOR_P1_FR2.24 (P24)
- new net L2: 5C_FR1_1.2, CONECTOR_P1_FR1.60 (P60)
- new net L3: 5C_FR2_.2, CONECTOR_P1_FR2.60 (P60)
- new net L4: 5B_FR1_1.1, CONECTOR_P1_FR1.27 (P27)
- new net L5: 5B_FR2_.1, CONECTOR_P1_FR2.27 (P27)
- new net L6: 5A_FR1_1.1, CONECTOR_P1_FR1.29 (P29)
- new net L7: 5A_FR2_.1, CONECTOR_P1_FR2.29 (P29)
- new net L/R: 5A_FR1_1.13, 5A_FR2_.13, 5B_FR1_1.13, 5B_FR2_.13, 5C_FR1_1.13, 5C_FR1_1.3, 5C_FR2_.13, 5C_FR2_.3, CONECTOR_P1_FR1.25, CONECTOR_P1_FR2.25
- new net RD0: 3F_FR1_.6 (~{Q}), CONECTOR_P1_FR1.14 (P14)
- new net RD1: 3F_FR2_.6 (~{Q}), CONECTOR_P1_FR2.14 (P14)
- new net RD2: 3F_FR1_.8 (~{Q}), CONECTOR_P1_FR1.54 (P54)
- new net RD3: 3F_FR2_.8 (~{Q}), CONECTOR_P1_FR2.54 (P54)
- new net RD4: 3E_FR1_.6 (~{Q}), CONECTOR_P1_FR1.15 (P15)
- new net RD5: 3E_FR2_.6 (~{Q}), CONECTOR_P1_FR2.15 (P15)
- new net RD6: 3E_FR1_.8 (~{Q}), CONECTOR_P1_FR1.21 (P21)
- new net RD7: 3E_FR2_.8 (~{Q}), CONECTOR_P1_FR2.21 (P21)
- new net RE0: 1C_FR1_.5 (Q), 1E_FR1_.2, CONECTOR_P1_FR1.37 (P37)
- new net RE1: 1C_FR2_.5 (Q), 1E_FR2_.2, CONECTOR_P1_FR2.37 (P37)
- new net RE10: 1A_FR1_.9 (Q), 1D_FR1_.1, CONECTOR_P1_FR1.42 (P42)
- new net RE11: 1A_FR2_.9 (Q), 1D_FR2_.1, CONECTOR_P1_FR2.42 (P42)
- new net RE2: 1C_FR1_.9 (Q), 1E_FR1_.5, CONECTOR_P1_FR1.2 (P2)
- new net RE3: 1C_FR2_.9 (Q), 1E_FR2_.5, CONECTOR_P1_FR2.2 (P2)
- new net RE4: 1B_FR1_.5 (Q), 1E_FR1_.12, CONECTOR_P1_FR1.13 (P13)
- new net RE5: 1B_FR2_.5 (Q), 1E_FR2_.12, CONECTOR_P1_FR2.13 (P13)
- new net RE6: 1B_FR1_.9 (Q), 1E_FR1_.9, CONECTOR_P1_FR1.12 (P12)
- new net RE7: 1B_FR2_.9 (Q), 1E_FR2_.9, CONECTOR_P1_FR2.12 (P12)
- new net RE8: 1A_FR1_.5 (Q), 1D_FR1_.3, CONECTOR_P1_FR1.7 (P7)
- new net RE9: 1A_FR2_.5 (Q), 1D_FR2_.3, CONECTOR_P1_FR2.7 (P7)
- new net RE/I: 1D_FR1_.13, 1D_FR1_.2, 1D_FR2_.13, 1D_FR2_.2, 1E_FR1_.1, 1E_FR1_.10, 1E_FR1_.13, 1E_FR1_.4, 1E_FR2_.1, 1E_FR2_.10, 1E_FR2_.13, 1E_FR2_.4, CONECTOR_P1_FR1.36 (P36), CONECTOR_P1_FR2.36 (P36)
- new net RI0: 5F_FR1_.6 (~{Q}), CONECTOR_P1_FR1.22 (P22)
- new net RI1: 5F_FR2_.6 (~{Q}), CONECTOR_P1_FR2.22 (P22)
- new net RI2: 5F_FR1_.8 (~{Q}), CONECTOR_P1_FR1.58 (P58)
- new net RI3: 5F_FR2_.8 (~{Q}), CONECTOR_P1_FR2.58 (P58)
- new net RI4: 5E_FR1_.6 (~{Q}), CONECTOR_P1_FR1.23 (P23)
- new net RI5: 5E_FR2_.6 (~{Q}), CONECTOR_P1_FR2.23 (P23)
- new net RI6: 5E_FR1_.8 (~{Q}), CONECTOR_P1_FR1.59 (P59)
- new net RI7: 5E_FR2_.8 (~{Q}), CONECTOR_P1_FR2.59 (P59)
- new net SOMETHING/I: 1D_FR1_.10, 1D_FR1_.9
- new net U0: 1C_FR1_.2 (D), 3C_FR1_.2 (D), CONECTOR_P1_FR1.4 (P4)
- new net U0_pino_63: 5B_FR1_1.2, CONECTOR_P1_FR1.63 (P63)
- new net U1: 1C_FR2_.2 (D), 3C_FR2_.2 (D), CONECTOR_P1_FR2.4 (P4)
- new net U1_pino_63: 5B_FR2_.2, CONECTOR_P1_FR2.63 (P63)
- new net U2: 1C_FR1_.12 (D), 3C_FR1_.12 (D), CONECTOR_P1_FR1.46 (P46)
- new net U2_pino_66: 5A_FR1_1.2, CONECTOR_P1_FR1.66 (P66)
- new net U3: 1C_FR2_.12 (D), 3C_FR2_.12 (D), CONECTOR_P1_FR2.46 (P46)
- new net U3_pino_66: 5A_FR2_.2, CONECTOR_P1_FR2.66 (P66)
- new net U/R: 5A_FR1_1.3, 5A_FR2_.3, 5B_FR1_1.3, 5B_FR2_.3, CONECTOR_P1_FR1.28 (P28), CONECTOR_P1_FR2.28 (P28)
- new net VCC: 1A_FR1_.14 (VCC), 1A_FR1_.14 (VCC), 1A_FR2_.14 (VCC), 1A_FR2_.14 (VCC), 1B_FR1_.14 (VCC), 1B_FR1_.14 (VCC), 1B_FR2_.14 (VCC), 1B_FR2_.14 (VCC), 1C_FR1_.14 (VCC), 1C_FR1_.14 (VCC), 1C_FR2_.14 (VCC), 1C_FR2_.14 (VCC), 1E_FR1_.14 (VCC), 1E_FR1_.14 (VCC), 1E_FR1_.14 (VCC), 1E_FR1_.14 (VCC), 1E_FR2_.14 (VCC), 1E_FR2_.14 (VCC), 1E_FR2_.14 (VCC), 1E_FR2_.14 (VCC), 3A_FR1_.14 (VCC), 3A_FR1_.14 (VCC), 3A_FR2_.14 (VCC), 3A_FR2_.14 (VCC), 3B_FR1_.14 (VCC), 3B_FR1_.14 (VCC), 3B_FR2_.14 (VCC), 3B_FR2_.14 (VCC), 3C_FR1_.14 (VCC), 3C_FR1_.14 (VCC), 3C_FR2_.14 (VCC), 3C_FR2_.14 (VCC), 3E_FR1_.14 (VCC), 3E_FR1_.14 (VCC), 3E_FR2_.14 (VCC), 3E_FR2_.14 (VCC), 3F_FR1_.14 (VCC), 3F_FR1_.14 (VCC), 3F_FR2_.14 (VCC), 3F_FR2_.14 (VCC), 5E_FR1_.14 (VCC), 5E_FR1_.14 (VCC), 5E_FR2_.14 (VCC), 5E_FR2_.14 (VCC), 5F_FR1_.14 (VCC), 5F_FR1_.14 (VCC), 5F_FR2_.14 (VCC), 5F_FR2_.14 (VCC), CONECTOR_P1_FR1.1 (P1), CONECTOR_P1_FR2.1 (P1)
- new net Z0: 1B_FR1_.2 (D), 3B_FR1_.2 (D), CONECTOR_P1_FR1.10 (P10)
- new net Z0_pino_65: 5C_FR1_1.10, CONECTOR_P1_FR1.65 (P65)
- new net Z1: 1B_FR2_.2 (D), 3B_FR2_.2 (D), CONECTOR_P1_FR2.10 (P10)
- new net Z1_pino_65: 5C_FR2_.10, CONECTOR_P1_FR2.65 (P65)
- new net Z2: 1B_FR1_.12 (D), 3B_FR1_.12 (D), CONECTOR_P1_FR1.45 (P45)
- new net Z2_pino_61: 5C_FR1_1.4, CONECTOR_P1_FR1.61 (P61)
- new net Z3: 1B_FR2_.12 (D), 3B_FR2_.12 (D), CONECTOR_P1_FR2.45 (P45)
- new net Z3_pino_61: 5C_FR2_.4, CONECTOR_P1_FR2.61 (P61)
- new net Z4: 1A_FR1_.2 (D), 3A_FR1_.2 (D)
- new net Z4_pino_67: 5B_FR1_1.10, CONECTOR_P1_FR1.67 (P67)
- new net Z5: 1A_FR2_.2 (D), 3A_FR2_.2 (D), CONECTOR_P1_FR1.41 (P41), CONECTOR_P1_FR2.41 (P41)
- new net Z5_pino_67: 5B_FR2_.10, CONECTOR_P1_FR2.67 (P67)
- new net Z6: 1A_FR1_.12 (D), 3A_FR1_.12 (D), 5A_FR1_1.10, CONECTOR_P1_FR1.8 (P8)
- new net Z6_pino_31: CONECTOR_P1_FR1.31 (P31)
- new net Z7: 1A_FR2_.12 (D), 3A_FR2_.12 (D), CONECTOR_P1_FR2.8 (P8)
- new net Z7_pino_31: 5A_FR2_.10, CONECTOR_P1_FR2.31 (P31)
- new net Z/R: 5A_FR1_1.9, 5A_FR2_.9, 5B_FR1_1.9, 5B_FR2_.9, 5C_FR1_1.5, 5C_FR1_1.9, 5C_FR2_.5, 5C_FR2_.9, CONECTOR_P1_FR1.26 (P26), CONECTOR_P1_FR2.26 (P26)
- no-connect marks 0 -> 118
Other:
- note added: "CI"
- note added: "FR1-1"
- note added: "FR2-2"
- note added: "PS4"
- note added: "PS5"
- note added: "RD"
- note added: "RE"
- note added: "RI"
- moved on the sheet: CONECTOR_P1_FR2
