File: FS1-3/FS1-3.kicad_sch (KiCad schematic)
At the start: 21 parts

Commit message: FS1-3 + FS2-4
Parts:
- added 1A_FS2_, 1D_FS2_, 1E_FS2_, 1F_FS2_, 3A_FS2_, 3D_FS2_, 3F_FS2_, 5D_FS2_, 5E_FS2_, 5F_FS2_: 74LS51, symbol 74xx:74LS51
- added 1B_FS2_, 3B_FS2_, 5A_FS2_, 5B_FS2_: 74LS54, symbol 74xx:74LS54
- added 1C_FS2_, 3E_FS2_, 5C_FS2_: 74AHC04, symbol 74xx:74AHC04
- added 2C_FS2_, 3C_FS2_: 74HC02, symbol 74xx:74HC02
- added 4C_FS2_: 74HC00, symbol 74xx:74HC00
- added CONECTOR_P2_FS2: CONN_35X2, symbol FS1-3-rescue:CONN_35X2-conn_35x2
- renumbered 1A_P2A_ to 1A_FS1_, 1B_P2A_ to 1B_FS1_, 1C_P2A_ to 1C_FS1_, 1D_P2A_ to 1D_FS1_, 1E_P2A_ to 1E_FS1_, 1F_P2A_ to 1F_FS1_, 2C_P2A_ to 2C_FS1_, 3A_P2A_ to 3A_FS1_, 3B_P2A_ to 3B_FS1_, 3C_P2A_ to 3C_FS1_, 3D_P2A_ to 3D_FS1_, 3E_P2A_ to 3E_FS1_, 3F_P2A_ to 3F_FS1_, 4C_P2A_ to 4C_FS1_, 5A_P2A_ to 5A_FS1_, 5B_P2A_ to 5B_FS1_, 5C_P2A_ to 5C_FS1_, 5D_P2A_ to 5D_FS1_, 5E_P2A_ to 5E_FS1_, 5F_P2A_ to 5F_FS1_, CONECTOR_P2A to CONECTOR_P2_FS1
Connections:
- net C1/X is gone; now on net CI/X: 1B_FS1_.4, 3B_FS1_.4, 5A_FS1_.4, 5B_FS1_.5
- net +NAND: now also 1F_FS2_.1, 1F_FS2_.2, 3F_FS2_.4, 3F_FS2_.9, CONECTOR_P2_FS2.60 (P60)
- net +SOXOR: now also 1F_FS2_.10, 1F_FS2_.4, 3F_FS2_.1, 3F_FS2_.2, CONECTOR_P2_FS2.34 (P34)
- net +VUR: now also 1E_FS2_.1, 1E_FS2_.4, 3E_FS2_.3, CONECTOR_P2_FS2.2 (P2)
- net -AC/X: now also 1B_FS2_.2, 3B_FS2_.2, 5A_FS2_.2, 5B_FS2_.2, CONECTOR_P2_FS2.65 (P65)
- net -XOR: now also 1E_FS2_.9, 4C_FS2_.10, 4C_FS2_.12, 5E_FS2_.13, CONECTOR_P2_FS2.61 (P61)
- net AC/X: now also 1B_FS2_.13, 3B_FS2_.13, 5A_FS2_.1, 5B_FS2_.13, CONECTOR_P2_FS2.33 (P33)
- net CI/X: now also 1B_FS2_.4, 3B_FS2_.4, 5A_FS2_.4, 5B_FS2_.5, CONECTOR_P2_FS2.29 (P29)
- net GND: now also CONECTOR_P2_FS2.70 (P70)
- net P/Y: now also 1A_FS2_.13, 1A_FS2_.3, 3A_FS2_.13, 3A_FS2_.2, CONECTOR_P2_FS2.5 (P5)
- net RD/Y: now also 1A_FS2_.10, 1A_FS2_.5, 3A_FS2_.10, 3A_FS2_.5, CONECTOR_P2_FS2.7 (P7)
- net RE/X: now also 1B_FS2_.10, 3B_FS2_.10, 5A_FS2_.10, 5B_FS2_.9, CONECTOR_P2_FS2.32 (P32)
- net VCC: now also CONECTOR_P2_FS2.1 (P1)
- net at 3E_FS1_.6: now also 3D_FS1_.2; no longer 3D_FS1_.3
- net at 1C_FS1_.8: now also 3D_FS1_.3; no longer 3D_FS1_.2
- new net: 1E_FS2_.10, 1F_FS2_.3, 3C_FS2_.1
- new net: 1E_FS2_.13, 4C_FS2_.3
- new net: 1E_FS2_.8, 3D_FS2_.1, 3D_FS2_.4, 3E_FS2_.5
- new net: 1C_FS2_.11, 1D_FS2_.8, 1E_FS2_.2
- new net: 1E_FS2_.3, 3E_FS2_.4
- new net: 1C_FS2_.10, 1E_FS2_.5
- new net: 1E_FS2_.6, 1F_FS2_.5
- new net: 3E_FS2_.13, 5D_FS2_.6, 5E_FS2_.2
- new net: 3E_FS2_.10, 5E_FS2_.3
- new net: 3E_FS2_.12, 5E_FS2_.4
- new net: 3D_FS2_.8, 3E_FS2_.11, 5E_FS2_.10, 5E_FS2_.5
- new net: 3F_FS2_.13, 5E_FS2_.6
- new net: 4C_FS2_.6, 5E_FS2_.9
- new net: 5C_FS2_.12, 5F_FS2_.1
- new net: 5C_FS2_.13, 5D_FS2_.8, 5F_FS2_.10
- new net: 3C_FS2_.4, 3F_FS2_.10, 5E_FS2_.1
- new net: 5C_FS2_.6, 5D_FS2_.2
- new net: 5C_FS2_.10, 5D_FS2_.9
- new net: 1C_FS2_.4, 1D_FS2_.9
- new net: 3D_FS2_.13, 4C_FS2_.11
- new net: 1F_FS2_.13, 2C_FS2_.13, 4C_FS2_.13
- new net: 3E_FS2_.8, 5F_FS2_.13
- new net: 1C_FS2_.8, 3D_FS2_.3
- new net: 1C_FS2_.9, 1D_FS2_.6, 3D_FS2_.5
- new net: 3D_FS2_.2, 3E_FS2_.6
- new net: 1F_FS2_.9, 3D_FS2_.6
- new net: 5C_FS2_.8, 5D_FS2_.10
- new net: 1C_FS2_.2, 1D_FS2_.10
- new net: 3F_FS2_.3, 5F_FS2_.8
- new net: 3C_FS2_.10, 3F_FS2_.5, 4C_FS2_.9
- new net: 4C_FS2_.8, 5F_FS2_.5
- new net: 5C_FS2_.4, 5D_FS2_.3
- new net: 1C_FS2_.12, 1D_FS2_.2
- new net: 1C_FS2_.6, 1D_FS2_.3
- new net +AC0: 5B_FS2_.1, CONECTOR_P2_FS2.62 (P62)
- new net +AC1: 5A_FS2_.13, CONECTOR_P2_FS2.66 (P66)
- new net +AC2: 3B_FS2_.1, CONECTOR_P2_FS2.15 (P15)
- new net +AC3: 1B_FS2_.1, CONECTOR_P2_FS2.38 (P38)
- new net +C0: CONECTOR_P2_FS2.57 (P57)
- new net +CI4: 5B_FS2_.4, CONECTOR_P2_FS2.63 (P63)
- new net +CI5: 5A_FS2_.5, CONECTOR_P2_FS2.64 (P64)
- new net +CI6: 3B_FS2_.5, CONECTOR_P2_FS2.16 (P16)
- new net +CI7: 1B_FS2_.5, CONECTOR_P2_FS2.39 (P39)
- new net +P4: 3A_FS2_.1, CONECTOR_P2_FS2.52 (P52)
- new net +P5: 3A_FS2_.3, CONECTOR_P2_FS2.17 (P17)
- new net +P6: 1A_FS2_.2, CONECTOR_P2_FS2.40 (P40)
- new net +P7: 1A_FS2_.1, CONECTOR_P2_FS2.4 (P4)
- new net +RD0: 3A_FS2_.9, CONECTOR_P2_FS2.55 (P55)
- new net +RD1: 3A_FS2_.4, CONECTOR_P2_FS2.53 (P53)
- new net +RD2: 1A_FS2_.4, CONECTOR_P2_FS2.41 (P41)
- new net +RD3: 1A_FS2_.9, CONECTOR_P2_FS2.42 (P42)
- new net +RE4: 5B_FS2_.10, CONECTOR_P2_FS2.67 (P67)
- new net +RE5: 5A_FS2_.9, CONECTOR_P2_FS2.31 (P31)
- new net +RE6: 3B_FS2_.9, CONECTOR_P2_FS2.20 (P20)
- new net +RE7: 1B_FS2_.9, CONECTOR_P2_FS2.43 (P43)
- new net +Z0: 3F_FS2_.6, CONECTOR_P2_FS2.56 (P56)
- new net +Z1: 3F_FS2_.8, CONECTOR_P2_FS2.58 (P58)
- new net +Z2: 1F_FS2_.8, CONECTOR_P2_FS2.47 (P47)
- new net +Z3: 1F_FS2_.6, CONECTOR_P2_FS2.37 (P37)
- new net -AC0: 5B_FS2_.3, CONECTOR_P2_FS2.28 (P28)
- new net -AC1: 5A_FS2_.3, CONECTOR_P2_FS2.30 (P30)
- new net -AC2: 3B_FS2_.3, CONECTOR_P2_FS2.51 (P51)
- new net -AC3: 1B_FS2_.3, CONECTOR_P2_FS2.3 (P3)
- new net -C1: 3E_FS2_.9, 5E_FS2_.8, 5F_FS2_.4, 5F_FS2_.9, CONECTOR_P2_FS2.68 (P68)
- new net -X0: 3C_FS2_.9, 5B_FS2_.8, 5C_FS2_.11, 5D_FS2_.1, 5F_FS2_.3
- new net -X1: 3C_FS2_.5, 4C_FS2_.4, 5A_FS2_.8, 5C_FS2_.5, 5D_FS2_.4
- new net -X2: 1C_FS2_.13, 1D_FS2_.4, 2C_FS2_.12, 3B_FS2_.8, 3D_FS2_.10
- new net -X3: 1B_FS2_.8, 1C_FS2_.1, 1D_FS2_.13, 3C_FS2_.2, 4C_FS2_.1
- new net -Y0: 3A_FS2_.8, 3C_FS2_.8, 5C_FS2_.9, 5D_FS2_.13, 5F_FS2_.2
- new net -Y1: 3A_FS2_.6, 3C_FS2_.6, 4C_FS2_.5, 5C_FS2_.3, 5D_FS2_.5
- new net -Y2: 1A_FS2_.6, 1C_FS2_.5, 1D_FS2_.5, 2C_FS2_.11, 3D_FS2_.9
- new net -Y3: 1A_FS2_.8, 1C_FS2_.3, 1D_FS2_.1, 3C_FS2_.3, 4C_FS2_.2
- new net C0: 5F_FS2_.6
- no-connect marks 48 -> 96
Other:
- moved on the sheet: 1A_FS1_A, 1A_FS1_B, 1B_FS1_A, 1C_FS1_A, 1C_FS1_B, 1C_FS1_C, 1C_FS1_D, 1C_FS1_E, 1C_FS1_F, 1D_FS1_A, 1D_FS1_B, 1E_FS1_A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
