File: backplane/backplane.kicad_sch (KiCad schematic)
At the start: 19 parts

Commit message: FAC-5
Parts:
- added CONECTOR_FAC_5: CONN_35X2, symbol FAC-5-rescue:CONN_35X2-conn_35x2
Connections:
- net +AC0: now also CONECTOR_FAC_5.41 (P41)
- net +AC1: now also CONECTOR_FAC_5.45 (P45)
- net +AC2: now also CONECTOR_FAC_5.46 (P46)
- net +AC3: now also CONECTOR_FAC_5.52 (P52)
- net +AC4: now also CONECTOR_FAC_5.53 (P53)
- net +AC5: now also CONECTOR_FAC_5.59 (P59)
- net +AC6: now also CONECTOR_FAC_5.25
- net +AC7: now also CONECTOR_FAC_5.28 (P28)
- net +RD2: now also CONECTOR_FAC_5.67 (P67)
- net +RD3: now also CONECTOR_FAC_5.2 (P2)
- net +T: now also CONECTOR_FAC_5.40 (P40)
- net +TR: now also CONECTOR_FAC_5.68 (P68)
- net -AC0: now also CONECTOR_FAC_5.42 (P42)
- net -AC1: now also CONECTOR_FAC_5.10 (P10)
- net -AC2: now also CONECTOR_FAC_5.47 (P47)
- net -AC3: now also CONECTOR_FAC_5.51 (P51)
- net -AC4: now also CONECTOR_FAC_5.54 (P54)
- net -AC5: now also CONECTOR_FAC_5.58 (P58)
- net -AC6: now also CONECTOR_FAC_5.61 (P61)
- net -AC7: now also CONECTOR_FAC_5.62 (P62)
- net -D-OVF: now also CONECTOR_FAC_5.66 (P66)
- net -SHIAC: now also CONECTOR_FAC_5.49 (P49)
- net GND: now also CONECTOR_FAC_5.70 (P70)
- net T/T: now also CONECTOR_FAC_5.4 (P4)
- net VCC: now also CONECTOR_FAC_5.1 (P1)
- new net +OVR: CONECTOR_FAC_5.29 (P29)
- new net +RESET: CONECTOR_FAC_5.7 (P7)
- new net +SET: CONECTOR_FAC_5.6 (P6)
- new net +SL: CONECTOR_FAC_5.56 (P56)
- new net +SR: CONECTOR_FAC_5.17 (P17)
- new net -A0: CONECTOR_FAC_5.37 (P37)
- new net -A1: CONECTOR_FAC_5.43 (P43)
- new net -A2: CONECTOR_FAC_5.44 (P44)
- new net -A3: CONECTOR_FAC_5.48 (P48)
- new net -A4: CONECTOR_FAC_5.50 (P50)
- new net -A5: CONECTOR_FAC_5.69 (P69)
- new net -A6: CONECTOR_FAC_5.57 (P57)
- new net -A7: CONECTOR_FAC_5.33 (P33)
- new net -C-AC: CONECTOR_FAC_5.55 (P55)
- new net -C-OVF: CONECTOR_FAC_5.65 (P65)
- new net -CLEAR-OVF: CONECTOR_FAC_5.63 (P63)
- new net -CLEAR-T: CONECTOR_FAC_5.3 (P3)
- new net -OVR: CONECTOR_FAC_5.64 (P64)
- new net -SET-OVF: CONECTOR_FAC_5.32 (P32)
- new net -SET-T: CONECTOR_FAC_5.39 (P39)
- new net -T: CONECTOR_FAC_5.38 (P38)
- new net DUPLSINAL: CONECTOR_FAC_5.60 (P60)
- new net TR/T: CONECTOR_FAC_5.30 (P30)
- no-connect marks 327 -> 349
Other:
- note added: "Placa FAC-5: Acumulador."
